File: test_project_01/VUSB_Li-ion_BMS_to_3v3.kicad_sch (KiCad schematic)
At the start: 1 part

Commit message: v
Parts:
- added BT1: Battery_Cell, symbol Device:Battery_Cell
- added C2, C3, C4: C_Small, symbol Device:C_Small
- added D1: D_Shockley, symbol Device:D_Shockley
- added F1: 1.5 2A, symbol Device:Fuse
- added R11: 3k, symbol Device:R_Small
- added R12: 10k, symbol Device:R_Small
- added U4: MCP73831-2-OT, Package_TO_SOT_SMD:SOT-23-5, symbol Battery_Management:MCP73831-2-OT
- added U5: IFX27001TFV33, Package_TO_SOT_SMD:TO-252-3_TabPin2, symbol Regulator_Linear:IFX27001TFV33
- gave numbers to parts that had none: 1
Connections:
- net +5V: now also F1.1
- net +VDC: now reaches Q1.1 (D)
- net +VDC: now also D1.1 (K), U5.3 (I)
- net at Q1.2 (G): now also D1.2 (A), F1.2, R12.1, U4.4 (VDD)
- net +BATT: now reaches Q1.3 (S)
- net +BATT: now also BT1.1 (+), U4.3 (VBAT)
- new net: R11.1, U4.5 (PROG)
- new net +3V3: U5.2 (Q)
- new net GND: BT1.2 (-), R11.2, R12.2, U4.2 (VSS)
Other:
- note added: "150% rating so 1.5A 2A for me"
- note added: "400-500mA+ pe parte asta cand se transmite RF"
- moved on the sheet: Q1

Commit message: f
Parts:
- removed Q1: Q_PMOS_DGS, symbol Device:Q_PMOS_DGS
- removed U4: MCP73831-2-OT, Package_TO_SOT_SMD:SOT-23-5, symbol Battery_Management:MCP73831-2-OT
- removed U5: IFX27001TFV33, Package_TO_SOT_SMD:TO-252-3_TabPin2, symbol Regulator_Linear:IFX27001TFV33
- added C12: 1u, symbol Device:C_Small
- added D2, D3: LED_Small, symbol Device:LED_Small
- added IC2: MCP73834T-FCI_UN, SOP50P490X110-10N, symbol SamacSys_Parts:MCP73834T-FCI_UN
- added IC3: AP2112M-3.3TRG1, SOIC127P600X170-8N, symbol SamacSys_Parts:AP2112M-3.3TRG1
- added Q1: MCQ9435-TP, Package_SO:SOP-8_3.76x4.96mm_P1.27mm, symbol My_custom_lib:MCQ9435-TP
- added R13: 470, symbol Device:R_Small
- added R14: <1k, symbol Device:R_Small
- added R15: 10k, symbol Device:R_Small
- C2, C4: value C_Small -> 1u
- C3: value C_Small -> 4.7u
- D1: footprint (none) -> Diode_THT:D_DO-15_P15.24mm_Horizontal
- R11: value 3k -> 470
Connections:
- net +3V3: now also C12.1, IC3.1 (VOUT)
- net +BATT: now also C3.1, IC2.10 (VBAT_2), IC2.9 (VBAT_1), Q1.5 (D), Q1.6 (D), Q1.7 (D), Q1.8 (D)
- net +VDC: now also C4.1, IC3.5 (EN), IC3.8 (VIN), Q1.1 (S), Q1.2 (S), Q1.3 (S)
- net GND: now also C2.2, C3.2, C4.2, C12.2, IC2.5 (VSS), IC3.6 (GND_1), IC3.7 (GND_2), R14.1, R15.1; no longer R11.2
- net at D1.2 (A), F1.2, R12.1: now also C2.1, D2.2 (A), D3.2 (A), IC2.1 (VDD_1), IC2.2 (VDD_2), Q1.4 (G)
- net at R11.1: now also D2.1 (K)
- new net: IC2.6 (PROG), R14.2
- new net: D3.1 (K), R13.1
- new net: IC2.4 (STAT2), R13.2
- new net: IC2.3 (STAT1), R11.2
- new net: IC2.8 (THERM), R15.2
- no-connect marks 0 -> 3
Other:
- note added: "TE uses 1.8V logic active high activates a timer"
- note added: "active high"
- moved on the sheet: BT1, F1

Commit message: d
Other:
- title: (none) -> ESP32 audio power meter SD dataloger
Changed lines of the file:
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@@
 (kicad_sch (version 20211123) (generator eeschema)
   (paper "A4")
+  (title_block
+    (title "ESP32 audio power meter SD dataloger")
+    (rev "1")
+  )
   (junction (at 200.66 50.8) (diameter 0) (color 0 0 0 0)
   )

Commit message: j
Parts:
- added BT?: Battery_Cell, symbol Device:Battery_Cell
- added C? (x3): 1u, symbol Device:C_Small
- added C?: 4.7u, symbol Device:C_Small
- added D? (x2): LED_Small, symbol Device:LED_Small
- added D?: 2.6-2.8V, symbol Device:D_Zener
- added D?: D_Shockley, Diode_THT:D_DO-15_P15.24mm_Horizontal, symbol Device:D_Shockley
- added F?: 1.5 2A, symbol Device:Fuse
- added IC?: AP2112M-3.3TRG1, SOIC127P600X170-8N, symbol SamacSys_Parts:AP2112M-3.3TRG1
- added IC?: MCP73834T-FCI_UN, SOP50P490X110-10N, symbol SamacSys_Parts:MCP73834T-FCI_UN
- added Q? (x2): MCQ9435-TP, Package_SO:SOP-8_3.76x4.96mm_P1.27mm, symbol My_custom_lib:MCQ9435-TP
- added R? (x3): 10k, symbol Device:R_Small
- added R? (x2): 470, symbol Device:R_Small
- added R?: <1k, symbol Device:R_Small
Connections:
- net +3V3: now also C?.1, IC?.1 (VOUT)
- net +5V: now also F?.1
- net +BATT: now also BT?.1 (+), C?.1, D?.1 (K), IC?.10 (VBAT_2), IC?.9 (VBAT_1), Q?.5 (D), Q?.6 (D), Q?.7 (D), Q?.8 (D)
- net +VDC: now also C?.1, D?.1 (K), IC?.5 (EN), IC?.8 (VIN), Q?.1 (S), Q?.2 (S), Q?.3 (S)
- net GND: now also BT?.2 (-), C?.2, C?.2, C?.2, C?.2, IC?.5 (VSS), IC?.6 (GND_1), IC?.7 (GND_2), R?.1, R?.1, R?.2, R?.2
- new net: D?.1 (K), R?.1 (x2)
- new net: C?.1, D?.2 (A), D?.2 (A), D?.2 (A), F?.2, IC?.1 (VDD_1), IC?.2 (VDD_2), Q?.4 (G), R?.1
- new net: IC?.4 (STAT2), R?.2
- new net: Q?.1 (S), Q?.2 (S), Q?.3 (S), Q?.5 (D), Q?.6 (D), Q?.7 (D), Q?.8 (D)
- new net: D?.2 (A), Q?.4 (G), R?.1
- new net: IC?.8 (THERM), R?.2
- new net: IC?.3 (STAT1), R?.2
- new net: IC?.6 (PROG), R?.2
- no-connect marks 3 -> 6

Commit message: h
Parts:
- removed BT?: Battery_Cell, symbol Device:Battery_Cell
- removed C? (x3): 1u, symbol Device:C_Small
- removed C?: 4.7u, symbol Device:C_Small
- removed D? (x2): LED_Small, symbol Device:LED_Small
- removed D?: 2.6-2.8V, symbol Device:D_Zener
- removed D?: D_Shockley, Diode_THT:D_DO-15_P15.24mm_Horizontal, symbol Device:D_Shockley
- removed F1, F?: 1.5 2A, symbol Device:Fuse
- removed IC?: AP2112M-3.3TRG1, SOIC127P600X170-8N, symbol SamacSys_Parts:AP2112M-3.3TRG1
- removed IC?: MCP73834T-FCI_UN, SOP50P490X110-10N, symbol SamacSys_Parts:MCP73834T-FCI_UN
- removed Q? (x2): MCQ9435-TP, Package_SO:SOP-8_3.76x4.96mm_P1.27mm, symbol My_custom_lib:MCQ9435-TP
- removed R14, R?: <1k, symbol Device:R_Small
- removed R? (x3): 10k, symbol Device:R_Small
- removed R? (x2): 470, symbol Device:R_Small
- added D9: LED_Small, LED_SMD:LED_0603_1608Metric_Pad1.05x0.95mm_HandSolder, symbol Device:LED_Small
- added J4: Conn_01x02, Connector_PinHeader_2.54mm:PinHeader_1x02_P2.54mm_Vertical, symbol Connector_Generic:Conn_01x02
- added R36: 470, Resistor_SMD:R_0603_1608Metric_Pad0.98x0.95mm_HandSolder, symbol Device:R_Small
- added R37: 10k, Resistor_SMD:R_0603_1608Metric_Pad0.98x0.95mm_HandSolder, symbol Device:R_Small
- added RV1: R_Potentiometer, Z_mycustom_footprint_lib:2002102255, symbol Device:R_Potentiometer
- added SW3: RA12131100, Z_mycustom_footprint_lib:RA12131100, symbol My_custom_lib:RA12131100
- BT1: footprint (none) -> Connector_PinHeader_2.54mm:PinHeader_1x02_P2.54mm_Vertical
- C12, C2, C3, C4: footprint (none) -> Capacitor_SMD:C_0603_1608Metric_Pad1.08x0.95mm_HandSolder
- D2, D3: footprint (none) -> LED_SMD:LED_0603_1608Metric_Pad1.05x0.95mm_HandSolder
- IC2: footprint SOP50P490X110-10N -> SamacSys_Parts:SOP50P490X110-10N
- IC3: footprint SOIC127P600X170-8N -> SamacSys_Parts:SOIC127P600X170-8N
- R11, R12, R13, R15: footprint (none) -> Resistor_SMD:R_0603_1608Metric_Pad0.98x0.95mm_HandSolder
Connections:
- net +5V: now also C2.1, D1.2 (A), D2.2 (A), D3.2 (A), IC2.1 (VDD_1), IC2.2 (VDD_2), Q1.4 (G), R12.1
- net +VDC: now also D9.2 (A), SW3.1; no longer C4.1, IC3.5 (EN), IC3.8 (VIN)
- net GND: now also J4.2 (Pin_2), R36.2, RV1.2
- net at IC2.6 (PROG): now also RV1.3
- new net: J4.1 (Pin_1), RV1.1
- new net: C4.1, IC3.8 (VIN), R37.1, SW3.2
- new net: D9.1 (K), R36.1
- new net LOW_BATT: IC3.5 (EN), R37.2
- no-connect marks 6 -> 3
Other:
- moved on the sheet: D1, D2, D3, Q1, R12
