File: test_project_01/test_project_01.kicad_pcb (KiCad board)
At the start: 2 copper layers, 2 parts, among them IC1 ESP32-C3

Commit message: j
Parts:
- removed AE1: Antenna_Shield, RF_Antenna:Texas_SWRA117D_2.4GHz_Right
- added J1: Conn_01x02_Female, Connector_Wire:SolderWire-1sqmm_1x02_P5.4mm_D1.4mm_OD2.7mm, F.Cu at (54.3, 41.0)
- added J4: Conn_01x02_Female, Connector_Wire:SolderWire-1sqmm_1x02_P5.4mm_D1.4mm_OD2.7mm, F.Cu at (54.3, 36.2)
- added J6: Conn_01x02_Female, Connector_Wire:SolderWire-0.75sqmm_1x02_P4.8mm_D1.25mm_OD2.3mm, F.Cu at (64.8, 36.1)
- added U1: LM7171xIM, Package_SO:SOIC-8_3.9x4.9mm_P1.27mm, F.Cu at (55.9, 46.6)
- added U2: LM7171xIM, Package_SO:SOIC-8_3.9x4.9mm_P1.27mm, F.Cu at (66.6, 41.6)
- moved IC1 16.6 mm to (55.4, 57.7), turned to 0 degrees

Commit message: v
Parts:
- added U3: ESP32-C3-MINI-1, Espressif:ESP32-C3-MINI-1_Hand-Soldering, F.Cu at (110.2, 55.4)
- added U4: MCP73831-2-OT, Package_TO_SOT_SMD:SOT-23-5, F.Cu at (134.4, 54.0)
- added U5: IFX27001TFV33, Package_TO_SOT_SMD:TO-252-3_TabPin2, F.Cu at (137.9, 47.8)

Commit message: f
Parts:
- removed U5: IFX27001TFV33, Package_TO_SOT_SMD:TO-252-3_TabPin2
- added D1: D_Shockley, Diode_THT:D_DO-15_P15.24mm_Horizontal, F.Cu at (94.9, 43.1)
- added FB1: HI1806T600R-10, SamacSys_Parts:BEADC4516X185N, F.Cu at (128.9, 68.0)
- added FB2: HI1806T600R-10, SamacSys_Parts:BEADC4516X185N, F.Cu at (83.7, 99.5)
- added IC2: MCP73834T-FCI_UN, SamacSys_Parts:SOP50P490X110-10N, F.Cu at (116.5, 68.5)
- added IC3: AP2112M-3.3TRG1, SamacSys_Parts:SOIC127P600X170-8N, F.Cu at (108.6, 69.5)
- added IC4: FT260S-U, SamacSys_Parts:SOP65P640X120-28N, F.Cu at (49.2, 59.2)
- added IC5: INA2181A4QDGSRQ1, SamacSys_Parts:SOP50P490X110-10N, F.Cu at (96.6, 63.7)
- added J8: MEM2051-00-195-00-A, SamacSys_Parts:MEM20510019500A, F.Cu at (78.4, 49.9)
- added Q1: MCQ9435-TP, Package_SO:SOP-8_3.76x4.96mm_P1.27mm, F.Cu at (97.2, 48.9)
- added S1: DS01C-254-S-08BE, SamacSys_Parts:DS01C254S08BE, F.Cu at (48.3, 50.8)
- IC1: value ESP32-C3 -> STM32L010K4T6; footprint SamacSys_Parts:QFN50P500X500X90-33N-D -> SamacSys_Parts:QFP80P900X900X160-32N
- U4: value MCP73831-2-OT -> iqs625; footprint Package_TO_SOT_SMD:SOT-23-5 -> Package_SO:TSSOP-8_4.4x3mm_P0.65mm
- moved U4 76.8 mm to (58.0, 61.7)
- moved IC1 56.5 mm to (92.6, 100.2)
- moved J1 43.3 mm to (72.0, 80.5)
- moved J4 43.3 mm to (72.0, 75.7)
- moved J6 43.3 mm to (82.4, 75.6)
- moved U1 43.3 mm to (73.6, 86.1)
- moved U2 43.3 mm to (84.2, 81.1)
- moved U3 43.3 mm to (127.9, 94.9)
Connections:
- IC1 pad 1: Net-(AE1-Pad1) -> +3V3
- IC1 pad 16: unconnected-(IC1-Pad16) -> GND
- IC1 pad 17: unconnected-(IC1-Pad17) -> +3V3
- IC1 pad 32: unconnected-(IC1-Pad32) -> GND
- IC1 pad 5: unconnected-(IC1-Pad5) -> +3.3VA
- U4 pad 2: GND -> unconnected-(U4-Pad2)
- U4 pad 3: +BATT -> unconnected-(U4-Pad3)
- U4 pad 4: Net-(D1-Pad2) -> unconnected-(U4-Pad4)
- U4 pad 5: Net-(R11-Pad1) -> unconnected-(U4-Pad5)

Commit message: d
Parts:
- removed FB2: HI1806T600R-10, SamacSys_Parts:BEADC4516X185N
- removed IC1: STM32L010K4T6, SamacSys_Parts:QFP80P900X900X160-32N
- removed IC4: FT260S-U, SamacSys_Parts:SOP65P640X120-28N
- removed U2: LM7171xIM, Package_SO:SOIC-8_3.9x4.9mm_P1.27mm
- added J10: Conn_02x10_Odd_Even, Connector_PinHeader_2.54mm:PinHeader_2x10_P2.54mm_Vertical, F.Cu at (147.1, 116.5)
- added J9: STX-3120-5B, SamacSys_Parts:STX31205B, F.Cu at (205.7, 149.9)
- added U6: D1213A-02SM, Package_TO_SOT_SMD:SOT-23-5, F.Cu at (264.2, 81.3)
- added U7: Adafruit_MAX98357, Z_mycustom_footprint_lib:Adafruit MAX98357 I2S Class-D Mono, F.Cu at (233.7, 132.1)
- U1: value LM7171xIM -> LM2902; footprint Package_SO:SOIC-8_3.9x4.9mm_P1.27mm -> Package_SO:SOIC-14_3.9x8.7mm_P1.27mm
- moved D1 140.0 mm to (232.0, 71.0)
- moved J1 140.0 mm to (209.2, 108.4)
- moved J4 140.0 mm to (209.2, 103.6)
- moved J8 140.0 mm to (215.6, 77.9)
- moved FB1 140.0 mm to (266.1, 95.9)
- moved IC2 140.0 mm to (253.6, 96.4)
- moved IC3 140.0 mm to (245.7, 97.4)
- moved IC5 140.0 mm to (233.7, 91.6)
- moved J6 140.0 mm to (219.6, 103.5)
- moved Q1 140.0 mm to (234.4, 76.8)
- moved S1 140.0 mm to (185.4, 78.7)
- moved U4 140.0 mm to (195.2, 89.6)
- moved U1 118.7 mm to (190.5, 106.7)
- moved U3 71.6 mm to (190.5, 129.5)
Connections:
- net /power_measurement/mini_power_out renamed /power_measurement/ext_5v
- net Net-(R2-Pad2) renamed op_amp-
- net Net-(R3-Pad2) renamed op_amp+
- IC5 pad 1: unconnected-(IC5-Pad1) -> INA218_OUT
- IC5 pad 10: unconnected-(IC5-Pad10) -> +3V3
- IC5 pad 2: unconnected-(IC5-Pad2) -> INA218_IN-
- IC5 pad 3: unconnected-(IC5-Pad3) -> INA218_IN+
- IC5 pad 4: unconnected-(IC5-Pad4) -> GND
- IC5 pad 5: unconnected-(IC5-Pad5) -> GND
- IC5 pad 6: unconnected-(IC5-Pad6) -> GND
- IC5 pad 7: unconnected-(IC5-Pad7) -> /power_measurement/source_vcc
- IC5 pad 8: unconnected-(IC5-Pad8) -> /power_measurement/load_vcc
- IC5 pad 9: unconnected-(IC5-Pad9) -> ADC_CH1
- J1 pad 1: /power_measurement/input+ -> GND
- J1 pad 2: GND -> /power_measurement/load_vcc
- J4 pad 1: /power_measurement/output+ -> GND
- J4 pad 2: GND -> /power_measurement/source_vcc
- J8 pad MP1: unconnected-(J8-PadMP1) -> GND
- J8 pad MP2: unconnected-(J8-PadMP2) -> /SD_sening
- J8 pad MP3: unconnected-(J8-PadMP3) -> GND
- J8 pad MP4: unconnected-(J8-PadMP4) -> GND
- J8 pad MP5: unconnected-(J8-PadMP5) -> GND
- J8 pad P2: unconnected-(J8-PadP2) -> /SS1
- J8 pad P3: unconnected-(J8-PadP3) -> /SPI_MOSI
- J8 pad P4: unconnected-(J8-PadP4) -> +3V3
- J8 pad P5: unconnected-(J8-PadP5) -> /SPI_CLK
- J8 pad P7: unconnected-(J8-PadP7) -> /SPI_MISO
- U1 pad 1: unconnected-(U1-Pad1) -> op_amp_out
- U1 pad 4: GND -> +3V3
- U1 pad 6: /power_measurement/V_sense1 -> unconnected-(U1-Pad6)
- U1 pad 7: +3V3 -> V_sense2
- U1 pad 8: unconnected-(U1-Pad8) -> V_sense1
- U3 pad 30: unconnected-(U3-Pad30) -> /RX
- U3 pad 31: unconnected-(U3-Pad31) -> /TX
- U3 pad 8: unconnected-(U3-Pad8) -> Net-(C7-Pad1)
- U4 pad 1: unconnected-(U4-Pad1) -> +3V3
- U4 pad 2: unconnected-(U4-Pad2) -> /I2C_SDA
- U4 pad 8: unconnected-(U4-Pad8) -> /I2C_CLK
Other:
- board outline added: 101.6 x 101.6 mm

Commit message: h
Parts:
- removed U4: iqs625, Package_SO:TSSOP-8_4.4x3mm_P0.65mm
- added BT1: Battery_Cell, Connector_PinHeader_2.54mm:PinHeader_1x02_P2.54mm_Vertical, F.Cu at (-6.48, 46.5)
- added C1: 1u, Capacitor_SMD:C_0603_1608Metric_Pad1.08x0.95mm_HandSolder, F.Cu at (61.0, 102.9)
- added C10: 0.1u, Capacitor_SMD:C_0603_1608Metric_Pad1.08x0.95mm_HandSolder, F.Cu at (124.2, 34.8)
- added C11: 1u, Capacitor_SMD:C_0603_1608Metric_Pad1.08x0.95mm_HandSolder, F.Cu at (178.4, 97.7)
- added C12: 1u, Capacitor_SMD:C_0603_1608Metric_Pad1.08x0.95mm_HandSolder, F.Cu at (80.7, 123.2)
- added C2: 1u, Capacitor_SMD:C_0603_1608Metric_Pad1.08x0.95mm_HandSolder, F.Cu at (83.7, 120.6)
- added C3: 4.7u, Capacitor_SMD:C_0603_1608Metric_Pad1.08x0.95mm_HandSolder, F.Cu at (88.5, 112.4)
- added C4: 1u, Capacitor_SMD:C_0603_1608Metric_Pad1.08x0.95mm_HandSolder, F.Cu at (90.2, 114.9)
- added C5: 10u, Capacitor_SMD:C_0603_1608Metric_Pad1.08x0.95mm_HandSolder, F.Cu at (190.8, 97.9)
- added C6: 0.1u, Capacitor_SMD:C_0603_1608Metric_Pad1.08x0.95mm_HandSolder, F.Cu at (192.4, 97.9)
- added C7: 1u, Capacitor_SMD:C_0603_1608Metric_Pad1.08x0.95mm_HandSolder, F.Cu at (56.6, 105.4)
- added C8: 1u, Capacitor_SMD:C_0603_1608Metric_Pad1.08x0.95mm_HandSolder, F.Cu at (67.8, 82.7)
- added C9: 0.1u, Capacitor_SMD:C_0603_1608Metric_Pad1.08x0.95mm_HandSolder, F.Cu at (133.2, 32.9)
- added D2: LED_Small, LED_SMD:LED_0603_1608Metric_Pad1.05x0.95mm_HandSolder, F.Cu at (-17.5, 50.5)
- added D3: LED_Small, LED_SMD:LED_0603_1608Metric_Pad1.05x0.95mm_HandSolder, F.Cu at (-17.5, 52.3)
- added D9: LED_Small, LED_SMD:LED_0603_1608Metric_Pad1.05x0.95mm_HandSolder, F.Cu at (309.9, 109.9)
- added J11: SS-52100-001, SamacSys_Parts:SS52100001, F.Cu at (232.5, 107.8)
- added J2: Conn_01x02_Female, Connector_BarrelJack:BarrelJack_GCT_DCJ200-10-A_Horizontal, F.Cu at (78.4, 29.1)
- added J3: Conn_01x02, Connector_PinHeader_2.54mm:PinHeader_1x02_P2.54mm_Vertical, F.Cu at (87.5, 29.4)
- added J5: 10033527-N3112MLF, SamacSys_Parts:10033527N3112MLF, F.Cu at (239.6, 72.5)
- added J7: Conn_01x10, Connector_PinHeader_2.54mm:PinHeader_1x10_P2.54mm_Vertical, F.Cu at (184.2, 90.6)
- added JP1: Jumper_3_Open, Connector_PinHeader_2.54mm:PinHeader_1x03_P2.54mm_Vertical, F.Cu at (129.9, 19.2)
- added R1: 50k, Resistor_SMD:R_0603_1608Metric_Pad0.98x0.95mm_HandSolder, F.Cu at (119.1, 27.6)
- added R10: 1, Resistor_THT:R_Axial_DIN0309_L9.0mm_D3.2mm_P15.24mm_Horizontal, F.Cu at (128.6, 35.4)
- added R11: 470, Resistor_SMD:R_0603_1608Metric_Pad0.98x0.95mm_HandSolder, F.Cu at (-14.0, 50.5)
- added R12: 10k, Resistor_SMD:R_0603_1608Metric_Pad0.98x0.95mm_HandSolder, F.Cu at (104.9, 101.2)
- added R13: 470, Resistor_SMD:R_0603_1608Metric_Pad0.98x0.95mm_HandSolder, F.Cu at (-14.0, 52.3)
- added R14: 0.05, Resistor_THT:R_Axial_DIN0309_L9.0mm_D3.2mm_P15.24mm_Horizontal, F.Cu at (56.0, 34.2)
- added R15: 10k, Resistor_SMD:R_0603_1608Metric_Pad0.98x0.95mm_HandSolder, F.Cu at (-3.56, 50.4)
- added R16: 10k, Resistor_SMD:R_0603_1608Metric_Pad0.98x0.95mm_HandSolder, F.Cu at (69.5, 85.2)
- added R17: 50k, Resistor_SMD:R_0603_1608Metric_Pad0.98x0.95mm_HandSolder, F.Cu at (128.9, 32.9)
- added R18: 50k, Resistor_SMD:R_0603_1608Metric_Pad0.98x0.95mm_HandSolder, F.Cu at (134.4, 25.3)
- added R19: 50k, Resistor_SMD:R_0603_1608Metric_Pad0.98x0.95mm_HandSolder, F.Cu at (109.5, 40.3)
- added R2: 50k, Resistor_SMD:R_0603_1608Metric_Pad0.98x0.95mm_HandSolder, F.Cu at (128.6, 40.4)
- added R20: 50k, Resistor_SMD:R_0603_1608Metric_Pad0.98x0.95mm_HandSolder, F.Cu at (133.2, 27.9)
- added R21: 10k, Resistor_SMD:R_0603_1608Metric_Pad0.98x0.95mm_HandSolder, F.Cu at (209.6, 147.3)
- added R22: 470, Resistor_SMD:R_0603_1608Metric_Pad0.98x0.95mm_HandSolder, F.Cu at (210.6, 101.9)
- added R23: 470, Resistor_SMD:R_0603_1608Metric_Pad0.98x0.95mm_HandSolder, F.Cu at (210.6, 100.3)
- added R24: 10k, Resistor_SMD:R_0603_1608Metric_Pad0.98x0.95mm_HandSolder, F.Cu at (56.6, 102.9)
- added R25: 10k, Resistor_SMD:R_0603_1608Metric_Pad0.98x0.95mm_HandSolder, F.Cu at (73.8, 82.7)
- added R26: 0.05, Resistor_THT:R_Axial_DIN0309_L9.0mm_D3.2mm_P15.24mm_Horizontal, F.Cu at (56.0, 38.9)
- added R27: 1, Resistor_THT:R_Axial_DIN0309_L9.0mm_D3.2mm_P15.24mm_Horizontal, F.Cu at (56.0, 29.4)
- added R3: 50k, Resistor_SMD:R_0603_1608Metric_Pad0.98x0.95mm_HandSolder, F.Cu at (128.6, 37.9)
- added R36: 470, Resistor_SMD:R_0603_1608Metric_Pad0.98x0.95mm_HandSolder, F.Cu at (313.4, 109.9)
- added R37: 10k, Resistor_SMD:R_0603_1608Metric_Pad0.98x0.95mm_HandSolder, F.Cu at (239.3, 118.6)
- added R4: 1M, Resistor_SMD:R_0603_1608Metric_Pad0.98x0.95mm_HandSolder, F.Cu at (105.1, 41.1)
- added R5: 0.05, Resistor_THT:R_Axial_DIN0309_L9.0mm_D3.2mm_P15.24mm_Horizontal, F.Cu at (124.2, 39.8)
- added R6: 50k, Resistor_SMD:R_0603_1608Metric_Pad0.98x0.95mm_HandSolder, F.Cu at (128.9, 27.8)
- added R7: 50k, Resistor_SMD:R_0603_1608Metric_Pad0.98x0.95mm_HandSolder, F.Cu at (133.2, 30.4)
- added R8: 50k, Resistor_SMD:R_0603_1608Metric_Pad0.98x0.95mm_HandSolder, F.Cu at (128.9, 30.4)
- added R9: 150k, Resistor_SMD:R_0603_1608Metric_Pad0.98x0.95mm_HandSolder, F.Cu at (124.2, 37.3)
- added RV1: R_Potentiometer, Z_mycustom_footprint_lib:2002102255, F.Cu at (4.10, 62.2)
- added SW2: RA12131100, Z_mycustom_footprint_lib:RA12131100, F.Cu at (66.8, 4.45)
- added SW3: RA12131100, Z_mycustom_footprint_lib:RA12131100, F.Cu at (15.4, 27.8)
- added U5: MCP3204, Package_DIP:DIP-14_W7.62mm_LongPads, F.Cu at (178.4, 135.4)
- J1: footprint Connector_Wire:SolderWire-1sqmm_1x02_P5.4mm_D1.4mm_OD2.7mm -> Connector_BarrelJack:BarrelJack_GCT_DCJ200-10-A_Horizontal
- J10: value Conn_02x10_Odd_Even -> Conn_01x10; footprint Connector_PinHeader_2.54mm:PinHeader_2x10_P2.54mm_Vertical -> Connector_PinHeader_2.54mm:PinHeader_1x10_P2.54mm_Vertical
- J4: value Conn_01x02_Female -> Conn_01x02; footprint Connector_Wire:SolderWire-1sqmm_1x02_P5.4mm_D1.4mm_OD2.7mm -> Connector_PinHeader_2.54mm:PinHeader_1x02_P2.54mm_Vertical
- moved IC2 266.2 mm to (-8.64, 50.9)
- moved J4 223.8 mm to (-10.2, 59.2), turned to 180 degrees
- moved IC5 141.0 mm to (109.3, 25.3)
- moved J6 132.3 mm to (105.4, 36.8)
- moved J1 126.4 mm to (119.6, 19.3)
- moved U1 102.3 mm to (117.8, 34.7)
- moved J9 69.1 mm to (168.9, 91.4), turned to -90 degrees
- moved J8 67.4 mm to (200.0, 143.5), turned to 180 degrees
- moved U7 65.2 mm to (172.0, 111.0), turned to 90 degrees
- moved Q1 57.9 mm to (239.3, 134.5)
- moved S1 50.4 mm to (209.8, 122.8), turned to 180 degrees
- moved D1 49.8 mm to (232.0, 120.8), turned to -90 degrees
- moved U6 42.8 mm to (228.1, 104.3), turned to 90 degrees
- moved J10 42.3 mm to (189.2, 113.3), turned to 90 degrees
- moved FB1 40.8 mm to (229.9, 114.7), turned to 180 degrees
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Connections:
- D1 pad 2: Net-(C2-Pad1) -> +5V
- FB1 pad 1: Net-(FB1-Pad1) -> VBUS
- FB1 pad 2: +5V -> Net-(F1-Pad1)
- IC2 pad 1: Net-(C2-Pad1) -> +5V
- IC2 pad 2: Net-(C2-Pad1) -> +5V
- IC3 pad 5: +VDC -> LOW_BATT
- IC3 pad 8: +VDC -> Net-(C4-Pad1)
- J1 pad 2: /power_measurement/load_vcc -> /power_measurement/source_vcc
- J10 pad 1: /TX -> /DATA_IN
- J10 pad 10: unconnected-(J10-Pad10) -> /SD_sening
- J10 pad 2: +5V -> /LRC
- J10 pad 3: /RX -> /BCLK
- J10 pad 4: GND -> /GPIO10
- J10 pad 5: unconnected-(J10-Pad5) -> /GPIO4
- J10 pad 6: unconnected-(J10-Pad6) -> /GPIO5
- J10 pad 7: unconnected-(J10-Pad7) -> /GPIO6
- J10 pad 8: unconnected-(J10-Pad8) -> /GPIO7
- J10 pad 9: unconnected-(J10-Pad9) -> /GPIO8
- J4 pad 1: GND -> Net-(J4-Pad1)
- J4 pad 2: /power_measurement/source_vcc -> GND
- J8 pad P2: /SS1 -> /SPI2_SS2
- J8 pad P3: /SPI_MOSI -> /SPI2_MOSI
- J8 pad P5: /SPI_CLK -> /SPI2_CLK
- J8 pad P7: /SPI_MISO -> /SPI2_MISO
- J9 pad 1: unconnected-(J9-Pad1) -> GND
- J9 pad 2: unconnected-(J9-Pad2) -> Net-(C11-Pad1)
- J9 pad 5: unconnected-(J9-Pad5) -> Net-(C11-Pad1)
- J9 pad MH1: unconnected-(J9-PadMH1) -> GND
- J9 pad MH2: unconnected-(J9-PadMH2) -> GND
- J9 pad MH3: unconnected-(J9-PadMH3) -> GND
- Q1 pad 4: Net-(C2-Pad1) -> +5V
- S1 pad 1: unconnected-(S1-Pad1) -> /GPIO8
- S1 pad 10: unconnected-(S1-Pad10) -> /SPI2_MOSI
- S1 pad 11: unconnected-(S1-Pad11) -> Net-(R24-Pad2)
- S1 pad 12: unconnected-(S1-Pad12) -> +3V3
- S1 pad 13: unconnected-(S1-Pad13) -> /gain
- S1 pad 14: unconnected-(S1-Pad14) -> GND
- S1 pad 15: unconnected-(S1-Pad15) -> Net-(R25-Pad2)
- S1 pad 16: unconnected-(S1-Pad16) -> GND
- S1 pad 2: unconnected-(S1-Pad2) -> /SPI2_SS1
- S1 pad 3: unconnected-(S1-Pad3) -> /GPIO7
- S1 pad 4: unconnected-(S1-Pad4) -> /SPI2_SS2
- S1 pad 5: unconnected-(S1-Pad5) -> /GPIO6
- S1 pad 6: unconnected-(S1-Pad6) -> /SPI2_MISO
- S1 pad 7: unconnected-(S1-Pad7) -> /GPIO5
- S1 pad 8: unconnected-(S1-Pad8) -> /SPI2_CLK
- S1 pad 9: unconnected-(S1-Pad9) -> /GPIO4
- U1 pad 5: unconnected-(U1-Pad5) -> Net-(R3-Pad2)
- U1 pad 6: unconnected-(U1-Pad6) -> Net-(R2-Pad2)
- U1 pad 7: V_sense2 -> ADC_CH2
- U1 pad 8: V_sense1 -> ADC_CH0
- U3 pad 12: unconnected-(U3-Pad12) -> /LRC
- U3 pad 13: unconnected-(U3-Pad13) -> /BCLK
- U3 pad 16: unconnected-(U3-Pad16) -> /GPIO10
- U3 pad 18: unconnected-(U3-Pad18) -> /GPIO4
- U3 pad 19: unconnected-(U3-Pad19) -> /GPIO5
- U3 pad 20: unconnected-(U3-Pad20) -> /GPIO6
- U3 pad 21: unconnected-(U3-Pad21) -> /GPIO7
- U3 pad 22: unconnected-(U3-Pad22) -> /GPIO8
- U3 pad 23: unconnected-(U3-Pad23) -> /SD_sening
- U3 pad 30: /RX -> Net-(R22-Pad1)
- U3 pad 31: /TX -> Net-(R23-Pad1)
- U3 pad 5: unconnected-(U3-Pad5) -> /gpio2
- U3 pad 6: unconnected-(U3-Pad6) -> /DATA_IN
- U3 pad 8: Net-(C7-Pad1) -> /reset
- U6 pad 5: +5V -> VBUS
- U7 pad 1: unconnected-(U7-Pad1) -> Net-(C11-Pad2)
- U7 pad 2: unconnected-(U7-Pad2) -> GND
- U7 pad 3: GND -> +VDC
- U7 pad 4: +VDC -> GND
- U7 pad 5: unconnected-(U7-Pad5) -> /LRC
- U7 pad 6: unconnected-(U7-Pad6) -> /BCLK
- U7 pad 7: unconnected-(U7-Pad7) -> /DATA_IN
- U7 pad 8: unconnected-(U7-Pad8) -> /gain
- U7 pad 9: unconnected-(U7-Pad9) -> /on/off+mode
Other:
- board outline removed
