File: test_project_01/test_project_01.kicad_pcb (KiCad board)
At the start: 2 copper layers, 72 parts, among them IC2 MCP73834T-FCI_UN, IC3 AP2112M-3.3TRG1, IC5 INA2181A4QDGSRQ1, J1 Conn_01x02_Female, J10 Conn_01x10, J11 SS-52100-001, J2 Conn_01x02_Female, J3 Conn_01x02, J4 Conn_01x02, J5 10033527-N3112MLF, J6 Conn_01x02_Female, J7 Conn_01x10, J8 MEM2051-00-195-00-A, J9 STX-3120-5B, Q1 MCQ9435-TP, SW2 RA12131100, SW3 RA12131100, U1 LM2902, U3 ESP32-C3-MINI-1, U5 MCP3204, U6 D1213A-02SM, U7 Adafruit_MAX98357

Commit message: r
Parts:
- removed BT1: Battery_Cell, Connector_PinHeader_2.54mm:PinHeader_1x02_P2.54mm_Vertical
- removed D9: LED_Small, LED_SMD:LED_0603_1608Metric_Pad1.05x0.95mm_HandSolder
- removed R36: 470, Resistor_SMD:R_0603_1608Metric_Pad0.98x0.95mm_HandSolder
- removed R37: 10k, Resistor_SMD:R_0603_1608Metric_Pad0.98x0.95mm_HandSolder
- removed SW3: RA12131100, Z_mycustom_footprint_lib:RA12131100
- added C13: 22u, Capacitor_THT:CP_Radial_D5.0mm_P2.00mm, F.Cu at (-47.6, 41.0)
- added C14: 22p optional, Capacitor_SMD:C_0603_1608Metric_Pad1.08x0.95mm_HandSolder, F.Cu at (-41.7, 45.8)
- added C15: 22u, Capacitor_THT:CP_Radial_D5.0mm_P2.00mm, F.Cu at (-39.6, 34.7)
- added C16: 22u, Capacitor_THT:CP_Radial_D5.0mm_P2.00mm, F.Cu at (-41.0, 41.3)
- added D4: LED_Small Green, LED_SMD:LED_0603_1608Metric_Pad1.05x0.95mm_HandSolder, F.Cu at (-33.7, -15.2)
- added D5: LED_Small Green, LED_SMD:LED_0603_1608Metric_Pad1.05x0.95mm_HandSolder, F.Cu at (-47.7, -4.22)
- added D6: LED_Small Green, LED_SMD:LED_0603_1608Metric_Pad1.05x0.95mm_HandSolder, F.Cu at (-47.7, -1.63)
- added F1: 1.5 A, Fuse:Fuse_0603_1608Metric_Pad1.05x0.95mm_HandSolder, F.Cu at (80.1, -44.5)
- added IC1: XRA1203IG24TR-F, SamacSys_Parts:SOP65P640X120-24N, F.Cu at (73.4, -41.0)
- added J12: Conn_02x05_Odd_Even, Connector_PinHeader_2.54mm:PinHeader_2x05_P2.54mm_Vertical, F.Cu at (-47.6, 7.61)
- added J13: Conn_01x03, Connector_PinHeader_2.54mm:PinHeader_1x03_P2.54mm_Vertical, F.Cu at (-28.5, -19.3)
- added L1: NRH3012T2R2MN 2,2uH, SamacSys_Parts:NRH3012T220MNV, F.Cu at (-46.9, 47.3)
- added R28: 10k, Resistor_SMD:R_0603_1608Metric_Pad0.98x0.95mm_HandSolder, F.Cu at (-47.8, 0.92)
- added R29: 4.7k, Resistor_THT:R_Axial_DIN0204_L3.6mm_D1.6mm_P2.54mm_Vertical, F.Cu at (-39.9, -14.9)
- added R30: 10k+ pullup, Resistor_SMD:R_0603_1608Metric_Pad0.98x0.95mm_HandSolder, F.Cu at (-39.3, -12.1)
- added R31: 330, Resistor_SMD:R_0603_1608Metric_Pad0.98x0.95mm_HandSolder, F.Cu at (-43.4, -4.26)
- added R32: 330, Resistor_SMD:R_0603_1608Metric_Pad0.98x0.95mm_HandSolder, F.Cu at (-43.4, -1.75)
- added RR1: R_Small, Resistor_THT:R_Axial_DIN0204_L3.6mm_D1.6mm_P5.08mm_Horizontal, F.Cu at (-48.5, 33.0)
- added RR2: R_Small, Resistor_THT:R_Axial_DIN0204_L3.6mm_D1.6mm_P5.08mm_Horizontal, F.Cu at (-48.5, 36.2)
- added S2: EG1224 SPDT switch, SamacSys_Parts:EG1224, F.Cu at (36.0, -41.6)
- added U2: 1043, SamacSys_Parts:1043, F.Cu at (-44.6, -33.7)
- added U4: APX810S05, Package_TO_SOT_SMD:SOT-23, F.Cu at (-47.5, -7.74)
- added U8: DIO6012BCST6, Package_TO_SOT_SMD:SOT-23-6_Handsoldering, F.Cu at (-32.4, 33.8)
- added U9: LM324A, Package_SO:SOIC-14_3.9x8.7mm_P1.27mm, F.Cu at (-38.5, 10.4)
- C12, C4: footprint Capacitor_SMD:C_0603_1608Metric_Pad1.08x0.95mm_HandSolder -> Capacitor_SMD:C_0805_2012Metric_Pad1.18x1.45mm_HandSolder
- Q1: value MCQ9435-TP -> DMG9933USD-13; footprint Package_SO:SOP-8_3.76x4.96mm_P1.27mm -> SamacSys_Parts:SOIC127P600X175-8N
- moved IC3 315.5 mm to (-45.7, -13.2), turned to 0 degrees
- moved D1 313.0 mm to (-48.0, -19.0), turned to 0 degrees
- moved Q1 258.1 mm to (35.8, -24.3)
- moved C4 181.3 mm to (-42.7, -8.46)
- moved R12 179.1 mm to (-35.0, -10.7)
- moved C12 177.3 mm to (-23.7, -20.1)
- moved C1 74.3 mm to (24.7, 38.1)
- moved C3 74.3 mm to (52.2, 47.5)
- moved C7 74.3 mm to (20.3, 40.6)
- moved R16 74.3 mm to (33.2, 20.3)
- moved R24 74.3 mm to (20.3, 38.1)
- moved R25 74.3 mm to (37.5, 17.8)
- moved C2 74.3 mm to (47.5, 55.7)
- moved C8 74.3 mm to (31.5, 17.8)
Connections:
- C12 pad 1: +3V3 -> /Power-IN-OUT-BMS/lin_reg
- C4 pad 1: Net-(C4-Pad1) -> +VDC
- IC3 pad 1: +3V3 -> /Power-IN-OUT-BMS/lin_reg
- IC3 pad 5: LOW_BATT -> 3v3_enable
- IC3 pad 8: Net-(C4-Pad1) -> +VDC
- Q1 pad 1: +VDC -> +BATT
- Q1 pad 2: +VDC -> Net-(Q1-Pad2)
- Q1 pad 5: +BATT -> /Power-IN-OUT-BMS/Drains
- Q1 pad 6: +BATT -> /Power-IN-OUT-BMS/Drains
- Q1 pad 7: +BATT -> /Power-IN-OUT-BMS/Drains
- Q1 pad 8: +BATT -> /Power-IN-OUT-BMS/Drains
- R12 pad 1: +5V -> GND
- R12 pad 2: GND -> Net-(Q1-Pad2)

Commit message: h
Parts:
- removed J1: Conn_01x02_Female, Connector_BarrelJack:BarrelJack_GCT_DCJ200-10-A_Horizontal
- removed J7: Conn_01x10, Connector_PinHeader_2.54mm:PinHeader_1x10_P2.54mm_Vertical
- removed SW2: RA12131100, Z_mycustom_footprint_lib:RA12131100
- removed U1: LM2902, Package_SO:SOIC-14_3.9x8.7mm_P1.27mm
- added J16: Conn_01x03, Connector_PinSocket_2.54mm:PinSocket_1x03_P2.54mm_Vertical, F.Cu at (484.4, 27.3)
- added J17: Conn_01x02, TestPoint:TestPoint_2Pads_Pitch5.08mm_Drill1.3mm, F.Cu at (493.1, 15.1)
- J10: value Conn_01x10 -> Conn_01x02; footprint Connector_PinHeader_2.54mm:PinHeader_1x10_P2.54mm_Vertical -> TestPoint:TestPoint_2Pads_Pitch5.08mm_Drill1.3mm
- J12: value Conn_02x05_Odd_Even -> Conn_01x03; footprint Connector_PinHeader_2.54mm:PinHeader_2x05_P2.54mm_Vertical -> Connectors:SCREWTERMINAL-5MM-3
- J2: value Conn_01x02_Female -> Conn_01x02; footprint Connector_BarrelJack:BarrelJack_GCT_DCJ200-10-A_Horizontal -> TestPoint:TestPoint_2Pads_Pitch5.08mm_Drill1.3mm
- J6: value Conn_01x02_Female -> Conn_01x03; footprint Connector_Wire:SolderWire-0.75sqmm_1x02_P4.8mm_D1.25mm_OD2.3mm -> Connectors:SCREWTERMINAL-5MM-3
- R1, R17, R2, R20: value 50k -> 10k
- R10: value 1 -> 1ohm 3W; footprint Resistor_THT:R_Axial_DIN0309_L9.0mm_D3.2mm_P15.24mm_Horizontal -> Resistor_THT:R_Axial_DIN0207_L6.3mm_D2.5mm_P15.24mm_Horizontal
- R14: value 0.05 -> 1ohm 3W; footprint Resistor_THT:R_Axial_DIN0309_L9.0mm_D3.2mm_P15.24mm_Horizontal -> Resistor_THT:R_Axial_DIN0207_L6.3mm_D2.5mm_P15.24mm_Horizontal
- R18: value 50k -> 1ohm 3W; footprint Resistor_SMD:R_0603_1608Metric_Pad0.98x0.95mm_HandSolder -> Resistor_THT:R_Axial_DIN0207_L6.3mm_D2.5mm_P15.24mm_Horizontal
- R19: value 50k -> 0.5ohm 2W; footprint Resistor_SMD:R_0603_1608Metric_Pad0.98x0.95mm_HandSolder -> Resistor_THT:R_Axial_DIN0207_L6.3mm_D2.5mm_P15.24mm_Horizontal
- R26: value 0.05 -> 10k; footprint Resistor_THT:R_Axial_DIN0309_L9.0mm_D3.2mm_P15.24mm_Horizontal -> Resistor_SMD:R_0603_1608Metric_Pad0.98x0.95mm_HandSolder
- R27: value 1 -> 10k; footprint Resistor_THT:R_Axial_DIN0309_L9.0mm_D3.2mm_P15.24mm_Horizontal -> Resistor_SMD:R_0603_1608Metric_Pad0.98x0.95mm_HandSolder
- R3: value 50k -> 4k
- R4: value 1M -> 40k
- R5: value 0.05 -> 400k; footprint Resistor_THT:R_Axial_DIN0309_L9.0mm_D3.2mm_P15.24mm_Horizontal -> Resistor_SMD:R_0603_1608Metric_Pad0.98x0.95mm_HandSolder
- R6: value 50k -> 1k
- R7, R8: value 50k -> 100k
- R9: value 150k -> 0.5ohm 2W; footprint Resistor_SMD:R_0603_1608Metric_Pad0.98x0.95mm_HandSolder -> Resistor_THT:R_Axial_DIN0207_L6.3mm_D2.5mm_P15.24mm_Horizontal
- moved J12 506.0 mm to (458.1, 26.3)
- moved C14 475.5 mm to (433.7, 37.7)
- moved C15 475.5 mm to (435.8, 26.7)
- moved L1 475.5 mm to (428.5, 39.3)
- moved RR1 475.5 mm to (426.9, 25.0)
- moved RR2 475.5 mm to (426.9, 28.1)
- moved U8 475.5 mm to (443.0, 25.7)
- moved C13 475.5 mm to (427.8, 33.0)
- moved C16 475.5 mm to (434.4, 33.2)
- moved C4 454.5 mm to (409.7, 35.0)
- moved R28 445.3 mm to (394.9, 48.8)
- moved C7 444.3 mm to (462.4, 85.2)
- moved R31 432.9 mm to (386.2, 48.8)
- moved R32 432.9 mm to (386.2, 51.3)
- moved U9 427.3 mm to (380.8, 92.4)
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Connections:
- C10 pad 1: +3V3 -> GND
- C10 pad 2: GND -> +3V3
- IC5 pad 7: /power_measurement/source_vcc -> /POWER_MEASUREMENTS/mini_power_source
- IC5 pad 8: /power_measurement/load_vcc -> /POWER_MEASUREMENTS/mini_power_load
- J10 pad 1: /DATA_IN -> GND
- J10 pad 2: /LRC -> /POWER_MEASUREMENTS/load_vcc
- J12 pad 1: +3V3 -> unconnected-(J12-Pad1)
- J12 pad 2: +3V3 -> GND
- J12 pad 3: GND -> unconnected-(J12-Pad3)
- J2 pad 2: /power_measurement/source_vcc -> /POWER_MEASUREMENTS/source_vcc
- J3 pad 1: /power_measurement/mini_power_source -> /POWER_MEASUREMENTS/mini_power_source
- J5 pad 1: /power_measurement/ext_5v -> /POWER_MEASUREMENTS/ext_5v
- J6 pad 1: /power_measurement/ext_5v -> /POWER_MEASUREMENTS/source_vcc
- JP1 pad 2: /power_measurement/mini_power_source -> /POWER_MEASUREMENTS/mini_power_source
- JP1 pad 3: /power_measurement/ext_5v -> /POWER_MEASUREMENTS/ext_5v
- R1 pad 1: ADC_CH2 -> ADC_CH3
- R1 pad 2: GND -> Net-(U9-Pad5)
- R10 pad 1: /power_measurement/mini_power_source -> /POWER_MEASUREMENTS/load_vcc
- R10 pad 2: Net-(J3-Pad2) -> Net-(J16-Pad2)
- R14 pad 1: Net-(R14-Pad1) -> Net-(J16-Pad2)
- R14 pad 2: /power_measurement/load_vcc -> /POWER_MEASUREMENTS/load_vcc
- R17 pad 2: /power_measurement/mini_power_source -> /POWER_MEASUREMENTS/mini_power_source
- R18 pad 1: /power_measurement/mini_power_load -> Net-(J3-Pad2)
- R18 pad 2: Net-(R18-Pad2) -> /POWER_MEASUREMENTS/mini_power_source
- R19 pad 1: ADC_CH3 -> /POWER_MEASUREMENTS/mini_power_load
- R19 pad 2: Net-(R17-Pad1) -> Net-(J3-Pad2)
- R2 pad 1: ADC_CH2 -> Net-(U9-Pad6)
- R2 pad 2: Net-(R2-Pad2) -> GND
- R20 pad 1: Net-(R18-Pad2) -> ADC_CH0
- R20 pad 2: GND -> Net-(R17-Pad1)
- R26 pad 1: Net-(R14-Pad1) -> Net-(U9-Pad9)
- R26 pad 2: /power_measurement/load_vcc -> GND
- R27 pad 1: Net-(J3-Pad2) -> GND
- R27 pad 2: /power_measurement/mini_power_load -> Net-(U9-Pad9)
- R3 pad 1: GND -> Net-(J15-Pad2)
- R3 pad 2: Net-(R3-Pad2) -> Net-(U9-Pad2)
- R4 pad 1: Net-(R3-Pad2) -> Net-(J15-Pad4)
- R4 pad 2: /power_measurement/source_vcc -> Net-(U9-Pad2)
- R5 pad 1: /power_measurement/source_vcc -> Net-(J15-Pad6)
- R5 pad 2: /power_measurement/load_vcc -> Net-(U9-Pad2)
- R6 pad 1: ADC_CH0 -> GND
- R6 pad 2: GND -> Net-(U9-Pad2)
- R7 pad 1: ADC_CH0 -> Net-(U9-Pad5)
- R7 pad 2: Net-(R7-Pad2) -> /POWER_MEASUREMENTS/source_vcc
- R8 pad 2: Net-(R8-Pad2) -> Net-(U9-Pad6)
- R9 pad 1: Net-(R8-Pad2) -> /POWER_MEASUREMENTS/source_vcc
- R9 pad 2: /power_measurement/mini_power_source -> /POWER_MEASUREMENTS/load_vcc
- S1 pad 1: /GPIO8 -> unconnected-(S1-Pad1)
- S1 pad 10: /SPI2_MOSI -> unconnected-(S1-Pad10)
- S1 pad 2: /SPI2_SS1 -> unconnected-(S1-Pad2)
- S1 pad 3: /GPIO7 -> unconnected-(S1-Pad3)
- S1 pad 4: /SPI2_SS2 -> unconnected-(S1-Pad4)
- S1 pad 5: /GPIO6 -> unconnected-(S1-Pad5)
- S1 pad 6: /SPI2_MISO -> unconnected-(S1-Pad6)
- S1 pad 7: /GPIO5 -> unconnected-(S1-Pad7)
- S1 pad 8: /SPI2_CLK -> unconnected-(S1-Pad8)
- S1 pad 9: /GPIO4 -> unconnected-(S1-Pad9)
- U3 pad 12: /LRC -> /GPIO0
- U3 pad 13: /BCLK -> /GPIO1
- U3 pad 23: /SD_sening -> /GPIO9
- U3 pad 5: /gpio2 -> /GPIO2
- U3 pad 6: /DATA_IN -> /GPIO3
- U9 pad 1: unconnected-(U9-Pad1) -> ADC_CH2
- U9 pad 10: unconnected-(U9-Pad10) -> Net-(R17-Pad1)
- U9 pad 11: unconnected-(U9-Pad11) -> GND
- U9 pad 2: unconnected-(U9-Pad2) -> Net-(U9-Pad2)
- U9 pad 3: unconnected-(U9-Pad3) -> /POWER_MEASUREMENTS/source_vcc
- U9 pad 4: unconnected-(U9-Pad4) -> +3V3
- U9 pad 5: unconnected-(U9-Pad5) -> Net-(U9-Pad5)
- U9 pad 6: unconnected-(U9-Pad6) -> Net-(U9-Pad6)
- U9 pad 7: unconnected-(U9-Pad7) -> ADC_CH3
- U9 pad 8: unconnected-(U9-Pad8) -> ADC_CH0
- U9 pad 9: unconnected-(U9-Pad9) -> Net-(U9-Pad9)

Commit message: f
Parts:
- removed C1, C11, C2, C7, C8: 1u, Capacitor_SMD:C_0603_1608Metric_Pad1.08x0.95mm_HandSolder
- removed C10, C6, C9: 0.1u, Capacitor_SMD:C_0603_1608Metric_Pad1.08x0.95mm_HandSolder
- removed C12, C4: 1u, Capacitor_SMD:C_0805_2012Metric_Pad1.18x1.45mm_HandSolder
- removed C13, C15, C16: 22u, Capacitor_THT:CP_Radial_D5.0mm_P2.00mm
- removed C14: 22p optional, Capacitor_SMD:C_0603_1608Metric_Pad1.08x0.95mm_HandSolder
- removed C3: 4.7u, Capacitor_SMD:C_0603_1608Metric_Pad1.08x0.95mm_HandSolder
- removed C5: 10u, Capacitor_SMD:C_0603_1608Metric_Pad1.08x0.95mm_HandSolder
- removed D1: D_Shockley, Diode_THT:D_DO-15_P15.24mm_Horizontal
- removed D2, D3: LED_Small, LED_SMD:LED_0603_1608Metric_Pad1.05x0.95mm_HandSolder
- removed D4, D5, D6: LED_Small Green, LED_SMD:LED_0603_1608Metric_Pad1.05x0.95mm_HandSolder
- removed F1: 1.5 A, Fuse:Fuse_0603_1608Metric_Pad1.05x0.95mm_HandSolder
- removed FB1: HI1806T600R-10, SamacSys_Parts:BEADC4516X185N
- removed IC1: XRA1203IG24TR-F, SamacSys_Parts:SOP65P640X120-24N
- removed IC2: MCP73834T-FCI_UN, SamacSys_Parts:SOP50P490X110-10N
- removed IC3: AP2112M-3.3TRG1, SamacSys_Parts:SOIC127P600X170-8N
- removed IC5: INA2181A4QDGSRQ1, SamacSys_Parts:SOP50P490X110-10N
- removed J10, J17, J2: Conn_01x02, TestPoint:TestPoint_2Pads_Pitch5.08mm_Drill1.3mm
- removed J11: SS-52100-001, SamacSys_Parts:SS52100001
- removed J12, J6: Conn_01x03, Connectors:SCREWTERMINAL-5MM-3
- removed J13: Conn_01x03, Connector_PinHeader_2.54mm:PinHeader_1x03_P2.54mm_Vertical
- removed J16: Conn_01x03, Connector_PinSocket_2.54mm:PinSocket_1x03_P2.54mm_Vertical
- removed J3, J4: Conn_01x02, Connector_PinHeader_2.54mm:PinHeader_1x02_P2.54mm_Vertical
- removed J5: 10033527-N3112MLF, SamacSys_Parts:10033527N3112MLF
- removed J8: MEM2051-00-195-00-A, SamacSys_Parts:MEM20510019500A
- removed J9: STX-3120-5B, SamacSys_Parts:STX31205B
- removed JP1: Jumper_3_Open, Connector_PinHeader_2.54mm:PinHeader_1x03_P2.54mm_Vertical
- removed L1: NRH3012T2R2MN 2,2uH, SamacSys_Parts:NRH3012T220MNV
- removed Q1: DMG9933USD-13, SamacSys_Parts:SOIC127P600X175-8N
- removed R1, R12, R15, R16, R17, R2, R20, R21, R24, R25, R26, R27, R28: 10k, Resistor_SMD:R_0603_1608Metric_Pad0.98x0.95mm_HandSolder
- removed R10, R14, R18: 1ohm 3W, Resistor_THT:R_Axial_DIN0207_L6.3mm_D2.5mm_P15.24mm_Horizontal
- removed R11, R13, R22, R23: 470, Resistor_SMD:R_0603_1608Metric_Pad0.98x0.95mm_HandSolder
- removed R19, R9: 0.5ohm 2W, Resistor_THT:R_Axial_DIN0207_L6.3mm_D2.5mm_P15.24mm_Horizontal
- removed R29: 4.7k, Resistor_THT:R_Axial_DIN0204_L3.6mm_D1.6mm_P2.54mm_Vertical
- removed R3: 4k, Resistor_SMD:R_0603_1608Metric_Pad0.98x0.95mm_HandSolder
- removed R30: 10k+ pullup, Resistor_SMD:R_0603_1608Metric_Pad0.98x0.95mm_HandSolder
- removed R31, R32: 330, Resistor_SMD:R_0603_1608Metric_Pad0.98x0.95mm_HandSolder
- removed R4: 40k, Resistor_SMD:R_0603_1608Metric_Pad0.98x0.95mm_HandSolder
- removed R5: 400k, Resistor_SMD:R_0603_1608Metric_Pad0.98x0.95mm_HandSolder
- removed R6: 1k, Resistor_SMD:R_0603_1608Metric_Pad0.98x0.95mm_HandSolder
- removed R7, R8: 100k, Resistor_SMD:R_0603_1608Metric_Pad0.98x0.95mm_HandSolder
- removed RR1, RR2: R_Small, Resistor_THT:R_Axial_DIN0204_L3.6mm_D1.6mm_P5.08mm_Horizontal
- removed RV1: R_Potentiometer, Z_mycustom_footprint_lib:2002102255
- removed S1: DS01C-254-S-08BE, SamacSys_Parts:DS01C254S08BE
- removed S2: EG1224 SPDT switch, SamacSys_Parts:EG1224
- removed U2: 1043, SamacSys_Parts:1043
- removed U3: ESP32-C3-MINI-1, Espressif:ESP32-C3-MINI-1_Hand-Soldering
- removed U4: APX810S05, Package_TO_SOT_SMD:SOT-23
- removed U5: MCP3204, Package_DIP:DIP-14_W7.62mm_LongPads
- removed U6: D1213A-02SM, Package_TO_SOT_SMD:SOT-23-5
- removed U7: Adafruit_MAX98357, Z_mycustom_footprint_lib:Adafruit MAX98357 I2S Class-D Mono
- removed U8: DIO6012BCST6, Package_TO_SOT_SMD:SOT-23-6_Handsoldering
- removed U9: LM324A, Package_SO:SOIC-14_3.9x8.7mm_P1.27mm
- added C101: 10u, Capacitor_SMD:C_0603_1608Metric_Pad1.08x0.95mm_HandSolder, F.Cu at (232.2, 101.7)
- added C102: 1u, Capacitor_SMD:C_0603_1608Metric_Pad1.08x0.95mm_HandSolder, F.Cu at (248.7, 97.7)
- added C103: 10u, Capacitor_SMD:C_0603_1608Metric_Pad1.08x0.95mm_HandSolder, F.Cu at (263.1, 82.7)
- added C104: 0.1u, Capacitor_SMD:C_0603_1608Metric_Pad1.08x0.95mm_HandSolder, F.Cu at (240.9, 106.7)
- added C105: 0.1u, Capacitor_SMD:C_0603_1608Metric_Pad1.08x0.95mm_HandSolder, F.Cu at (240.9, 101.7)
- added C106: 10u, Capacitor_SMD:C_0603_1608Metric_Pad1.08x0.95mm_HandSolder, F.Cu at (267.9, 80.2)
- added C107: 1u, Capacitor_SMD:C_0603_1608Metric_Pad1.08x0.95mm_HandSolder, F.Cu at (240.9, 104.2)
- added C201: 0.1u, Capacitor_SMD:C_0603_1608Metric_Pad1.08x0.95mm_HandSolder, F.Cu at (288.5, 102.9)
- added C202: 1u, Capacitor_SMD:C_0603_1608Metric_Pad1.08x0.95mm_HandSolder, F.Cu at (301.7, 121.2)
- added C203: 0.1u, Capacitor_SMD:C_0603_1608Metric_Pad1.08x0.95mm_HandSolder, F.Cu at (300.2, 113.7)
- added C301: 1u, Capacitor_SMD:C_0603_1608Metric_Pad1.08x0.95mm_HandSolder, F.Cu at (267.8, 44.8)
- added C302: 4.7u, Capacitor_SMD:C_0603_1608Metric_Pad1.08x0.95mm_HandSolder, F.Cu at (272.1, 42.3)
- added C303: 1u, Capacitor_SMD:C_0805_2012Metric_Pad1.18x1.45mm_HandSolder, F.Cu at (245.8, 49.8)
- added C304: 1u, Capacitor_SMD:C_0805_2012Metric_Pad1.18x1.45mm_HandSolder, F.Cu at (250.5, 40.1)
- added C401: 22u, Capacitor_THT:CP_Radial_D5.0mm_P2.00mm, F.Cu at (272.5, 96.8)
- added C402: 22p optional, Capacitor_SMD:C_0603_1608Metric_Pad1.08x0.95mm_HandSolder, F.Cu at (278.5, 101.5)
- added C403: 22u, Capacitor_THT:CP_Radial_D5.0mm_P2.00mm, F.Cu at (280.6, 90.5)
- added C404: 22u, Capacitor_THT:CP_Radial_D5.0mm_P2.00mm, F.Cu at (279.2, 97.0)
- added D101: LED_Small Green, LED_SMD:LED_0603_1608Metric_Pad1.05x0.95mm_HandSolder, F.Cu at (209.5, 106.3)
- added D301: LED_Small, LED_SMD:LED_0603_1608Metric_Pad1.05x0.95mm_HandSolder, F.Cu at (263.5, 39.9)
- added D302: LED_Small, LED_SMD:LED_0603_1608Metric_Pad1.05x0.95mm_HandSolder, F.Cu at (250.3, 42.9)
- added D303: D_Shockley, Diode_THT:D_DO-15_P15.24mm_Horizontal, F.Cu at (209.3, 41.1)
- added D304: LED_Small Green, LED_SMD:LED_0603_1608Metric_Pad1.05x0.95mm_HandSolder, F.Cu at (254.7, 42.9)
- added D305: LED_Small Green, LED_SMD:LED_0603_1608Metric_Pad1.05x0.95mm_HandSolder, F.Cu at (255.1, 39.9)
- added D306: LED_Small Green, LED_SMD:LED_0603_1608Metric_Pad1.05x0.95mm_HandSolder, F.Cu at (259.1, 42.5)
- added F101: 1.5 A, Fuse:Fuse_0603_1608Metric_Pad1.05x0.95mm_HandSolder, F.Cu at (264.4, 88.5)
- added FB101: HI1806T600R-10, SamacSys_Parts:BEADC4516X185N, F.Cu at (215.5, 106.5)
- added H101: MountingHole_Pad, MountingHole:MountingHole_3.2mm_M3, F.Cu at (230.1, 95.3)
- added H102: MountingHole_Pad, MountingHole:MountingHole_3.2mm_M3, F.Cu at (230.1, 87.4)
- added H103: MountingHole_Pad, MountingHole:MountingHole_3.2mm_M3, F.Cu at (238.1, 87.4)
- added H104: MountingHole_Pad, MountingHole:MountingHole_3.2mm_M3, F.Cu at (238.1, 95.3)
- added IC101: XRA1203IG24TR-F, SamacSys_Parts:SOP65P640X120-24N, F.Cu at (216.4, 100.1)
- added IC301: MCP73834T-FCI_UN, SamacSys_Parts:SOP50P490X110-10N, F.Cu at (211.0, 52.5)
- added IC302: AP2112M-3.3TRG1, SamacSys_Parts:SOIC127P600X170-8N, F.Cu at (211.5, 47.0)
- added J101: STX-3120-5B, SamacSys_Parts:STX31205B, F.Cu at (251.8, 88.7)
- added J102: SS-52100-001, SamacSys_Parts:SS52100001, F.Cu at (267.3, 64.9)
- added J103: MEM2051-00-195-00-A, SamacSys_Parts:MEM20510019500A, F.Cu at (252.6, 71.5)
- added J201: Barrel_Jack_Switch, Z_mycustom_footprint_lib:DC plug jack 5.5-2.5mm, F.Cu at (199.9, 20.1)
- added J202: Conn_01x03, Connectors:SCREWTERMINAL-5MM-3, F.Cu at (230.0, 114.7)
- added J203: Barrel_Jack_Switch, Connector_BarrelJack:BarrelJack_Wuerth_6941xx301002, F.Cu at (209.8, 10.0)
- added J204: Conn_01x03, Connectors:SCREWTERMINAL-5MM-3, F.Cu at (230.0, 123.4)
- added J206: Conn_01x03, Connector_PinSocket_2.54mm:PinSocket_1x03_P2.54mm_Vertical, F.Cu at (288.3, 116.9)
- added J207: Conn_01x03, Connector_PinSocket_2.54mm:PinSocket_1x03_P2.54mm_Vertical, F.Cu at (283.7, 116.9)
- added J208: USB_A, Connector_USB:USB_A_Molex_67643_Horizontal, F.Cu at (290.2, 43.1)
- added J209: Conn_01x02, Connector_PinSocket_2.54mm:PinSocket_1x02_P2.54mm_Vertical, F.Cu at (283.7, 126.6)
- added J210: 10033527-N3112MLF, SamacSys_Parts:10033527N3112MLF, F.Cu at (269.7, 120.6)
- added J211: Conn_01x02, TestPoint:TestPoint_2Pads_Pitch5.08mm_Drill1.3mm, F.Cu at (255.1, 124.4)
- added J212: Conn_01x02, TestPoint:TestPoint_2Pads_Pitch5.08mm_Drill1.3mm, F.Cu at (255.0, 103.1)
- added J213: Conn_01x02, Connector_PinHeader_2.54mm:PinHeader_1x02_P2.54mm_Vertical, F.Cu at (279.0, 126.6)
- added J301: Conn_01x02, Connector_PinHeader_2.54mm:PinHeader_1x02_P2.54mm_Vertical, F.Cu at (217.0, 52.5)
- added J302: Conn_01x02, Connector_PinHeader_2.54mm:PinHeader_1x02_P2.54mm_Vertical, F.Cu at (221.6, 52.5)
- added J303: Conn_01x03, Connector_PinHeader_2.54mm:PinHeader_1x03_P2.54mm_Vertical, F.Cu at (245.7, 40.9)
- added JP101: Jumper_2_Bridged, Jumper:SolderJumper-2_P1.3mm_Bridged_RoundedPad1.0x1.5mm, F.Cu at (245.2, 103.3)
- added JP201: Jumper_3_Open, Connector_PinHeader_2.54mm:PinHeader_1x03_P2.54mm_Vertical, F.Cu at (279.0, 116.9)
- added L401: NRH3012T2R2MN 2,2uH, SamacSys_Parts:NRH3012T220MNV, F.Cu at (273.2, 103.1)
- added Q301: DMG9933USD-13, SamacSys_Parts:SOIC127P600X175-8N, F.Cu at (220.0, 47.0)
- added R101: 10k, Resistor_SMD:R_0603_1608Metric_Pad0.98x0.95mm_HandSolder, F.Cu at (318.2, 41.0)
- added R102: 10k, Resistor_SMD:R_0603_1608Metric_Pad0.98x0.95mm_HandSolder, F.Cu at (232.2, 104.2)
- added R103: 10k, Resistor_SMD:R_0603_1608Metric_Pad0.98x0.95mm_HandSolder, F.Cu at (236.5, 104.2)
- added R104: 10k, Resistor_SMD:R_0603_1608Metric_Pad0.98x0.95mm_HandSolder, F.Cu at (263.6, 80.2)
- added R105: 10k, Resistor_SMD:R_0603_1608Metric_Pad0.98x0.95mm_HandSolder, F.Cu at (236.5, 106.7)
- added R106: 10k, Resistor_SMD:R_0603_1608Metric_Pad0.98x0.95mm_HandSolder, F.Cu at (282.4, 63.3)
- added R107: 10k+ pullup, Resistor_SMD:R_0603_1608Metric_Pad0.98x0.95mm_HandSolder, F.Cu at (245.2, 100.2)
- added R108: 10k, Resistor_SMD:R_0603_1608Metric_Pad0.98x0.95mm_HandSolder, F.Cu at (244.3, 97.7)
- added R109: 10k, Resistor_SMD:R_0603_1608Metric_Pad0.98x0.95mm_HandSolder, F.Cu at (232.2, 106.7)
- added R110: 10k, Resistor_SMD:R_0603_1608Metric_Pad0.98x0.95mm_HandSolder, F.Cu at (266.8, -2.94)
- added R111: 10k, Resistor_SMD:R_0603_1608Metric_Pad0.98x0.95mm_HandSolder, F.Cu at (291.6, -15.9)
- added R112: 330, Resistor_SMD:R_0603_1608Metric_Pad0.98x0.95mm_HandSolder, F.Cu at (236.5, 101.7)
- added R113: 10k, Resistor_SMD:R_0603_1608Metric_Pad0.98x0.95mm_HandSolder, F.Cu at (282.4, 65.8)
- added R201: 10k, Resistor_SMD:R_0603_1608Metric_Pad0.98x0.95mm_HandSolder, F.Cu at (272.0, 128.0)
- added R202: 100k, Resistor_SMD:R_0603_1608Metric_Pad0.98x0.95mm_HandSolder, F.Cu at (280.9, 3.76)
- added R203: 100k, Resistor_SMD:R_0603_1608Metric_Pad0.98x0.95mm_HandSolder, F.Cu at (275.5, 13.1)
- added R204: 10k, Resistor_SMD:R_0603_1608Metric_Pad0.98x0.95mm_HandSolder, F.Cu at (266.8, 13.1)
- added R205: 10k, Resistor_SMD:R_0603_1608Metric_Pad0.98x0.95mm_HandSolder, F.Cu at (280.9, 6.27)
- added R206: 100k, Resistor_SMD:R_0603_1608Metric_Pad0.98x0.95mm_HandSolder, F.Cu at (300.2, 116.2)
- added R207: 47k, Resistor_SMD:R_0603_1608Metric_Pad0.98x0.95mm_HandSolder, F.Cu at (297.3, 120.9)
- added R208: 0.5ohm 2W, Resistor_THT:R_Axial_DIN0207_L6.3mm_D2.5mm_P5.08mm_Vertical, F.Cu at (245.9, 120.0)
- added R209: 1ohm 3W, Resistor_THT:R_Axial_DIN0207_L6.3mm_D2.5mm_P5.08mm_Vertical, F.Cu at (254.7, 107.4)
- added R210: 1ohm 3W, Resistor_THT:R_Axial_DIN0207_L6.3mm_D2.5mm_P5.08mm_Vertical, F.Cu at (264.3, 112.0)
- added R211: 1M, Resistor_SMD:R_0603_1608Metric_Pad0.98x0.95mm_HandSolder, F.Cu at (288.5, 105.4)
- added R212: 1ohm 3W, Resistor_THT:R_Axial_DIN0207_L6.3mm_D2.5mm_P5.08mm_Vertical, F.Cu at (227.3, 129.3)
- added R213: 0.5ohm 2W, Resistor_THT:R_Axial_DIN0207_L6.3mm_D2.5mm_P5.08mm_Vertical, F.Cu at (245.9, 112.0)
- added R214: 10k, Resistor_SMD:R_0603_1608Metric_Pad0.98x0.95mm_HandSolder, F.Cu at (301.7, 118.7)
- added R215: 10k, Resistor_SMD:R_0603_1608Metric_Pad0.98x0.95mm_HandSolder, F.Cu at (272.0, 130.5)
- added R216: 100k, Resistor_SMD:R_0603_1608Metric_Pad0.98x0.95mm_HandSolder, F.Cu at (276.5, 3.76)
- added R217: 100k, Resistor_SMD:R_0603_1608Metric_Pad0.98x0.95mm_HandSolder, F.Cu at (271.2, 13.1)
- added R218: 10k, Resistor_SMD:R_0603_1608Metric_Pad0.98x0.95mm_HandSolder, F.Cu at (276.5, 8.78)
- added R219: 10k, Resistor_SMD:R_0603_1608Metric_Pad0.98x0.95mm_HandSolder, F.Cu at (276.5, 6.27)
- added R301: 470, Resistor_SMD:R_0603_1608Metric_Pad0.98x0.95mm_HandSolder, F.Cu at (276.5, 42.3)
- added R302: 470, Resistor_SMD:R_0603_1608Metric_Pad0.98x0.95mm_HandSolder, F.Cu at (276.5, 39.8)
- added R303: 1k, Resistor_SMD:R_0603_1608Metric_Pad0.98x0.95mm_HandSolder, F.Cu at (250.4, 47.4)
- added R304: 10k, Resistor_SMD:R_0603_1608Metric_Pad0.98x0.95mm_HandSolder, F.Cu at (272.1, 44.8)
- added R305: 10k, Resistor_SMD:R_0603_1608Metric_Pad0.98x0.95mm_HandSolder, F.Cu at (267.8, 39.8)
- added R306: 10k, Resistor_SMD:R_0603_1608Metric_Pad0.98x0.95mm_HandSolder, F.Cu at (267.8, 42.3)
- added R307: 4.7k, Resistor_THT:R_Axial_DIN0204_L3.6mm_D1.6mm_P2.54mm_Vertical, F.Cu at (208.9, 56.4)
- added R308: 330, Resistor_SMD:R_0603_1608Metric_Pad0.98x0.95mm_HandSolder, F.Cu at (272.1, 39.8)
- added R309: 330, Resistor_SMD:R_0603_1608Metric_Pad0.98x0.95mm_HandSolder, F.Cu at (263.4, 44.8)
- added RR401: R_Small, Resistor_THT:R_Axial_DIN0204_L3.6mm_D1.6mm_P5.08mm_Horizontal, F.Cu at (271.7, 88.8)
- added RR402: R_Small, Resistor_THT:R_Axial_DIN0204_L3.6mm_D1.6mm_P5.08mm_Horizontal, F.Cu at (271.7, 91.9)
- added RV301: R_Potentiometer, Z_mycustom_footprint_lib:2002102255, F.Cu at (208.6, 110.7)
- added S101: DS01C-254-S-08BE, SamacSys_Parts:DS01C254S08BE, F.Cu at (268.2, -6.89)
- added S102: DS01C-254-S-08BE, SamacSys_Parts:DS01C254S08BE, F.Cu at (210.9, 72.4)
- added S301: EG1224 SPDT switch, SamacSys_Parts:EG1224, F.Cu at (231.0, 42.7)
- added SW101: SW_SPST, SamacSys_Parts:PTS526SM15SMTR2LFS, F.Cu at (225.5, 104.3)
- added U101: ESP32-C3-MINI-1, Espressif:ESP32-C3-MINI-1_Hand-Soldering, F.Cu at (173.9, 85.9)
- added U102: LM4132xMF-3.0, Package_TO_SOT_SMD:SOT-23-5, F.Cu at (223.5, 97.6)
- added U103: MCP3204, Package_DIP:DIP-14_W7.62mm_LongPads, F.Cu at (234.1, 64.2)
- added U104: Adafruit_MAX98357, Z_mycustom_footprint_lib:Adafruit MAX98357 I2S Class-D Mono, F.Cu at (216.8, 85.8)
- added U105: D1213A-02SM, Package_TO_SOT_SMD:SOT-23-5, F.Cu at (228.9, 77.3)
- added U201: LM324A, Package_SO:SOIC-14_3.9x8.7mm_P1.27mm, F.Cu at (248.6, 127.2)
- added U301: 1043, SamacSys_Parts:1043, F.Cu at (170.5, -16.0)
- added U302: APX810S05, Package_TO_SOT_SMD:SOT-23, F.Cu at (210.1, 122.3)
- added U401: DIO6012BCST6, Package_TO_SOT_SMD:SOT-23-6_Handsoldering, F.Cu at (287.8, 89.5)
Routing:
- added copper zone on B.Cu, net GND
Other:
- board outline added: 100 x 100 mm

Commit message: r
Parts:
- removed D306: LED_Small Green, LED_SMD:LED_0603_1608Metric_Pad1.05x0.95mm_HandSolder
- removed J303: Conn_01x03, Connector_PinHeader_2.54mm:PinHeader_1x03_P2.54mm_Vertical
- removed R107: 10k+ pullup, Resistor_SMD:R_0603_1608Metric_Pad0.98x0.95mm_HandSolder
- removed R309: 330, Resistor_SMD:R_0603_1608Metric_Pad0.98x0.95mm_HandSolder
- added R114: 10k+ pulldown, Resistor_SMD:R_0603_1608Metric_Pad0.98x0.95mm_HandSolder, F.Cu at (232.4, 55.4)
- R101: value 10k -> 1k
- U301: moved to B.Cu
- moved S101 207.7 mm to (74.4, 68.1), turned to -90 degrees
- moved J101 198.9 mm to (53.2, 99.3)
- moved U401 197.9 mm to (95.6, 136.9)
- moved C403 196.5 mm to (91.9, 145.4), turned to -90 degrees
- moved J103 193.7 mm to (59.1, 79.1), turned to 90 degrees
- moved H104 189.7 mm to (55.0, 145.0)
- moved L401 186.4 mm to (90.4, 139.3), turned to -90 degrees
- moved C404 185.9 mm to (99.6, 145.3), turned to -90 degrees
- moved C401 181.4 mm to (96.8, 141.7), turned to 180 degrees
- moved C402 181.2 mm to (100.9, 138.1), turned to 180 degrees
- moved S301 180.6 mm to (82.6, 145.8), turned to 180 degrees
- moved H101 179.7 mm to (55.0, 55.0)
- moved RR401 179.4 mm to (100.0, 141.2), turned to 90 degrees
- moved IC302 175.6 mm to (65.7, 144.7), turned to 180 degrees
- moved SW101 175.2 mm to (54.4, 66.8)
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Connections:
- S102 pad 10: Net-(R107-Pad2) -> unconnected-(S102-Pad10)
- S102 pad 7: unconnected-(S102-Pad7) -> 3v3_enable
- S102 pad 8: unconnected-(S102-Pad8) -> GND
- S102 pad 9: 3v3_enable -> unconnected-(S102-Pad9)
- U102 pad 3: unconnected-(U102-Pad3) -> Net-(R101-Pad2)
Routing:
- added copper zone on F.Cu, net GND

Commit message: k
Parts:
- removed the J207 at (283.7, 116.9)
- removed the J209 at (283.7, 126.6)
- removed J213: Conn_01x02, Connector_PinHeader_2.54mm:PinHeader_1x02_P2.54mm_Vertical
- removed the J301 at (212.6, 65.2)
- removed the R202 at (246.5, 49.7)
- removed the R203 at (241.1, 59.0)
- removed the R204 at (232.4, 59.0)
- removed the R205 at (246.5, 52.2)
- removed R209, R210: 1ohm 3W, Resistor_THT:R_Axial_DIN0207_L6.3mm_D2.5mm_P5.08mm_Vertical
- removed R213: 0.5ohm 2W, Resistor_THT:R_Axial_DIN0207_L6.3mm_D2.5mm_P5.08mm_Vertical
- removed R216, R217: 100k, Resistor_SMD:R_0603_1608Metric_Pad0.98x0.95mm_HandSolder
- removed R218, R219: 10k, Resistor_SMD:R_0603_1608Metric_Pad0.98x0.95mm_HandSolder
- removed the R303 at (216.0, 93.3)
- removed U201: LM324A, Package_SO:SOIC-14_3.9x8.7mm_P1.27mm
- added C104: 100n, Capacitor_SMD:C_0603_1608Metric_Pad1.08x0.95mm_HandSolder, F.Cu at (199.8, 46.2)
- added C106: 100n, Capacitor_SMD:C_0603_1608Metric_Pad1.08x0.95mm_HandSolder, F.Cu at (204.7, 41.7)
- added C204: 1u, Capacitor_SMD:C_0603_1608Metric_Pad1.08x0.95mm_HandSolder, F.Cu at (213.3, 46.4)
- added C205: 100n, Capacitor_SMD:C_0603_1608Metric_Pad1.08x0.95mm_HandSolder, F.Cu at (213.3, 48.9)
- added FB401: FerriteBead_Small, Resistor_SMD:R_0402_1005Metric_Pad0.72x0.64mm_HandSolder, F.Cu at (201.3, 57.0)
- added IC201: INA2181A4QDGSRQ1, SamacSys_Parts:SOP50P490X110-10N, F.Cu at (214.8, 42.8)
- added R304: 10k, Resistor_SMD:R_0603_1608Metric_Pad0.98x0.95mm_HandSolder, F.Cu at (191.4, 57.3)
- added R305: 10k, Resistor_SMD:R_0603_1608Metric_Pad0.98x0.95mm_HandSolder, F.Cu at (191.4, 59.8)
- C105: renamed from C104; value 0.1u -> 100n
- C107: renamed from C105; value 0.1u -> 100n
- C203: value 0.1u -> 100n
- R204: renamed from R208; value 0.5ohm 2W -> 5m; footprint Resistor_THT:R_Axial_DIN0207_L6.3mm_D2.5mm_P5.08mm_Vertical -> Resistor_SMD:R_0612_1632Metric_Pad1.18x3.40mm_HandSolder
- R208: renamed from R212; value 1ohm 3W -> 30m; footprint Resistor_THT:R_Axial_DIN0207_L6.3mm_D2.5mm_P5.08mm_Vertical -> Resistor_SMD:R_0402_1005Metric_Pad0.72x0.64mm_HandSolder
- RV301: footprint Z_mycustom_footprint_lib:2002102255 -> Potentiometer_THT:Potentiometer_Bourns_3386F_Vertical
- U102: value LM4132xMF-3.0 -> LM4040DBZ-3; footprint Package_TO_SOT_SMD:SOT-23-5 -> Package_TO_SOT_SMD:SOT-23
- U103: value MCP3204 -> MCP3208; footprint Package_DIP:DIP-14_W7.62mm_LongPads -> Package_SO:SOIC-16_3.9x9.9mm_P1.27mm
- moved U103 100.4 mm to (193.4, 46.2), turned to 0 degrees
- moved U102 59.6 mm to (200.1, 42.7)
- renumbered C106 to C108, C107 to C109, J203 to J202, J202 to J203, J206 to J205, J208 to J206, J210 to J207, J211 to J208, J212 to J209, J302 to J301, R114 to R103, R103 to R104, R104 to R105, R105 to R106, R106 to R107, R206 to R202, R207 to R203, R211 to R205, R214 to R206, R215 to R207, R304 to R303, R305 to R306, R306 to R307, R307 to R308, R308 to R309
Connections:
- net /SD_sening renamed /SD_sense
- net Net-(Q301-Pad2) renamed /Power-IN-OUT-BMS/low_batt_shutoff
- C202 pad 1: +3V3 -> +VDC
- C203 pad 2: +3V3 -> +VDC
- C401 pad 1: +VDC -> Net-(C401-Pad1)
- IC301 pad 6: Net-(IC301-Pad6) -> /Power-IN-OUT-BMS/Set_charge_current
- R101 pad 2: Net-(R101-Pad2) -> /Vref
- R208 pad 1: Net-(J213-Pad2) -> /POWER_MEASUREMENTS/mini_power_load
- RV301 pad 3: Net-(J301-Pad2) -> /Power-IN-OUT-BMS/Set_charge_current
- U102 pad 1: unconnected-(U102-Pad1) -> /Vref
- U102 pad 3: Net-(R101-Pad2) -> (no net)
- U103 pad 10: /SPI1_MISO -> /SPI1_SS1
- U103 pad 11: /SPI1_CLK -> /SPI1_MOSI
- U103 pad 12: GND -> /SPI1_MISO
- U103 pad 13: Net-(U102-Pad5) -> /SPI1_CLK
- U103 pad 14: +VDC -> GND
- U103 pad 5: unconnected-(U103-Pad5) -> ADC_CH4
- U103 pad 7: GND -> unconnected-(U103-Pad7)
- U103 pad 8: /SPI1_SS1 -> unconnected-(U103-Pad8)
- U103 pad 9: /SPI1_MOSI -> GND
- U401 pad 4: +VDC -> Net-(C401-Pad1)
Other:
- board size 100 x 100 mm -> 18.7 x 2 mm
