File: test_project_01/test_project_01.kicad_pcb (KiCad board)
At the start: 2 copper layers, 18.7 x 2 mm, 101 parts, among them IC101 XRA1203IG24TR-F, IC201 INA2181A4QDGSRQ1, IC301 MCP73834T-FCI_UN, IC302 AP2112M-3.3TRG1, J101 STX-3120-5B, J102 SS-52100-001, J103 MEM2051-00-195-00-A, J201 Barrel_Jack_Switch, J202 Barrel_Jack_Switch, J203 Conn_01x03, J204 Conn_01x03, J205 Conn_01x03, J206 USB_A, J207 10033527-N3112MLF, J208 Conn_01x02, J209 Conn_01x02, J301 Conn_01x02, Q301 DMG9933USD-13, SW101 SW_SPST, U101 ESP32-C3-MINI-1, U102 LM4040DBZ-3, U103 MCP3208, U104 Adafruit_MAX98357, U105 D1213A-02SM, U301 1043, U302 APX810S05, U401 DIO6012BCST6

Commit message: i
Parts:
- added R201: 10k, Resistor_SMD:R_0603_1608Metric_Pad0.98x0.95mm_HandSolder, F.Cu at (202.2, 126.2)
- added R202: 10k, Resistor_SMD:R_0603_1608Metric_Pad0.98x0.95mm_HandSolder, F.Cu at (210.9, 123.7)
- added R203: 1k, Resistor_SMD:R_0603_1608Metric_Pad0.98x0.95mm_HandSolder, F.Cu at (206.5, 123.7)
- added R204: 1k, Resistor_SMD:R_0603_1608Metric_Pad0.98x0.95mm_HandSolder, F.Cu at (202.2, 128.7)
- added R205: 100k, Resistor_SMD:R_0603_1608Metric_Pad0.98x0.95mm_HandSolder, F.Cu at (202.2, 123.7)
- added R206: 100k, Resistor_SMD:R_0603_1608Metric_Pad0.98x0.95mm_HandSolder, F.Cu at (206.5, 126.2)
- added R308: 5m, Resistor_SMD:R_0612_1632Metric_Pad1.18x3.40mm_HandSolder, F.Cu at (220.7, 124.9)
- moved J209 35.4 mm to (249.2, 89.5)
- moved J210 35.4 mm to (249.1, 68.2)
- moved C201 27.6 mm to (261.1, 105.2)
- moved C203 27.6 mm to (272.7, 115.9)
- moved R209 27.6 mm to (269.9, 123.1)
- moved J206 27.6 mm to (260.8, 119.1)
- moved R208 27.6 mm to (272.7, 118.4)
- moved R211 27.6 mm to (261.1, 107.7)
- moved JP201 27.6 mm to (251.6, 119.1)
- moved R207 27.6 mm to (244.6, 130.2)
- moved R213 27.6 mm to (244.6, 132.7)
- moved R212 27.6 mm to (274.2, 120.9)
- moved C202 27.6 mm to (274.2, 123.4)
- moved U104 3.20 mm to (72.2, 99.3)
- renumbered J205 to J206, J206 to J207, J207 to J208, J208 to J209, J209 to J210, R201 to R207, R202 to R208, R203 to R209, R204 to R210, R205 to R211, R206 to R212, R207 to R213, R208 to R214, R308 to R309, R309 to R310
Connections:
- C106 pad 1: +VDC -> Power_in-
- C107 pad 2: +VDC -> Power_in-
- C108 pad 1: +VDC -> Power_in-
- C202 pad 1: +VDC -> Power_in-
- C203 pad 2: +VDC -> Power_in-
- C303 pad 1: +VDC -> Power_in-
- D303 pad 1: +VDC -> Power_in+
- FB401 pad 1: +VDC -> Power_in-
- IC302 pad 8: +VDC -> Power_in-
- Q301 pad 3: +VDC -> Power_in+
- R101 pad 1: +VDC -> Power_in-
- R103 pad 2: +VDC -> Power_in-
- U103 pad 16: +VDC -> Power_in-
- U103 pad 6: unconnected-(U103-Pad6) -> ADC_CH5
- U103 pad 7: unconnected-(U103-Pad7) -> ADC_CH6
- U104 pad 3: +VDC -> Power_in-
Other:
- board size 18.7 x 2 mm -> 100 x 100 mm

Commit message: y
Parts:
- added R105: 10k, Resistor_SMD:R_0603_1608Metric_Pad0.98x0.95mm_HandSolder, B.Cu at (59.2, 80.6)
- added R107: 10k, Resistor_SMD:R_0603_1608Metric_Pad0.98x0.95mm_HandSolder, B.Cu at (59.2, 82.1)
- added R110: 10k, Resistor_SMD:R_0603_1608Metric_Pad0.98x0.95mm_HandSolder, B.Cu at (59.2, 83.7)
- added R111: 10k, Resistor_SMD:R_0603_1608Metric_Pad0.98x0.95mm_HandSolder, B.Cu at (59.2, 85.2)
- added R112: 10k, Resistor_SMD:R_0603_1608Metric_Pad0.98x0.95mm_HandSolder, F.Cu at (82.5, 34.5)
- added R113: 10k, Resistor_SMD:R_0603_1608Metric_Pad0.98x0.95mm_HandSolder, F.Cu at (82.5, 32.9)
- added R114: 10k, Resistor_SMD:R_0603_1608Metric_Pad0.98x0.95mm_HandSolder, B.Cu at (59.2, 79.0)
- added R115: 10k, Resistor_SMD:R_0603_1608Metric_Pad0.98x0.95mm_HandSolder, B.Cu at (59.2, 86.8)
- added U201: LM324A, Package_SO:SOIC-14_3.9x8.7mm_P1.27mm, F.Cu at (117.1, 98.3)
- D303: footprint Diode_THT:D_DO-15_P15.24mm_Horizontal -> Diode_THT:D_DO-15_P5.08mm_Vertical_AnodeUp
- R309: footprint Resistor_THT:R_Axial_DIN0204_L3.6mm_D1.6mm_P2.54mm_Vertical -> Resistor_SMD:R_0805_2012Metric
- moved C103 205.8 mm to (58.3, 62.3), turned to 180 degrees
- moved C102 193.2 mm to (61.2, 51.3), turned to 180 degrees
- moved R121 190.6 mm to (56.5, 71.2), turned to 180 degrees
- moved C105 187.6 mm to (61.2, 52.8), turned to 180 degrees
- moved R102 179.3 mm to (58.3, 60.7)
- moved C101 177.4 mm to (61.2, 54.3), turned to 180 degrees
- moved R109 164.6 mm to (91.2, 110.5), turned to -90 degrees
- moved JP101 157.5 mm to (89.9, 77.6), turned to 90 degrees
- moved F101 156.3 mm to (110.3, 62.4)
- moved C202 153.6 mm to (122.8, 97.6)
- moved R116 152.4 mm to (93.8, 74.1)
- moved R119 152.1 mm to (88.5, 84.4), turned to -90 degrees
- moved C203 150.9 mm to (122.8, 99.1), turned to 180 degrees
- moved R118 150.8 mm to (90.1, 84.4), turned to 90 degrees
- moved R120 148.2 mm to (89.8, 81.3)
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- renumbered R105 to R106, R106 to R108, R107 to R109, R108 to R116, R109 to R117, R110 to R118, R111 to R119, R112 to R120, R113 to R121, R306 to R304, R307 to R305, R308 to R306, R304 to R307, R305 to R308
Connections:
- R307 pad 2: +BATT -> Power_in-
Routing:
- net +3V3: track 0.00 -> 185.8 mm, vias 0 -> 1
- net +5V: track 0.00 -> 55.6 mm, vias 0 -> 1
- net /Power-IN-OUT-BMS/buck_out: track 0.00 -> 38.2 mm
- net 3v3_enable: track 0.00 -> 34.1 mm, vias 0 -> 2
- net D-: track 0.00 -> 32.8 mm
- net D+: track 0.00 -> 30.1 mm
- net +BATT: track 0.00 -> 24.7 mm
- net /POWER_MEASUREMENTS/D2+: track 0.00 -> 24.1 mm, vias 0 -> 2
- net GND: track 0.00 -> 23.9 mm, vias 0 -> 13
- net /A1: track 0.00 -> 22.0 mm, vias 0 -> 1
- net /POWER_MEASUREMENTS/D2-: track 0.00 -> 21.7 mm
- net Net-(J101-Pad2): track 0.00 -> 21.4 mm
- net Net-(C201-Pad1): track 0.00 -> 18.3 mm
- net /SD_sense: track 0.00 -> 16.7 mm, vias 0 -> 2
- net Net-(C402-Pad2): track 0.00 -> 14.3 mm, vias 0 -> 1
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
Commit message: r
Parts:
- removed D101, D304, D305: LED_Small Green, LED_SMD:LED_0603_1608Metric_Pad1.05x0.95mm_HandSolder
- removed J206: Conn_01x03, Connector_PinSocket_2.54mm:PinSocket_1x03_P2.54mm_Vertical
- removed R120, R310: 330, Resistor_SMD:R_0603_1608Metric_Pad0.98x0.95mm_HandSolder
- removed R209: 47k, Resistor_SMD:R_0603_1608Metric_Pad0.98x0.95mm_HandSolder
- removed R309: 4.7k, Resistor_SMD:R_0805_2012Metric
- added C23: 100n, Capacitor_SMD:C_0603_1608Metric_Pad1.08x0.95mm_HandSolder, F.Cu at (97.8, 75.8)
- added D1: LED_Small Green, LED_SMD:LED_0603_1608Metric_Pad1.05x0.95mm_HandSolder, F.Cu at (113.8, 65.8)
- added D5: LED_Small Green, LED_SMD:LED_0603_1608Metric_Pad1.05x0.95mm_HandSolder, F.Cu at (88.6, 126.2)
- added D6: LED_Small Green, LED_SMD:LED_0603_1608Metric_Pad1.05x0.95mm_HandSolder, F.Cu at (86.6, 69.7)
- added F2: 1.5 A, Fuse:Fuse_0603_1608Metric_Pad1.05x0.95mm_HandSolder, F.Cu at (109.9, 110.5)
- added R20: 4.7k, Resistor_SMD:R_0805_2012Metric, F.Cu at (112.1, 67.7)
- added R44: 330, Resistor_SMD:R_0603_1608Metric_Pad0.98x0.95mm_HandSolder, F.Cu at (88.6, 124.4)
- added R45: 330, Resistor_SMD:R_0603_1608Metric_Pad0.98x0.95mm_HandSolder, F.Cu at (88.3, 69.7)
- R3: renamed from R103; value 10k+ pulldown -> 20k
- R42: renamed from R307; value 10k -> 1Meg
- R43: renamed from R308; value 10k -> 1Meg
- moved C8 180.4 mm to (88.5, 99.1), turned to -90 degrees
- moved R6 173.4 mm to (90.8, 94.7), turned to 180 degrees
- moved R3 159.9 mm to (93.2, 133.9), turned to 180 degrees
- moved C17 159.7 mm to (60.7, 148.5), turned to 180 degrees
- moved C18 158.1 mm to (69.5, 145.4), turned to 90 degrees
- moved R29 148.5 mm to (125.8, 85.6)
- moved R4 146.0 mm to (90.8, 96.3), turned to 180 degrees
- moved R28 126.3 mm to (125.9, 87.2), turned to 180 degrees
- moved R24 100.3 mm to (109.9, 96.8)
- moved R27 100.2 mm to (111.2, 94.5), turned to 0 degrees
- moved R25 88.5 mm to (110.8, 100.0), turned to 180 degrees
- moved R26 88.5 mm to (110.8, 98.4), turned to 180 degrees
- moved R13 40.2 mm to (95.6, 71.0), turned to 180 degrees
- moved R12 40.2 mm to (95.6, 72.5), turned to 180 degrees
- moved R41 15.8 mm to (111.7, 106.7)
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- renumbered C101 to C1, C201 to C10, C202 to C11, C203 to C12, C204 to C13, C205 to C14, C301 to C15, C302 to C16, C303 to C17, C304 to C18, C401 to C19, C102 to C2, C402 to C20, C403 to C21, C404 to C22, C103 to C3, C104 to C4, C105 to C5, C106 to C6, C107 to C7, C108 to C8, C109 to C9, D301 to D2, D302 to D3, D303 to D4, F101 to F1, FB101 to FB1, FB401 to FB2, H101 to H1, H102 to H2, H103 to H3, H104 to H4, IC101 to IC1, IC201 to IC2, IC301 to IC3, IC302 to IC4, J101 to J1, J208 to J10, J209 to J11, J210 to J12, J301 to J13, J102 to J2, J103 to J3, J201 to J4, J202 to J5, J203 to J6, J204 to J7, J207 to J9, JP101 to JP1, JP201 to JP2, L401 to L1, Q301 to Q1, R101 to R1, R110 to R10, R111 to R11, R112 to R12, R113 to R13, R114 to R14, R115 to R15, R116 to R16, R117 to R17, R118 to R18, R119 to R19, R102 to R2, R121 to R21, R201 to R22, R202 to R23, R203 to R24, R204 to R25, R205 to R26, R206 to R27, R207 to R28, R208 to R29, R210 to R31, R211 to R32, R212 to R33, R213 to R34, R214 to R35, R301 to R36, R302 to R37, R303 to R38, R304 to R39, R104 to R4, R305 to R40, R306 to R41, R105 to R5, R106 to R6, R107 to R7, R108 to R8, R109 to R9, RR401 to RR1, RR402 to RR2, RV301 to RV1, S101 to S1, S102 to S2, S301 to S3, SW101 to SW1, U101 to U1, U401 to U10, U102 to U2, U103 to U3, U104 to U4, U105 to U5, U201 to U6, U301 to U7, U302 to U8
Connections:
- C11 pad 1: Power_in- -> +VDC
- C12 pad 2: Power_in- -> +VDC
- C17 pad 1: Power_in- -> +VDC
- C6 pad 1: Power_in- -> +VDC
- C7 pad 2: Power_in- -> +VDC
- C8 pad 1: Power_in- -> +VDC
- FB2 pad 1: Power_in- -> +VDC
- IC4 pad 8: Power_in- -> +VDC
- R1 pad 1: Power_in- -> +VDC
- R3 pad 2: Power_in- -> GND
- R42 pad 1: ADC_CH4 -> Net-(R42-Pad1)
- R42 pad 2: Power_in- -> +VDC
- R43 pad 2: ADC_CH4 -> Net-(R42-Pad1)
- S2 pad 7: 3v3_enable -> +VDC
- S2 pad 8: GND -> 3v3_enable
- U3 pad 16: Power_in- -> +VDC
- U4 pad 3: Power_in- -> +VDC
- U6 pad 12: Net-(J205-Pad4) -> Net-(R42-Pad1)
- U6 pad 13: Net-(J205-Pad3) -> ADC_CH4
- U6 pad 14: Net-(J205-Pad2) -> ADC_CH4
- U6 pad 4: Power_in- -> +VDC
Routing:
- net GND: track 23.9 -> 230.7 mm, vias 13 -> 105
- net +VDC: track 0.00 -> 170.1 mm, vias 0 -> 12
- net +3V3: track 185.8 -> 265.0 mm, vias 1 -> 12
- net Power_in+: track 11.7 -> 85.5 mm, vias 1 -> 9
- net +5V: track 55.6 -> 117.1 mm, vias 1 -> 9
- net TE: track 1.66 -> 62.2 mm, vias 0 -> 2
- net /SPI1_MOSI: track 0.00 -> 58.6 mm, vias 0 -> 6
- net /POWER_MEASUREMENTS/source_vcc: track 0.00 -> 57.2 mm
- net /SPI1_CLK: track 0.00 -> 53.1 mm, vias 0 -> 5
- net Net-(R33-Pad2): track 1.55 -> 54.1 mm, vias 0 -> 2
- net /SPI1_MISO: track 0.00 -> 49.9 mm, vias 0 -> 5
- net /GPIO9: track 8.67 -> 53.5 mm, vias 0 -> 3
- net SDA: track 0.00 -> 42.9 mm, vias 0 -> 2
- net SCL: track 0.00 -> 42.7 mm, vias 0 -> 2
- net 3v3_enable: track 34.1 -> 76.4 mm
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- added copper zone on F.Cu, net (none)
- added copper zone on F.Cu, net +VDC
- added copper zone on F.Cu, net /Power-IN-OUT-BMS/buck/inductor_buck
- added copper zone on F.Cu, net /Power-IN-OUT-BMS/buck_out
- added copper zone on F.Cu, net /Power-IN-OUT-BMS/lin_reg
