File: test_project_01/test_project_01.kicad_pcb (KiCad board)
At the start: 2 copper layers, 100 x 100 mm, 117 parts, among them IC1 XRA1203IG24TR-F, IC2 INA2181A4QDGSRQ1, IC3 MCP73834T-FCI_UN, IC4 AP2112M-3.3TRG1, J1 STX-3120-5B, J10 10033527-N3112MLF, J11 Conn_01x02, J12 Conn_01x02, J13 Conn_01x02, J2 SS-52100-001, J3 MEM2051-00-195-00-A, J4 Barrel_Jack_Switch, J5 Barrel_Jack_Switch, J6 Conn_01x03, J7 Conn_01x03, J9 USB_A, Q1 DMG9933USD-13, SW1 SW_SPST, U1 ESP32-C3-MINI-1, U10 DIO6012BCST6, U2 LM4040DBZ-3, U3 MCP3208, U4 Adafruit_MAX98357, U5 D1213A-02SM, U6 LM324A, U7 1043, U8 APX810S05

Commit message: H
Parts:
- added FID1: Fiducial, Fiducial:Fiducial_0.5mm_Mask1mm, F.Cu at (138.0, 53.7)
- added FID2: Fiducial, Symbol:Polarity_Center_Positive_6mm_SilkScreen, F.Cu at (136.7, 75.0)
- added FID3: Fiducial, Symbol:OSHW-Logo_5.7x6mm_SilkScreen, F.Cu at (70.8, 123.9)
- added FID4: Fiducial, Symbol:KiCad-Logo2_6mm_SilkScreen, F.Cu at (114.9, 144.4)
- added FID5: Fiducial, Symbol:WEEE-Logo_5.6x8mm_SilkScreen, B.Cu at (106.2, 144.4)
- added J8: Conn_01x06, Connector_PinHeader_2.54mm:PinHeader_1x06_P2.54mm_Vertical, F.Cu at (120.2, 53.7)
- added kibuzzard-62BCC557: G***, kibuzzard-62BCC557, F.Cu at (51.8, 60.8)
- added kibuzzard-62BCC581: G***, kibuzzard-62BCC581, F.Cu at (67.3, 138.2)
- added kibuzzard-62BCC683: G***, kibuzzard-62BCC683, F.Cu at (91.2, 109.2)
- added kibuzzard-62BCC6A1: G***, kibuzzard-62BCC6A1, F.Cu at (56.8, 128.7)
- added kibuzzard-62BCC6A1: G***, kibuzzard-62BCC6A1, F.Cu at (75.8, 103.4)
- added kibuzzard-62BCC6D2: G***, kibuzzard-62BCC6D2, F.Cu at (140.0, 90.6)
- added kibuzzard-62BCC6D2: G***, kibuzzard-62BCC6D2, F.Cu at (116.7, 53.8)
- added kibuzzard-62BCC6D2: G***, kibuzzard-62BCC6D2, F.Cu at (139.9, 107.1)
- added kibuzzard-62BCC6DA: G***, kibuzzard-62BCC6DA, F.Cu at (117.1, 56.2)
- added kibuzzard-62BCC6E5: G***, kibuzzard-62BCC6E5, F.Cu at (117.1, 58.9)
- added kibuzzard-62BCC6EE: G***, kibuzzard-62BCC6EE, F.Cu at (116.7, 61.3)
- added kibuzzard-62BCC6FB: G***, kibuzzard-62BCC6FB, F.Cu at (116.7, 66.4)
- added kibuzzard-62BCC715: G***, kibuzzard-62BCC715, F.Cu at (116.7, 63.9)
- added kibuzzard-62BCCB31: G***, kibuzzard-62BCCB31, F.Cu at (137.7, 127.5)
- added kibuzzard-62BCCBA4: G***, kibuzzard-62BCCBA4, F.Cu at (74.1, 90.8)
- added kibuzzard-62BCCBB0: G***, kibuzzard-62BCCBB0, F.Cu at (81.8, 91.2)
- RR1: value R_Small -> 91k; footprint Resistor_THT:R_Axial_DIN0204_L3.6mm_D1.6mm_P5.08mm_Horizontal -> Resistor_SMD:R_0805_2012Metric_Pad1.20x1.40mm_HandSolder
- RR2: value R_Small -> 20k; footprint Resistor_THT:R_Axial_DIN0204_L3.6mm_D1.6mm_P5.08mm_Horizontal -> Resistor_SMD:R_0805_2012Metric_Pad1.20x1.40mm_HandSolder
- moved RR1 9.53 mm to (95.2, 143.3), turned to 180 degrees
- moved FB2 5.92 mm to (97.5, 130.3), turned to 0 degrees
- moved C20 5.53 mm to (95.0, 141.5)
- moved RR2 5.06 mm to (95.2, 139.8)
- moved J2 4.04 mm to (107.0, 60.9)
- moved U5 3.74 mm to (103.6, 65.2)
- moved C19 3.73 mm to (99.4, 140.4)
- moved FB1 3.48 mm to (107.1, 68.4)
- moved C22 3.07 mm to (95.4, 146.0)
- moved R9 2.88 mm to (88.3, 110.3)
- moved R20 2.24 mm to (112.0, 69.9)
- moved D1 2.22 mm to (113.6, 68.0)
- moved F1 2.19 mm to (110.2, 64.6)
- moved C9 2.16 mm to (112.0, 66.3)
- moved C21 1.98 mm to (89.6, 145.5)
Connections:
- net Net-(C19-Pad1) renamed /Power-IN-OUT-BMS/buck/buck_input_filtered
Routing:
- net /reset: track 12.2 -> 95.7 mm, vias 2 -> 10
- net /DATA0: track 31.1 -> 105.0 mm, vias 1 -> 9
- net /RX: track 0.00 -> 45.3 mm
- net /TX: track 0.00 -> 44.6 mm
- net +3V3: track 265.0 -> 296.7 mm, vias 12 -> 14
- net /Power-IN-OUT-BMS/buck/buck_input_filtered: track 0.27 -> 15.8 mm
- net /Power-IN-OUT-BMS/buck_out: track 30.3 -> 23.7 mm
- net GND: track 230.7 -> 236.3 mm, vias 105 -> 126
- net Net-(C20-Pad2): track 14.3 -> 9.07 mm, vias 1 -> 0
- net +VDC: track 170.1 -> 165.5 mm
- net Net-(R9-Pad2): track 4.10 -> 7.04 mm
- net /SPI1_MISO: track 49.9 -> 48.2 mm, vias 5 -> 3
- net /GPIO5: track 36.6 -> 38.1 mm, vias 2 -> 4
- net +5V: track 117.1 -> 115.7 mm, vias 9 -> 11
- net Net-(F1-Pad1): track 2.54 -> 3.86 mm
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- added copper zone on F.Cu, net /POWER_MEASUREMENTS/source_vcc
- added copper zone on F.Cu, net /Power-IN-OUT-BMS/Drains
- added copper zone on F.Cu, net /Power-IN-OUT-BMS/buck/buck_input_filtered
