File: test_project_01/test_project_01.kicad_sch (KiCad schematic)
At the start: 2 parts

Commit message: j
Parts:
- removed AE?: Antenna_Shield, symbol Device:Antenna_Shield
- removed IC?: ESP32-C3, QFN50P500X500X90-33N-D, symbol SamacSys_Parts:ESP32-C3
- added J7: USB_B_Mini, symbol Connector:USB_B_Mini
- added J8: Micro_SD_Card_Det, symbol Connector:Micro_SD_Card_Det
- added J?: Conn_01x10_Male, symbol Connector:Conn_01x10_Male
Connections:
- net GND: now also J7.5 (GND)
- new net +5V: J7.1 (VBUS)
- no-connect marks 0 -> 1
Other:
- added sheet VUSB_Li-ion_BMS_to_3v3 (VUSB_Li-ion_BMS_to_3v3.kicad_sch)

Commit message: v
Parts:
- removed J?: Conn_01x10_Male, symbol Connector:Conn_01x10_Male
- added C1: C_Small, symbol Device:C_Small
- added FB1: FerriteBead, symbol Device:FerriteBead
- added U3: ESP32-C3-MINI-1, Espressif:ESP32-C3-MINI-1_Hand-Soldering, symbol Espressif:ESP32-C3-MINI-1
Connections:
- net +5V: now also C1.1, FB1.2; no longer J7.1 (VBUS)
- net GND: now also J7.4 (ID), C1.2, U3.1 (GND), U3.11 (GND), U3.14 (GND), U3.2 (GND), U3.36 (GND)
- net D-: now reaches J7.2 (D-)
- net D-: now also U3.26 (GPIO18/USB_D-)
- net D+: now reaches J7.3 (D+)
- net D+: now also U3.27 (GPIO19/USB_D+)
- new net: FB1.1, J7.1 (VBUS)
- new net +3V3: U3.3 (3V3)
Other:
- moved on the sheet: J7, J8

Commit message: f
Parts:
- removed FB1: FerriteBead, symbol Device:FerriteBead
- removed J8: Micro_SD_Card_Det, symbol Connector:Micro_SD_Card_Det
- added FB1: HI1806T600R-10, BEADC4516X185N, symbol SamacSys_Parts:HI1806T600R-10
- added IC4: FT260S-U, SOP65P640X120-28N, symbol SamacSys_Parts:FT260S-U
- added J8: MEM2051-00-195-00-A, MEM20510019500A, symbol SamacSys_Parts:MEM2051-00-195-00-A
- added S1: DS01C-254-S-08BE, DS01C254S08BE, symbol SamacSys_Parts:DS01C-254-S-08BE
- added U4: iqs625, Package_SO:TSSOP-8_4.4x3mm_P0.65mm, symbol My_custom_lib:iqs625
- added U5: MCP3204, symbol Analog_ADC:MCP3204
Connections:
- net +5V: now also FB1.2
- net GND: now also IC4.23 (GND), J8.P6 (VSS), U4.7 (VSS), U5.12 (AGND), U5.7 (DGND)
- net at J7.1 (VBUS): now also FB1.1
Other:
- added sheet STM32_stuff (STM32_stuff.kicad_sch)
- note added: "DIP SWITCHES"
- note added: "SD CARD ADAPTER"
- note added: "USB BRIDGE IC"

Commit message: h
Connections:
- net GND: now also IC4.28 (AGND)
Other:
- removed sheet STM32_stuff
- moved on the sheet: C1, FB1, IC4, J7

Commit message: d
Parts:
- removed IC4: FT260S-U, SOP65P640X120-28N, symbol SamacSys_Parts:FT260S-U
- added C5: 10u, symbol Device:C_Small
- added C6: 0.1u, symbol Device:C_Small
- added C7, C8: 1u, symbol Device:C_Small
- added C?: 10u, Capacitor_SMD:C_0603_1608Metric, symbol Device:C
- added J10: Conn_02x10_Odd_Even, Connector_PinHeader_2.54mm:PinHeader_2x10_P2.54mm_Vertical, symbol Connector_Generic:Conn_02x10_Odd_Even
- added J9: STX-3120-5B, STX31205B, symbol SamacSys_Parts:STX-3120-5B
- added J?: MEM2051-00-195-00-A, MEM20510019500A, symbol SamacSys_Parts:MEM2051-00-195-00-A
- added R16, R? (x2): 10k, symbol Device:R_Small
- added R21: 1M, symbol Device:R_Small
- added R?: 1M, Capacitor_SMD:C_0402_1005Metric, symbol Device:R
- added R? (x3): 10k, Resistor_SMD:R_0402_1005Metric, symbol Device:R
- added SW1: SW_SPST, symbol Switch:SW_SPST
- added U6: D1213A-02SM, Package_TO_SOT_SMD:SOT-23-5, symbol My_custom_lib:D1213A-02SM
- added U7: Adafruit_MAX98357, Z_mycustom_footprint_lib:Adafruit MAX98357 I2S Class-D Mono, symbol My_custom_lib:Adafruit_MAX98357
Connections:
- net +3V3: now also J8.P4 (VDD), S1.12 (NO_6), U4.1 (VDD), U5.13 (Vref), U5.14 (Vdd), C5.1, C6.1, C?.1, J?.P4 (VDD), R16.1, R21.2, R?.2, R?.2, R?.2
- net +5V: now also J10.2 (Pin_2), U6.5 (VCC)
- net D+: now also U6.4 (CH2)
- net D-: now also U6.3 (CH1)
- net GND: now also J8.MP1, J8.MP3, J8.MP4, J8.MP5, S1.14 (NO_7), S1.16 (NO_8), C5.2, C6.2, C7.2, C8.1, C?.2, J10.4 (Pin_4), J?.MP1, J?.MP3, J?.MP4, J?.MP5, J?.P6 (VSS), R?.2, SW1.1 (A), U6.2 (VSS), U7.3 (VDD)
- net SPI2_MISO: now reaches U5.10 (Dout)
- net SPI2_CLK: now reaches U5.11 (CLK)
- net ADC_CH1: now reaches U5.2 (CH1)
- net ADC_CH3: now reaches U5.4 (CH3)
- net SPI2_MOSI: now reaches U5.9 (Din)
- net I2C_SDA: now reaches U4.2 (SDA)
- net I2C_CLK: now reaches U4.8 (SCL)
- net at S1.11 (COM_6): now also R?.2
- net gain: now reaches S1.13 (COM_7)
- net gain: now also R?.1, U7.8 (GAIN)
- net at S1.15 (COM_8): now also R?.2
- net SD_sening: now reaches J8.MP2
- net SD_sening: now also R21.1
- net SS1: now reaches J8.P2 (CD/DAT3)
- net SPI_MOSI: now reaches J8.P3 (CMD)
- net SPI_CLK: now reaches J8.P5 (CLK)
- net SPI_MISO: now reaches J8.P7 (DAT0)
- net RX: now reaches U3.30 (GPIO20/U0RXD)
- net RX: now also J10.3 (Pin_3)
- net TX: now reaches U3.31 (GPIO21/U0TXD)
- net TX: now also J10.1 (Pin_1)
- net at U3.8 (EN/CHIP_PU): now also C7.1, R16.2, SW1.2 (B)
- new net: J?.P5 (CLK), R?.1
- new net +VDC: C8.2, U7.4 (VSS)
- new net BCLK: U7.6 (BCLK_(Bit_Clock))
- new net DATA_IN: U7.7 (DIN_(Data_In))
- new net GPIO18: J?.P3 (CMD)
- new net GPIO19: J?.P7 (DAT0)
- new net GPIO22: J?.P2 (CD/DAT3)
- new net LRC: U7.5 (LRC_(Left/Right_Clock)
- new net SD_DAT1: J?.P1 (DAT2), R?.1
- new net SD_DAT2: J?.P8 (DAT1), R?.1
- new net SD_detect: J?.MP2, R?.1
- new net on/off+mode: R?.1, U7.9 (SD_/_MODE)
- no-connect marks 1 -> 4
Other:
- note added: "Audio jack"
- note added: "ESD protection IC"
- note added: "MCU can: push 40mA out pull 28mA in"
- note added: "SS"
- note added: "exemplu SD rp2040"
- note added: "sensor"
- note removed: "USB BRIDGE IC"
- title: (none) -> ESP32 audio power meter SD dataloger
- moved on the sheet: S1, U3, U4

Commit message: h
Parts:
- removed C?: 10u, Capacitor_SMD:C_0603_1608Metric, symbol Device:C
- removed J10: Conn_02x10_Odd_Even, Connector_PinHeader_2.54mm:PinHeader_2x10_P2.54mm_Vertical, symbol Connector_Generic:Conn_02x10_Odd_Even
- removed J7: USB_B_Mini, symbol Connector:USB_B_Mini
- removed J?: MEM2051-00-195-00-A, MEM20510019500A, symbol SamacSys_Parts:MEM2051-00-195-00-A
- removed R?: 1M, Capacitor_SMD:C_0402_1005Metric, symbol Device:R
- removed R? (x3): 10k, Resistor_SMD:R_0402_1005Metric, symbol Device:R
- removed U4: iqs625, Package_SO:TSSOP-8_4.4x3mm_P0.65mm, symbol My_custom_lib:iqs625
- added C11: 1u, Capacitor_SMD:C_0603_1608Metric_Pad1.08x0.95mm_HandSolder, symbol Device:C_Small
- added F1: 1.5 2A, symbol Device:Fuse
- added J10, J7: Conn_01x10, Connector_PinHeader_2.54mm:PinHeader_1x10_P2.54mm_Vertical, symbol Connector_Generic:Conn_01x10
- added J11: SS-52100-001, SamacSys_Parts:SS52100001, symbol SamacSys_Parts:SS-52100-001
- added R22, R23: 470, Resistor_SMD:R_0603_1608Metric_Pad0.98x0.95mm_HandSolder, symbol Device:R_Small
- C1: value C_Small -> 1u; footprint (none) -> Capacitor_SMD:C_0603_1608Metric_Pad1.08x0.95mm_HandSolder
- C5, C6, C7, C8: footprint (none) -> Capacitor_SMD:C_0603_1608Metric_Pad1.08x0.95mm_HandSolder
- FB1: footprint BEADC4516X185N -> SamacSys_Parts:BEADC4516X185N
- J8: footprint MEM20510019500A -> SamacSys_Parts:MEM20510019500A
- J9: footprint STX31205B -> SamacSys_Parts:STX31205B
- R16: footprint (none) -> Resistor_SMD:R_0603_1608Metric_Pad0.98x0.95mm_HandSolder
- R21: value 1M -> 10k; footprint (none) -> Resistor_SMD:R_0603_1608Metric_Pad0.98x0.95mm_HandSolder
- R24, R25: renamed from R?; footprint (none) -> Resistor_SMD:R_0603_1608Metric_Pad0.98x0.95mm_HandSolder
- S1: footprint DS01C254S08BE -> SamacSys_Parts:DS01C254S08BE
- U5: footprint (none) -> Package_DIP:DIP-14_W7.62mm_LongPads
Connections:
- net SPI_CLK is gone; now on net SPI2_CLK: J8.P5 (CLK)
- net SPI_MISO is gone; now on net SPI2_MISO: J8.P7 (DAT0)
- net SPI_MOSI is gone; now on net SPI2_MOSI: J8.P3 (CMD)
- net SS1 is gone; now on net SPI2_SS2: J8.P2 (CD/DAT3)
- net +3V3: now also J7.3 (Pin_3), J7.4 (Pin_4)
- net +5V: now also F1.2, J7.1 (Pin_1), J7.2 (Pin_2); no longer FB1.2, U6.5 (VCC)
- net +VDC: now also C8.1, U7.3 (VDD), J7.6 (Pin_6); no longer C8.2, U7.4 (VSS)
- net BCLK: now also U3.13 (GPIO1/ADC1_CH1/XTAL_32K_N), J10.3 (Pin_3)
- net D+: now also J11.3
- net D-: now also J11.2
- net DATA_IN: now also U3.6 (GPIO3/ADC1_CH3), J10.1 (Pin_1)
- net GND: now also C8.2, J9.1, J9.MH1, J9.MH2, J9.MH3, U7.2 (speaker-), U7.4 (VSS), J11.4, J11.MH1, J11.MH2, J7.5 (Pin_5), J7.7 (Pin_7); no longer C8.1, U7.3 (VDD)
- net LRC: now also U3.12 (GPIO0/ADC1_CH0/XTAL_32K_P), J10.2 (Pin_2)
- net RX: now also J7.10 (Pin_10), R22.2; no longer U3.30 (GPIO20/U0RXD)
- net SD_sening: now also U3.23 (GPIO9), J10.10 (Pin_10)
- net SPI2_CLK: now also S1.8 (NO_4)
- net SPI2_MISO: now also S1.6 (NO_3)
- net SPI2_MOSI: now also S1.10 (NO_5)
- net TX: now also J7.9 (Pin_9), R23.2; no longer U3.31 (GPIO21/U0TXD)
- net ADC_CH0: now reaches U5.1 (CH0)
- net ADC_CH2: now reaches U5.3 (CH2)
- net SPI2_SS1: now reaches U5.8 (~{CS}/SHDN)
- net SPI2_SS1: now also S1.2 (NO_1)
- net GPIO8: now reaches S1.1 (COM_1)
- net GPIO8: now also U3.22 (GPIO8), J10.9 (Pin_9)
- net GPIO7: now reaches S1.3 (COM_2)
- net GPIO7: now also U3.21 (GPIO7), J10.8 (Pin_8)
- net SPI2_SS2: now reaches S1.4 (NO_2)
- net GPIO6: now reaches S1.5 (COM_3)
- net GPIO6: now also U3.20 (GPIO6), J10.7 (Pin_7)
- net GPIO5: now reaches S1.7 (COM_4)
- net GPIO5: now also U3.19 (GPIO5/ADC2_CH0), J10.6 (Pin_6)
- net GPIO4: now reaches S1.9 (COM_5)
- net GPIO4: now also U3.18 (GPIO4/ADC1_CH4), J10.5 (Pin_5)
- net at U7.1 (speaker+): now also C11.2
- net reset: now reaches C7.1, R16.2, SW1.2 (B), U3.8 (EN/CHIP_PU)
- net at J9.2: now also J9.5, C11.1
- net VBUS: now reaches FB1.1
- net VBUS: now also U6.5 (VCC), J11.1
- net GPIO10: now reaches U3.16 (GPIO10)
- net GPIO10: now also J10.4 (Pin_4)
- net gpio2: now reaches U3.5 (GPIO2/ADC1_CH2)
- net gpio2: now also J7.8 (Pin_8)
- new net: R23.1, U3.31 (GPIO21/U0TXD)
- new net: R22.1, U3.30 (GPIO20/U0RXD)
- new net: F1.1, FB1.2
- no-connect marks 4 -> 9
Other:
- note added: "acording to DC doc: https://docs.espressif.com/projects/esp-idf/en/latest/esp32/api-reference/peripherals/sdmmc_host.html"
- note removed: "SS"
- note removed: "exemplu SD rp2040"
- note removed: "sensor"
- moved on the sheet: C1, J8, J9, R21, R24, R25, S1

Commit message: h
Parts:
- added IC?: XRA1203IG24TR-F, SOP65P640X120-24N, symbol SamacSys_Parts:XRA1203IG24TR-F
