File: test_project_01/test_project_01.kicad_sch (KiCad schematic)
At the start: 26 parts, among them J10 Conn_01x10, J11 SS-52100-001, J7 Conn_01x10, J8 MEM2051-00-195-00-A, J9 STX-3120-5B, SW1 SW_SPST, U3 ESP32-C3-MINI-1, U5 MCP3204, U6 D1213A-02SM, U7 Adafruit_MAX98357

Commit message: v
Parts:
- added BT?: Battery, symbol Device:Battery
- added C? (x2): 1u, Capacitor_SMD:C_0805_2012Metric_Pad1.18x1.45mm_HandSolder, symbol Device:C_Small
- added D? (x3): LED_Small Green, LED_SMD:LED_0603_1608Metric_Pad1.05x0.95mm_HandSolder, symbol Device:LED_Small
- added D?: D_Shockley, Diode_THT:D_DO-15_P15.24mm_Horizontal, symbol Device:D_Shockley
- added F?: Polyfuse_Small, Fuse:Fuse_1812_4532Metric_Pad1.30x3.40mm_HandSolder, symbol Device:Polyfuse_Small
- added FB?: HI1806T600R-10, SamacSys_Parts:BEADC4516X185N, symbol SamacSys_Parts:HI1806T600R-10
- added IC?: AP2112M-3.3TRG1, SamacSys_Parts:SOIC127P600X170-8N, symbol SamacSys_Parts:AP2112M-3.3TRG1
- added J?: Conn_01x03, Connector_PinHeader_2.54mm:PinHeader_1x03_P2.54mm_Vertical, symbol Connector_Generic:Conn_01x03
- added J?: Conn_01x02_Male, Connector_PinHeader_2.54mm:PinHeader_1x02_P2.54mm_Vertical, symbol Connector:Conn_01x02_Male
- added J?: USB_B_Mini, Connector_USB:USB_Mini-B_Lumberg_2486_01_Horizontal, symbol Connector:USB_B_Mini
- added Q?: DMG9933USD-13, SamacSys_Parts:SOIC127P600X175-8N, symbol SamacSys_Parts:DMG9933USD-13
- added R? (x2): 330, Resistor_SMD:R_0603_1608Metric_Pad0.98x0.95mm_HandSolder, symbol Device:R
- added R?: 10k+ pullup, Resistor_SMD:R_0603_1608Metric_Pad0.98x0.95mm_HandSolder, symbol Device:R
- added R?: 10k, Resistor_SMD:R_0603_1608Metric_Pad0.98x0.95mm_HandSolder, symbol Device:R
- added R?: 4.7k, Resistor_THT:R_Axial_DIN0204_L3.6mm_D1.6mm_P2.54mm_Vertical, symbol Device:R
- added S?: EG1224 SPDT switch, SamacSys_Parts:EG1224, symbol SamacSys_Parts:EG1224
- added U?: D1213A-02SM, Package_TO_SOT_SMD:SOT-23-5_HandSoldering, symbol My_custom_lib:D1213A-02SM
Connections:
- net +3V3: now also R?.2, S?.2 (COM)
- net +VDC: now also C?.1, D?.1 (K), IC?.8 (VIN), J?.3 (Pin_3), Q?.3 (S2), R?.2
- net D+: now also J?.3 (D+), U?.4 (CH2)
- net D-: now also J?.2 (D-), U?.3 (CH1)
- net GND: now also BT?.2 (-), C?.2, C?.2, D?.1 (K), D?.1 (K), D?.1 (K), IC?.6 (GND_1), IC?.7 (GND_2), J?.2 (Pin_2), J?.5 (GND), J?.6 (Shield), R?.1, S?.MH1, S?.MH2, S?.MH3, S?.MH4, U?.2 (VSS)
- net VBUS: now also D?.2 (A), FB?.2, Q?.2 (G1), Q?.4 (G2), R?.2, R?.2, U?.5 (VCC)
- new net: D?.2 (A), R?.1 (x3)
- new net: J?.2 (Pin_2), R?.2
- new net +BATT: BT?.1 (+), J?.1 (Pin_1), J?.1 (Pin_1), Q?.1 (S1)
- new net 3v3_enable: IC?.5 (EN), R?.1
- new net Drains: Q?.5 (D2_1), Q?.6 (D2_2), Q?.7 (D1_1), Q?.8 (D1_2)
- new net VBUS_RAW: F?.1, J?.1 (VBUS)
- new net VBUS_RAW2: F?.2, FB?.1
- new net buck_out: S?.1 (PIN1)
- new net lin_reg: C?.1, IC?.1 (VOUT), S?.3 (PIN2)
- no-connect marks 9 -> 14
Other:
- added sheet buck (buck.kicad_sch)
- note added: "200-300mA <100 typical"
- note added: "400-500mA+ max power usage of MCU"
- note added: "BATT TO USB POWER AUTO SHITCHING WITH REVERSE POWER PROTECTION"
- note added: "Linear regulator just in case the buck fails or i need lower noise power"
- note added: "Power"
- note added: "Power indicator leds"
- note added: "USB Data+Power Input filtering and fuse"
- note added: "active high"

Commit message: f
Parts:
- removed BT?: Battery, symbol Device:Battery
- removed C? (x2): 1u, Capacitor_SMD:C_0805_2012Metric_Pad1.18x1.45mm_HandSolder, symbol Device:C_Small
- removed D? (x3): LED_Small Green, LED_SMD:LED_0603_1608Metric_Pad1.05x0.95mm_HandSolder, symbol Device:LED_Small
- removed D?: D_Shockley, Diode_THT:D_DO-15_P15.24mm_Horizontal, symbol Device:D_Shockley
- removed F?: Polyfuse_Small, Fuse:Fuse_1812_4532Metric_Pad1.30x3.40mm_HandSolder, symbol Device:Polyfuse_Small
- removed FB?: HI1806T600R-10, SamacSys_Parts:BEADC4516X185N, symbol SamacSys_Parts:HI1806T600R-10
- removed IC?: AP2112M-3.3TRG1, SamacSys_Parts:SOIC127P600X170-8N, symbol SamacSys_Parts:AP2112M-3.3TRG1
- removed J?: Conn_01x03, Connector_PinHeader_2.54mm:PinHeader_1x03_P2.54mm_Vertical, symbol Connector_Generic:Conn_01x03
- removed J?: Conn_01x02_Male, Connector_PinHeader_2.54mm:PinHeader_1x02_P2.54mm_Vertical, symbol Connector:Conn_01x02_Male
- removed J?: USB_B_Mini, Connector_USB:USB_Mini-B_Lumberg_2486_01_Horizontal, symbol Connector:USB_B_Mini
- removed Q?: DMG9933USD-13, SamacSys_Parts:SOIC127P600X175-8N, symbol SamacSys_Parts:DMG9933USD-13
- removed R? (x2): 330, Resistor_SMD:R_0603_1608Metric_Pad0.98x0.95mm_HandSolder, symbol Device:R
- removed R?: 10k+ pullup, Resistor_SMD:R_0603_1608Metric_Pad0.98x0.95mm_HandSolder, symbol Device:R
- removed R?: 10k, Resistor_SMD:R_0603_1608Metric_Pad0.98x0.95mm_HandSolder, symbol Device:R
- removed R?: 4.7k, Resistor_THT:R_Axial_DIN0204_L3.6mm_D1.6mm_P2.54mm_Vertical, symbol Device:R
- removed S?: EG1224 SPDT switch, SamacSys_Parts:EG1224, symbol SamacSys_Parts:EG1224
- removed U?: D1213A-02SM, Package_TO_SOT_SMD:SOT-23-5_HandSoldering, symbol My_custom_lib:D1213A-02SM
- F1: value 1.5 2A -> (none)
Connections:
- no-connect marks 14 -> 3
Other:
- sheet VUSB_Li-ion_BMS_to_3v3 renamed Power-IN-OUT-BMS
- removed sheet buck
- sheet Power-IN-OUT-BMS: file VUSB_Li-ion_BMS_to_3v3.kicad_sch -> Power-IN-OUT-BMS.kicad_sch
- note added: "150% rating so 1.5A 2A for me"
- note removed: "200-300mA <100 typical"
- note removed: "400-500mA+ max power usage of MCU"
- note removed: "BATT TO USB POWER AUTO SHITCHING WITH REVERSE POWER PROTECTION"
- note removed: "Linear regulator just in case the buck fails or i need lower noise power"
- note removed: "Power"
- note removed: "Power indicator leds"
- note removed: "USB Data+Power Input filtering and fuse"
- note removed: "active high"
- moved on the sheet: C11, IC?, J8, R21, R24, R25, S1, U5, U6
Changed lines of the file:
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@@
 (kicad_sch (version 20211123) (generator eeschema)
-  (paper "A4")
+  (paper "A3")
   (title_block
     (title "ESP32 audio power meter SD dataloger")

Commit message: r
Parts:
- gave numbers to parts that had none: 1

Commit message: j
Parts:
- F1: value (none) -> 1.5 A; footprint (none) -> Fuse:Fuse_0603_1608Metric_Pad1.05x0.95mm_HandSolder

Commit message: h
Parts:
- removed J10, J7: Conn_01x10, Connector_PinHeader_2.54mm:PinHeader_1x10_P2.54mm_Vertical, symbol Connector_Generic:Conn_01x10
Connections:
- net BCLK: no longer U3.13 (GPIO1/ADC1_CH1/XTAL_32K_N)
- net DATA_IN: no longer U3.6 (GPIO3/ADC1_CH3)
- net GPIO4: no longer S1.9 (COM_5)
- net GPIO5: no longer S1.7 (COM_4)
- net GPIO6: no longer S1.5 (COM_3)
- net GPIO7: no longer S1.3 (COM_2)
- net GPIO8: no longer S1.1 (COM_1)
- net LRC: no longer U3.12 (GPIO0/ADC1_CH0/XTAL_32K_P)
- net SD_sening: no longer U3.23 (GPIO9)
- net SPI2_CLK: no longer S1.8 (NO_4)
- net SPI2_MISO: no longer S1.6 (NO_3)
- net SPI2_MOSI: no longer S1.10 (NO_5)
- net SPI2_SS1: no longer S1.2 (NO_1)
- net SPI2_SS2: no longer S1.4 (NO_2)
- net gpio2 renamed GPIO2
- new net GPIO0: U3.12 (GPIO0/ADC1_CH0/XTAL_32K_P)
- new net GPIO1: U3.13 (GPIO1/ADC1_CH1/XTAL_32K_N)
- new net GPIO3: U3.6 (GPIO3/ADC1_CH3)
- new net GPIO9: U3.23 (GPIO9)
Other:
- sheet power_measurement renamed POWER_MEASUREMENTS
- note added: "AUDIO PART"
- note added: "USB POWER+DATA"
- moved on the sheet: C1, C11, C5, C6, C7, C8, F1, FB1, IC1, J11, J8, J9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

Commit message: f
Parts:
- removed C11: 1u, Capacitor_SMD:C_0603_1608Metric_Pad1.08x0.95mm_HandSolder, symbol Device:C_Small
- removed R22, R23: 470, Resistor_SMD:R_0603_1608Metric_Pad0.98x0.95mm_HandSolder, symbol Device:R_Small
- added C102: 1u, Capacitor_SMD:C_0603_1608Metric_Pad1.08x0.95mm_HandSolder, symbol Device:C_Small
- added C105: 0.1u, Capacitor_SMD:C_0603_1608Metric_Pad1.08x0.95mm_HandSolder, symbol Device:C_Small
- added D101: LED_Small Green, LED_SMD:LED_0603_1608Metric_Pad1.05x0.95mm_HandSolder, symbol Device:LED_Small
- added H101, H102, H103, H104: MountingHole_Pad, MountingHole:MountingHole_3.2mm_M3, symbol Mechanical:MountingHole_Pad
- added JP101: Jumper_2_Bridged, Jumper:SolderJumper-2_P1.3mm_Bridged_RoundedPad1.0x1.5mm, symbol Jumper:Jumper_2_Bridged
- added R101, R103, R104, R108, R109, R110, R111: 10k, Resistor_SMD:R_0603_1608Metric_Pad0.98x0.95mm_HandSolder, symbol Device:R_Small
- added R107: 10k+ pullup, Resistor_SMD:R_0603_1608Metric_Pad0.98x0.95mm_HandSolder, symbol Device:R
- added R112: 330, Resistor_SMD:R_0603_1608Metric_Pad0.98x0.95mm_HandSolder, symbol Device:R
- added S101: DS01C-254-S-08BE, SamacSys_Parts:DS01C254S08BE, symbol SamacSys_Parts:DS01C-254-S-08BE
- added U102: LM4132xMF-3.0, Package_TO_SOT_SMD:SOT-23-5, symbol Reference_Voltage:LM4132xMF-3.0
- C103: renamed from C7; value 1u -> 10u
- C106: renamed from C8; value 1u -> 10u
- IC101: renamed from IC1; footprint SOP65P640X120-24N -> SamacSys_Parts:SOP65P640X120-24N
- SW101: renamed from SW1; footprint (none) -> SamacSys_Parts:PTS526SM15SMTR2LFS
- renumbered C5 to C101, C6 to C104, C1 to C107, F1 to F101, FB1 to FB101, J9 to J101, J11 to J102, J8 to J103, R16 to R102, R24 to R105, R25 to R106, R21 to R113, S1 to S102, U3 to U101, U5 to U103, U7 to U104, U6 to U105
Connections:
- net GPIO3 is gone; now on net DATA2: U101.6 (GPIO3/ADC1_CH3)
- net GPIO4 is gone; now on net DATA1: U101.18 (GPIO4/ADC1_CH4)
- net GPIO6 is gone; now on net SDA: U101.20 (GPIO6)
- net GPIO7 is gone; now on net SCL: U101.21 (GPIO7)
- net SPI2_SS2 is gone; now on net DATA3: J103.P2 (CD/DAT3)
- net +3V3: now also IC101.24 (VCC), C102.1, R103.2, R104.2, R108.2, R109.2; no longer U103.13 (Vref), U103.14 (Vdd)
- net +VDC: now also U103.14 (Vdd), C105.2, R101.1, R107.1
- net BCLK: now also S101.12 (NO_6)
- net DATA_IN: now also S101.8 (NO_4)
- net GND: now also IC101.12 (GND), S102.2 (NO_1), S102.4 (NO_2), S102.6 (NO_3), C102.2, C105.1, D101.1 (K), R111.1, U102.2 (GND)
- net GPIO1: now also J103.P5 (CLK)
- net GPIO10: now also S101.14 (NO_7), S101.15 (COM_8)
- net GPIO2: now also J103.P3 (CMD)
- net GPIO5: now also IC101.1 (IRQ#), R109.1
- net GPIO8: now also S101.6 (NO_3), S101.7 (COM_4)
- net GPIO9: now also S102.1 (COM_1), S101.10 (NO_5), S101.11 (COM_6)
- net LRC: now also S101.16 (NO_8)
- net RX: now also U101.30 (GPIO20/U0RXD)
- net SD_sening: now also IC101.6 (P2)
- net SPI2_SS1: now also IC101.4 (P0); no longer U103.8 (~{CS}/SHDN)
- net TX: now also U101.31 (GPIO21/U0TXD)
- net at IC101.10 (P6): now also R110.2
- net A1: now reaches IC101.2 (A1)
- net A1: now also S102.3 (COM_2), R104.1
- net A0: now reaches IC101.21 (A0)
- net A0: now also S102.5 (COM_3), R103.1
- net SCL: now reaches IC101.22 (SCL)
- net SDA: now reaches IC101.23 (SDA)
- net at IC101.3 (RESET#): now also JP101.1 (A), R108.1
- net DATA3: now reaches IC101.5 (P1)
- net P3: now reaches IC101.7 (P3)
- net P3: now also R112.2
- net at IC101.9 (P5): now also JP101.2 (B)
- net at S102.10 (NO_5): now also R107.2
- net 3v3_enable: now reaches S102.9 (COM_5)
- net at U104.1 (speaker+): now also J101.2, J101.5
- net DATA2: now reaches J103.P1 (DAT2)
- net DATA1: now reaches J103.P8 (DAT1)
- net GPIO0 renamed DATA0
- net DATA0: now also J103.P7 (DAT0)
- net SPI2_CLK renamed SPI1_CLK
- net SPI1_CLK: now also S101.9 (COM_5); no longer J103.P5 (CLK)
- net SPI2_MISO renamed SPI1_MISO
- net SPI1_MISO: now also S101.5 (COM_3); no longer J103.P7 (DAT0)
- net SPI2_MOSI renamed SPI1_MOSI
- net SPI1_MOSI: now also S101.13 (COM_7); no longer J103.P3 (CMD)
- new net: U102.5 (VREF), U103.13 (Vref)
- new net: D101.2 (A), R112.1
- new net: R101.2, U102.4 (VIN)
- new net SPI1_SS1: U103.8 (~{CS}/SHDN)
- new net TE: R110.1, R111.2
- no-connect marks 3 -> 21
Other:
- note added: "A1 A0 I2C adredd GND GND 0x40 (0100 000X) GND VCC 0x42 (0100 001X) VCC GND 0x44 (0100 010X) VCC VCC 0x46 (0100 011X)"
- note added: "ADC"
- note added: "AUDIO Board + JACK"
- note added: "DIP SWITCH"
- note added: "GPIO EXTENDER"
- note added: "I2C bus"
- note added: "I2S pins/ SPI1 for ADC"
- note added: "SD +SPI"
- note added: "SD CARD"
- note added: "interupt pin to MCU"
- note removed: "AUDIO PART"
- note removed: "DIP SWITCHES"
- moved on the sheet: C103, C104, C106, IC101, J101, J103, R102, R105, R106, R113, S102, U103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

Commit message: r
Parts:
- removed R107: 10k+ pullup, Resistor_SMD:R_0603_1608Metric_Pad0.98x0.95mm_HandSolder, symbol Device:R
- added R114: 10k+ pulldown, Resistor_SMD:R_0603_1608Metric_Pad0.98x0.95mm_HandSolder, symbol Device:R
- R101: value 10k -> (none); footprint Resistor_SMD:R_0603_1608Metric_Pad0.98x0.95mm_HandSolder -> (none)
Connections:
- net +VDC: now also R114.2
- net 3v3_enable: now also S102.7 (COM_4), R114.1; no longer S102.9 (COM_5)
- net GND: now also S102.8 (NO_4)
- net at U102.3 (EN): now also R101.2, U102.4 (VIN)
- no-connect marks 21 -> 37
Other:
- note added: "DIP SWITCHES"
- note added: "https://www.espressif.com/sites/default/files/documentation/esp32-c3_hardware_design_guidelines_en.pdf anteena is on the left"
- note added: "this board has screw terminals at thee audio autpur"
- note removed: "DIP SWITCH"
- moved on the sheet: C105, R101, U102
