File: test_project_01/test_project_01.kicad_sch (KiCad schematic)
At the start: 40 parts, among them IC101 XRA1203IG24TR-F, J101 STX-3120-5B, J102 SS-52100-001, J103 MEM2051-00-195-00-A, SW101 SW_SPST, U101 ESP32-C3-MINI-1, U102 LM4132xMF-3.0, U103 MCP3204, U104 Adafruit_MAX98357, U105 D1213A-02SM

Commit message: h
Parts:
- removed U102: LM4132xMF-3.0, Package_TO_SOT_SMD:SOT-23-5, symbol Reference_Voltage:LM4132xMF-3.0
- removed U103: MCP3204, Package_DIP:DIP-14_W7.62mm_LongPads, symbol Analog_ADC:MCP3204
- added C104: (no value), Capacitor_SMD:C_0603_1608Metric_Pad1.08x0.95mm_HandSolder, symbol Device:C_Small
- added C106: 100n, Capacitor_SMD:C_0603_1608Metric_Pad1.08x0.95mm_HandSolder, symbol Device:C_Small
- added U102: LM4040DBZ-3, Package_TO_SOT_SMD:SOT-23, symbol Reference_Voltage:LM4040DBZ-3
- added U103: (no value), symbol Analog_ADC:MCP3208
- C105: renamed from C104; value 0.1u -> (none); footprint Capacitor_SMD:C_0603_1608Metric_Pad1.08x0.95mm_HandSolder -> (none)
- C107: renamed from C105; value 0.1u -> (none)
- R101: value (none) -> 1k; footprint (none) -> Resistor_SMD:R_0603_1608Metric_Pad0.98x0.95mm_HandSolder
- renumbered C106 to C108, C107 to C109, R114 to R103, R103 to R104, R104 to R105, R105 to R106, R106 to R107
Connections:
- net +VDC: now also C106.1, U103.16 (Vdd)
- net ADC_CH0: now also U103.1 (CH0)
- net ADC_CH1: now also U103.2 (CH1)
- net ADC_CH2: now also U103.3 (CH2)
- net ADC_CH3: now also U103.4 (CH3)
- net GND: now also C104.1, C106.2, U102.2 (A), U103.14 (AGND), U103.9 (DGND)
- net SPI1_CLK: now also U103.13 (CLK)
- net SPI1_MISO: now also U103.12 (Dout)
- net SPI1_MOSI: now also U103.11 (Din)
- net SPI1_SS1: now also U103.10 (~{CS}/SHDN)
- net Vref: now reaches R101.2
- net Vref: now also C104.2, U102.1 (K), U103.15 (Vref)
- net SD_sening renamed SD_sense
- new net ADC_CH4: U103.5 (CH4)
- no-connect marks 37 -> 40
Other:
- note added: "1.2mA max at 4.2V 0.3mA min at 3V3"
- note added: "SD +SPI2"
- note added: "https://www.espressif.com/sites/default/files/documentation/esp32-c3_hardware_design_guidelines_en.pdf anteena is on the left pull up/down resitors are 45k"
- note removed: "SD +SPI"
- note removed: "https://www.espressif.com/sites/default/files/documentation/esp32-c3_hardware_design_guidelines_en.pdf anteena is on the left"
- moved on the sheet: C107, R104, R105

Commit message: k
Parts:
- C104, C107: value (none) -> 100n
- C105: value (none) -> 100n; footprint (none) -> Capacitor_SMD:C_0603_1608Metric_Pad1.08x0.95mm_HandSolder
- U103: value (none) -> MCP3208; footprint (none) -> Package_SO:SOIC-16_3.9x9.9mm_P1.27mm

Commit message: i
Connections:
- net ADC_CH5: now reaches U103.6 (CH5)
- net ADC_CH6: now reaches U103.7 (CH6)
- no-connect marks 40 -> 38
Other:
- note added: "MCU"

Commit message: y
Parts:
- added R105, R107, R110, R111, R112, R113, R114, R115: 10k, Resistor_SMD:R_0603_1608Metric_Pad0.98x0.95mm_HandSolder, symbol Device:R_Small
- renumbered R105 to R106, R106 to R108, R107 to R109, R108 to R116, R109 to R117, R110 to R118, R111 to R119, R112 to R120, R113 to R121
Connections:
- net +3V3: now also R105.2, R107.2, R110.2, R111.2, R112.2, R113.2, R114.2, R115.2
- net DATA0: now also R111.1
- net DATA1: now also R115.1
- net DATA2: now also R114.1
- net DATA3: now also R105.1
- net GPIO1: now also R110.1
- net GPIO2: now also R107.1
- net SCL: now also R113.1
- net SDA: now also R112.1
Other:
- note added: "150% rating so 1.5A-2A for me"
- note added: "Pull ups"
- note removed: "150% rating so 1.5A 2A for me"
- moved on the sheet: C101, C102, C105, C109, F101, FB101, H101, H102, H103, H104, J102, U105

Commit message: r
Parts:
- removed D101: LED_Small Green, LED_SMD:LED_0603_1608Metric_Pad1.05x0.95mm_HandSolder, symbol Device:LED_Small
- removed R120: 330, Resistor_SMD:R_0603_1608Metric_Pad0.98x0.95mm_HandSolder, symbol Device:R
- added C23: 100n, Capacitor_SMD:C_0603_1608Metric_Pad1.08x0.95mm_HandSolder, symbol Device:C_Small
- added D1, D5, D6: LED_Small Green, LED_SMD:LED_0603_1608Metric_Pad1.05x0.95mm_HandSolder, symbol Device:LED_Small
- added R20: 4.7k, Resistor_SMD:R_0805_2012Metric, symbol Device:R
- added R44, R45: 330, Resistor_SMD:R_0603_1608Metric_Pad0.98x0.95mm_HandSolder, symbol Device:R
- IC1: renamed from IC101; value XRA1203IG24TR-F -> (none); footprint SamacSys_Parts:SOP65P640X120-24N -> (none)
- R3: renamed from R103; value 10k+ pulldown -> (none); footprint Resistor_SMD:R_0603_1608Metric_Pad0.98x0.95mm_HandSolder -> (none)
- renumbered C101 to C1, C102 to C2, C103 to C3, C104 to C4, C105 to C5, C106 to C6, C107 to C7, C108 to C8, C109 to C9, F101 to F1, FB101 to FB1, H101 to H1, H102 to H2, H103 to H3, H104 to H4, J101 to J1, J102 to J2, J103 to J3, JP101 to JP1, R101 to R1, R110 to R10, R111 to R11, R112 to R12, R113 to R13, R114 to R14, R115 to R15, R116 to R16, R117 to R17, R118 to R18, R119 to R19, R102 to R2, R121 to R21, R104 to R4, R105 to R5, R106 to R6, R107 to R7, R108 to R8, R109 to R9, S101 to S1, S102 to S2, SW101 to SW1, U101 to U1, U102 to U2, U103 to U3, U104 to U4, U105 to U5
Connections:
- net +3V3: now also C23.2, R44.2
- net +5V: now also R20.2
- net +VDC: now also S2.7 (COM_4); no longer R3.2
- net 3v3_enable: now also S2.8 (NO_4); no longer S2.7 (COM_4)
- net GND: now also R3.2, C23.1, D1.1 (K), D5.1 (K), D6.1 (K); no longer S2.8 (NO_4)
- net P3: now also R45.2
- new net: D1.2 (A), R20.1
- new net: D6.2 (A), R45.1
- new net: D5.2 (A), R44.1
Other:
- note added: "Power indicator leds"
- note added: "pull down since this way it is by default off and it doent draw power as oposed to a pull up that is turned off when tied to GND"
- moved on the sheet: R3, R4, R6, R8, R9, S1, S2

Commit message: H
Parts:
- added FID1, FID2, FID3, FID4, FID5: (no value), symbol Mechanical:Fiducial
- added J8: (no value), symbol Connector_Generic:Conn_01x06
Connections:
- net +3V3: now also J8.6 (Pin_6)
- net DATA0: now also J8.5 (Pin_5)
- net GND: now also J8.1 (Pin_1)
- net RX: now also J8.3 (Pin_3)
- net TX: now also J8.2 (Pin_2)
- net reset: now also J8.4 (Pin_4)

Commit message: r
Parts:
- added C26: 10u, Capacitor_SMD:C_0603_1608Metric_Pad1.08x0.95mm_HandSolder, symbol Device:C_Small
- added D7, D8, D9: LED_Small Green, LED_SMD:LED_0603_1608Metric_Pad1.05x0.95mm_HandSolder, symbol Device:LED_Small
- added R30, R46, R47: 330, Resistor_SMD:R_0603_1608Metric_Pad0.98x0.95mm_HandSolder, symbol Device:R
- added TP1, TP2, TP3: TestPoint, TestPoint:TestPoint_Pad_1.0x1.0mm, symbol Connector:TestPoint
- FID1: value (none) -> Fiducial; footprint (none) -> Fiducial:Fiducial_0.5mm_Mask1mm
- FID2: value (none) -> Fiducial; footprint (none) -> Symbol:Polarity_Center_Positive_6mm_SilkScreen
- FID3: value (none) -> Fiducial; footprint (none) -> Symbol:OSHW-Logo_5.7x6mm_SilkScreen
- FID4: value (none) -> Fiducial; footprint (none) -> Symbol:KiCad-Logo2_6mm_SilkScreen
- FID5: value (none) -> Fiducial; footprint (none) -> Symbol:WEEE-Logo_5.6x8mm_SilkScreen
- IC1: value (none) -> XRA1203IG24TR-F; footprint (none) -> SamacSys_Parts:SOP65P640X120-24N
- J8: value (none) -> Conn_01x06; footprint (none) -> Connector_PinHeader_2.54mm:PinHeader_1x06_P2.54mm_Vertical
- R3: value (none) -> 20k; footprint (none) -> Resistor_SMD:R_0603_1608Metric_Pad0.98x0.95mm_HandSolder
Connections:
- net +3V3: now also C26.1
- net GND: now also C26.2, D7.1 (K), D8.1 (K), D9.1 (K)
- net at IC1.13 (P8): now also R47.2
- net at IC1.15 (P10): now also TP3.1
- net at IC1.16 (P11): now also R46.2
- net at IC1.17 (P12): now also TP2.1
- net at IC1.19 (P14): now also TP1.1
- net at IC1.20 (P15): now also R30.2
- new net: D7.2 (A), R30.1
- new net: D8.2 (A), R46.1
- new net: D9.2 (A), R47.1
- no-connect marks 38 -> 32
Other:
- moved on the sheet: C23, IC1, JP1, R10, R11, R12, R13, R14, R15, R16, R17, R18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

Commit message: Y
Connections:
- net ADC_CH0 renamed POWER_MEASUREMENTS/ADC_CH0
- net ADC_CH1 renamed POWER_MEASUREMENTS/ADC_CH1
- net ADC_CH2 renamed POWER_MEASUREMENTS/ADC_CH2
- net ADC_CH3 renamed POWER_MEASUREMENTS/ADC_CH3
- net ADC_CH5 renamed POWER_MEASUREMENTS/ADC_CH5
- net ADC_CH6 renamed POWER_MEASUREMENTS/ADC_CH6
Other:
- sheet POWER_MEASUREMENTS ports: added ADC_CH0, ADC_CH1, ADC_CH2, ADC_CH3, ADC_CH5, ADC_CH6; removed none
- sheet Power-IN-OUT-BMS ports: added 5v; removed none
- note added: "ADC ON SIDE"
- note added: "AUDIO ON SIDE"
- note added: "MCU can: push 40mA out pull 28mA in 350mA max consumption (wifi)"
- note added: "USD CARD SOCKET"
- note added: "graphics+ mechanical"
- note added: "test points for bodges later one"
- note removed: "MCU can: push 40mA out pull 28mA in"
- note removed: "SD CARD ADAPTER"
- title: ESP32 audio power meter SD dataloger -> ESP32 MP3 player/web radio+power meter+uSD dataloger
- moved on the sheet: C8, D1, D5, D6, FID1, FID2, FID3, FID4, FID5, H1, H2, H3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
Changed lines of the file:
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@@
   (paper "A3")
   (title_block
-    (title "ESP32 audio power meter SD dataloger")
-    (rev "1")
+    (title "ESP32 MP3 player/web radio+power meter+uSD dataloger")
+    (date "2022-06-30")
+    (rev "2")
   )
