File: test_project_01/untitled.kicad_sch (KiCad schematic)
At the start: 12 parts

Commit message: j
Parts:
- removed J? (x3): Conn_01x02_Female, symbol Connector:Conn_01x02_Female
- removed R?: 0.01, symbol Device:R_Small
- added J4: Conn_01x02_Female, Connector_Wire:SolderWire-1sqmm_1x02_P5.4mm_D1.4mm_OD2.7mm, symbol Connector:Conn_01x02_Female
- added JP1: Jumper_3_Open, symbol Jumper:Jumper_3_Open
- added R1, R2, R6, R7, R8: 50k, symbol Device:R_Small
- added R10: 0.01, symbol Device:R_Small
- added R9: 150k, symbol Device:R_Small
- added U1, U2: LM7171xIM, Package_SO:SOIC-8_3.9x4.9mm_P1.27mm, symbol Amplifier_Operational:LM7171xIM
- J1: renamed from J?; footprint (none) -> Connector_Wire:SolderWire-1sqmm_1x02_P5.4mm_D1.4mm_OD2.7mm
- J6: renamed from J?; footprint (none) -> Connector_Wire:SolderWire-0.75sqmm_1x02_P4.8mm_D1.25mm_OD2.3mm
- R3: renamed from R?; value R_Small -> 50k
- R4: renamed from R?; value R_Small -> 1M
- gave numbers to parts that had none: 4
Connections:
- net GND: now also J1.2 (Pin_2), J2.2 (Pin_2), J3.2 (Pin_2), J5.4 (GND), J5.5 (Shield), J6.2 (Pin_2), R3.1, J4.2 (Pin_2), R1.2, R6.2, R8.1, U1.4 (V-), U2.4 (V-)
- net input+: now reaches J1.1 (Pin_1), J2.1 (Pin_1), J3.1 (Pin_1)
- net input+: now also R4.2, R5.1
- net at R4.1: now also R3.2, U1.3 (+)
- net output+: now reaches R5.2
- net output+: now also J4.1 (Pin_1)
- net mini_power_out: now reaches J5.1 (VBUS), J6.1 (Pin_1)
- net mini_power_out: now also R10.2
- net at J5.2 (D-): now also J5.3 (D+)
- new net: R8.2, R9.1, U2.3 (+)
- new net: R2.2, U1.2 (-)
- new net: JP1.2 (C), R10.1, R9.2
- new net: R7.2, U2.2 (-)
- new net +3V3: JP1.3 (B), U1.7 (V+), U2.7 (V+)
- new net +5V: JP1.1 (A)
- new net V_sense1: R1.1, R2.1, R6.1, R7.1, U1.6, U2.6
Other:
- note added: "2 tyoes of jack and 1 open pads 5 12 24V max 3A for all"
- note added: "3A so 30mV 100mA so 1mV so max amplification is x100 ADC 12bit 3v3 can sense steps of 0.73mV"
- note added: "50/1050 so 1/21 so max 1.14V"
- note added: "5V with 500mA to 1uA ?"
- note added: "INA IC available gains 20 50 100 200 ; 1 2 4 channels available"
- note added: "P=I^2 * R so 9*0.01 => 0.09W"
- note added: "X2 amplification and opamp isolation so 2.28V max"
- note added: "drop on 0.01 500mA 5mV 5mA 0.05mV 5uA 10^-8V"
- note added: "drop on 0.1 500mA 50mV 5mA 0.5mV 5uA 5*10^-7V"
- note added: "drop on 1 500mA 500mV 5mA 5mV 5uA 5*10^-6V"
- note added: "isolation and scaling down 2*( 1/4) = 1/2 so 2.5V max"
- note removed: "2 tyoes of jack and 1 open pads"
- moved on the sheet: J1, J2, J3, J5, J6, R3, R4, R5

Commit message: v
Other:
- note added: "drop on 1 500mA 500mV 5mA 5mV 50uA 0.05mV"
- note added: "so if i use +-1% sense resistor and a sense op amp with a gain of 100 and +-100uV ADC 12bit 3v3 can sense steps of 0.73mV then over a 0.1 ohm Rsense ill have : drop on 0.1 500mA 50mV so 495-505mV +-0.1 neglectable error i think 5mA 0.5mV 4.95-5.05 mV+-0.1 6-7 divisions on the ADC so still sort of ok i think 0.5mA 0.05mV 0.495-0.505mV+-0.1 , going under ADC So i think for me the min unit i cam mea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"
- note removed: "drop on 1 500mA 500mV 5mA 5mV 5uA 5*10^-6V"
- moved on the sheet: JP1, R10, R6, R7, R8, R9, U2

Commit message: f
Parts:
- added IC5: INA2181A4QDGSRQ1, SOP50P490X110-10N, symbol SamacSys_Parts:INA2181A4QDGSRQ1

Commit message: d
Parts:
- removed U1, U2: LM7171xIM, Package_SO:SOIC-8_3.9x4.9mm_P1.27mm, symbol Amplifier_Operational:LM7171xIM
- added C10, C9: 0.1u, symbol Device:C_Small
- added R17, R18, R19, R20: 50k, symbol Device:R_Small
- added U1: LM2902, Package_SO:SOIC-14_3.9x8.7mm_P1.27mm, symbol Amplifier_Operational:LM2902
- R10: value 0.01 -> 1
- R5: value 0.01 -> 0.05
Connections:
- net +3V3: now also IC5.10 (VS), C10.1, C9.1, U1.4 (V+); no longer JP1.3 (B)
- net GND: now also IC5.4 (GND), IC5.5 (REF1), IC5.6 (REF2), J1.1 (Pin_1), J2.1 (Pin_1), J3.1 (Pin_1), J4.1 (Pin_1), C10.2, C9.2, R20.2, U1.11 (V-); no longer J1.2 (Pin_2), J2.2 (Pin_2), J3.2 (Pin_2), J4.2 (Pin_2)
- net V_sense1: now also U1.8; no longer R1.1, R2.1
- net at R8.2, R9.1: now also U1.10 (+)
- net INA218_OUT: now reaches IC5.1 (OUT1)
- net INA218_IN-: now reaches IC5.2 (IN-1)
- net INA218_IN+: now reaches IC5.3 (IN+1)
- net source_vcc: now reaches IC5.7 (IN+2)
- net source_vcc: now also J4.2 (Pin_2), R4.2, R5.1
- net load_vcc: now reaches IC5.8 (IN-2)
- net load_vcc: now also J1.2 (Pin_2), J2.2 (Pin_2), J3.2 (Pin_2), R5.2
- net ADC_CH1: now reaches IC5.9 (OUT2)
- net mini_power_source: now reaches JP1.2 (C), R10.1, R9.2
- net mini_power_source: now also R17.2
- net at R7.2: now also U1.9 (-)
- removed net input+: J1.1 (Pin_1), J2.1 (Pin_1), J3.1 (Pin_1), R4.2, R5.1
- net mini_power_out renamed ext_5v
- net ext_5v: now also JP1.3 (B); no longer R10.2
- removed net output+: J4.1 (Pin_1), R5.2
- new net: R17.1, R19.2, U1.13 (-)
- new net: R18.2, R20.1, U1.12 (+)
- new net ADC_CH3: R19.1, U1.14
- new net V_sense2: R1.1, R2.1, U1.7
- new net mini_power_load: R10.2, R18.1
- new net op_amp+: U1.3 (+)
- new net op_amp-: U1.2 (-)
- new net op_amp_out: U1.1
Other:
- note added: "50/1050 so 1/21"
- note added: "ADC 12bit 3v3 can sense steps of 0.73mV INA is X200"
- note added: "P=I^2 * R so 9*0.05 => 0.45W"
- note added: "R=0.05 INA X200 5V max 3A so 150mV so 30 V 1A so 50mV so 10 V 0.1A so 5mV so 1 V 0.01A so 0.5mV so 0.1V"
- note added: "R=1 INA is x200 100mA 0.1v so 20v 10mA 0.01v so 2v 1mA 0.001v so 0.2v 0.1mA 0.0001v so 0.02v 0.01mA 0.00001v so 0.002v"
- note added: "X2 amplification and opamp isolation so: 24V 24/21*2 so 2.29V 12V 1.15V 5V 0.48V"
- note removed: "3A so 30mV 100mA so 1mV so max amplification is x100 ADC 12bit 3v3 can sense steps of 0.73mV"
- note removed: "50/1050 so 1/21 so max 1.14V"
- note removed: "INA IC available gains 20 50 100 200 ; 1 2 4 channels available"
- note removed: "P=I^2 * R so 9*0.01 => 0.09W"
- note removed: "X2 amplification and opamp isolation so 2.28V max"
- note removed: "drop on 0.01 500mA 5mV 5mA 0.05mV 5uA 10^-8V"
- note removed: "drop on 0.1 500mA 50mV 5mA 0.5mV 5uA 5*10^-7V"
- note removed: "drop on 1 500mA 500mV 5mA 5mV 50uA 0.05mV"
- title: (none) -> ESP32 audio power meter SD dataloger
- moved on the sheet: IC5, J4

Commit message: h
Parts:
- removed J3: Conn_01x02_Female, symbol Connector:Conn_01x02_Female
- removed J4: Conn_01x02_Female, Connector_Wire:SolderWire-1sqmm_1x02_P5.4mm_D1.4mm_OD2.7mm, symbol Connector:Conn_01x02_Female
- removed J5: USB_A, symbol Connector:USB_A
- added J12: Conn_02x05_Odd_Even, Connector_PinHeader_2.54mm:PinHeader_2x05_P2.54mm_Vertical, symbol Connector_Generic:Conn_02x05_Odd_Even
- added J3: Conn_01x02, Connector_PinHeader_2.54mm:PinHeader_1x02_P2.54mm_Vertical, symbol Connector_Generic:Conn_01x02
- added J5: 10033527-N3112MLF, SamacSys_Parts:10033527N3112MLF, symbol SamacSys_Parts:10033527-N3112MLF
- added R14, R26: 0.05, Resistor_THT:R_Axial_DIN0309_L9.0mm_D3.2mm_P15.24mm_Horizontal, symbol Device:R_Small
- added R27: 1, Resistor_THT:R_Axial_DIN0309_L9.0mm_D3.2mm_P15.24mm_Horizontal, symbol Device:R_Small
- added SW2: RA12131100, Z_mycustom_footprint_lib:RA12131100, symbol My_custom_lib:RA12131100
- C10, C9: footprint (none) -> Capacitor_SMD:C_0603_1608Metric_Pad1.08x0.95mm_HandSolder
- IC5: footprint SOP50P490X110-10N -> SamacSys_Parts:SOP50P490X110-10N
- J1: footprint Connector_Wire:SolderWire-1sqmm_1x02_P5.4mm_D1.4mm_OD2.7mm -> Connector_BarrelJack:BarrelJack_GCT_DCJ200-10-A_Horizontal
- J2: footprint (none) -> Connector_BarrelJack:BarrelJack_GCT_DCJ200-10-A_Horizontal
- JP1: footprint (none) -> Connector_PinHeader_2.54mm:PinHeader_1x03_P2.54mm_Vertical
- R1, R17, R18, R19, R2, R20, R3, R4, R6, R7, R8, R9: footprint (none) -> Resistor_SMD:R_0603_1608Metric_Pad0.98x0.95mm_HandSolder
- R10, R5: footprint (none) -> Resistor_THT:R_Axial_DIN0309_L9.0mm_D3.2mm_P15.24mm_Horizontal
Connections:
- net +3V3: now also J12.1 (Pin_1), J12.2 (Pin_2)
- net GND: now also J12.3 (Pin_3), J12.4 (Pin_4), J5.4, J5.5, J5.MP1, J5.MP2, J5.MP3, J5.MP4
- net ext_5v: now also J5.1
- net load_vcc: now also R14.2, R26.2; no longer J1.2 (Pin_2), J2.2 (Pin_2)
- net mini_power_load: now also R27.2; no longer R10.2
- net mini_power_source: now also J3.1 (Pin_1)
- net op_amp+: now also J12.5 (Pin_5), J12.6 (Pin_6)
- net op_amp-: now also J12.10 (Pin_10), J12.9 (Pin_9)
- net op_amp_out: now also J12.7 (Pin_7), J12.8 (Pin_8)
- net source_vcc: now also J1.2 (Pin_2), J2.2 (Pin_2), SW2.1
- net at R3.2, R4.1: now also U1.5 (+)
- net at U1.6 (-): now also R2.2
- net V_sense1 renamed ADC_CH0
- net V_sense2 renamed ADC_CH2
- new net: J3.2 (Pin_2), R10.2, R27.1
- new net: R14.1, R26.1, SW2.2
- new net: J5.2, J5.3
Other:
- note added: "R=0.05 INA X200 5V max 1/3 3A so 150mV so 30 V so 10V 1A so 50mV so 10 V so 3V3 0.1A so 5mV so 1 V so 0.33V 0.01A so 0.5mV so 0.1V so 0.003V"
- note removed: "R=0.05 INA X200 5V max 3A so 150mV so 30 V 1A so 50mV so 10 V 0.1A so 5mV so 1 V 0.01A so 0.5mV so 0.1V"
- moved on the sheet: C10, C9, J1, J6, JP1, R10, R17, R18, R19, R20, R6, R7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

Commit message: r
Parts:
- added U9: (no value), symbol Amplifier_Operational:LM324A
Connections:
- net +3V3: now also C10.2, U9.4 (V+); no longer C10.1, U1.4 (V+)
- net GND: now also C10.1, U9.11 (V-); no longer C10.2, U1.11 (V-)
Other:
- moved on the sheet: C10, C9, IC5, J1, J12, J2, J3, J5, J6, JP1, R1, R10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

Commit message: j
Parts:
- U9: value (none) -> LM324A; footprint (none) -> Package_SO:SOIC-14_3.9x8.7mm_P1.27mm
- U9: value (none) -> LM324A
Other:
- note added: "Extra op amp"
- note added: "USB input for power only"
- moved on the sheet: J12, J5, J6
