File: test_project_01/untitled.kicad_sch (KiCad schematic)
At the start: 30 parts, among them IC5 INA2181A4QDGSRQ1, J1 Conn_01x02_Female, J12 Conn_02x05_Odd_Even, J2 Conn_01x02_Female, J3 Conn_01x02, J5 10033527-N3112MLF, J6 Conn_01x02_Female, SW2 RA12131100, U1 LM2902, U9 LM324A

Commit message: h
Parts:
- removed J1, J2: Conn_01x02_Female, Connector_BarrelJack:BarrelJack_GCT_DCJ200-10-A_Horizontal, symbol Connector:Conn_01x02_Female
- removed J12: Conn_02x05_Odd_Even, Connector_PinHeader_2.54mm:PinHeader_2x05_P2.54mm_Vertical, symbol Connector_Generic:Conn_02x05_Odd_Even
- removed J6: Conn_01x02_Female, Connector_Wire:SolderWire-0.75sqmm_1x02_P4.8mm_D1.25mm_OD2.3mm, symbol Connector:Conn_01x02_Female
- removed R10: 1, Resistor_THT:R_Axial_DIN0309_L9.0mm_D3.2mm_P15.24mm_Horizontal, symbol Device:R_Small
- removed R14: 0.05, Resistor_THT:R_Axial_DIN0309_L9.0mm_D3.2mm_P15.24mm_Horizontal, symbol Device:R_Small
- removed R18, R19: 50k, Resistor_SMD:R_0603_1608Metric_Pad0.98x0.95mm_HandSolder, symbol Device:R_Small
- removed R9: 150k, Resistor_SMD:R_0603_1608Metric_Pad0.98x0.95mm_HandSolder, symbol Device:R_Small
- removed SW2: RA12131100, Z_mycustom_footprint_lib:RA12131100, symbol My_custom_lib:RA12131100
- removed U1: LM2902, Package_SO:SOIC-14_3.9x8.7mm_P1.27mm, symbol Amplifier_Operational:LM2902
- added J1, J7: Conn_01x02, symbol Connector_Generic:Conn_01x02
- added J10, J17: Conn_01x02, TestPoint:TestPoint_2Pads_Pitch5.08mm_Drill1.3mm, symbol Connector_Generic:Conn_01x02
- added J12: Conn_01x03, Connectors:SCREWTERMINAL-5MM-3, symbol Connector_Generic:Conn_01x03
- added J14, J2: (no value), symbol Connector_Generic:Conn_01x02
- added J15: (no value), symbol Connector_Generic:Conn_02x03_Odd_Even
- added J16, J6: (no value), symbol Connector_Generic:Conn_01x03
- added R10, R18: 1ohm 3W, Resistor_THT:R_Axial_DIN0207_L6.3mm_D2.5mm_P15.24mm_Horizontal, symbol Device:R
- added R14, R9: (no value), symbol Device:R
- added R19: 0.5ohm 2W, Resistor_THT:R_Axial_DIN0207_L6.3mm_D2.5mm_P15.24mm_Horizontal, symbol Device:R
- R1, R20: value 50k -> 10k
- R17, R2, R3, R6, R7, R8: value 50k -> (none); footprint Resistor_SMD:R_0603_1608Metric_Pad0.98x0.95mm_HandSolder -> (none)
- R26: value 0.05 -> 10k; footprint Resistor_THT:R_Axial_DIN0309_L9.0mm_D3.2mm_P15.24mm_Horizontal -> Resistor_SMD:R_0603_1608Metric_Pad0.98x0.95mm_HandSolder
- R27: value 1 -> 10k; footprint Resistor_THT:R_Axial_DIN0309_L9.0mm_D3.2mm_P15.24mm_Horizontal -> Resistor_SMD:R_0603_1608Metric_Pad0.98x0.95mm_HandSolder
- R4: value 1M -> (none)
- R5: value 0.05 -> (none); footprint Resistor_THT:R_Axial_DIN0309_L9.0mm_D3.2mm_P15.24mm_Horizontal -> (none)
Connections:
- net ADC_CH0: now also R20.1, U9.8; no longer R6.1, R7.1
- net ADC_CH2: now also U9.1, J15.1 (Pin_1), J15.3 (Pin_3), J15.5 (Pin_5); no longer R1.1, R2.1
- net ADC_CH3: now also R1.1, U9.7
- net GND: now also R2.2, R26.2, R27.1, R6.1, J1.1 (Pin_1), J10.1 (Pin_1), J12.2 (Pin_2), J17.2 (Pin_2), J2.1 (Pin_1), J6.2 (Pin_2), J7.1 (Pin_1); no longer R1.2, R20.2, R3.1, R6.2
- net ext_5v: now also J17.1 (Pin_1)
- net load_vcc: now also J10.2 (Pin_2), J7.2 (Pin_2), R10.1, R14.2, R9.2; no longer IC5.8 (IN-2), R26.2, R5.2
- net mini_power_load: now also IC5.8 (IN-2), R19.1; no longer R27.2
- net mini_power_source: now also IC5.7 (IN+2), R18.2
- net source_vcc: now also R7.2, U9.3 (+), J1.2 (Pin_2), J16.1 (Pin_1), J2.2 (Pin_2), J6.1 (Pin_1), R9.1; no longer IC5.7 (IN+2), R4.2, R5.1
- net at R4.1: now also J15.4 (Pin_4); no longer R3.2
- net at R17.1: now also R20.2, U9.10 (+)
- net at J3.2 (Pin_2): now also R18.1, R19.2; no longer R27.1
- net at R8.2: now also R2.1, U9.6 (-)
- net at R26.1: now also R27.2, U9.9 (-)
- net at U9.2 (-): now also R3.2, R4.2, R5.2, R6.2
- net at U9.5 (+): now also R1.2, R7.1
- new net: J16.2 (Pin_2), R10.2, R14.1
- new net: J15.6 (Pin_6), R5.1
- new net: J15.2 (Pin_2), R3.1
- no-connect marks 0 -> 3
Other:
- note added: "0.25ohm 3A so 750mV 1A so 250mV 0.1A so 25mV 0.01A so 2.5mV So amplification can be between 4 and 1300 with 0.5 ohm (jumper off) 3A so 1.5V 1A so 0.5V 0.1A so 50mV 0.01A so 5mV so amplification can be 2 to 650"
- note added: "1/10 voltage ratio"
- note added: "LARGE CURRENT 24V 3A MAX"
- note added: "P=I^2 * R so 9*0.25 => 2.25W 0.75V max"
- note added: "R=0.05 INA X200 5V max 0.25ohm 3A so 150mV so 30 V so 10V 1A so 50mV so 10 V so 3V3 0.1A so 5mV so 1 V so 0.33V 0.01A so 0.5mV so 0.1V so 0.003V"
- note added: "R=0.5 INA is x200 1A 0.5V so 100V 100mA 0.05v so 10v 10mA 0.005v so 1v 1mA 0.0005v so 0.1v 0.1mA 0.00005v so 0.01v 0.01mA 0.000005v so 0.001v"
- note added: "SMALL CURRENT 5V OR LESS"
- note added: "input port"
- note added: "or if 1ohm is on 10mA 0.015v so 3v 1mA 0.0015v so 0.3v 0.1mA 0.00015v so 0.03v"
- note added: "output port"
- note added: "ratio 1+ Rhigh/Rlow x5 x50 x500"
- note removed: "2 tyoes of jack and 1 open pads 5 12 24V max 3A for all"
- note removed: "50/1050 so 1/21"
- note removed: "Extra op amp"
- note removed: "P=I^2 * R so 9*0.05 => 0.45W"
- note removed: "R=0.05 INA X200 5V max 1/3 3A so 150mV so 30 V so 10V 1A so 50mV so 10 V so 3V3 0.1A so 5mV so 1 V so 0.33V 0.01A so 0.5mV so 0.1V so 0.003V"
- note removed: "R=1 INA is x200 100mA 0.1v so 20v 10mA 0.01v so 2v 1mA 0.001v so 0.2v 0.1mA 0.0001v so 0.02v 0.01mA 0.00001v so 0.002v"
- note removed: "X2 amplification and opamp isolation so: 24V 24/21*2 so 2.29V 12V 1.15V 5V 0.48V"
- note removed: "isolation and scaling down 2*( 1/4) = 1/2 so 2.5V max"
- note removed: "load"
- note removed: "source"
- moved on the sheet: C10, C9, IC5, J3, J5, JP1, R17, U9A, U9B, U9C, U9D, U9E

Commit message: j
Parts:
- removed R2, R8: (no value), symbol Device:R_Small
- removed R26, R27: 10k, Resistor_SMD:R_0603_1608Metric_Pad0.98x0.95mm_HandSolder, symbol Device:R_Small
- added J?: Conn_01x03, Connector_PinSocket_2.54mm:PinSocket_1x03_P2.54mm_Vertical, symbol Connector_Generic:Conn_01x03
- added R?: 47k, Resistor_SMD:R_0603_1608Metric_Pad0.98x0.95mm_HandSolder, symbol Device:R_Small
- J14: value (none) -> Conn_01x02
- J15: value (none) -> jumper selector
- J16: value (none) -> Conn_01x03; footprint (none) -> Connector_PinSocket_2.54mm:PinSocket_1x03_P2.54mm_Vertical
- J2: value (none) -> Conn_01x02; footprint (none) -> TestPoint:TestPoint_2Pads_Pitch5.08mm_Drill1.3mm
- J6: value (none) -> Conn_01x03; footprint (none) -> Connectors:SCREWTERMINAL-5MM-3
- R14: value (none) -> 1ohm 3W; footprint (none) -> Resistor_THT:R_Axial_DIN0207_L6.3mm_D2.5mm_P15.24mm_Horizontal
- R17: value (none) -> 10k; footprint (none) -> Resistor_SMD:R_0603_1608Metric_Pad0.98x0.95mm_HandSolder
- R3: value (none) -> 4k; footprint (none) -> Resistor_SMD:R_0603_1608Metric_Pad0.98x0.95mm_HandSolder
- R4: value (none) -> 40k
- R5: value (none) -> 400k; footprint (none) -> Resistor_SMD:R_0603_1608Metric_Pad0.98x0.95mm_HandSolder
- R6: value (none) -> 1k; footprint (none) -> Resistor_SMD:R_0603_1608Metric_Pad0.98x0.95mm_HandSolder
- R7: value (none) -> 100k; footprint (none) -> Resistor_SMD:R_0603_1608Metric_Pad0.98x0.95mm_HandSolder
- R9: value (none) -> 0.5ohm 2W; footprint (none) -> Resistor_THT:R_Axial_DIN0207_L6.3mm_D2.5mm_P15.24mm_Horizontal
Connections:
- net ADC_CH0: now also U9.9 (-); no longer R20.1
- net ADC_CH3: now also U9.6 (-); no longer R1.1
- net GND: now also R1.1, R20.1
- net source_vcc: now also J?.2 (Pin_2)
- net at R1.2, R7.1, U9.5 (+): now also R?.1
- new net: J?.1 (Pin_1), R?.2
- no-connect marks 3 -> 4
Other:
- note added: "when ok ratio is about 10/32"

Commit message: f
Parts:
- removed C9: 0.1u, Capacitor_SMD:C_0603_1608Metric_Pad1.08x0.95mm_HandSolder, symbol Device:C_Small
- removed IC5: INA2181A4QDGSRQ1, SamacSys_Parts:SOP50P490X110-10N, symbol SamacSys_Parts:INA2181A4QDGSRQ1
- removed J1, J7: Conn_01x02, symbol Connector_Generic:Conn_01x02
- removed J10, J2: Conn_01x02, TestPoint:TestPoint_2Pads_Pitch5.08mm_Drill1.3mm, symbol Connector_Generic:Conn_01x02
- removed J15: jumper selector, symbol Connector_Generic:Conn_02x03_Odd_Even
- removed R10: 1ohm 3W, Resistor_THT:R_Axial_DIN0207_L6.3mm_D2.5mm_P15.24mm_Horizontal, symbol Device:R
- removed R3: 4k, Resistor_SMD:R_0603_1608Metric_Pad0.98x0.95mm_HandSolder, symbol Device:R_Small
- removed R4: 40k, Resistor_SMD:R_0603_1608Metric_Pad0.98x0.95mm_HandSolder, symbol Device:R_Small
- removed R5: 400k, Resistor_SMD:R_0603_1608Metric_Pad0.98x0.95mm_HandSolder, symbol Device:R_Small
- removed R6: 1k, Resistor_SMD:R_0603_1608Metric_Pad0.98x0.95mm_HandSolder, symbol Device:R_Small
- added C201: 0.1u, Capacitor_SMD:C_0603_1608Metric_Pad1.08x0.95mm_HandSolder, symbol Device:C_Small
- added C202: 1u, Capacitor_SMD:C_0603_1608Metric_Pad1.08x0.95mm_HandSolder, symbol Device:C_Small
- added J201: Barrel_Jack_Switch, Z_mycustom_footprint_lib:DC plug jack 5.5-2.5mm, symbol Connector:Barrel_Jack_Switch
- added J203: Barrel_Jack_Switch, Connector_BarrelJack:BarrelJack_Wuerth_6941xx301002, symbol Connector:Barrel_Jack_Switch
- added J208: USB_A, Connector_USB:USB_A_Molex_67643_Horizontal, symbol Connector:USB_A
- added J212: Conn_01x02, TestPoint:TestPoint_2Pads_Pitch5.08mm_Drill1.3mm, symbol Connector_Generic:Conn_01x02
- added R202, R203, R216, R217: 100k, Resistor_SMD:R_0603_1608Metric_Pad0.98x0.95mm_HandSolder, symbol Device:R_Small
- added R204, R205, R218, R219: 10k, Resistor_SMD:R_0603_1608Metric_Pad0.98x0.95mm_HandSolder, symbol Device:R_Small
- added R209: 1ohm 3W, Resistor_THT:R_Axial_DIN0207_L6.3mm_D2.5mm_P5.08mm_Vertical, symbol Device:R
- added R211: 1M, Resistor_SMD:R_0603_1608Metric_Pad0.98x0.95mm_HandSolder, symbol Device:R_Small
- J209: renamed from J14; footprint (none) -> Connector_PinSocket_2.54mm:PinSocket_1x02_P2.54mm_Vertical
- R208: renamed from R9; footprint Resistor_THT:R_Axial_DIN0207_L6.3mm_D2.5mm_P15.24mm_Horizontal -> Resistor_THT:R_Axial_DIN0207_L6.3mm_D2.5mm_P5.08mm_Vertical
- R210: renamed from R14; footprint Resistor_THT:R_Axial_DIN0207_L6.3mm_D2.5mm_P15.24mm_Horizontal -> Resistor_THT:R_Axial_DIN0207_L6.3mm_D2.5mm_P5.08mm_Vertical
- R212: renamed from R18; footprint Resistor_THT:R_Axial_DIN0207_L6.3mm_D2.5mm_P15.24mm_Horizontal -> Resistor_THT:R_Axial_DIN0207_L6.3mm_D2.5mm_P5.08mm_Vertical
- R213: renamed from R19; footprint Resistor_THT:R_Axial_DIN0207_L6.3mm_D2.5mm_P15.24mm_Horizontal -> Resistor_THT:R_Axial_DIN0207_L6.3mm_D2.5mm_P5.08mm_Vertical
- U201: renamed from U9; footprint (none) -> Package_SO:SOIC-14_3.9x8.7mm_P1.27mm
- gave numbers to parts that had none: 2
- renumbered C10 to C203, J6 to J202, J12 to J204, J16 to J207, J5 to J210, J17 to J211, J3 to J213, JP1 to JP201, R1 to R201, R7 to R206, R20 to R214, R17 to R215, U9 to U201
Connections:
- net +3V3: now also C202.1
- net ADC_CH1: now also U201.14, R216.1
- net ADC_CH2: now also R202.1
- net GND: now also C201.2, C202.2, J201.2, J203.2, J208.4 (GND), J212.1 (Pin_1), R203.1, R211.1, R217.1; no longer J210.5
- net load_vcc: now also J204.1 (Pin_1), R205.2, R209.1
- net mini_power_load: now also J208.1 (VBUS), J212.2 (Pin_2), R218.2
- net mini_power_source: now also R219.2
- net source_vcc: now also J201.1, J203.1, R204.2; no longer U201.3 (+)
- net at U201.2 (-): now also R202.2, R205.1
- net at J207.2 (Pin_2), R210.1: now also R209.2
- net at U201.12 (+): now also R217.2, R219.1
- net at U201.13 (-): now also R216.2, R218.1
- net D2+: now reaches J210.3
- net D2+: now also J208.3 (D+); no longer J210.2
- new net: R203.2, R204.1, U201.3 (+)
- new net: C201.1, J208.5 (Shield), R211.2
- new net D2-: J208.2 (D-), J210.2
- no-connect marks 4 -> 7
Other:
- note added: "optimusdigital USB2 normal"
- note added: "x10 gain"
- note removed: "5V with 500mA to 1uA ?"
- note removed: "ADC 12bit 3v3 can sense steps of 0.73mV INA is X200"
- note removed: "R=0.5 INA is x200 1A 0.5V so 100V 100mA 0.05v so 10v 10mA 0.005v so 1v 1mA 0.0005v so 0.1v 0.1mA 0.00005v so 0.01v 0.01mA 0.000005v so 0.001v"
- note removed: "or if 1ohm is on 10mA 0.015v so 3v 1mA 0.0015v so 0.3v 0.1mA 0.00015v so 0.03v"
- note removed: "ratio 1+ Rhigh/Rlow x5 x50 x500"
- moved on the sheet: C203, J202, J204, J209, J213, JP201, R212, R213, R214, R215, U201C, U201D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
