File: test_project_01/untitled.kicad_sch (KiCad schematic)
At the start: 25 parts, among them IC201 INA2181A4QDGSRQ1, J201 Barrel_Jack_Switch, J202 Barrel_Jack_Switch, J203 Conn_01x03, J204 Conn_01x03, J205 Conn_01x03, J206 USB_A, J207 10033527-N3112MLF, J208 Conn_01x02, J209 Conn_01x02, U201 LM324A

Commit message: i
Parts:
- added J205: (no value), symbol Connector_Generic:Conn_01x04
- added R201, R202: 10k, Resistor_SMD:R_0603_1608Metric_Pad0.98x0.95mm_HandSolder, symbol Device:R_Small
- added R203, R204, R205, R206: (no value), symbol Device:R_Small
- R210: renamed from R204; value (none) -> 5m; footprint (none) -> Resistor_SMD:R_0612_1632Metric_Pad1.18x3.40mm_HandSolder
- renumbered J205 to J206, J206 to J207, J207 to J208, J208 to J209, J209 to J210, R201 to R207, R202 to R208, R203 to R209, R205 to R211, R206 to R212, R207 to R213, R208 to R214
Connections:
- net GND: now also J205.1 (Pin_1), R202.1, R205.1
- net at U201.12 (+): now also J205.4 (Pin_4)
- net at U201.13 (-): now also J205.3 (Pin_3)
- net at U201.14: now also J205.2 (Pin_2)
- net at U201.10 (+): now also R203.2, R206.1
- net ADC_CH5: now reaches U201.8
- net ADC_CH5: now also R206.2
- net at U201.9 (-): now also R204.2, R205.2
- new net ADC_CH6: R201.1, R202.2
- new net Power_in+: R201.2, R204.1
- new net Power_in-: R203.1
Other:
- note added: "100 gain"
- note added: "5m shunt with 2A max current so 10mV drop so max gain is 3/0.01= 300 so 100-300 gain is fine"
- moved on the sheet: U201C, U201D

Commit message: y
Parts:
- J205: value (none) -> Conn_01x04
- R203, R204: value (none) -> 1k; footprint (none) -> Resistor_SMD:R_0603_1608Metric_Pad0.98x0.95mm_HandSolder
- R205, R206: value (none) -> 100k; footprint (none) -> Resistor_SMD:R_0603_1608Metric_Pad0.98x0.95mm_HandSolder
- U201: value LM324A -> (none)
Other:
- moved on the sheet: J206, R207, R208, R209, R210, U201B

Commit message: r
Parts:
- removed J205: Conn_01x04, symbol Connector_Generic:Conn_01x04
- removed J206: Conn_01x03, Connector_PinSocket_2.54mm:PinSocket_1x03_P2.54mm_Vertical, symbol Connector_Generic:Conn_01x03
- removed R209: 47k, Resistor_SMD:R_0603_1608Metric_Pad0.98x0.95mm_HandSolder, symbol Device:R_Small
- removed unit 4 of U201
- R29: renamed from R208; value 100k -> (none); footprint Resistor_SMD:R_0603_1608Metric_Pad0.98x0.95mm_HandSolder -> (none)
- renumbered C201 to C10, C202 to C11, C203 to C12, C204 to C13, C205 to C14, IC201 to IC2, J208 to J10, J209 to J11, J210 to J12, J201 to J4, J202 to J5, J203 to J6, J204 to J7, J207 to J9, JP201 to JP2, R201 to R22, R202 to R23, R203 to R24, R204 to R25, R205 to R26, R206 to R27, R207 to R28, R210 to R31, R211 to R32, R212 to R33, R213 to R34, R214 to R35, U201 to U6
Connections:
- no-connect marks 6 -> 5
Other:
- note added: "1/11 voltage ratio"
- note removed: "1/10 voltage ratio"
- note removed: "when ok ratio is about 10/32"

Commit message: r
Parts:
- R29: value (none) -> 100k; footprint (none) -> Resistor_SMD:R_0603_1608Metric_Pad0.98x0.95mm_HandSolder
- U6: value (none) -> LM324A; footprint (none) -> Package_SO:SOIC-14_3.9x8.7mm_P1.27mm
Changed lines of the file:
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@@
     (in_bom yes) (on_board yes)
     (property "Reference" "U6" (id 0) (at 112.395 58.42 0))
-    (property "Value" "" (id 1) (at 112.395 60.96 0))
-    (property "Footprint" "" (id 2) (at 118.11 52.705 0)
+    (property "Value" "LM324A" (id 1) (at 112.395 60.96 0))
+    (property "Footprint" "Package_SO:SOIC-14_3.9x8.7mm_P1.27mm" (id 2) (at 118.11 52.705 0)
       (effects (font (size 1.27 1.27)) hide)
     )
@@
     (in_bom yes) (on_board yes)
     (property "Reference" "R29" (id 0) (at 133.35 45.72 90))
-    (property "Value" "" (id 1) (at 133.35 43.18 90))
-    (property "Footprint" "" (id 2) (at 133.35 48.26 0)
+    (property "Value" "100k" (id 1) (at 133.35 43.18 90))
+    (property "Footprint" "Resistor_SMD:R_0603_1608Metric_Pad0.98x0.95mm_HandSolder" (id 2) (at 133.35 48.26 0)
       (effects (font (size 1.27 1.27)) hide)
     )
@@
     (in_bom yes) (on_board yes)
     (property "Reference" "U6" (id 0) (at 355.6 34.925 0))
-    (property "Value" "" (id 1) (at 355.6 37.465 0))
-    (property "Footprint" "" (id 2) (at 362.585 28.575 0)
+    (property "Value" "LM324A" (id 1) (at 355.6 37.465 0))
+    (property "Footprint" "Package_SO:SOIC-14_3.9x8.7mm_P1.27mm" (id 2) (at 362.585 28.575 0)
       (effects (font (size 1.27 1.27)) hide)
     )
@@
       (effects (font (size 1.27 1.27)) (justify left))
     )
-    (property "Value" "" (id 1) (at 288.925 213.9949 0)
-      (effects (font (size 1.27 1.27)) (justify left))
-    )
-    (property "Footprint" "" (id 2) (at 289.56 210.185 0)
+    (property "Value" "LM324A" (id 1) (at 288.925 213.9949 0)
+      (effects (font (size 1.27 1.27)) (justify left))
+    )
+    (property "Footprint" "Package_SO:SOIC-14_3.9x8.7mm_P1.27mm" (id 2) (at 289.56 210.185 0)
       (effects (font (size 1.27 1.27)) hide)
     )
@@
     (in_bom yes) (on_board yes)
     (property "Reference" "U6" (id 0) (at 77.47 180.975 0))
-    (property "Value" "" (id 1) (at 77.47 183.515 0))
-    (property "Footprint" "" (id 2) (at 71.755 174.625 0)
-      (effects (font (size 1.27 1.27)) hide)
-    )
+    (property "Value" "LM324A" (id 1) (at 77.47 183.515 0))
+    (property "Footprint" "Package_SO:SOIC-14_3.9x8.7mm_P1.27mm" (id 2) (at 71.755 174.625 0)
+      (effects (font (size 1.27 1.27)) hide)
+    )

Commit message: Y
Other:
- note added: "MAIN ICs POWER AND CIRCUITRY"
- note added: "SELF POWER CONSUMPTION + LI ION CHARGEING CURRENT"
- title: ESP32 audio power meter SD dataloger -> ESP32 MP3 player/web radio+power meter+uSD dataloger
- moved on the sheet: R22, R23, R24, R25, R26, R27, U6C

Commit message: f
Parts:
- R32: value 1M -> 1Meg
Changed lines of the file:
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@@
     (in_bom yes) (on_board yes)
     (property "Reference" "R32" (id 0) (at 257.429 136.525 0))
-    (property "Value" "1M" (id 1) (at 257.429 139.065 0))
+    (property "Value" "1Meg" (id 1) (at 257.429 139.065 0))
     (property "Footprint" "Resistor_SMD:R_0603_1608Metric_Pad0.98x0.95mm_HandSolder" (id 2) (at 253.365 137.795 0)
       (effects (font (size 1.27 1.27)) hide)
