File: test_project_01/_autosave-untitled.kicad_sch (KiCad schematic)
At the start: 25 parts, among them IC201 INA2181A4QDGSRQ1, J201 Barrel_Jack_Switch, J202 Barrel_Jack_Switch, J203 Conn_01x03, J204 Conn_01x03, J205 Conn_01x03, J206 USB_A, J207 10033527-N3112MLF, J208 Conn_01x02, J209 Conn_01x02, U201 LM324A

Commit message: h
Parts:
- R208: value (none) -> 30m; footprint (none) -> Resistor_SMD:R_0402_1005Metric_Pad0.72x0.64mm_HandSolder
Changed lines of the file:
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@@
       (effects (font (size 1.27 1.27)) (justify right))
     )
-    (property "Value" "" (id 1) (at 371.475 77.47 0)
+    (property "Value" "30m" (id 1) (at 371.475 77.47 0)
       (effects (font (size 1.27 1.27)) (justify right))
     )
-    (property "Footprint" "" (id 2) (at 380.238 76.2 90)
+    (property "Footprint" "Resistor_SMD:R_0402_1005Metric_Pad0.72x0.64mm_HandSolder" (id 2) (at 380.238 76.2 90)
       (effects (font (size 1.27 1.27)) hide)
     )
