File: test_project_01/Power-IN-OUT-BMS.kicad_sch (KiCad schematic)
At the start: 28 parts

Commit message: r
Parts:
- gave numbers to parts that had none: 18

Commit message: j
Parts:
- C2: value (none) -> 1u; footprint (none) -> Capacitor_SMD:C_0603_1608Metric_Pad1.08x0.95mm_HandSolder
- C3: value (none) -> 4.7u; footprint (none) -> Capacitor_SMD:C_0603_1608Metric_Pad1.08x0.95mm_HandSolder
- D2, D3: value (none) -> LED_Small; footprint (none) -> LED_SMD:LED_0603_1608Metric_Pad1.05x0.95mm_HandSolder
- IC2: value (none) -> MCP73834T-FCI_UN; footprint (none) -> SamacSys_Parts:SOP50P490X110-10N
- J4: value (none) -> Conn_01x02; footprint (none) -> Connector_PinHeader_2.54mm:PinHeader_1x02_P2.54mm_Vertical
- R11, R13: value (none) -> 470; footprint (none) -> Resistor_SMD:R_0603_1608Metric_Pad0.98x0.95mm_HandSolder
- R15: value (none) -> 10k; footprint (none) -> Resistor_SMD:R_0603_1608Metric_Pad0.98x0.95mm_HandSolder
- RV1: value (none) -> R_Potentiometer; footprint (none) -> Z_mycustom_footprint_lib:2002102255
Changed lines of the file:
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@@
     (in_bom yes) (on_board yes) (fields_autoplaced)
     (property "Reference" "RV1" (id 0) (at 96.52 86.36 90))
-    (property "Value" "" (id 1) (at 96.52 88.9 90))
-    (property "Footprint" "" (id 2) (at 96.52 92.71 0)
+    (property "Value" "R_Potentiometer" (id 1) (at 96.52 88.9 90))
+    (property "Footprint" "Z_mycustom_footprint_lib:2002102255" (id 2) (at 96.52 92.71 0)
       (effects (font (size 1.27 1.27)) hide)
     )
@@
       (effects (font (size 1.27 1.27)) hide)
     )
-    (property "Value" "" (id 1) (at 57.15 92.71 0)
+    (property "Value" "GND" (id 1) (at 57.15 92.71 0)
       (effects (font (size 1.27 1.27)) hide)
     )
@@
       (effects (font (size 1.27 1.27)) (justify left))
     )
-    (property "Value" "" (id 1) (at 103.505 102.235 0)
-      (effects (font (size 1.27 1.27)) (justify left))
-    )
-    (property "Footprint" "" (id 2) (at 107.95 92.71 0)
+    (property "Value" "Conn_01x02" (id 1) (at 103.505 102.235 0)
+      (effects (font (size 1.27 1.27)) (justify left))
+    )
+    (property "Footprint" "Connector_PinHeader_2.54mm:PinHeader_1x02_P2.54mm_Vertical" (id 2) (at 107.95 92.71 0)
       (effects (font (size 1.27 1.27)) hide)
     )
@@
       (effects (font (size 1.27 1.27)) (justify right))
     )
-    (property "Value" "" (id 1) (at 46.99 87.63 0)
-      (effects (font (size 1.27 1.27)) (justify right))
-    )
-    (property "Footprint" "" (id 2) (at 45.72 82.55 0)
+    (property "Value" "470" (id 1) (at 46.99 87.63 0)
+      (effects (font (size 1.27 1.27)) (justify right))
+    )
+    (property "Footprint" "Resistor_SMD:R_0603_1608Metric_Pad0.98x0.95mm_HandSolder" (id 2) (at 45.72 82.55 0)
       (effects (font (size 1.27 1.27)) hide)
     )
@@
       (effects (font (size 1.27 1.27)) hide)
     )
-    (property "Value" "" (id 1) (at 109.22 80.01 0)
+    (property "Value" "GND" (id 1) (at 109.22 80.01 0)
       (effects (font (size 1.27 1.27)) hide)
     )
@@
     (in_bom yes) (on_board yes)
     (property "Reference" "D3" (id 0) (at 38.1 88.9 0))
-    (property "Value" "" (id 1) (at 38.1 86.36 0))
-    (property "Footprint" "" (id 2) (at 38.1 82.55 90)
+    (property "Value" "LED_Small" (id 1) (at 38.1 86.36 0))
+    (property "Footprint" "LED_SMD:LED_0603_1608Metric_Pad1.05x0.95mm_HandSolder" (id 2) (at 38.1 82.55 90)
       (effects (font (size 1.27 1.27)) hide)
     )
@@
     (in_bom yes) (on_board yes) (fields_autoplaced)
     (property "Reference" "IC2" (id 0) (at 74.93 67.31 0))
-    (property "Value" "" (id 1) (at 74.93 69.85 0))
-    (property "Footprint" "" (id 2) (at 88.9 72.39 0)
+    (property "Value" "MCP73834T-FCI_UN" (id 1) (at 74.93 69.85 0))
+    (property "Footprint" "SamacSys_Parts:SOP50P490X110-10N" (id 2) (at 88.9 72.39 0)
       (effects (font (size 1.27 1.27)) (justify left) hide)
     )
@@
       (effects (font (size 1.27 1.27)) (justify left))
     )
-    (property "Value" "" (id 1) (at 111.76 86.36 0)
-      (effects (font (size 1.27 1.27)) (justify left))
-    )
-    (property "Footprint" "" (id 2) (at 114.3 85.09 0)
+    (property "Value" "4.7u" (id 1) (at 111.76 86.36 0)
+      (effects (font (size 1.27 1.27)) (justify left))
+    )
+    (property "Footprint" "Capacitor_SMD:C_0603_1608Metric_Pad1.08x0.95mm_HandSolder" (id 2) (at 114.3 85.09 0)
       (effects (font (size 1.27 1.27)) hide)
     )
@@
       (effects (font (size 1.27 1.27)) hide)
     )
-    (property "Value" "" (id 1) (at 114.3 95.25 0)
+    (property "Value" "GND" (id 1) (at 114.3 95.25 0)
       (effects (font (size 1.27 1.27)) hide)
     )
@@
       (effects (font (size 1.27 1.27)) hide)
     )
-    (property "Value" "" (id 1) (at 40.64 69.85 0)
+    (property "Value" "GND" (id 1) (at 40.64 69.85 0)
       (effects (font (size 1.27 1.27)) hide)
     )
@@
       (effects (font (size 1.27 1.27)) (justify right))
     )
-    (property "Value" "" (id 1) (at 46.99 78.74 0)
-      (effects (font (size 1.27 1.27)) (justify right))
-    )
-    (property "Footprint" "" (id 2) (at 45.72 80.01 0)
+    (property "Value" "470" (id 1) (at 46.99 78.74 0)
+      (effects (font (size 1.27 1.27)) (justify right))
+    )
+    (property "Footprint" "Resistor_SMD:R_0603_1608Metric_Pad0.98x0.95mm_HandSolder" (id 2) (at 45.72 80.01 0)
       (effects (font (size 1.27 1.27)) hide)
     )
@@
       (effects (font (size 1.27 1.27)) hide)
     )
-    (property "Value" "" (id 1) (at 96.52 104.14 0)
+    (property "Value" "GND" (id 1) (at 96.52 104.14 0)
       (effects (font (size 1.27 1.27)) hide)
     )
@@
       (effects (font (size 1.27 1.27)) hide)
     )
-    (property "Value" "" (id 1) (at 33.02 57.15 0))
+    (property "Value" "+5V" (id 1) (at 33.02 57.15 0))
     (property "Footprint" "" (id 2) (at 33.02 62.23 0)
       (effects (font (size 1.27 1.27)) hide)
@@
       (effects (font (size 1.27 1.27)) (justify left))
     )
-    (property "Value" "" (id 1) (at 49.53 67.31 0)
-      (effects (font (size 1.27 1.27)) (justify left))
-    )
-    (property "Footprint" "" (id 2) (at 50.8 69.85 0)
+    (property "Value" "1u" (id 1) (at 49.53 67.31 0)
+      (effects (font (size 1.27 1.27)) (justify left))
+    )
+    (property "Footprint" "Capacitor_SMD:C_0603_1608Metric_Pad1.08x0.95mm_HandSolder" (id 2) (at 50.8 69.85 0)
       (effects (font (size 1.27 1.27)) hide)
     )
@@
       (effects (font (size 1.27 1.27)) hide)
     )
-    (property "Value" "" (id 1) (at 127 67.31 0))
+    (property "Value" "+BATT" (id 1) (at 127 67.31 0))
     (property "Footprint" "" (id 2) (at 127 72.39 0)
       (effects (font (size 1.27 1.27)) hide)
@@
       (effects (font (size 1.27 1.27)) (justify right))
     )
-    (property "Value" "" (id 1) (at 97.79 74.93 0)
-      (effects (font (size 1.27 1.27)) (justify right))
-    )
-    (property "Footprint" "" (id 2) (at 99.06 80.01 0)
+    (property "Value" "10k" (id 1) (at 97.79 74.93 0)
+      (effects (font (size 1.27 1.27)) (justify right))
+    )
+    (property "Footprint" "Resistor_SMD:R_0603_1608Metric_Pad0.98x0.95mm_HandSolder" (id 2) (at 99.06 80.01 0)
       (effects (font (size 1.27 1.27)) hide)
     )
@@
     (in_bom yes) (on_board yes) (fields_autoplaced)
     (property "Reference" "D2" (id 0) (at 38.0365 73.66 0))
-    (property "Value" "" (id 1) (at 38.0365 76.2 0))
-    (property "Footprint" "" (id 2) (at 38.1 80.01 90)
-      (effects (font (size 1.27 1.27)) hide)
-    )
+    (property "Value" "LED_Small" (id 1) (at 38.0365 76.2 0))
+    (property "Footprint" "LED_SMD:LED_0603_1608Metric_Pad1.05x0.95mm_HandSolder" (id 2) (at 38.1 80.01 90)
+      (effects (font (size 1.27 1.27)) hide)
+    )

Commit message: j
Other:
- note added: "18650 cell holder"
Changed lines of the file:
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@@
+    (effects (font (size 1.27 1.27)) (justify left bottom))
+  )
+  (text "18650 cell\nholder" (at 129.794 96.266 0)
     (effects (font (size 1.27 1.27)) (justify left bottom))
   )

Commit message: f
Parts:
- removed R30: 10k+ pullup, Resistor_SMD:R_0603_1608Metric_Pad0.98x0.95mm_HandSolder, symbol Device:R
- added J301: Conn_01x02, Connector_PinHeader_2.54mm:PinHeader_1x02_P2.54mm_Vertical, symbol Connector_Generic:Conn_01x02
- added R303: 1k, Resistor_SMD:R_0603_1608Metric_Pad0.98x0.95mm_HandSolder, symbol Device:R_Small
- U301: renamed from U2; footprint 1043 -> SamacSys_Parts:1043
- renumbered C2 to C301, C3 to C302, C4 to C303, C12 to C304, D2 to D301, D3 to D302, D1 to D303, D4 to D304, D5 to D305, D6 to D306, IC2 to IC301, IC3 to IC302, J4 to J302, J13 to J303, Q1 to Q301, R11 to R301, R13 to R302, R15 to R304, R12 to R305, R28 to R306, R29 to R307, R31 to R308, R32 to R309, RV1 to RV301, S2 to S301, U4 to U302
Connections:
- net at IC301.6 (PROG): now also J301.1 (Pin_1), R303.2; no longer RV301.3
- net TE: now reaches IC301.7 (~{PG(}TE))
- new net: J301.2 (Pin_2), R303.1, RV301.3
Other:
- note added: "timer enable"
- moved on the sheet: J302, RV301

Commit message: r
Parts:
- removed D306: LED_Small Green, LED_SMD:LED_0603_1608Metric_Pad1.05x0.95mm_HandSolder, symbol Device:LED_Small
- removed J303: Conn_01x03, Connector_PinHeader_2.54mm:PinHeader_1x03_P2.54mm_Vertical, symbol Connector_Generic:Conn_01x03
- removed R309: 330, Resistor_SMD:R_0603_1608Metric_Pad0.98x0.95mm_HandSolder, symbol Device:R

Commit message: h
Parts:
- removed J301: Conn_01x02, Connector_PinHeader_2.54mm:PinHeader_1x02_P2.54mm_Vertical, symbol Connector_Generic:Conn_01x02
- removed R303: 1k, Resistor_SMD:R_0603_1608Metric_Pad0.98x0.95mm_HandSolder, symbol Device:R_Small
- added R304, R305: 10k, Resistor_SMD:R_0603_1608Metric_Pad0.98x0.95mm_HandSolder, symbol Device:R_Small
- RV301: footprint Z_mycustom_footprint_lib:2002102255 -> Potentiometer_THT:Potentiometer_Bourns_3386F_Vertical
- renumbered J302 to J301, R304 to R303, R305 to R306, R306 to R307, R307 to R308, R308 to R309
Connections:
- net +BATT: now also R304.2
- net GND: now also R305.1
- net Set_charge_current: now reaches IC301.6 (PROG)
- net Set_charge_current: now also RV301.3
- net low_batt_shutoff: now reaches Q301.2 (G1), R306.2, U302.1 (RESET)
- new net ADC_CH4: R304.1, R305.2
Other:
- moved on the sheet: C301, C302, D301, D302, IC301, J301, R301, R302, R303, RV301

Commit message: i
Parts:
- added R308: 5m, Resistor_SMD:R_0612_1632Metric_Pad1.18x3.40mm_HandSolder, symbol Device:R
- renumbered R308 to R309, R309 to R310
Connections:
- net +VDC: now also R308.2; no longer D303.1 (K), Q301.3 (S2)
- new net Power_in+: D303.1 (K), Q301.3 (S2), R308.1
Changed lines of the file:
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@@
     (stroke (width 0) (type default) (color 0 0 0 0))
   )
-  (wire (pts (xy 199.39 81.915) (xy 207.01 81.915))
+  (wire (pts (xy 199.39 81.915) (xy 205.105 81.915))
     (stroke (width 0) (type default) (color 0 0 0 0))
   )
@@
   )
   (wire (pts (xy 38.1 82.55) (xy 46.99 82.55))
+    (stroke (width 0) (type default) (color 0 0 0 0))
+  )
+  (wire (pts (xy 212.725 81.915) (xy 222.885 81.915))
     (stroke (width 0) (type default) (color 0 0 0 0))
   )
@@
     )
   )
+  (global_label "Power_in-" (shape input) (at 215.265 81.915 90) (fields_autoplaced)
+    (effects (font (size 1.27 1.27)) (justify left))
+    (property "Intersheet References" "${INTERSHEET_REFS}" (id 0) (at 215.1856 69.5838 90)
+      (effects (font (size 1.27 1.27)) (justify left) hide)
+    )
+  )
+  (global_label "Power_in+" (shape input) (at 203.835 81.915 90) (fields_autoplaced)
+    (effects (font (size 1.27 1.27)) (justify left))
+    (property "Intersheet References" "${INTERSHEET_REFS}" (id 0) (at 203.7556 69.5838 90)
+      (effects (font (size 1.27 1.27)) (justify left) hide)
+    )
+  )
   (global_label "TE" (shape input) (at 86.36 82.55 0) (fields_autoplaced)
     (effects (font (size 1.27 1.27)) (justify left))
@@
   (symbol (lib_id "Device:R") (at 314.96 173.355 0) (mirror x) (unit 1)
     (in_bom yes) (on_board yes)
-    (property "Reference" "R309" (id 0) (at 311.15 172.085 0))
+    (property "Reference" "R310" (id 0) (at 311.15 172.085 0))
     (property "Value" "330" (id 1) (at 311.15 174.625 0))
     (property "Footprint" "Resistor_SMD:R_0603_1608Metric_Pad0.98x0.95mm_HandSolder" (id 2) (at 313.182 173.355 90)
@@
     (pin "1")
   )
+  (symbol (lib_id "Device:R") (at 208.915 81.915 90) (unit 1)
+    (in_bom yes) (on_board yes)
+    (property "Reference" "R308" (id 0) (at 210.82 78.105 90)
+      (effects (font (size 1.27 1.27)) (justify left))
+    )
+    (property "Value" "5m" (id 1) (at 210.82 75.565 90)
+      (effects (font (size 1.27 1.27)) (justify left))
+    )
+    (property "Footprint" "Resistor_SMD:R_0612_1632Metric_Pad1.18x3.40mm_HandSolder" (id 2) (at 208.915 83.693 90)
+      (effects (font (size 1.27 1.27)) hide)
+    )
+    (property "Datasheet" "https://ro.mouser.com/ProductDetail/Vishay/WFCP06125L000FE66?qs=sGAEpiMZZMtlubZbdhIBIJBDgjsVQBFlUYEtiJor9t8%3D" (id 3) (at 208.915 81.915 0)
+      (effects (font (size 1.27 1.27)) hide)
+    )
+    (pin "1")
+    (pin "2")
+  )
   (symbol (lib_id "power:GND") (at 93.98 80.01 90) (mirror x) (unit 1)
     (in_bom yes) (on_board yes) (fields_autoplaced)
@@
   (symbol (lib_id "Device:R") (at 289.56 173.355 0) (mirror x) (unit 1)
     (in_bom yes) (on_board yes)
-    (property "Reference" "R308" (id 0) (at 285.75 172.085 0))
+    (property "Reference" "R309" (id 0) (at 285.75 172.085 0))
     (property "Value" "4.7k" (id 1) (at 285.75 174.625 0))
     (property "Footprint" "Resistor_THT:R_Axial_DIN0204_L3.6mm_D1.6mm_P2.54mm_Vertical" (id 2) (at 287.782 173.355 90)
@@
   (symbol (lib_id "power:+5V") (at 215.9 96.52 0) (unit 1)
     (in_bom yes) (on_board yes) (fields_autoplaced)
-    (property "Reference" "#PWR0313" (id 0) (at 215.9 100.33 0)
+    (property "Reference" "#PWR0312" (id 0) (at 215.9 100.33 0)
       (effects (font (size 1.27 1.27)) hide)
     )
@@
     (pin "2")
   )
-  (symbol (lib_id "power:+VDC") (at 207.01 81.915 0) (unit 1)
-    (in_bom yes) (on_board yes) (fields_autoplaced)
-    (property "Reference" "#PWR0312" (id 0) (at 207.01 84.455 0)
-      (effects (font (size 1.27 1.27)) hide)
-    )
-    (property "Value" "+VDC" (id 1) (at 207.01 74.295 0))
-    (property "Footprint" "" (id 2) (at 207.01 81.915 0)
-      (effects (font (size 1.27 1.27)) hide)
-    )
-    (property "Datasheet" "" (id 3) (at 207.01 81.915 0)
-      (effects (font (size 1.27 1.27)) hide)
-    )
+  (symbol (lib_id "power:+VDC") (at 222.885 81.915 0) (unit 1)
+    (in_bom yes) (on_board yes) (fields_autoplaced)
+    (property "Reference" "#PWR0313" (id 0) (at 222.885 84.455 0)
+      (effects (font (size 1.27 1.27)) hide)
+    )
+    (property "Value" "+VDC" (id 1) (at 222.885 74.295 0))
+    (property "Footprint" "" (id 2) (at 222.885 81.915 0)
+      (effects (font (size 1.27 1.27)) hide)
+    )
+    (property "Datasheet" "" (id 3) (at 222.885 81.915 0)
+      (effects (font (size 1.27 1.27)) hide)
+    )

Commit message: y
Parts:
- D303: value D_Shockley -> (none); footprint Diode_THT:D_DO-15_P15.24mm_Horizontal -> (none)
- R309: value 4.7k -> (none); footprint Resistor_THT:R_Axial_DIN0204_L3.6mm_D1.6mm_P2.54mm_Vertical -> (none)
- renumbered R306 to R304, R307 to R305, R308 to R306, R304 to R307, R305 to R308
Connections:
- net +BATT: no longer R307.2
- net +VDC: now also R307.2
Other:
- moved on the sheet: R307, R308
