File: test_project_01/Power-IN-OUT-BMS.kicad_sch (KiCad schematic)
At the start: 27 parts, among them IC301 MCP73834T-FCI_UN, IC302 AP2112M-3.3TRG1, J301 Conn_01x02, Q301 DMG9933USD-13, U301 1043, U302 APX810S05

Commit message: r
Parts:
- removed D304, D305: LED_Small Green, LED_SMD:LED_0603_1608Metric_Pad1.05x0.95mm_HandSolder, symbol Device:LED_Small
- removed R309: (no value), symbol Device:R
- removed R310: 330, Resistor_SMD:R_0603_1608Metric_Pad0.98x0.95mm_HandSolder, symbol Device:R
- added F2: 1.5 A, Fuse:Fuse_0603_1608Metric_Pad1.05x0.95mm_HandSolder, symbol Device:Fuse
- added U6: (no value), symbol Amplifier_Operational:LM324A
- D4: renamed from D303; value (none) -> D_Shockley; footprint (none) -> Diode_THT:D_DO-15_P5.08mm_Vertical_AnodeUp
- R42: renamed from R307; value 10k -> (none); footprint Resistor_SMD:R_0603_1608Metric_Pad0.98x0.95mm_HandSolder -> (none)
- R43: renamed from R308; value 10k -> (none); footprint Resistor_SMD:R_0603_1608Metric_Pad0.98x0.95mm_HandSolder -> (none)
- renumbered C301 to C15, C302 to C16, C303 to C17, C304 to C18, D301 to D2, D302 to D3, IC301 to IC3, IC302 to IC4, J301 to J13, Q301 to Q1, R301 to R36, R302 to R37, R303 to R38, R304 to R39, R305 to R40, R306 to R41, RV301 to RV1, S301 to S3, U301 to U7, U302 to U8
Connections:
- net +VDC: now also F2.2; no longer R41.2
- net ADC_CH4: now also U6.13 (-), U6.14; no longer R42.1, R43.2
- new net: R42.1, R43.2, U6.12 (+)
- new net Power_in-: F2.1, R41.2
Other:
- note removed: "Power indicator leds"
- moved on the sheet: R42, R43

Commit message: r
Parts:
- R42, R43: value (none) -> 1Meg; footprint (none) -> Resistor_SMD:R_0603_1608Metric_Pad0.98x0.95mm_HandSolder
- U6: value (none) -> LM324A; footprint (none) -> Package_SO:SOIC-14_3.9x8.7mm_P1.27mm
Changed lines of the file:
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@@
     (in_bom yes) (on_board yes)
     (property "Reference" "U6" (id 0) (at 219.075 109.22 0))
-    (property "Value" "" (id 1) (at 219.075 111.76 0))
-    (property "Footprint" "" (id 2) (at 222.25 102.87 0)
+    (property "Value" "LM324A" (id 1) (at 219.075 111.76 0))
+    (property "Footprint" "Package_SO:SOIC-14_3.9x8.7mm_P1.27mm" (id 2) (at 222.25 102.87 0)
       (effects (font (size 1.27 1.27)) hide)
     )
@@
       (effects (font (size 1.27 1.27)) (justify right))
     )
-    (property "Value" "" (id 1) (at 225.425 93.345 0)
-      (effects (font (size 1.27 1.27)) (justify right))
-    )
-    (property "Footprint" "" (id 2) (at 232.41 92.71 0)
+    (property "Value" "1Meg" (id 1) (at 225.425 93.345 0)
+      (effects (font (size 1.27 1.27)) (justify right))
+    )
+    (property "Footprint" "Resistor_SMD:R_0603_1608Metric_Pad0.98x0.95mm_HandSolder" (id 2) (at 232.41 92.71 0)
       (effects (font (size 1.27 1.27)) hide)
     )
@@
       (effects (font (size 1.27 1.27)) (justify right))
     )
-    (property "Value" "" (id 1) (at 224.79 116.84 0)
-      (effects (font (size 1.27 1.27)) (justify right))
-    )
-    (property "Footprint" "" (id 2) (at 232.41 116.205 0)
-      (effects (font (size 1.27 1.27)) hide)
-    )
+    (property "Value" "1Meg" (id 1) (at 224.79 116.84 0)
+      (effects (font (size 1.27 1.27)) (justify right))
+    )
+    (property "Footprint" "Resistor_SMD:R_0603_1608Metric_Pad0.98x0.95mm_HandSolder" (id 2) (at 232.41 116.205 0)
+      (effects (font (size 1.27 1.27)) hide)
+    )

Commit message: Y
Other:
- note added: "BMS+POWER SOURCE AUTO SWITCHING"
- note added: "BUCK"
- note added: "LDO"
- note removed: "Power"
- title: ESP32 audio power meter SD dataloger -> ESP32 MP3 player/web radio+power meter+uSD dataloger
Changed lines of the file:
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@@
   (paper "A3")
   (title_block
-    (title "ESP32 audio power meter SD dataloger")
-    (rev "1")
+    (title "ESP32 MP3 player/web radio+power meter+uSD dataloger")
+    (rev "2")
   )
   (junction (at 22.86 62.23) (diameter 0) (color 0 0 0 0)
@@
     (effects (font (size 1.27 1.27)) (justify left bottom))
   )
+  (text "BUCK" (at 297.18 88.9 0)
+    (effects (font (size 5 5)) (justify left bottom))
+  )
   (text "TE uses 1.8V logic\nactive high\nactivates a timer" (at 53.34 95.25 0)
     (effects (font (size 1.27 1.27)) (justify left bottom))
@@
   )
   (text "Linear regulator\njust in case the buck fails \nor i need lower noise power"
-    (at 295.91 38.1 0)
-    (effects (font (size 1.27 1.27)) (justify left bottom))
-  )
-  (text "Power" (at 187.96 27.94 0)
+    (at 316.865 72.39 0)
+    (effects (font (size 1.27 1.27)) (justify left bottom))
+  )
+  (text "BATT TO USB POWER AUTO SHITCHING\n WITH REVERSE POWER PROTECTION\nAND PROTECTED CHARGEING CCCV"
+    (at 77.47 59.055 0)
+    (effects (font (size 1.27 1.27)) (justify left bottom))
+  )
+  (text "18650 cell\nholder" (at 129.794 96.266 0)
+    (effects (font (size 1.27 1.27)) (justify left bottom))
+  )
+  (text "LDO" (at 295.275 40.64 0)
     (effects (font (size 5 5)) (justify left bottom))
   )
-  (text "BATT TO USB POWER AUTO SHITCHING\n WITH REVERSE POWER PROTECTION\nAND PROTECTED CHARGEING CCCV"
-    (at 123.19 48.26 0)
-    (effects (font (size 1.27 1.27)) (justify left bottom))
-  )
-  (text "18650 cell\nholder" (at 129.794 96.266 0)
-    (effects (font (size 1.27 1.27)) (justify left bottom))
-  )
   (text "200-300mA\n<100 typical" (at 339.09 114.3 0)
     (effects (font (size 1.27 1.27)) (justify left bottom))
+  )
+  (text "BMS+POWER SOURCE AUTO SWITCHING" (at 50.165 47.625 0)
+    (effects (font (size 5 5)) (justify left bottom))
   )
   (label "Drains" (at 192.405 52.705 0)
@@
     )
   )
+  (hierarchical_label "5v" (shape input) (at 27.94 62.23 90)
+    (effects (font (size 1.27 1.27)) (justify left))
+  )
   (symbol (lib_id "Device:R") (at 187.96 105.41 0) (mirror x) (unit 1)
