File: test_project_01/buck.kicad_sch (KiCad schematic)
At the start: 8 parts

Commit message: f
Other:
- title: (none) -> ESP32 audio power meter SD dataloger
Changed lines of the file:
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@@
 (kicad_sch (version 20211123) (generator eeschema)
-  (paper "A4")
+  (paper "A3")
+  (title_block
+    (title "ESP32 audio power meter SD dataloger")
+    (rev "1")
+  )
   (junction (at 154.305 66.675) (diameter 0) (color 0 0 0 0)
   )

Commit message: j
Parts:
- gave numbers to parts that had none: 8
Changed lines of the file:
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@@
   (symbol (lib_id "power:GND") (at 140.335 83.82 0) (unit 1)
     (in_bom yes) (on_board yes) (fields_autoplaced)
-    (property "Reference" "#PWR?" (id 0) (at 140.335 90.17 0)
+    (property "Reference" "#PWR040" (id 0) (at 140.335 90.17 0)
       (effects (font (size 1.27 1.27)) hide)
     )
@@
   (symbol (lib_id "power:GND") (at 61.595 74.93 0) (unit 1)
     (in_bom yes) (on_board yes) (fields_autoplaced)
-    (property "Reference" "#PWR?" (id 0) (at 61.595 81.28 0)
+    (property "Reference" "#PWR038" (id 0) (at 61.595 81.28 0)
       (effects (font (size 1.27 1.27)) hide)
     )
@@
   (symbol (lib_id "Device:R_Small") (at 140.335 71.12 0) (unit 1)
     (in_bom yes) (on_board yes) (fields_autoplaced)
-    (property "Reference" "RR?" (id 0) (at 142.24 69.8499 0)
+    (property "Reference" "RR1" (id 0) (at 142.24 69.8499 0)
       (effects (font (size 1.27 1.27)) (justify left))
     )
@@
   (symbol (lib_id "My_custom_lib:DIO6012BCST6") (at 84.455 66.675 0) (unit 1)
     (in_bom yes) (on_board yes) (fields_autoplaced)
-    (property "Reference" "U?" (id 0) (at 84.455 55.88 0))
+    (property "Reference" "U8" (id 0) (at 84.455 55.88 0))
     (property "Value" "DIO6012BCST6" (id 1) (at 84.455 58.42 0))
     (property "Footprint" "Package_TO_SOT_SMD:SOT-23-6_Handsoldering" (id 2) (at 81.915 59.055 0)
@@
   (symbol (lib_id "Device:C_Small") (at 154.305 70.485 0) (unit 1)
     (in_bom yes) (on_board yes) (fields_autoplaced)
-    (property "Reference" "C?" (id 0) (at 156.845 69.2212 0)
+    (property "Reference" "C15" (id 0) (at 156.845 69.2212 0)
       (effects (font (size 1.27 1.27)) (justify left))
     )
@@
   (symbol (lib_id "power:GND") (at 81.915 77.47 0) (unit 1)
     (in_bom yes) (on_board yes) (fields_autoplaced)
-    (property "Reference" "#PWR?" (id 0) (at 81.915 83.82 0)
+    (property "Reference" "#PWR039" (id 0) (at 81.915 83.82 0)
       (effects (font (size 1.27 1.27)) hide)
     )
@@
   (symbol (lib_id "power:GND") (at 161.925 75.565 0) (unit 1)
     (in_bom yes) (on_board yes) (fields_autoplaced)
-    (property "Reference" "#PWR?" (id 0) (at 161.925 81.915 0)
+    (property "Reference" "#PWR042" (id 0) (at 161.925 81.915 0)
       (effects (font (size 1.27 1.27)) hide)
     )
@@
   (symbol (lib_id "Device:C_Small") (at 61.595 70.485 0) (unit 1)
     (in_bom yes) (on_board yes) (fields_autoplaced)
-    (property "Reference" "C?" (id 0) (at 64.135 69.2212 0)
+    (property "Reference" "C13" (id 0) (at 64.135 69.2212 0)
       (effects (font (size 1.27 1.27)) (justify left))
     )
@@
   (symbol (lib_id "Device:R_Small") (at 140.335 79.375 0) (unit 1)
     (in_bom yes) (on_board yes) (fields_autoplaced)
-    (property "Reference" "RR?" (id 0) (at 142.875 78.1049 0)
+    (property "Reference" "RR2" (id 0) (at 142.875 78.1049 0)
       (effects (font (size 1.27 1.27)) (justify left))
     )
@@
   (symbol (lib_id "Device:C_Small") (at 161.925 70.485 0) (unit 1)
     (in_bom yes) (on_board yes) (fields_autoplaced)
-    (property "Reference" "C?" (id 0) (at 164.465 69.2212 0)
+    (property "Reference" "C16" (id 0) (at 164.465 69.2212 0)
       (effects (font (size 1.27 1.27)) (justify left))
     )
@@
   (symbol (lib_id "Device:C_Small") (at 131.445 70.485 0) (unit 1)
     (in_bom yes) (on_board yes)
-    (property "Reference" "C?" (id 0) (at 125.095 69.215 0)
+    (property "Reference" "C14" (id 0) (at 125.095 69.215 0)
       (effects (font (size 1.27 1.27)) (justify left))
     )
@@
   (symbol (lib_id "power:GND") (at 154.305 75.565 0) (unit 1)
     (in_bom yes) (on_board yes) (fields_autoplaced)
-    (property "Reference" "#PWR?" (id 0) (at 154.305 81.915 0)
+    (property "Reference" "#PWR041" (id 0) (at 154.305 81.915 0)
       (effects (font (size 1.27 1.27)) hide)
     )
@@
   (symbol (lib_id "SamacSys_Parts:NRH3012T2R2MN") (at 98.425 66.675 0) (unit 1)
     (in_bom yes) (on_board yes) (fields_autoplaced)
-    (property "Reference" "L?" (id 0) (at 108.585 60.325 0))
+    (property "Reference" "L1" (id 0) (at 108.585 60.325 0))
     (property "Value" "NRH3012T2R2MN  2,2uH" (id 1) (at 108.585 62.865 0))
     (property "Footprint" "SamacSys_Parts:NRH3012T220MNV" (id 2) (at 114.935 65.405 0)

Commit message: f
Parts:
- renumbered C13 to C401, C14 to C402, C15 to C403, C16 to C404, L1 to L401, RR1 to RR401, RR2 to RR402, U8 to U401
Changed lines of the file:
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@@
   (symbol (lib_id "power:GND") (at 140.335 83.82 0) (unit 1)
     (in_bom yes) (on_board yes) (fields_autoplaced)
-    (property "Reference" "#PWR040" (id 0) (at 140.335 90.17 0)
+    (property "Reference" "#PWR0403" (id 0) (at 140.335 90.17 0)
       (effects (font (size 1.27 1.27)) hide)
     )
@@
   (symbol (lib_id "power:GND") (at 61.595 74.93 0) (unit 1)
     (in_bom yes) (on_board yes) (fields_autoplaced)
-    (property "Reference" "#PWR038" (id 0) (at 61.595 81.28 0)
+    (property "Reference" "#PWR0401" (id 0) (at 61.595 81.28 0)
       (effects (font (size 1.27 1.27)) hide)
     )
@@
   (symbol (lib_id "Device:R_Small") (at 140.335 71.12 0) (unit 1)
     (in_bom yes) (on_board yes) (fields_autoplaced)
-    (property "Reference" "RR1" (id 0) (at 142.24 69.8499 0)
+    (property "Reference" "RR401" (id 0) (at 142.24 69.8499 0)
       (effects (font (size 1.27 1.27)) (justify left))
     )
@@
   (symbol (lib_id "My_custom_lib:DIO6012BCST6") (at 84.455 66.675 0) (unit 1)
     (in_bom yes) (on_board yes) (fields_autoplaced)
-    (property "Reference" "U8" (id 0) (at 84.455 55.88 0))
+    (property "Reference" "U401" (id 0) (at 84.455 55.88 0))
     (property "Value" "DIO6012BCST6" (id 1) (at 84.455 58.42 0))
     (property "Footprint" "Package_TO_SOT_SMD:SOT-23-6_Handsoldering" (id 2) (at 81.915 59.055 0)
@@
   (symbol (lib_id "Device:C_Small") (at 154.305 70.485 0) (unit 1)
     (in_bom yes) (on_board yes) (fields_autoplaced)
-    (property "Reference" "C15" (id 0) (at 156.845 69.2212 0)
+    (property "Reference" "C403" (id 0) (at 156.845 69.2212 0)
       (effects (font (size 1.27 1.27)) (justify left))
     )
@@
   (symbol (lib_id "power:GND") (at 81.915 77.47 0) (unit 1)
     (in_bom yes) (on_board yes) (fields_autoplaced)
-    (property "Reference" "#PWR039" (id 0) (at 81.915 83.82 0)
+    (property "Reference" "#PWR0402" (id 0) (at 81.915 83.82 0)
       (effects (font (size 1.27 1.27)) hide)
     )
@@
   (symbol (lib_id "power:GND") (at 161.925 75.565 0) (unit 1)
     (in_bom yes) (on_board yes) (fields_autoplaced)
-    (property "Reference" "#PWR042" (id 0) (at 161.925 81.915 0)
+    (property "Reference" "#PWR0405" (id 0) (at 161.925 81.915 0)
       (effects (font (size 1.27 1.27)) hide)
     )
@@
   (symbol (lib_id "Device:C_Small") (at 61.595 70.485 0) (unit 1)
     (in_bom yes) (on_board yes) (fields_autoplaced)
-    (property "Reference" "C13" (id 0) (at 64.135 69.2212 0)
+    (property "Reference" "C401" (id 0) (at 64.135 69.2212 0)
       (effects (font (size 1.27 1.27)) (justify left))
     )
@@
   (symbol (lib_id "Device:R_Small") (at 140.335 79.375 0) (unit 1)
     (in_bom yes) (on_board yes) (fields_autoplaced)
-    (property "Reference" "RR2" (id 0) (at 142.875 78.1049 0)
+    (property "Reference" "RR402" (id 0) (at 142.875 78.1049 0)
       (effects (font (size 1.27 1.27)) (justify left))
     )
@@
   (symbol (lib_id "Device:C_Small") (at 161.925 70.485 0) (unit 1)
     (in_bom yes) (on_board yes) (fields_autoplaced)
-    (property "Reference" "C16" (id 0) (at 164.465 69.2212 0)
+    (property "Reference" "C404" (id 0) (at 164.465 69.2212 0)
       (effects (font (size 1.27 1.27)) (justify left))
     )
@@
   (symbol (lib_id "Device:C_Small") (at 131.445 70.485 0) (unit 1)
     (in_bom yes) (on_board yes)
-    (property "Reference" "C14" (id 0) (at 125.095 69.215 0)
+    (property "Reference" "C402" (id 0) (at 125.095 69.215 0)
       (effects (font (size 1.27 1.27)) (justify left))
     )
@@
   (symbol (lib_id "power:GND") (at 154.305 75.565 0) (unit 1)
     (in_bom yes) (on_board yes) (fields_autoplaced)
-    (property "Reference" "#PWR041" (id 0) (at 154.305 81.915 0)
+    (property "Reference" "#PWR0404" (id 0) (at 154.305 81.915 0)
       (effects (font (size 1.27 1.27)) hide)
     )
@@
   (symbol (lib_id "SamacSys_Parts:NRH3012T2R2MN") (at 98.425 66.675 0) (unit 1)
     (in_bom yes) (on_board yes) (fields_autoplaced)
-    (property "Reference" "L1" (id 0) (at 108.585 60.325 0))
+    (property "Reference" "L401" (id 0) (at 108.585 60.325 0))
     (property "Value" "NRH3012T2R2MN  2,2uH" (id 1) (at 108.585 62.865 0))
     (property "Footprint" "SamacSys_Parts:NRH3012T220MNV" (id 2) (at 114.935 65.405 0)

Commit message: h
Parts:
- added FB401: FerriteBead_Small, Resistor_SMD:R_0402_1005Metric_Pad0.72x0.64mm_HandSolder, symbol Device:FerriteBead_Small
Connections:
- net BUCK_INPUT: now also FB401.1; no longer C401.1, U401.4 (IN)
- new net: C401.1, FB401.2, U401.4 (IN)
Changed lines of the file:
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@@
     (stroke (width 0) (type default) (color 0 0 0 0))
   )
-  (wire (pts (xy 59.055 66.675) (xy 61.595 66.675))
+  (wire (pts (xy 38.1 66.675) (xy 45.085 66.675))
+    (stroke (width 0) (type default) (color 0 0 0 0))
+  )
+  (wire (pts (xy 50.165 66.675) (xy 61.595 66.675))
     (stroke (width 0) (type default) (color 0 0 0 0))
   )
@@
     (effects (font (size 1.27 1.27)) (justify left bottom))
   )
-  (hierarchical_label "BUCK_INPUT" (shape input) (at 59.055 66.675 180)
+  (hierarchical_label "BUCK_INPUT" (shape input) (at 38.1 66.675 180)
     (effects (font (size 1.27 1.27)) (justify right))
   )
@@
     (pin "1")
   )
+  (symbol (lib_id "Device:FerriteBead_Small") (at 47.625 66.675 90) (unit 1)
+    (in_bom yes) (on_board yes) (fields_autoplaced)
+    (property "Reference" "FB401" (id 0) (at 47.5869 59.69 90))
+    (property "Value" "FerriteBead_Small" (id 1) (at 47.5869 62.23 90))
+    (property "Footprint" "Resistor_SMD:R_0402_1005Metric_Pad0.72x0.64mm_HandSolder" (id 2) (at 47.625 68.453 90)
+      (effects (font (size 1.27 1.27)) hide)
+    )
+    (property "Datasheet" "~" (id 3) (at 47.625 66.675 0)
+      (effects (font (size 1.27 1.27)) hide)
+    )
+    (pin "1")
+    (pin "2")
+  )
   (symbol (lib_id "SamacSys_Parts:NRH3012T2R2MN") (at 98.425 66.675 0) (unit 1)

Commit message: y
Other:
- moved on the sheet: C404
Changed lines of the file:
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@@
   (junction (at 154.305 66.675) (diameter 0) (color 0 0 0 0)
   )
-  (junction (at 161.925 66.675) (diameter 0) (color 0 0 0 0)
+  (junction (at 165.735 66.675) (diameter 0) (color 0 0 0 0)
   )
   (junction (at 131.445 66.675) (diameter 0) (color 0 0 0 0)
@@
     (stroke (width 0) (type default) (color 0 0 0 0))
   )
-  (wire (pts (xy 161.925 73.025) (xy 161.925 75.565))
+  (wire (pts (xy 165.735 73.025) (xy 165.735 75.565))
     (stroke (width 0) (type default) (color 0 0 0 0))
   )
@@
     (stroke (width 0) (type default) (color 0 0 0 0))
   )
-  (wire (pts (xy 161.925 66.675) (xy 167.64 66.675))
+  (wire (pts (xy 165.735 66.675) (xy 179.07 66.675))
     (stroke (width 0) (type default) (color 0 0 0 0))
   )
@@
     (stroke (width 0) (type default) (color 0 0 0 0))
   )
-  (wire (pts (xy 161.925 66.675) (xy 161.925 67.945))
-    (stroke (width 0) (type default) (color 0 0 0 0))
-  )
-  (wire (pts (xy 154.305 66.675) (xy 161.925 66.675))
+  (wire (pts (xy 154.305 66.675) (xy 165.735 66.675))
     (stroke (width 0) (type default) (color 0 0 0 0))
   )
@@
   )
   (wire (pts (xy 50.165 66.675) (xy 61.595 66.675))
+    (stroke (width 0) (type default) (color 0 0 0 0))
+  )
+  (wire (pts (xy 165.735 66.675) (xy 165.735 67.945))
     (stroke (width 0) (type default) (color 0 0 0 0))
   )
@@
     (effects (font (size 1.27 1.27)) (justify right))
   )
-  (hierarchical_label "BUCK_OUTPUT" (shape input) (at 167.64 66.675 0)
+  (hierarchical_label "BUCK_OUTPUT" (shape input) (at 179.07 66.675 0)
     (effects (font (size 1.27 1.27)) (justify left))
   )
@@
     (pin "1")
   )
-  (symbol (lib_id "power:GND") (at 161.925 75.565 0) (unit 1)
-    (in_bom yes) (on_board yes) (fields_autoplaced)
-    (property "Reference" "#PWR0405" (id 0) (at 161.925 81.915 0)
-      (effects (font (size 1.27 1.27)) hide)
-    )
-    (property "Value" "GND" (id 1) (at 161.925 80.645 0)
-      (effects (font (size 1.27 1.27)) hide)
-    )
-    (property "Footprint" "" (id 2) (at 161.925 75.565 0)
-      (effects (font (size 1.27 1.27)) hide)
-    )
-    (property "Datasheet" "" (id 3) (at 161.925 75.565 0)
+  (symbol (lib_id "power:GND") (at 165.735 75.565 0) (unit 1)
+    (in_bom yes) (on_board yes) (fields_autoplaced)
+    (property "Reference" "#PWR0405" (id 0) (at 165.735 81.915 0)
+      (effects (font (size 1.27 1.27)) hide)
+    )
+    (property "Value" "GND" (id 1) (at 165.735 80.645 0)
+      (effects (font (size 1.27 1.27)) hide)
+    )
+    (property "Footprint" "" (id 2) (at 165.735 75.565 0)
+      (effects (font (size 1.27 1.27)) hide)
+    )
+    (property "Datasheet" "" (id 3) (at 165.735 75.565 0)
       (effects (font (size 1.27 1.27)) hide)
     )
@@
     (pin "2")
   )
-  (symbol (lib_id "Device:C_Small") (at 161.925 70.485 0) (unit 1)
-    (in_bom yes) (on_board yes) (fields_autoplaced)
-    (property "Reference" "C404" (id 0) (at 164.465 69.2212 0)
-      (effects (font (size 1.27 1.27)) (justify left))
-    )
-    (property "Value" "22u" (id 1) (at 164.465 71.7612 0)
-      (effects (font (size 1.27 1.27)) (justify left))
-    )
-    (property "Footprint" "Capacitor_THT:CP_Radial_D5.0mm_P2.00mm" (id 2) (at 161.925 70.485 0)
-      (effects (font (size 1.27 1.27)) hide)
-    )
-    (property "Datasheet" "~" (id 3) (at 161.925 70.485 0)
+  (symbol (lib_id "Device:C_Small") (at 165.735 70.485 0) (unit 1)
+    (in_bom yes) (on_board yes) (fields_autoplaced)
+    (property "Reference" "C404" (id 0) (at 168.275 69.2212 0)
+      (effects (font (size 1.27 1.27)) (justify left))
+    )
+    (property "Value" "22u" (id 1) (at 168.275 71.7612 0)
+      (effects (font (size 1.27 1.27)) (justify left))
+    )
+    (property "Footprint" "Capacitor_THT:CP_Radial_D5.0mm_P2.00mm" (id 2) (at 165.735 70.485 0)
+      (effects (font (size 1.27 1.27)) hide)
+    )
+    (property "Datasheet" "~" (id 3) (at 165.735 70.485 0)
       (effects (font (size 1.27 1.27)) hide)
     )
@@
   (symbol (lib_id "Device:C_Small") (at 131.445 70.485 0) (unit 1)
     (in_bom yes) (on_board yes)
-    (property "Reference" "C402" (id 0) (at 125.095 69.215 0)
+    (property "Reference" "C402" (id 0) (at 121.285 69.215 0)
       (effects (font (size 1.27 1.27)) (justify left))
     )
@@
   )
   (symbol (lib_id "SamacSys_Parts:NRH3012T2R2MN") (at 98.425 66.675 0) (unit 1)
-    (in_bom yes) (on_board yes) (fields_autoplaced)
-    (property "Reference" "L401" (id 0) (at 108.585 60.325 0))
-    (property "Value" "NRH3012T2R2MN  2,2uH" (id 1) (at 108.585 62.865 0))
+    (in_bom yes) (on_board yes)
+    (property "Reference" "L401" (id 0) (at 113.03 60.325 0))
+    (property "Value" "NRH3012T2R2MN  2,2uH" (id 1) (at 113.03 62.865 0))
     (property "Footprint" "SamacSys_Parts:NRH3012T220MNV" (id 2) (at 114.935 65.405 0)
       (effects (font (size 1.27 1.27)) (justify left) hide)

Commit message: r
Parts:
- renumbered C401 to C19, C402 to C20, C403 to C21, C404 to C22, FB401 to FB2, L401 to L1, RR401 to RR1, RR402 to RR2, U401 to U10
Changed lines of the file:
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@@
   (symbol (lib_id "power:GND") (at 140.335 83.82 0) (unit 1)
     (in_bom yes) (on_board yes) (fields_autoplaced)
-    (property "Reference" "#PWR0403" (id 0) (at 140.335 90.17 0)
+    (property "Reference" "#PWR083" (id 0) (at 140.335 90.17 0)
       (effects (font (size 1.27 1.27)) hide)
     )
@@
   (symbol (lib_id "power:GND") (at 61.595 74.93 0) (unit 1)
     (in_bom yes) (on_board yes) (fields_autoplaced)
-    (property "Reference" "#PWR0401" (id 0) (at 61.595 81.28 0)
+    (property "Reference" "#PWR081" (id 0) (at 61.595 81.28 0)
       (effects (font (size 1.27 1.27)) hide)
     )
@@
   (symbol (lib_id "Device:R_Small") (at 140.335 71.12 0) (unit 1)
     (in_bom yes) (on_board yes) (fields_autoplaced)
-    (property "Reference" "RR401" (id 0) (at 142.24 69.8499 0)
+    (property "Reference" "RR1" (id 0) (at 142.24 69.8499 0)
       (effects (font (size 1.27 1.27)) (justify left))
     )
@@
   (symbol (lib_id "My_custom_lib:DIO6012BCST6") (at 84.455 66.675 0) (unit 1)
     (in_bom yes) (on_board yes) (fields_autoplaced)
-    (property "Reference" "U401" (id 0) (at 84.455 55.88 0))
+    (property "Reference" "U10" (id 0) (at 84.455 55.88 0))
     (property "Value" "DIO6012BCST6" (id 1) (at 84.455 58.42 0))
     (property "Footprint" "Package_TO_SOT_SMD:SOT-23-6_Handsoldering" (id 2) (at 81.915 59.055 0)
@@
   (symbol (lib_id "Device:C_Small") (at 154.305 70.485 0) (unit 1)
     (in_bom yes) (on_board yes) (fields_autoplaced)
-    (property "Reference" "C403" (id 0) (at 156.845 69.2212 0)
+    (property "Reference" "C21" (id 0) (at 156.845 69.2212 0)
       (effects (font (size 1.27 1.27)) (justify left))
     )
@@
   (symbol (lib_id "power:GND") (at 81.915 77.47 0) (unit 1)
     (in_bom yes) (on_board yes) (fields_autoplaced)
-    (property "Reference" "#PWR0402" (id 0) (at 81.915 83.82 0)
+    (property "Reference" "#PWR082" (id 0) (at 81.915 83.82 0)
       (effects (font (size 1.27 1.27)) hide)
     )
@@
   (symbol (lib_id "power:GND") (at 165.735 75.565 0) (unit 1)
     (in_bom yes) (on_board yes) (fields_autoplaced)
-    (property "Reference" "#PWR0405" (id 0) (at 165.735 81.915 0)
+    (property "Reference" "#PWR085" (id 0) (at 165.735 81.915 0)
       (effects (font (size 1.27 1.27)) hide)
     )
@@
   (symbol (lib_id "Device:C_Small") (at 61.595 70.485 0) (unit 1)
     (in_bom yes) (on_board yes) (fields_autoplaced)
-    (property "Reference" "C401" (id 0) (at 64.135 69.2212 0)
+    (property "Reference" "C19" (id 0) (at 64.135 69.2212 0)
       (effects (font (size 1.27 1.27)) (justify left))
     )
@@
   (symbol (lib_id "Device:R_Small") (at 140.335 79.375 0) (unit 1)
     (in_bom yes) (on_board yes) (fields_autoplaced)
-    (property "Reference" "RR402" (id 0) (at 142.875 78.1049 0)
+    (property "Reference" "RR2" (id 0) (at 142.875 78.1049 0)
       (effects (font (size 1.27 1.27)) (justify left))
     )
@@
   (symbol (lib_id "Device:C_Small") (at 165.735 70.485 0) (unit 1)
     (in_bom yes) (on_board yes) (fields_autoplaced)
-    (property "Reference" "C404" (id 0) (at 168.275 69.2212 0)
+    (property "Reference" "C22" (id 0) (at 168.275 69.2212 0)
       (effects (font (size 1.27 1.27)) (justify left))
     )
@@
   (symbol (lib_id "Device:C_Small") (at 131.445 70.485 0) (unit 1)
     (in_bom yes) (on_board yes)
-    (property "Reference" "C402" (id 0) (at 121.285 69.215 0)
+    (property "Reference" "C20" (id 0) (at 121.285 69.215 0)
       (effects (font (size 1.27 1.27)) (justify left))
     )
@@
   (symbol (lib_id "power:GND") (at 154.305 75.565 0) (unit 1)
     (in_bom yes) (on_board yes) (fields_autoplaced)
-    (property "Reference" "#PWR0404" (id 0) (at 154.305 81.915 0)
+    (property "Reference" "#PWR084" (id 0) (at 154.305 81.915 0)
       (effects (font (size 1.27 1.27)) hide)
     )
@@
   (symbol (lib_id "Device:FerriteBead_Small") (at 47.625 66.675 90) (unit 1)
     (in_bom yes) (on_board yes) (fields_autoplaced)
-    (property "Reference" "FB401" (id 0) (at 47.5869 59.69 90))
+    (property "Reference" "FB2" (id 0) (at 47.5869 59.69 90))
     (property "Value" "FerriteBead_Small" (id 1) (at 47.5869 62.23 90))
     (property "Footprint" "Resistor_SMD:R_0402_1005Metric_Pad0.72x0.64mm_HandSolder" (id 2) (at 47.625 68.453 90)
@@
   (symbol (lib_id "SamacSys_Parts:NRH3012T2R2MN") (at 98.425 66.675 0) (unit 1)
     (in_bom yes) (on_board yes)
-    (property "Reference" "L401" (id 0) (at 113.03 60.325 0))
+    (property "Reference" "L1" (id 0) (at 113.03 60.325 0))
     (property "Value" "NRH3012T2R2MN  2,2uH" (id 1) (at 113.03 62.865 0))
     (property "Footprint" "SamacSys_Parts:NRH3012T220MNV" (id 2) (at 114.935 65.405 0)
