File: test_project_01/buck.kicad_sch (KiCad schematic)
At the start: 9 parts, among them U10 DIO6012BCST6

Commit message: H
Parts:
- RR1, RR2: value R_Small -> (none); footprint Resistor_THT:R_Axial_DIN0204_L3.6mm_D1.6mm_P5.08mm_Horizontal -> (none)
Connections:
- net buck_input_filtered: now reaches C19.1, FB2.2, U10.4 (IN)
Other:
- note added: "RR1 RR2 81.81k 18.19k -100k pot 100k 450k 222k 1M 47k 211.5k 10k 2k22 47k 10k444 91k 20k222"
- note added: "for rr1 47k and rr2 10k we have : 3.42V"
- note added: "for rr1 91k and rr2 20k we have : 3.33V"
- note removed: "RR1 RR2 81.81k 18.19k -100k pot 100k 450k 222k 1M 47k 211.5k"
- moved on the sheet: C21, C22
Changed lines of the file:
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@@
     (stroke (width 0) (type default) (color 0 0 0 0))
   )
-  (wire (pts (xy 165.735 73.025) (xy 165.735 75.565))
+  (wire (pts (xy 165.735 77.47) (xy 165.735 81.915))
     (stroke (width 0) (type default) (color 0 0 0 0))
   )
@@
     (stroke (width 0) (type default) (color 0 0 0 0))
   )
-  (wire (pts (xy 165.735 66.675) (xy 179.07 66.675))
+  (wire (pts (xy 165.735 66.675) (xy 193.675 66.675))
     (stroke (width 0) (type default) (color 0 0 0 0))
   )
@@
     (stroke (width 0) (type default) (color 0 0 0 0))
   )
-  (wire (pts (xy 154.305 73.025) (xy 154.305 75.565))
+  (wire (pts (xy 154.305 77.47) (xy 154.305 81.915))
     (stroke (width 0) (type default) (color 0 0 0 0))
   )
@@
     (stroke (width 0) (type default) (color 0 0 0 0))
   )
-  (wire (pts (xy 165.735 66.675) (xy 165.735 67.945))
+  (wire (pts (xy 165.735 66.675) (xy 165.735 72.39))
     (stroke (width 0) (type default) (color 0 0 0 0))
   )
@@
     (stroke (width 0) (type default) (color 0 0 0 0))
   )
-  (wire (pts (xy 154.305 66.675) (xy 154.305 67.945))
+  (wire (pts (xy 154.305 66.675) (xy 154.305 72.39))
     (stroke (width 0) (type default) (color 0 0 0 0))
   )
@@
     (stroke (width 0) (type default) (color 0 0 0 0))
   )
-  (text "RR2=0,6*RR1/(Vout-0,6)" (at 144.78 85.725 0)
+  (text "for rr1 47k and rr2 10k we have : 3.42V" (at 231.14 92.71 0)
+    (effects (font (size 1.27 1.27)) (justify left bottom))
+  )
+  (text "for rr1 91k and rr2 20k we have : 3.33V" (at 231.14 95.885 0)
+    (effects (font (size 1.27 1.27)) (justify left bottom))
+  )
+  (text "RR2=0,6*RR1/(Vout-0,6)" (at 191.77 90.805 0)
     (effects (font (size 1.27 1.27)) (justify left bottom))
   )
@@
     (effects (font (size 1.27 1.27)) (justify left bottom))
   )
-  (text "RR1     RR2\n81.81k  18.19k  -100k pot\n100k    450k\n222k    1M\n47k     211.5k"
-    (at 145.415 98.425 0)
+  (text "RR1     RR2\n81.81k  18.19k  -100k pot\n100k    450k\n222k    1M\n47k     211.5k\n10k     2k22\n47k     10k444\n91k     20k222"
+    (at 191.77 110.49 0)
+    (effects (font (size 1.27 1.27)) (justify left bottom))
+  )
+  (label "buck_input_filtered" (at 53.34 66.675 0)
     (effects (font (size 1.27 1.27)) (justify left bottom))
   )
@@
     (effects (font (size 1.27 1.27)) (justify right))
   )
-  (hierarchical_label "BUCK_OUTPUT" (shape input) (at 179.07 66.675 0)
+  (hierarchical_label "BUCK_OUTPUT" (shape input) (at 193.675 66.675 0)
     (effects (font (size 1.27 1.27)) (justify left))
   )
@@
       (effects (font (size 1.27 1.27)) (justify left))
     )
-    (property "Value" "R_Small" (id 1) (at 142.24 72.3899 0)
-      (effects (font (size 1.27 1.27)) (justify left))
-    )
-    (property "Footprint" "Resistor_THT:R_Axial_DIN0204_L3.6mm_D1.6mm_P5.08mm_Horizontal" (id 2) (at 140.335 71.12 0)
+    (property "Value" "" (id 1) (at 142.24 72.3899 0)
+      (effects (font (size 1.27 1.27)) (justify left))
+    )
+    (property "Footprint" "" (id 2) (at 140.335 71.12 0)
       (effects (font (size 1.27 1.27)) hide)
     )
@@
     (pin "6")
   )
-  (symbol (lib_id "Device:C_Small") (at 154.305 70.485 0) (unit 1)
-    (in_bom yes) (on_board yes) (fields_autoplaced)
-    (property "Reference" "C21" (id 0) (at 156.845 69.2212 0)
-      (effects (font (size 1.27 1.27)) (justify left))
-    )
-    (property "Value" "22u" (id 1) (at 156.845 71.7612 0)
-      (effects (font (size 1.27 1.27)) (justify left))
-    )
-    (property "Footprint" "Capacitor_THT:CP_Radial_D5.0mm_P2.00mm" (id 2) (at 154.305 70.485 0)
-      (effects (font (size 1.27 1.27)) hide)
-    )
-    (property "Datasheet" "~" (id 3) (at 154.305 70.485 0)
+  (symbol (lib_id "Device:C_Small") (at 154.305 74.93 0) (unit 1)
+    (in_bom yes) (on_board yes) (fields_autoplaced)
+    (property "Reference" "C21" (id 0) (at 156.845 73.6662 0)
+      (effects (font (size 1.27 1.27)) (justify left))
+    )
+    (property "Value" "22u" (id 1) (at 156.845 76.2062 0)
+      (effects (font (size 1.27 1.27)) (justify left))
+    )
+    (property "Footprint" "Capacitor_THT:CP_Radial_D5.0mm_P2.00mm" (id 2) (at 154.305 74.93 0)
+      (effects (font (size 1.27 1.27)) hide)
+    )
+    (property "Datasheet" "~" (id 3) (at 154.305 74.93 0)
       (effects (font (size 1.27 1.27)) hide)
     )
@@
     (pin "1")
   )
-  (symbol (lib_id "power:GND") (at 165.735 75.565 0) (unit 1)
-    (in_bom yes) (on_board yes) (fields_autoplaced)
-    (property "Reference" "#PWR085" (id 0) (at 165.735 81.915 0)
-      (effects (font (size 1.27 1.27)) hide)
-    )
-    (property "Value" "GND" (id 1) (at 165.735 80.645 0)
-      (effects (font (size 1.27 1.27)) hide)
-    )
-    (property "Footprint" "" (id 2) (at 165.735 75.565 0)
-      (effects (font (size 1.27 1.27)) hide)
-    )
-    (property "Datasheet" "" (id 3) (at 165.735 75.565 0)
+  (symbol (lib_id "power:GND") (at 165.735 81.915 0) (unit 1)
+    (in_bom yes) (on_board yes) (fields_autoplaced)
+    (property "Reference" "#PWR085" (id 0) (at 165.735 88.265 0)
+      (effects (font (size 1.27 1.27)) hide)
+    )
+    (property "Value" "GND" (id 1) (at 165.735 86.995 0)
+      (effects (font (size 1.27 1.27)) hide)
+    )
+    (property "Footprint" "" (id 2) (at 165.735 81.915 0)
+      (effects (font (size 1.27 1.27)) hide)
+    )
+    (property "Datasheet" "" (id 3) (at 165.735 81.915 0)
       (effects (font (size 1.27 1.27)) hide)
     )
@@
       (effects (font (size 1.27 1.27)) (justify left))
     )
-    (property "Value" "R_Small" (id 1) (at 142.875 80.6449 0)
-      (effects (font (size 1.27 1.27)) (justify left))
-    )
-    (property "Footprint" "Resistor_THT:R_Axial_DIN0204_L3.6mm_D1.6mm_P5.08mm_Horizontal" (id 2) (at 140.335 79.375 0)
+    (property "Value" "" (id 1) (at 142.875 80.6449 0)
+      (effects (font (size 1.27 1.27)) (justify left))
+    )
+    (property "Footprint" "" (id 2) (at 140.335 79.375 0)
       (effects (font (size 1.27 1.27)) hide)
     )
@@
     (pin "2")
   )
-  (symbol (lib_id "Device:C_Small") (at 165.735 70.485 0) (unit 1)
-    (in_bom yes) (on_board yes) (fields_autoplaced)
-    (property "Reference" "C22" (id 0) (at 168.275 69.2212 0)
-      (effects (font (size 1.27 1.27)) (justify left))
-    )
-    (property "Value" "22u" (id 1) (at 168.275 71.7612 0)
-      (effects (font (size 1.27 1.27)) (justify left))
-    )
-    (property "Footprint" "Capacitor_THT:CP_Radial_D5.0mm_P2.00mm" (id 2) (at 165.735 70.485 0)
-      (effects (font (size 1.27 1.27)) hide)
-    )
-    (property "Datasheet" "~" (id 3) (at 165.735 70.485 0)
+  (symbol (lib_id "Device:C_Small") (at 165.735 74.93 0) (unit 1)
+    (in_bom yes) (on_board yes) (fields_autoplaced)
+    (property "Reference" "C22" (id 0) (at 168.275 73.6662 0)
+      (effects (font (size 1.27 1.27)) (justify left))
+    )
+    (property "Value" "22u" (id 1) (at 168.275 76.2062 0)
+      (effects (font (size 1.27 1.27)) (justify left))
+    )
+    (property "Footprint" "Capacitor_THT:CP_Radial_D5.0mm_P2.00mm" (id 2) (at 165.735 74.93 0)
+      (effects (font (size 1.27 1.27)) hide)
+    )
+    (property "Datasheet" "~" (id 3) (at 165.735 74.93 0)
       (effects (font (size 1.27 1.27)) hide)
     )
@@
     (pin "2")
   )
-  (symbol (lib_id "power:GND") (at 154.305 75.565 0) (unit 1)
-    (in_bom yes) (on_board yes) (fields_autoplaced)
-    (property "Reference" "#PWR084" (id 0) (at 154.305 81.915 0)
-      (effects (font (size 1.27 1.27)) hide)
-    )
-    (property "Value" "GND" (id 1) (at 154.305 80.645 0)
-      (effects (font (size 1.27 1.27)) hide)
-    )
-    (property "Footprint" "" (id 2) (at 154.305 75.565 0)
-      (effects (font (size 1.27 1.27)) hide)
-    )
-    (property "Datasheet" "" (id 3) (at 154.305 75.565 0)
-      (effects (font (size 1.27 1.27)) hide)
-    )
+  (symbol (lib_id "power:GND") (at 154.305 81.915 0) (unit 1)
+    (in_bom yes) (on_board yes) (fields_autoplaced)
+    (property "Reference" "#PWR084" (id 0) (at 154.305 88.265 0)
+      (effects (font (size 1.27 1.27)) hide)
+    )
+    (property "Value" "GND" (id 1) (at 154.305 86.995 0)
+      (effects (font (size 1.27 1.27)) hide)
+    )
+    (property "Footprint" "" (id 2) (at 154.305 81.915 0)
+      (effects (font (size 1.27 1.27)) hide)
+    )
+    (property "Datasheet" "" (id 3) (at 154.305 81.915 0)
+      (effects (font (size 1.27 1.27)) hide)
+    )
