File: test_project_01/buck.kicad_sch (KiCad schematic)
At the start: 9 parts, among them U10 DIO6012BCST6

Commit message: r
Parts:
- added C24, C25: 10u, Capacitor_SMD:C_0805_2012Metric, symbol Device:C_Small
- C21, C22: value 22u -> 10u; footprint Capacitor_THT:CP_Radial_D5.0mm_P2.00mm -> Capacitor_SMD:C_0805_2012Metric
- RR1: value (none) -> 91k; footprint (none) -> Resistor_SMD:R_0805_2012Metric_Pad1.20x1.40mm_HandSolder
- RR2: value (none) -> 20k; footprint (none) -> Resistor_SMD:R_0805_2012Metric_Pad1.20x1.40mm_HandSolder
Connections:
- net BUCK_OUTPUT: now also C24.1, C25.1
- net GND: now also C24.2, C25.2
Changed lines of the file:
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@@
     (rev "1")
   )
+  (junction (at 187.96 66.675) (diameter 0) (color 0 0 0 0)
+  )
   (junction (at 154.305 66.675) (diameter 0) (color 0 0 0 0)
   )
   (junction (at 165.735 66.675) (diameter 0) (color 0 0 0 0)
+  )
+  (junction (at 176.53 66.675) (diameter 0) (color 0 0 0 0)
   )
   (junction (at 131.445 66.675) (diameter 0) (color 0 0 0 0)
@@
     (stroke (width 0) (type default) (color 0 0 0 0))
   )
+  (wire (pts (xy 176.53 66.675) (xy 187.96 66.675))
+    (stroke (width 0) (type default) (color 0 0 0 0))
+  )
   (wire (pts (xy 94.615 69.215) (xy 94.615 75.565))
     (stroke (width 0) (type default) (color 0 0 0 0))
@@
     (stroke (width 0) (type default) (color 0 0 0 0))
   )
+  (wire (pts (xy 187.96 77.47) (xy 187.96 81.915))
+    (stroke (width 0) (type default) (color 0 0 0 0))
+  )
   (wire (pts (xy 94.615 66.675) (xy 98.425 66.675))
     (stroke (width 0) (type default) (color 0 0 0 0))
@@
     (stroke (width 0) (type default) (color 0 0 0 0))
   )
-  (wire (pts (xy 165.735 66.675) (xy 193.675 66.675))
+  (wire (pts (xy 165.735 66.675) (xy 176.53 66.675))
     (stroke (width 0) (type default) (color 0 0 0 0))
   )
@@
     (stroke (width 0) (type default) (color 0 0 0 0))
   )
+  (wire (pts (xy 187.96 66.675) (xy 193.675 66.675))
+    (stroke (width 0) (type default) (color 0 0 0 0))
+  )
   (wire (pts (xy 61.595 66.675) (xy 74.295 66.675))
     (stroke (width 0) (type default) (color 0 0 0 0))
@@
     (stroke (width 0) (type default) (color 0 0 0 0))
   )
+  (wire (pts (xy 176.53 77.47) (xy 176.53 81.915))
+    (stroke (width 0) (type default) (color 0 0 0 0))
+  )
   (wire (pts (xy 71.755 69.215) (xy 74.295 69.215))
     (stroke (width 0) (type default) (color 0 0 0 0))
   )
+  (wire (pts (xy 176.53 66.675) (xy 176.53 72.39))
+    (stroke (width 0) (type default) (color 0 0 0 0))
+  )
   (wire (pts (xy 140.335 66.675) (xy 154.305 66.675))
+    (stroke (width 0) (type default) (color 0 0 0 0))
+  )
+  (wire (pts (xy 187.96 66.675) (xy 187.96 72.39))
     (stroke (width 0) (type default) (color 0 0 0 0))
   )
@@
       (effects (font (size 1.27 1.27)) (justify left))
     )
-    (property "Value" "" (id 1) (at 142.24 72.3899 0)
-      (effects (font (size 1.27 1.27)) (justify left))
-    )
-    (property "Footprint" "" (id 2) (at 140.335 71.12 0)
+    (property "Value" "91k" (id 1) (at 142.24 72.3899 0)
+      (effects (font (size 1.27 1.27)) (justify left))
+    )
+    (property "Footprint" "Resistor_SMD:R_0805_2012Metric_Pad1.20x1.40mm_HandSolder" (id 2) (at 140.335 71.12 0)
       (effects (font (size 1.27 1.27)) hide)
     )
@@
   (symbol (lib_id "Device:C_Small") (at 154.305 74.93 0) (unit 1)
     (in_bom yes) (on_board yes) (fields_autoplaced)
-    (property "Reference" "C21" (id 0) (at 156.845 73.6662 0)
-      (effects (font (size 1.27 1.27)) (justify left))
-    )
-    (property "Value" "22u" (id 1) (at 156.845 76.2062 0)
-      (effects (font (size 1.27 1.27)) (justify left))
-    )
-    (property "Footprint" "Capacitor_THT:CP_Radial_D5.0mm_P2.00mm" (id 2) (at 154.305 74.93 0)
+    (property "Reference" "C21" (id 0) (at 157.48 73.6662 0)
+      (effects (font (size 1.27 1.27)) (justify left))
+    )
+    (property "Value" "10u" (id 1) (at 157.48 76.2062 0)
+      (effects (font (size 1.27 1.27)) (justify left))
+    )
+    (property "Footprint" "Capacitor_SMD:C_0805_2012Metric" (id 2) (at 154.305 74.93 0)
       (effects (font (size 1.27 1.27)) hide)
     )
@@
     (pin "1")
   )
+  (symbol (lib_id "power:GND") (at 176.53 81.915 0) (unit 1)
+    (in_bom yes) (on_board yes) (fields_autoplaced)
+    (property "Reference" "#PWR089" (id 0) (at 176.53 88.265 0)
+      (effects (font (size 1.27 1.27)) hide)
+    )
+    (property "Value" "GND" (id 1) (at 176.53 86.995 0)
+      (effects (font (size 1.27 1.27)) hide)
+    )
+    (property "Footprint" "" (id 2) (at 176.53 81.915 0)
+      (effects (font (size 1.27 1.27)) hide)
+    )
+    (property "Datasheet" "" (id 3) (at 176.53 81.915 0)
+      (effects (font (size 1.27 1.27)) hide)
+    )
+    (pin "1")
+  )
   (symbol (lib_id "power:GND") (at 165.735 81.915 0) (unit 1)
     (in_bom yes) (on_board yes) (fields_autoplaced)
@@
       (effects (font (size 1.27 1.27)) (justify left))
     )
-    (property "Value" "" (id 1) (at 142.875 80.6449 0)
-      (effects (font (size 1.27 1.27)) (justify left))
-    )
-    (property "Footprint" "" (id 2) (at 140.335 79.375 0)
+    (property "Value" "20k" (id 1) (at 142.875 80.6449 0)
+      (effects (font (size 1.27 1.27)) (justify left))
+    )
+    (property "Footprint" "Resistor_SMD:R_0805_2012Metric_Pad1.20x1.40mm_HandSolder" (id 2) (at 140.335 79.375 0)
       (effects (font (size 1.27 1.27)) hide)
     )
@@
     (pin "2")
   )
+  (symbol (lib_id "Device:C_Small") (at 187.96 74.93 0) (unit 1)
+    (in_bom yes) (on_board yes) (fields_autoplaced)
+    (property "Reference" "C25" (id 0) (at 190.5 73.6662 0)
+      (effects (font (size 1.27 1.27)) (justify left))
+    )
+    (property "Value" "10u" (id 1) (at 190.5 76.2062 0)
+      (effects (font (size 1.27 1.27)) (justify left))
+    )
+    (property "Footprint" "Capacitor_SMD:C_0805_2012Metric" (id 2) (at 187.96 74.93 0)
+      (effects (font (size 1.27 1.27)) hide)
+    )
+    (property "Datasheet" "~" (id 3) (at 187.96 74.93 0)
+      (effects (font (size 1.27 1.27)) hide)
+    )
+    (pin "1")
+    (pin "2")
+  )
   (symbol (lib_id "Device:C_Small") (at 165.735 74.93 0) (unit 1)
     (in_bom yes) (on_board yes) (fields_autoplaced)
@@
       (effects (font (size 1.27 1.27)) (justify left))
     )
-    (property "Value" "22u" (id 1) (at 168.275 76.2062 0)
-      (effects (font (size 1.27 1.27)) (justify left))
-    )
-    (property "Footprint" "Capacitor_THT:CP_Radial_D5.0mm_P2.00mm" (id 2) (at 165.735 74.93 0)
+    (property "Value" "10u" (id 1) (at 168.275 76.2062 0)
+      (effects (font (size 1.27 1.27)) (justify left))
+    )
+    (property "Footprint" "Capacitor_SMD:C_0805_2012Metric" (id 2) (at 165.735 74.93 0)
       (effects (font (size 1.27 1.27)) hide)
     )
@@
     (pin "1")
     (pin "2")
+  )
+  (symbol (lib_id "power:GND") (at 187.96 81.915 0) (unit 1)
+    (in_bom yes) (on_board yes) (fields_autoplaced)
+    (property "Reference" "#PWR090" (id 0) (at 187.96 88.265 0)
+      (effects (font (size 1.27 1.27)) hide)
+    )
+    (property "Value" "GND" (id 1) (at 187.96 86.995 0)
+      (effects (font (size 1.27 1.27)) hide)
+    )
+    (property "Footprint" "" (id 2) (at 187.96 81.915 0)
+      (effects (font (size 1.27 1.27)) hide)
+    )
+    (property "Datasheet" "" (id 3) (at 187.96 81.915 0)
+      (effects (font (size 1.27 1.27)) hide)
+    )
+    (pin "1")
   )
   (symbol (lib_id "Device:C_Small") (at 131.445 70.485 0) (unit 1)
@@
     (pin "1")
   )
+  (symbol (lib_id "Device:C_Small") (at 176.53 74.93 0) (unit 1)
+    (in_bom yes) (on_board yes) (fields_autoplaced)
+    (property "Reference" "C24" (id 0) (at 179.07 73.6662 0)
+      (effects (font (size 1.27 1.27)) (justify left))
+    )
+    (property "Value" "10u" (id 1) (at 179.07 76.2062 0)
+      (effects (font (size 1.27 1.27)) (justify left))
+    )
+    (property "Footprint" "Capacitor_SMD:C_0805_2012Metric" (id 2) (at 176.53 74.93 0)
+      (effects (font (size 1.27 1.27)) hide)
+    )
+    (property "Datasheet" "~" (id 3) (at 176.53 74.93 0)
+      (effects (font (size 1.27 1.27)) hide)
+    )
+    (pin "1")
+    (pin "2")
+  )
   (symbol (lib_id "Device:FerriteBead_Small") (at 47.625 66.675 90) (unit 1)

Commit message: Y
Other:
- title: ESP32 audio power meter SD dataloger -> ESP32 MP3 player/web radio+power meter+uSD dataloger
Changed lines of the file:
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@@
   (paper "A3")
   (title_block
-    (title "ESP32 audio power meter SD dataloger")
-    (rev "1")
+    (title "ESP32 MP3 player/web radio+power meter+uSD dataloger")
+    (rev "2")
   )
   (junction (at 187.96 66.675) (diameter 0) (color 0 0 0 0)
