File: V2/test_project_01.kicad_sch (KiCad schematic)
At the start: 71 parts, among them IC1 XRA1203IG24TR-F, J1 STX-3120-5B, J2 SS-52100-001, J3 MEM2051-00-195-00-A, J8 Conn_01x06, SW1 SW_SPST, U1 ESP32-C3-MINI-1, U2 LM4040DBZ-3, U3 MCP3208, U4 Adafruit_MAX98357, U5 D1213A-02SM

Commit message: Update test_project_01.kicad_sch
Parts:
- removed C1, C3: 10u, Capacitor_SMD:C_0603_1608Metric_Pad1.08x0.95mm_HandSolder, symbol Device:C_Small
- removed C2: 1u, Capacitor_SMD:C_0603_1608Metric_Pad1.08x0.95mm_HandSolder, symbol Device:C_Small
- removed C5: 100n, Capacitor_SMD:C_0603_1608Metric_Pad1.08x0.95mm_HandSolder, symbol Device:C_Small
- removed R2: 10k, Resistor_SMD:R_0603_1608Metric_Pad0.98x0.95mm_HandSolder, symbol Device:R_Small
- removed SW1: SW_SPST, SamacSys_Parts:PTS526SM15SMTR2LFS, symbol Switch:SW_SPST
- removed U1: ESP32-C3-MINI-1, Espressif:ESP32-C3-MINI-1_Hand-Soldering, symbol Espressif:ESP32-C3-MINI-1
Connections:
- no-connect marks 32 -> 21
Other:
- note removed: "MCU"
- note removed: "MCU can: push 40mA out pull 28mA in 350mA max consumption (wifi)"
- note removed: "acording to DC doc: https://docs.espressif.com/projects/esp-idf/en/latest/esp32/api-reference/peripherals/sdmmc_host.html"
- note removed: "https://www.espressif.com/sites/default/files/documentation/esp32-c3_hardware_design_guidelines_en.pdf anteena is on the left pull up/down resitors are 45k"
- moved on the sheet: C23, C26, C4, C6, C7, C8, C9, D1, D5, D6, D7, D8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

Commit message: Update test_project_01.kicad_sch
Parts:
- added C? (x2): 100n, Capacitor_SMD:C_0603_1608Metric_Pad1.08x0.95mm_HandSolder, symbol Device:C_Small
- added C?: 15n, Capacitor_SMD:C_0603_1608Metric_Pad1.08x0.95mm_HandSolder, symbol Device:C_Small
- added C?: 22u, Capacitor_SMD:C_0805_2012Metric_Pad1.18x1.45mm_HandSolder, symbol Device:C_Small
- added C?: DNP, Capacitor_SMD:C_0603_1608Metric_Pad1.08x0.95mm_HandSolder, symbol Device:C_Small
- added Q? (x2): BC847BS, Package_TO_SOT_SMD:SOT-363_SC-70-6_Handsoldering, symbol Device:Q_Dual_NPN_NPN_E1B1C2E2B2C1
- added R? (x3): 10k, Resistor_SMD:R_0603_1608Metric_Pad0.98x0.95mm_HandSolder, symbol Device:R_Small
- added SW?: MCU_RESET, SamacSys_Parts:PTS526SK15SMTR2LFS, symbol Switch:SW_SPST
- added U?: ESP32-S3-WROOM-1, Espressif:ESP32-S3-WROOM-1, symbol Espressif:ESP32-S3-WROOM-1
Connections:
- net +3V3: now also C?.1, C?.1, R?.2, U?.2 (3V3)
- net GND: now also C?.2, C?.2, C?.2, C?.2, C?.2, SW?.2 (B), U?.1 (GND), U?.40 (GND), U?.41 (GND)
- new net BASE1: Q?.2 (B1), R?.1
- new net BASE2: Q?.5 (B2), R?.2
- new net BOOT: C?.1, Q?.3 (C2), R?.1, U?.27 (GPIO0/BOOT)
- new net GPIO_01: U?.39 (GPIO1/TOUCH1/ADC1_CH0)
- new net GPIO_02: U?.38 (GPIO2/TOUCH2/ADC1_CH1)
- new net GPIO_03: U?.15 (GPIO3/TOUCH3/ADC1_CH2)
- new net GPIO_04: U?.4 (GPIO4/TOUCH4/ADC1_CH3)
- new net GPIO_05: U?.5 (GPIO5/TOUCH5/ADC1_CH4)
- new net GPIO_06: U?.6 (GPIO6/TOUCH6/ADC1_CH5)
- new net GPIO_07: U?.7 (GPIO7/TOUCH7/ADC1_CH6)
- new net GPIO_08: U?.12 (GPIO8/TOUCH8/ADC1_CH7/SUBSPICS1)
- new net GPIO_09: U?.17 (GPIO9/TOUCH9/ADC1_CH8/FSPIHD/SUBSPIHD)
- new net GPIO_10: U?.18 (GPIO10/TOUCH10/ADC1_CH9/FSPICS0/FSPIIO4/SUBSPICS0)
- new net GPIO_11: U?.19 (GPIO11/TOUCH11/ADC2_CH0/FSPID/FSPIIO5/SUBSPID)
- new net GPIO_12: U?.20 (GPIO12/TOUCH12/ADC2_CH1/FSPICLK/FSPIIO6/SUBSPICLK)
- new net GPIO_13: U?.21 (GPIO13/TOUCH13/ADC2_CH2/FSPIQ/FSPIIO7/SUBSPIQ)
- new net GPIO_14: U?.22 (GPIO14/TOUCH14/ADC2_CH3/FSPIWP/FSPIDQS/SUBSPIWP)
- new net GPIO_15: U?.8 (GPIO15/U0RTS/ADC2_CH4/XTAL_32K_P)
- new net GPIO_16: U?.9 (GPIO16/U0CTS/ADC2_CH5/XTAL_32K_NH5)
- new net GPIO_17: U?.10 (GPIO17/U1TXD/ADC2_CH6)
- new net GPIO_18: U?.11 (GPIO18/U1RXD/ADC2_CH7/CLK_OUT3)
- new net GPIO_21: U?.23 (GPIO21)
- new net GPIO_35: U?.28 (SPIIO6/GPIO35/FSPID/SUBSPID)
- new net GPIO_36: U?.29 (SPIIO7/GPIO36/FSPICLK/SUBSPICLK)
- new net GPIO_37: U?.30 (SPIDQS/GPIO37/FSPIQ/SUBSPIQ)
- new net GPIO_38: U?.31 (GPIO38/FSPIWP/SUBSPIWP)
- new net GPIO_39: U?.32 (MTCK/GPIO39/CLK_OUT3/SUBSPICS1)
- new net GPIO_40: U?.33 (MTDO/GPIO40/CLK_OUT2)
- new net GPIO_41: U?.34 (MTDI/GPIO41/CLK_OUT1)
- new net GPIO_42: U?.35 (MTMS/GPIO42)
- new net GPIO_45: U?.26 (GPIO45)
- new net GPIO_46: U?.16 (GPIO46)
- new net GPIO_47: U?.24 (GPIO47/SPICLK_P/SUBSPICLK_P_DIFF)
- new net GPIO_48: U?.25 (GPIO48/SPICLK_N/SUBSPICLK_N_DIFF)
- new net PG_3V3: C?.1, C?.1, Q?.6 (C1), SW?.1 (A), U?.3 (EN)
- new net UART0_RX: U?.36 (U0RXD/GPIO44/CLK_OUT2)
- new net UART0_TX: U?.37 (U0TXD/GPIO43/CLK_OUT1)
- new net USB_OTG_D+: U?.14 (GPIO20/U1CTS/ADC2_CH9/CLK_OUT1/USB_D+)
- new net USB_OTG_D-: U?.13 (GPIO19/U1RTS/ADC2_CH8/CLK_OUT2/USB_D-)
- new net ~{DTR}: Q?.4 (E2), R?.2
- new net ~{RTS}: Q?.1 (E1), R?.1
- no-connect marks 21 -> 24
Other:
- note added: "BOOOT & RESET"
- note added: "Danger free pins:"
- note added: "ESP32-S3 has four strapping pins: • GPIO0 • GPIO45 • GPIO46 • GPIO3 GPIO0, GPIO45 and GPIO46 are connected to the chip's internal weak pull-up/pull-down during the chip reset. GPIO3 is floating by default"
- note added: "Free safe pins:"
- note added: "Internal Pull-up/down 45k Max IC typical current: source 40mA sink 28mA EN pin TTL: 0.75*Vcc+ HIGH 0.25*Vcc- LOW"
- note added: "MCU"
- note added: "NOTE: PG 1Meg R so for delay in ms is cap rating in nF ex: 15ms => 15nF"
- note added: "RC delay recomanded min 10ms wanted 15-20ms"
