File: ESP32_power_meter_MP3_player_WIFI_radio_V2/ESP32_power_meter_MP3_player_WIFI_radio_V2.kicad_pcb (KiCad board)
At the start: 2 copper layers, 99.9 x 100 mm, 140 parts, among them IC1 XRA1203IG24TR-F, IC2 INA2181A4QDGSRQ1, IC3 MCP73834T-FCI_UN, IC4 AP2112M-3.3TRG1, J1 STX-3120-5B, J10 10033527-N3112MLF, J11 Conn_01x02, J12 Conn_01x02, J13 Conn_01x02, J2 SS-52100-001, J3 MEM2051-00-195-00-A, J4 Barrel_Jack_Switch, J5 Barrel_Jack_Switch, J6 Conn_01x03, J7 Conn_01x03, J8 Conn_01x06, J9 USB_A, Q1 DMG9933USD-13, Q2 BC847BS, SW1 MCU_RESET, U1 ESP32-S3-WROOM-1, U10 DIO6012BCST6, U2 LM4040DBZ-3, U3 MCP3208, U4 Adafruit_MAX98357, U5 D1213A-02SM, U6 LM324A, U7 1043, U8 APX810S05

Commit message: m
Parts:
- removed D8, D9: LED_Small Green, LED_SMD:LED_0603_1608Metric_Pad1.05x0.95mm_HandSolder
- removed JP2: Jumper_3_Open, Connector_PinHeader_2.54mm:PinHeader_1x03_P2.54mm_Vertical
- removed R41: 5m, Resistor_SMD:R_0612_1632Metric_Pad1.18x3.40mm_HandSolder
- removed R42, R43: 1Meg, Resistor_SMD:R_0603_1608Metric_Pad0.98x0.95mm_HandSolder
- removed R44, R45, R46, R47: 330, Resistor_SMD:R_0603_1608Metric_Pad0.98x0.95mm_HandSolder
- removed R48, R49, R50: 10k, Resistor_SMD:R_0603_1608Metric_Pad0.98x0.95mm_HandSolder
- removed S3: EG1224 SPDT switch, SamacSys_Parts:EG1224
- removed TP1, TP2, TP3: TestPoint, TestPoint:TestPoint_Pad_1.0x1.0mm
- removed U10: DIO6012BCST6, Package_TO_SOT_SMD:SOT-23-6_Handsoldering
- added SW2: MCU_RESET, SamacSys_Parts:PTS526SK15SMTR2LFS, F.Cu at (345.3, 138.5)
- added U9: DIO6012BCST6, Package_TO_SOT_SMD:SOT-23-6_Handsoldering, F.Cu at (418.0, 92.0)
- C1: value 22u -> 100n; footprint Capacitor_SMD:C_0805_2012Metric_Pad1.18x1.45mm_HandSolder -> Capacitor_SMD:C_0603_1608Metric_Pad1.08x0.95mm_HandSolder
- C10: value 0.1u -> 100n
- C11: value 1u -> DNP
- C12: value 100n -> 15n
- C13: value 1u -> 0.1u
- C14: value 100n -> 1u
- C15: value 1u -> 100n
- C16: value 4.7u -> 1u
- C17: value 1u -> 100n; footprint Capacitor_SMD:C_0805_2012Metric_Pad1.18x1.45mm_HandSolder -> Capacitor_SMD:C_0603_1608Metric_Pad1.08x0.95mm_HandSolder
- C19: value 22u -> 1u; footprint Capacitor_THT:CP_Radial_D5.0mm_P2.00mm -> Capacitor_SMD:C_0805_2012Metric_Pad1.18x1.45mm_HandSolder
- C20: value 22p optional -> 1u
- C21: value 10u -> 4.7u; footprint Capacitor_SMD:C_0805_2012Metric -> Capacitor_SMD:C_0603_1608Metric_Pad1.08x0.95mm_HandSolder
- C22: value 10u -> 22u; footprint Capacitor_SMD:C_0805_2012Metric -> Capacitor_THT:CP_Radial_D5.0mm_P2.00mm
- C23: value 100n -> 22p optional
- C26: footprint Capacitor_SMD:C_0603_1608Metric_Pad1.08x0.95mm_HandSolder -> Capacitor_SMD:C_0805_2012Metric
- C27: value 15n -> 10u; footprint Capacitor_SMD:C_0603_1608Metric_Pad1.08x0.95mm_HandSolder -> Capacitor_SMD:C_0805_2012Metric
- C4: value 100n -> 10u
- C5: value DNP -> 22u; footprint Capacitor_SMD:C_0603_1608Metric_Pad1.08x0.95mm_HandSolder -> Capacitor_SMD:C_0805_2012Metric_Pad1.18x1.45mm_HandSolder
- C7: value 100n -> 10u; footprint Capacitor_SMD:C_0603_1608Metric_Pad1.08x0.95mm_HandSolder -> Capacitor_SMD:C_0805_2012Metric
- C8: value 10u -> 100n
- D1: value LED_Small Green -> Green
- D2, D3: value LED_Small -> Green
- D4: value D_Shockley -> Green; footprint Diode_THT:D_DO-15_P5.08mm_Vertical_AnodeUp -> LED_SMD:LED_0603_1608Metric_Pad1.05x0.95mm_HandSolder
- D5, D6: value LED_Small Green -> LED_Small
- D7: value LED_Small Green -> D_Shockley; footprint LED_SMD:LED_0603_1608Metric_Pad1.05x0.95mm_HandSolder -> Diode_THT:D_DO-15_P5.08mm_Vertical_AnodeUp
- FID2: footprint Symbol:Polarity_Center_Positive_6mm_SilkScreen -> Symbol:KiCad-Logo2_6mm_SilkScreen
- FID3: footprint Symbol:OSHW-Logo_5.7x6mm_SilkScreen -> Symbol:Polarity_Center_Positive_6mm_SilkScreen
- FID4: footprint Symbol:KiCad-Logo2_6mm_SilkScreen -> Symbol:WEEE-Logo_5.6x8mm_SilkScreen
- FID5: footprint Symbol:WEEE-Logo_5.6x8mm_SilkScreen -> Symbol:OSHW-Logo_5.7x6mm_SilkScreen
- IC3: value MCP73834T-FCI_UN -> AP2112M-3.3TRG1; footprint SamacSys_Parts:SOP50P490X110-10N -> SamacSys_Parts:SOIC127P600X170-8N
- IC4: value AP2112M-3.3TRG1 -> MCP73834T-FCI_UN; footprint SamacSys_Parts:SOIC127P600X170-8N -> SamacSys_Parts:SOP50P490X110-10N
- J10: value 10033527-N3112MLF -> USB_A; footprint SamacSys_Parts:10033527N3112MLF -> Connector_USB:USB_A_Molex_67643_Horizontal
- J11: value Conn_01x02 -> Conn_01x03; footprint TestPoint:TestPoint_2Pads_Pitch5.08mm_Drill1.3mm -> Connectors:SCREWTERMINAL-5MM-3
- J2: value SS-52100-001 -> MEM2051-00-195-00-A; footprint SamacSys_Parts:SS52100001 -> SamacSys_Parts:MEM20510019500A
- J3: value MEM2051-00-195-00-A -> SS-52100-001; footprint SamacSys_Parts:MEM20510019500A -> SamacSys_Parts:SS52100001
- J4: value Barrel_Jack_Switch -> Conn_01x06; footprint Z_mycustom_footprint_lib:DC plug jack 5.5-2.5mm -> Connector_PinHeader_2.54mm:PinHeader_1x06_P2.54mm_Vertical
- J5: footprint Connector_BarrelJack:BarrelJack_Wuerth_6941xx301002 -> Z_mycustom_footprint_lib:DC plug jack 5.5-2.5mm
- J6: value Conn_01x03 -> Conn_01x02; footprint Connectors:SCREWTERMINAL-5MM-3 -> TestPoint:TestPoint_2Pads_Pitch5.08mm_Drill1.3mm
- J7: value Conn_01x03 -> 10033527-N3112MLF; footprint Connectors:SCREWTERMINAL-5MM-3 -> SamacSys_Parts:10033527N3112MLF
- J8: value Conn_01x06 -> Barrel_Jack_Switch; footprint Connector_PinHeader_2.54mm:PinHeader_1x06_P2.54mm_Vertical -> Connector_BarrelJack:BarrelJack_Wuerth_6941xx301002
- J9: value USB_A -> Conn_01x03; footprint Connector_USB:USB_A_Molex_67643_Horizontal -> Connectors:SCREWTERMINAL-5MM-3
- JP1: value Jumper_2_Bridged -> Jumper_3_Open; footprint Jumper:SolderJumper-2_P1.3mm_Bridged_RoundedPad1.0x1.5mm -> Connector_PinHeader_2.54mm:PinHeader_1x03_P2.54mm_Vertical
- Q1: value DMG9933USD-13 -> BC847BS; footprint SamacSys_Parts:SOIC127P600X175-8N -> Package_TO_SOT_SMD:SOT-363_SC-70-6_Handsoldering
- Q2: value BC847BS -> DMG9933USD-13; footprint Package_TO_SOT_SMD:SOT-363_SC-70-6_Handsoldering -> SamacSys_Parts:SOIC127P600X175-8N
- R10, R11, R12: value 10k -> 330
- R13: value 10k -> 20k
- R20: value 4.7k -> 10k; footprint Resistor_SMD:R_0805_2012Metric -> Resistor_SMD:R_0603_1608Metric_Pad0.98x0.95mm_HandSolder
- R23, R28: value 10k -> 100k
- R24: value 1k -> 5m; footprint Resistor_SMD:R_0603_1608Metric_Pad0.98x0.95mm_HandSolder -> Resistor_SMD:R_0612_1632Metric_Pad1.18x3.40mm_HandSolder
- R25: value 1k -> 30m; footprint Resistor_SMD:R_0603_1608Metric_Pad0.98x0.95mm_HandSolder -> Resistor_SMD:R_0402_1005Metric_Pad0.72x0.64mm_HandSolder
- R26: value 100k -> 1Meg
- R27, R29: value 100k -> 1k
- R3: value 20k -> 10k
- R30: value 330 -> 10k
- R31: value 5m -> 100k; footprint Resistor_SMD:R_0612_1632Metric_Pad1.18x3.40mm_HandSolder -> Resistor_SMD:R_0603_1608Metric_Pad0.98x0.95mm_HandSolder
- R32: value 1Meg -> 10k
- R33: value 10k -> 470
- R35: value 30m -> 5m; footprint Resistor_SMD:R_0402_1005Metric_Pad0.72x0.64mm_HandSolder -> Resistor_SMD:R_0612_1632Metric_Pad1.18x3.40mm_HandSolder
- R37: value 470 -> 1Meg
- R40: value 10k -> 1Meg
- R9: value 10k -> 4.7k; footprint Resistor_SMD:R_0603_1608Metric_Pad0.98x0.95mm_HandSolder -> Resistor_SMD:R_0805_2012Metric
- S2: value DS01C-254-S-08BE -> EG1224 SPDT switch; footprint SamacSys_Parts:DS01C254S08BE -> SamacSys_Parts:EG1224
- SW1: value MCU_RESET -> GPIO_RESET
- U1: value ESP32-S3-WROOM-1 -> LM4040DBZ-3; footprint Espressif:ESP32-S3-WROOM-1 -> Package_TO_SOT_SMD:SOT-23
- U2: value LM4040DBZ-3 -> MCP3208; footprint Package_TO_SOT_SMD:SOT-23 -> Package_SO:SOIC-16_3.9x9.9mm_P1.27mm
- U3: value MCP3208 -> Adafruit_MAX98357; footprint Package_SO:SOIC-16_3.9x9.9mm_P1.27mm -> Z_mycustom_footprint_lib:Adafruit MAX98357 I2S Class-D Mono
- U4: value Adafruit_MAX98357 -> ESP32-S3-WROOM-1; footprint Z_mycustom_footprint_lib:Adafruit MAX98357 I2S Class-D Mono -> Espressif:ESP32-S3-WROOM-1
- moved C15 283.5 mm to (483.2, 53.8)
- moved J8 261.6 mm to (481.9, 37.9)
- moved R21 259.5 mm to (471.2, 57.1)
- moved C17 252.1 mm to (458.2, 59.5)
- moved JP1 250.1 mm to (478.7, 54.9)
- moved C16 249.3 mm to (445.1, 59.3)
- moved R30 241.3 mm to (462.5, 59.5)
- moved Q2 213.7 mm to (395.7, 50.3)
- moved R20 205.5 mm to (453.8, 59.3)
- moved C23 199.6 mm to (415.3, 103.5)
- moved C26 193.5 mm to (423.1, 94.1)
- moved U1 188.3 mm to (385.7, 100.2)
- moved FID2 186.3 mm to (382.5, 93.1)
- moved C13 180.5 mm to (504.8, 37.2)
- moved J7 174.8 mm to (495.6, 42.6)
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Connections:
- C1 pad 1: +3V3 -> +VDC
- C10 pad 1: Net-(C10-Pad1) -> /BOOT
- C11 pad 1: +VDC -> /EN
- C12 pad 1: GND -> /EN
- C12 pad 2: +VDC -> GND
- C13 pad 1: +3V3 -> Net-(C13-Pad1)
- C15 pad 1: +5V -> +3V3
- C16 pad 1: +BATT -> +VDC
- C17 pad 1: +VDC -> GND
- C17 pad 2: GND -> +VDC
- C18 pad 1: /Power-IN-OUT-BMS/lin_reg -> +VDC
- C19 pad 1: /Power-IN-OUT-BMS/buck/buck_input_filtered -> /Power-IN-OUT-BMS/lin_reg
- C2 pad 1: +3V3 -> GND
- C2 pad 2: GND -> +VDC
- C20 pad 1: /Power-IN-OUT-BMS/buck_out -> +5V
- C20 pad 2: Net-(C20-Pad2) -> GND
- C21 pad 1: /Power-IN-OUT-BMS/buck_out -> +BATT
- C22 pad 1: /Power-IN-OUT-BMS/buck_out -> /Power-IN-OUT-BMS/buck/buck_input_filtered
- C23 pad 1: GND -> /Power-IN-OUT-BMS/buck_out
- C23 pad 2: +3V3 -> Net-(C23-Pad2)
- C26 pad 1: +3V3 -> /Power-IN-OUT-BMS/buck_out
- C27 pad 1: /EN -> /Power-IN-OUT-BMS/buck_out
- C3 pad 1: /BOOT -> GND
- C3 pad 2: GND -> /Vref
- C4 pad 1: GND -> +VDC
- C4 pad 2: /Vref -> GND
- C5 pad 1: /EN -> +3V3
- C6 pad 1: +VDC -> +3V3
- C7 pad 1: GND -> +3V3
- C7 pad 2: +VDC -> GND
- C8 pad 1: +VDC -> GND
- C8 pad 2: GND -> +3V3
- D2 pad 1: Net-(D2-Pad1) -> GND
- D2 pad 2: +5V -> Net-(R10-Pad1)
- D3 pad 1: Net-(D3-Pad1) -> GND
- D3 pad 2: +5V -> Net-(R11-Pad1)
- D4 pad 1: Power_in+ -> GND
- D4 pad 2: +5V -> Net-(D4-Pad2)
- D5 pad 1: GND -> Net-(D5-Pad1)
- D5 pad 2: Net-(D5-Pad2) -> +5V
- D6 pad 1: GND -> Net-(D6-Pad1)
- D6 pad 2: Net-(D6-Pad2) -> +5V
- D7 pad 1: GND -> Power_in+
- D7 pad 2: Net-(D7-Pad2) -> +5V
- IC1 pad 1: /GPIO5 -> /IRQ
- IC1 pad 10: Net-(IC1-Pad10) -> unconnected-(IC1-Pad10)
- IC1 pad 13: Net-(IC1-Pad13) -> unconnected-(IC1-Pad13)
- IC1 pad 15: Net-(IC1-Pad15) -> unconnected-(IC1-Pad15)
- IC1 pad 16: Net-(IC1-Pad16) -> unconnected-(IC1-Pad16)
- IC1 pad 17: Net-(IC1-Pad17) -> unconnected-(IC1-Pad17)
- IC1 pad 19: Net-(IC1-Pad19) -> unconnected-(IC1-Pad19)
- IC1 pad 20: Net-(IC1-Pad20) -> unconnected-(IC1-Pad20)
- IC1 pad 4: /SPI2_SS1 -> unconnected-(IC1-Pad4)
- IC1 pad 5: /DATA3 -> unconnected-(IC1-Pad5)
- IC1 pad 6: /SD_sense -> unconnected-(IC1-Pad6)
- IC1 pad 7: /P3 -> unconnected-(IC1-Pad7)
- IC1 pad 9: Net-(IC1-Pad9) -> unconnected-(IC1-Pad9)
- IC3 pad 1: +5V -> /Power-IN-OUT-BMS/lin_reg
- IC3 pad 2: +5V -> unconnected-(IC3-Pad2)
- IC3 pad 3: Net-(IC3-Pad3) -> unconnected-(IC3-Pad3)
- IC3 pad 4: Net-(IC3-Pad4) -> unconnected-(IC3-Pad4)
- IC3 pad 5: GND -> 3v3_enable
- IC3 pad 6: /Power-IN-OUT-BMS/Set_charge_current -> GND
- IC3 pad 7: TE -> GND
- IC3 pad 8: Net-(IC3-Pad8) -> +VDC
- IC4 pad 1: /Power-IN-OUT-BMS/lin_reg -> +5V
- IC4 pad 2: unconnected-(IC4-Pad2) -> +5V
- IC4 pad 3: unconnected-(IC4-Pad3) -> Net-(IC4-Pad3)
- IC4 pad 4: unconnected-(IC4-Pad4) -> Net-(IC4-Pad4)
- IC4 pad 5: 3v3_enable -> GND
- IC4 pad 6: GND -> /Power-IN-OUT-BMS/Set_charge_current
- IC4 pad 7: GND -> TE
- IC4 pad 8: +VDC -> Net-(IC4-Pad8)
- J10 pad 1: /POWER_MEASUREMENTS/ext_5v -> /POWER_MEASUREMENTS/mini_power_load
- J10 pad 5: unconnected-(J10-Pad5) -> Net-(C13-Pad1)
- J11 pad 1: /POWER_MEASUREMENTS/ext_5v -> /POWER_MEASUREMENTS/load_vcc
- J4 pad 1: /POWER_MEASUREMENTS/source_vcc -> GND
- J4 pad 2: GND -> /TX
- J4 pad 3: unconnected-(J4-Pad3) -> /RX
- J6 pad 1: /POWER_MEASUREMENTS/source_vcc -> /POWER_MEASUREMENTS/ext_5v
- J7 pad 1: /POWER_MEASUREMENTS/load_vcc -> /POWER_MEASUREMENTS/ext_5v
- J7 pad 2: GND -> /POWER_MEASUREMENTS/D2-
- J7 pad 3: unconnected-(J7-Pad3) -> /POWER_MEASUREMENTS/D2+
- J8 pad 1: GND -> /POWER_MEASUREMENTS/source_vcc
- J8 pad 2: /TX -> GND
- J8 pad 3: /RX -> unconnected-(J8-Pad3)
- J9 pad 1: /POWER_MEASUREMENTS/mini_power_load -> /POWER_MEASUREMENTS/source_vcc
- J9 pad 2: /POWER_MEASUREMENTS/D2- -> GND
- J9 pad 3: /POWER_MEASUREMENTS/D2+ -> unconnected-(J9-Pad3)
- JP1 pad 1: Net-(IC1-Pad3) -> +5V
- JP1 pad 2: Net-(IC1-Pad9) -> /POWER_MEASUREMENTS/mini_power_source
- Q1 pad 1: +BATT -> /~{RTS}
- Q1 pad 2: /Power-IN-OUT-BMS/low_batt_shutoff -> /BASE1
- Q1 pad 3: Power_in+ -> /BOOT
- Q1 pad 4: +5V -> /~{DTR}
- Q1 pad 5: /Power-IN-OUT-BMS/Drains -> /BASE2
- Q1 pad 6: /Power-IN-OUT-BMS/Drains -> /EN
- Q2 pad 1: /~{RTS} -> +BATT
- Q2 pad 2: /BASE1 -> /Power-IN-OUT-BMS/low_batt_shutoff
- Q2 pad 3: /BOOT -> Power_in+
- Q2 pad 4: /~{DTR} -> +5V
- Q2 pad 5: /BASE2 -> /Power-IN-OUT-BMS/Drains
- Q2 pad 6: /EN -> /Power-IN-OUT-BMS/Drains
- R10 pad 1: /GPIO1 -> Net-(R10-Pad1)
- R11 pad 1: /DATA0 -> Net-(R11-Pad1)
- R11 pad 2: +3V3 -> /P3
- R12 pad 1: SDA -> Net-(D4-Pad2)
- R12 pad 2: +3V3 -> /GPIO_14
- R13 pad 1: SCL -> unconnected-(R13-Pad1)
- R13 pad 2: +3V3 -> GND
- R14 pad 1: /DATA2 -> Net-(IC1-Pad3)
- R15 pad 1: /DATA1 -> /IRQ
- R16 pad 1: Net-(IC1-Pad3) -> /BASE1
- R16 pad 2: +3V3 -> /~{DTR}
- R17 pad 1: /GPIO5 -> /BOOT
- R18 pad 1: TE -> +3V3
- R18 pad 2: Net-(IC1-Pad10) -> /EN
- R19 pad 1: GND -> /~{RTS}
- R19 pad 2: TE -> /BASE2
- R2 pad 1: /BASE1 -> +3V3
- R2 pad 2: /~{DTR} -> /GPIO_41
- R20 pad 1: Net-(D1-Pad2) -> GND
- R20 pad 2: +5V -> Net-(R20-Pad2)
- R21 pad 1: /SD_sense -> Net-(R20-Pad2)
- R21 pad 2: +3V3 -> /POWER_MEASUREMENTS/mini_power_source
- R22 pad 1: /POWER_MEASUREMENTS/ADC_CH6 -> GND
- R22 pad 2: Power_in+ -> Net-(R22-Pad2)
- R23 pad 1: GND -> Net-(R22-Pad2)
- R23 pad 2: /POWER_MEASUREMENTS/ADC_CH6 -> /POWER_MEASUREMENTS/source_vcc
- R24 pad 1: Power_in- -> /POWER_MEASUREMENTS/source_vcc
- R24 pad 2: Net-(R24-Pad2) -> /POWER_MEASUREMENTS/load_vcc
- R25 pad 1: Power_in+ -> /POWER_MEASUREMENTS/mini_power_load
- R25 pad 2: Net-(R25-Pad2) -> /POWER_MEASUREMENTS/mini_power_source
- R26 pad 2: Net-(R25-Pad2) -> Net-(C13-Pad1)
- R27 pad 1: Net-(R24-Pad2) -> Power_in-
- R27 pad 2: /POWER_MEASUREMENTS/ADC_CH5 -> Net-(R27-Pad2)
- R28 pad 1: GND -> Net-(R27-Pad2)
- R28 pad 2: Net-(R28-Pad2) -> /POWER_MEASUREMENTS/ADC_CH5
- R29 pad 1: Net-(R28-Pad2) -> Power_in+
- R29 pad 2: /POWER_MEASUREMENTS/source_vcc -> Net-(R29-Pad2)
- R3 pad 1: 3v3_enable -> +3V3
- R3 pad 2: GND -> /GPIO_36
- R30 pad 1: Net-(D7-Pad2) -> /POWER_MEASUREMENTS/ADC_CH6
- R30 pad 2: Net-(IC1-Pad20) -> Power_in+
- R31 pad 1: /POWER_MEASUREMENTS/source_vcc -> GND
- R31 pad 2: /POWER_MEASUREMENTS/load_vcc -> Net-(R29-Pad2)
- R32 pad 2: Net-(C10-Pad1) -> /POWER_MEASUREMENTS/ADC_CH6
- R33 pad 1: GND -> Net-(D5-Pad1)
- R33 pad 2: Net-(R33-Pad2) -> Net-(IC4-Pad3)
- R34 pad 1: Net-(R33-Pad2) -> GND
- R34 pad 2: /POWER_MEASUREMENTS/mini_power_source -> Net-(IC4-Pad8)
- R35 pad 1: /POWER_MEASUREMENTS/mini_power_load -> Power_in+
- R35 pad 2: /POWER_MEASUREMENTS/mini_power_source -> Power_in-
- R36 pad 1: Net-(D2-Pad1) -> Net-(D6-Pad1)
- R36 pad 2: Net-(IC3-Pad3) -> Net-(IC4-Pad4)
- R37 pad 1: Net-(D3-Pad1) -> Net-(R37-Pad1)
- R37 pad 2: Net-(IC3-Pad4) -> +VDC
- R38 pad 2: Net-(IC3-Pad8) -> /Power-IN-OUT-BMS/low_batt_shutoff
- R39 pad 2: /Power-IN-OUT-BMS/low_batt_shutoff -> +5V
- R4 pad 1: /A0 -> +3V3
- R4 pad 2: +3V3 -> /GPIO_37
- R40 pad 2: +5V -> Net-(R37-Pad1)
- R5 pad 1: /DATA3 -> +3V3
- R5 pad 2: +3V3 -> /GPIO_38
- R6 pad 1: /A1 -> +3V3
- R6 pad 2: +3V3 -> /GPIO_39
- R7 pad 1: /GPIO2 -> +3V3
- R7 pad 2: +3V3 -> /GPIO_40
- R8 pad 1: /on/off+mode -> +3V3
- R8 pad 2: Net-(R8-Pad2) -> /GPIO_42
- R9 pad 1: /gain -> Net-(D1-Pad2)
- R9 pad 2: Net-(R9-Pad2) -> +5V
- RR1 pad 2: Net-(C20-Pad2) -> Net-(C23-Pad2)
- RR2 pad 1: Net-(C20-Pad2) -> Net-(C23-Pad2)
- S1 pad 10: /GPIO9 -> unconnected-(S1-Pad10)
- S1 pad 11: /GPIO9 -> unconnected-(S1-Pad11)
- S1 pad 12: /BCLK -> unconnected-(S1-Pad12)
- S1 pad 13: /SPI1_MOSI -> unconnected-(S1-Pad13)
- S1 pad 14: /GPIO10 -> unconnected-(S1-Pad14)
- S1 pad 15: /GPIO10 -> unconnected-(S1-Pad15)
- S1 pad 16: /LRC -> unconnected-(S1-Pad16)
- S1 pad 5: /SPI1_MISO -> unconnected-(S1-Pad5)
- S1 pad 6: /GPIO8 -> unconnected-(S1-Pad6)
- S1 pad 7: /GPIO8 -> unconnected-(S1-Pad7)
- S1 pad 8: /DATA_IN -> unconnected-(S1-Pad8)
- S1 pad 9: /SPI1_CLK -> unconnected-(S1-Pad9)
- S2 pad 1: /GPIO9 -> /Power-IN-OUT-BMS/buck_out
- S2 pad 2: GND -> +3V3
- S2 pad 3: /A1 -> /Power-IN-OUT-BMS/lin_reg
- SW1 pad 1: /EN -> Net-(IC1-Pad3)
- U1 pad 1: GND -> /Vref
- U1 pad 2: +3V3 -> GND
- U1 pad 3: /EN -> (no net)
- U2 pad 1: /Vref -> /POWER_MEASUREMENTS/ADC_CH0
- U2 pad 2: GND -> /POWER_MEASUREMENTS/ADC_CH1
- U2 pad 3: (no net) -> ADC_CH2
- U3 pad 1: unconnected-(U3-Pad1) -> Net-(J1-Pad2)
- U3 pad 2: unconnected-(U3-Pad2) -> GND
- U3 pad 3: unconnected-(U3-Pad3) -> +VDC
- U3 pad 4: unconnected-(U3-Pad4) -> GND
- U3 pad 5: ADC_CH4 -> /GPIO_09
- U3 pad 6: unconnected-(U3-Pad6) -> /BCLK
- U3 pad 7: unconnected-(U3-Pad7) -> /DATA_IN
- U3 pad 8: unconnected-(U3-Pad8) -> /gain
- U3 pad 9: GND -> /GPIO_06
- U4 pad 1: unconnected-(U4-Pad1) -> GND
- U4 pad 2: unconnected-(U4-Pad2) -> +3V3
- U4 pad 3: +VDC -> /EN
- U4 pad 4: GND -> SDA
- U4 pad 5: /LRC -> SCL
- U4 pad 6: /BCLK -> /GPIO_06
- U4 pad 8: /gain -> /GPIO_15
- U4 pad 9: /on/off+mode -> /GPIO_16
- U5 pad 2: unconnected-(U5-Pad2) -> GND
- U5 pad 5: unconnected-(U5-Pad5) -> VBUS
- U6 pad 10: Net-(R24-Pad2) -> Net-(R27-Pad2)
- U6 pad 12: Net-(R42-Pad1) -> Net-(R37-Pad1)
- U6 pad 3: Net-(R33-Pad2) -> Net-(R20-Pad2)
- U6 pad 5: Net-(R28-Pad2) -> Net-(R22-Pad2)
- U6 pad 9: Net-(R25-Pad2) -> Net-(R29-Pad2)

Commit message: f
Parts:
- added C28: 22u, Capacitor_SMD:C_0805_2012Metric, F.Cu at (72.4, 132.6)
- added C29: 22u, Capacitor_SMD:C_0805_2012Metric, F.Cu at (75.2, 131.8)
- added C30: 100n, Capacitor_SMD:C_0603_1608Metric, F.Cu at (75.2, 133.6)
- added R41: 470, Resistor_SMD:R_0603_1608Metric_Pad0.98x0.95mm_HandSolder, F.Cu at (125.4, 107.8)
- added R42: 5m, Resistor_SMD:R_0612_1632Metric_Pad1.18x3.40mm_HandSolder, F.Cu at (96.3, 116.1)
- added R43: 10k, Resistor_SMD:R_0603_1608Metric_Pad0.98x0.95mm_HandSolder, F.Cu at (121.4, 115.0)
- added R44: 10k, Resistor_SMD:R_0603_1608Metric_Pad0.98x0.95mm_HandSolder, F.Cu at (118.4, 117.2)
- C1: value 100n -> 10u; footprint Capacitor_SMD:C_0603_1608Metric_Pad1.08x0.95mm_HandSolder -> Capacitor_SMD:C_0805_2012Metric
- C12: value 15n -> 100n
- C13: value 0.1u -> 100n
- C14, C20: value 1u -> 100n
- C18: value 1u -> 100n; footprint Capacitor_SMD:C_0805_2012Metric_Pad1.18x1.45mm_HandSolder -> Capacitor_SMD:C_0603_1608Metric_Pad1.08x0.95mm_HandSolder
- C19: footprint Capacitor_SMD:C_0805_2012Metric_Pad1.18x1.45mm_HandSolder -> Capacitor_SMD:C_0603_1608Metric_Pad1.08x0.95mm_HandSolder
- C21: value 4.7u -> 100n
- C22: value 22u -> 1u; footprint Capacitor_THT:CP_Radial_D5.0mm_P2.00mm -> Capacitor_SMD:C_0805_2012Metric_Pad1.18x1.45mm_HandSolder
- C23: value 22p optional -> 1u; footprint Capacitor_SMD:C_0603_1608Metric_Pad1.08x0.95mm_HandSolder -> Capacitor_SMD:C_0805_2012Metric_Pad1.18x1.45mm_HandSolder
- C24: value 10u -> 1u; footprint Capacitor_SMD:C_0805_2012Metric -> Capacitor_SMD:C_0603_1608Metric_Pad1.08x0.95mm_HandSolder
- C25: value 10u -> 4.7u; footprint Capacitor_SMD:C_0805_2012Metric -> Capacitor_SMD:C_0603_1608Metric_Pad1.08x0.95mm_HandSolder
- C26: value 10u -> 22u
- C27: value 10u -> 22p optional; footprint Capacitor_SMD:C_0805_2012Metric -> Capacitor_SMD:C_0603_1608Metric_Pad1.08x0.95mm_HandSolder
- C4: footprint Capacitor_SMD:C_0603_1608Metric_Pad1.08x0.95mm_HandSolder -> Capacitor_SMD:C_0805_2012Metric
- F1, F2: footprint Fuse:Fuse_0603_1608Metric_Pad1.05x0.95mm_HandSolder -> Fuse:Fuse_1812_4532Metric
- FB2: footprint Resistor_SMD:R_0402_1005Metric_Pad0.72x0.64mm_HandSolder -> Resistor_SMD:R_0603_1608Metric_Pad0.98x0.95mm_HandSolder
- J10: value USB_A -> Conn_01x02; footprint Connector_USB:USB_A_Molex_67643_Horizontal -> TestPoint:TestPoint_2Pads_Pitch5.08mm_Drill1.3mm
- J11: value Conn_01x03 -> USB_A; footprint Connectors:SCREWTERMINAL-5MM-3 -> Connector_USB:USB_A_Molex_67643_Horizontal
- J12: value Conn_01x02 -> Conn_01x03; footprint TestPoint:TestPoint_2Pads_Pitch5.08mm_Drill1.3mm -> Connectors:SCREWTERMINAL-5MM-3
- J3: value SS-52100-001 -> USB_A; footprint SamacSys_Parts:SS52100001 -> Connector_USB:USB_A_Molex_67643_Horizontal
- J7: value 10033527-N3112MLF -> Barrel_Jack_Switch; footprint SamacSys_Parts:10033527N3112MLF -> Connector_BarrelJack:BarrelJack_Wuerth_6941xx301002
- J8: value Barrel_Jack_Switch -> USB_A; footprint Connector_BarrelJack:BarrelJack_Wuerth_6941xx301002 -> Connector_USB:USB_A_Molex_67643_Horizontal
- R13: value 20k -> 10k
- R16, R17, R20, R32: value 10k -> 100k
- R23: value 100k -> 10k
- R24, R35: value 5m -> 10k; footprint Resistor_SMD:R_0612_1632Metric_Pad1.18x3.40mm_HandSolder -> Resistor_SMD:R_0603_1608Metric_Pad0.98x0.95mm_HandSolder
- R25: value 30m -> 10k; footprint Resistor_SMD:R_0402_1005Metric_Pad0.72x0.64mm_HandSolder -> Resistor_SMD:R_0603_1608Metric_Pad0.98x0.95mm_HandSolder
- R26: value 1Meg -> 100k
- R27: value 1k -> 10k
- R28: value 100k -> 5m; footprint Resistor_SMD:R_0603_1608Metric_Pad0.98x0.95mm_HandSolder -> Resistor_SMD:R_0612_1632Metric_Pad1.18x3.40mm_HandSolder
- R29: value 1k -> 30m; footprint Resistor_SMD:R_0603_1608Metric_Pad0.98x0.95mm_HandSolder -> Resistor_SMD:R_0402_1005Metric_Pad0.72x0.64mm_HandSolder
- R30: value 10k -> 1Meg
- R31: value 100k -> 1k
- R33: value 470 -> 10k
- R34: value 10k -> 1k
- R36: value 470 -> 100k
- R37, R40: value 1Meg -> 10k
- R39: value 10k -> 470
- U5: footprint Package_TO_SOT_SMD:SOT-23-5 -> Package_TO_SOT_SMD:SOT-23-5_HandSoldering
- U6: value LM324A -> LM324
- moved R32 375.4 mm to (100.0, 115.6)
- moved J8 369.2 mm to (127.3, 140.6)
- moved JP1 365.9 mm to (121.9, 135.8), turned to 90 degrees
- moved FB2 364.9 mm to (65.6, 139.2)
- moved J7 360.5 mm to (135.8, 65.2), turned to 90 degrees
- moved R29 357.9 mm to (132.6, 132.1), turned to 180 degrees
- moved C26 357.4 mm to (68.4, 138.2), turned to 90 degrees
- moved RR2 352.3 mm to (74.4, 140.0), turned to -90 degrees
- moved U9 349.5 mm to (71.4, 137.4), turned to -90 degrees
- moved R22 348.2 mm to (133.4, 129.7), turned to 90 degrees
- moved R31 345.7 mm to (100.0, 117.2)
- moved L1 344.3 mm to (68.8, 132.4), turned to 90 degrees
- moved R23 341.3 mm to (131.8, 129.7), turned to -90 degrees
- moved J10 338.0 mm to (135.6, 120.5), turned to -90 degrees
- moved RR1 337.9 mm to (74.4, 136.2), turned to -90 degrees
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Connections:
- C13 pad 1: Net-(C13-Pad1) -> /POWER_MEASUREMENTS/ADC_CH0
- C14 pad 1: +3V3 -> /POWER_MEASUREMENTS/ADC_CH2
- C15 pad 1: +3V3 -> Net-(C15-Pad1)
- C16 pad 1: +VDC -> +3V3
- C17 pad 1: GND -> +3V3
- C17 pad 2: +VDC -> GND
- C18 pad 1: +VDC -> /POWER_MEASUREMENTS/ADC_CH5
- C19 pad 1: /Power-IN-OUT-BMS/lin_reg -> +VDC
- C20 pad 1: +5V -> GND
- C20 pad 2: GND -> +VDC
- C21 pad 1: +BATT -> /POWER_MEASUREMENTS/ADC_CH6
- C22 pad 1: /Power-IN-OUT-BMS/buck/buck_input_filtered -> +VDC
- C23 pad 1: /Power-IN-OUT-BMS/buck_out -> /Power-IN-OUT-BMS/lin_reg
- C23 pad 2: Net-(C23-Pad2) -> GND
- C24 pad 1: /Power-IN-OUT-BMS/buck_out -> +5V
- C25 pad 1: /Power-IN-OUT-BMS/buck_out -> +BATT
- C26 pad 1: /Power-IN-OUT-BMS/buck_out -> /Power-IN-OUT-BMS/buck/buck_input_filtered
- C27 pad 2: GND -> Net-(C27-Pad2)
- C4 pad 1: +VDC -> GND
- C4 pad 2: GND -> +VDC
- C7 pad 1: +3V3 -> +3.3V
- C8 pad 2: +3V3 -> +3.3V
- IC1 pad 24: +3V3 -> +3.3V
- J10 pad 1: /POWER_MEASUREMENTS/mini_power_load -> GND
- J10 pad 2: /POWER_MEASUREMENTS/D2- -> /POWER_MEASUREMENTS/mini_power_load
- J11 pad 1: /POWER_MEASUREMENTS/load_vcc -> /POWER_MEASUREMENTS/mini_power_load
- J11 pad 2: GND -> /POWER_MEASUREMENTS/D2-
- J11 pad 3: unconnected-(J11-Pad3) -> /POWER_MEASUREMENTS/D2+
- J12 pad 1: GND -> /POWER_MEASUREMENTS/load_vcc
- J12 pad 2: /POWER_MEASUREMENTS/mini_power_load -> GND
- J13 pad 1: Net-(J13-Pad1) -> GND
- J13 pad 2: GND -> Net-(J13-Pad2)
- J2 pad P4: +3V3 -> +3.3V
- J3 pad 2: D- -> D+
- J3 pad 3: D+ -> D-
- J4 pad 2: /TX -> UART0_TX
- J4 pad 3: /RX -> UART0_RX
- J4 pad 4: /reset -> /BOOT
- J4 pad 5: /GPIO0 -> /EN
- J4 pad 6: +3V3 -> +3.3V
- J6 pad 1: /POWER_MEASUREMENTS/ext_5v -> GND
- J6 pad 2: GND -> /POWER_MEASUREMENTS/ext_5v
- J7 pad 1: /POWER_MEASUREMENTS/ext_5v -> /POWER_MEASUREMENTS/source_vcc
- J7 pad 2: /POWER_MEASUREMENTS/D2- -> GND
- J7 pad 3: /POWER_MEASUREMENTS/D2+ -> unconnected-(J7-Pad3)
- J8 pad 1: /POWER_MEASUREMENTS/source_vcc -> /POWER_MEASUREMENTS/ext_5v
- J8 pad 2: GND -> /POWER_MEASUREMENTS/D2+
- J8 pad 3: unconnected-(J8-Pad3) -> /POWER_MEASUREMENTS/D2-
- R10 pad 2: +3V3 -> +3.3V
- R13 pad 1: unconnected-(R13-Pad1) -> Net-(IC1-Pad3)
- R13 pad 2: GND -> +3.3V
- R14 pad 1: Net-(IC1-Pad3) -> /IRQ
- R14 pad 2: +3V3 -> +3.3V
- R15 pad 1: /IRQ -> 3v3_enable
- R15 pad 2: +3V3 -> Net-(R15-Pad2)
- R16 pad 1: /BASE1 -> /gain
- R16 pad 2: /~{DTR} -> Net-(R16-Pad2)
- R17 pad 1: /BOOT -> Net-(R17-Pad1)
- R17 pad 2: +3V3 -> /gain
- R18 pad 1: +3V3 -> /BASE1
- R18 pad 2: /EN -> /~{DTR}
- R19 pad 1: /~{RTS} -> /BOOT
- R19 pad 2: /BASE2 -> +3V3
- R2 pad 1: +3V3 -> +3.3V
- R20 pad 1: GND -> +3V3
- R20 pad 2: Net-(R20-Pad2) -> /EN
- R21 pad 1: Net-(R20-Pad2) -> /~{RTS}
- R21 pad 2: /POWER_MEASUREMENTS/mini_power_source -> /BASE2
- R23 pad 2: /POWER_MEASUREMENTS/source_vcc -> /POWER_MEASUREMENTS/mini_power_source
- R24 pad 1: /POWER_MEASUREMENTS/source_vcc -> Net-(R24-Pad1)
- R24 pad 2: /POWER_MEASUREMENTS/load_vcc -> /POWER_MEASUREMENTS/ADC_CH0
- R25 pad 1: /POWER_MEASUREMENTS/mini_power_load -> GND
- R25 pad 2: /POWER_MEASUREMENTS/mini_power_source -> Net-(R25-Pad2)
- R26 pad 1: GND -> Net-(R25-Pad2)
- R26 pad 2: Net-(C13-Pad1) -> /POWER_MEASUREMENTS/source_vcc
- R27 pad 1: Power_in- -> Net-(R27-Pad1)
- R27 pad 2: Net-(R27-Pad2) -> /POWER_MEASUREMENTS/ADC_CH2
- R28 pad 1: Net-(R27-Pad2) -> /POWER_MEASUREMENTS/source_vcc
- R28 pad 2: /POWER_MEASUREMENTS/ADC_CH5 -> /POWER_MEASUREMENTS/load_vcc
- R29 pad 1: Power_in+ -> /POWER_MEASUREMENTS/mini_power_load
- R29 pad 2: Net-(R29-Pad2) -> /POWER_MEASUREMENTS/mini_power_source
- R3 pad 1: +3V3 -> +3.3V
- R30 pad 1: /POWER_MEASUREMENTS/ADC_CH6 -> GND
- R30 pad 2: Power_in+ -> Net-(C15-Pad1)
- R31 pad 1: GND -> Power_in-
- R31 pad 2: Net-(R29-Pad2) -> Net-(R31-Pad2)
- R32 pad 1: GND -> Net-(R31-Pad2)
- R32 pad 2: /POWER_MEASUREMENTS/ADC_CH6 -> Net-(R32-Pad2)
- R33 pad 1: Net-(D5-Pad1) -> Net-(R32-Pad2)
- R33 pad 2: Net-(IC4-Pad3) -> /POWER_MEASUREMENTS/ADC_CH5
- R34 pad 1: GND -> Power_in+
- R34 pad 2: Net-(IC4-Pad8) -> Net-(R34-Pad2)
- R35 pad 1: Power_in+ -> Net-(R35-Pad1)
- R35 pad 2: Power_in- -> Power_in+
- R36 pad 1: Net-(D6-Pad1) -> GND
- R36 pad 2: Net-(IC4-Pad4) -> Net-(R34-Pad2)
- R37 pad 1: Net-(R37-Pad1) -> Net-(R35-Pad1)
- R37 pad 2: +VDC -> /POWER_MEASUREMENTS/ADC_CH6
- R38 pad 2: /Power-IN-OUT-BMS/low_batt_shutoff -> Net-(R35-Pad1)
- R39 pad 1: GND -> Net-(D5-Pad1)
- R39 pad 2: +5V -> Net-(IC4-Pad3)
- R4 pad 1: +3V3 -> +3.3V
- R40 pad 2: Net-(R37-Pad1) -> Net-(IC4-Pad8)
- R5 pad 1: +3V3 -> +3.3V
- R6 pad 1: +3V3 -> +3.3V
- R7 pad 1: +3V3 -> +3.3V
- R8 pad 1: +3V3 -> +3.3V
- RR1 pad 2: Net-(C23-Pad2) -> Net-(C27-Pad2)
- RR2 pad 1: Net-(C23-Pad2) -> Net-(C27-Pad2)
- RV1 pad 1: Net-(J13-Pad1) -> Net-(J13-Pad2)
- S1 pad 1: unconnected-(S1-Pad1) -> Net-(R15-Pad2)
- S1 pad 2: unconnected-(S1-Pad2) -> +VDC
- S1 pad 3: unconnected-(S1-Pad3) -> Net-(R16-Pad2)
- S1 pad 4: unconnected-(S1-Pad4) -> +VDC
- S1 pad 5: unconnected-(S1-Pad5) -> /gain
- S1 pad 6: unconnected-(S1-Pad6) -> +VDC
- S1 pad 7: unconnected-(S1-Pad7) -> Net-(R17-Pad1)
- S1 pad 8: unconnected-(S1-Pad8) -> GND
- S2 pad 2: +3V3 -> +3.3V
- U2 pad 3: ADC_CH2 -> /POWER_MEASUREMENTS/ADC_CH2
- U5 pad 3: D- -> D+
- U5 pad 4: D+ -> D-
- U6 pad 1: /POWER_MEASUREMENTS/ADC_CH0 -> Net-(R24-Pad1)
- U6 pad 10: Net-(R27-Pad2) -> Net-(R31-Pad2)
- U6 pad 12: Net-(R37-Pad1) -> unconnected-(U6-Pad12)
- U6 pad 13: ADC_CH4 -> unconnected-(U6-Pad13)
- U6 pad 14: ADC_CH4 -> unconnected-(U6-Pad14)
- U6 pad 2: /POWER_MEASUREMENTS/ADC_CH0 -> Net-(R24-Pad1)
- U6 pad 3: Net-(R20-Pad2) -> Net-(R22-Pad2)
- U6 pad 5: Net-(R22-Pad2) -> Net-(R25-Pad2)
- U6 pad 6: ADC_CH2 -> Net-(R27-Pad1)
- U6 pad 7: ADC_CH2 -> Net-(R27-Pad1)
- U6 pad 8: /POWER_MEASUREMENTS/ADC_CH5 -> Net-(R32-Pad2)
- U6 pad 9: Net-(R29-Pad2) -> Net-(R34-Pad2)
- U9 pad 6: Net-(C23-Pad2) -> Net-(C27-Pad2)

Commit message: f
Parts:
- removed Q1: BC847BS, Package_TO_SOT_SMD:SOT-363_SC-70-6_Handsoldering
- removed R18, R21: 10k, Resistor_SMD:R_0603_1608Metric_Pad0.98x0.95mm_HandSolder
- R2, R3, R4, R5, R6, R7, R8: moved to B.Cu
- R9: value 4.7k -> 4k7; footprint Resistor_SMD:R_0805_2012Metric -> Resistor_SMD:R_0603_1608Metric_Pad0.98x0.95mm_HandSolder
- moved U1 173.1 mm to (109.8, 89.6), turned to 180 degrees
- moved C3 171.6 mm to (110.0, 92.2), turned to 0 degrees
- moved R1 167.8 mm to (111.6, 93.8), turned to 180 degrees
- moved U2 163.4 mm to (115.6, 86.8), turned to 180 degrees
- moved C2 161.5 mm to (115.0, 92.8), turned to 180 degrees
- moved C1 160.8 mm to (115.0, 94.6), turned to 0 degrees
- moved IC1 146.7 mm to (71.2, 120.0), turned to 90 degrees
- moved C6 133.7 mm to (89.2, 52.4), turned to 90 degrees
- moved R16 125.9 mm to (96.8, 96.7), turned to -90 degrees
- moved R7 109.9 mm to (119.8, 60.0), turned to 180 degrees
- moved R17 107.7 mm to (96.8, 93.3), turned to -90 degrees
- moved R15 107.5 mm to (97.6, 100.0), turned to 180 degrees
- moved R5 105.3 mm to (119.8, 63.2), turned to 180 degrees
- moved C5 104.3 mm to (87.4, 52.4), turned to 90 degrees
- moved R6 97.7 mm to (119.8, 61.6), turned to 180 degrees
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Connections:
- U4 pad 13: /USB_OTG_D- -> D-
- U4 pad 14: /USB_OTG_D+ -> D+
- U4 pad 36: UART0_RX -> unconnected-(U4-Pad36)
- U4 pad 37: UART0_TX -> unconnected-(U4-Pad37)
Routing:
- added copper zone on F.Cu, net GND
