File: ESP32_power_meter_MP3_player_WIFI_radio_V2/ESP32_power_meter_MP3_player_WIFI_radio_V2.kicad_sch (KiCad schematic)
At the start: 76 parts, among them IC1 XRA1203IG24TR-F, J1 STX-3120-5B, J2 SS-52100-001, J3 MEM2051-00-195-00-A, J8 Conn_01x06, U2 LM4040DBZ-3, U3 MCP3208, U4 Adafruit_MAX98357, U5 D1213A-02SM

Commit message: e
Parts:
- added R49: 10k, Resistor_SMD:R_0603_1608Metric_Pad0.98x0.95mm_HandSolder, symbol Device:R_Small
- gave numbers to parts that had none: 11
Connections:
- net +3V3: now also R49.1
- net GND: no longer U4.2 (speaker-), U5.2 (VSS)
- net POWER_MEASUREMENTS/ADC_CH0: no longer U3.1 (CH0)
- net POWER_MEASUREMENTS/ADC_CH1: no longer U3.2 (CH1)
- net POWER_MEASUREMENTS/ADC_CH2: no longer U3.3 (CH2)
- net POWER_MEASUREMENTS/ADC_CH3: no longer U3.4 (CH3)
- net POWER_MEASUREMENTS/ADC_CH5: no longer U3.6 (CH5)
- net POWER_MEASUREMENTS/ADC_CH6: no longer U3.7 (CH6)
- net VBUS: no longer U5.5 (VCC)
- net at J1.2, J1.5: no longer U4.1 (speaker+)
- net PG_3V3 renamed EN
- net EN: now also R49.2
Other:
- moved on the sheet: C1, C2, C23, C26, C27, C3, C4, C5, C6, C7, C8, C9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

Commit message: m
Parts:
- removed D5, D6, D7, D8, D9: LED_Small Green, LED_SMD:LED_0603_1608Metric_Pad1.05x0.95mm_HandSolder, symbol Device:LED_Small
- removed JP1: Jumper_2_Bridged, Jumper:SolderJumper-2_P1.3mm_Bridged_RoundedPad1.0x1.5mm, symbol Jumper:Jumper_2_Bridged
- removed R10, R11, R12, R13, R14, R15, R18, R19, R21, R9: 10k, Resistor_SMD:R_0603_1608Metric_Pad0.98x0.95mm_HandSolder, symbol Device:R_Small
- removed R30, R46, R47: 330, Resistor_SMD:R_0603_1608Metric_Pad0.98x0.95mm_HandSolder, symbol Device:R
- removed S2: DS01C-254-S-08BE, SamacSys_Parts:DS01C254S08BE, symbol SamacSys_Parts:DS01C-254-S-08BE
- removed TP1, TP2, TP3: TestPoint, TestPoint:TestPoint_Pad_1.0x1.0mm, symbol Connector:TestPoint
- added D2, D3, D4: Green, LED_SMD:LED_0603_1608Metric_Pad1.05x0.95mm_HandSolder, symbol Device:LED_Small
- added R12: 330, Resistor_SMD:R_0603_1608Metric_Pad0.98x0.95mm_HandSolder, symbol Device:R
- added R2, R3: 10k, Resistor_SMD:R_0603_1608Metric_Pad0.98x0.95mm_HandSolder, symbol Device:R_Small
- added SW1: GPIO_RESET, SamacSys_Parts:PTS526SK15SMTR2LFS, symbol Switch:SW_SPST
- C7: renamed from C26; footprint Capacitor_SMD:C_0603_1608Metric_Pad1.08x0.95mm_HandSolder -> Capacitor_SMD:C_0805_2012Metric
- D1: value LED_Small Green -> Green
- renumbered C6 to C1, C3 to C10, C5 to C11, C27 to C12, C7 to C2, C4 to C3, C8 to C4, C1 to C5, C2 to C6, C23 to C8, FID4 to FID2, FID2 to FID3, FID5 to FID4, FID3 to FID5, J3 to J2, J2 to J3, J8 to J4, Q2 to Q1, R44 to R10, R45 to R11, R3 to R13, R16 to R14, R17 to R15, R2 to R16, R48 to R17, R49 to R18, R50 to R19, R20 to R9, SW1 to SW2, U2 to U1, U3 to U2, U4 to U3, U1 to U4
Connections:
- net DATA1 is gone; now on net GPIO_37: J2.P8 (DAT1)
- net DATA2 is gone; now on net GPIO_38: J2.P1 (DAT2)
- net GPIO1 is gone; now on net GPIO_42: J2.P5 (CLK)
- net GPIO_04 is gone; now on net SDA: U4.4 (GPIO4/TOUCH4/ADC1_CH3)
- net GPIO_05 is gone; now on net SCL: U4.5 (GPIO5/TOUCH5/ADC1_CH4)
- net GPIO_07 is gone; now on net DATA_IN: U4.7 (GPIO7/TOUCH7/ADC1_CH6)
- net GPIO_08 is gone; now on net BCLK: U4.12 (GPIO8/TOUCH8/ADC1_CH7/SUBSPICS1)
- net SPI1_SS1 is gone; now on net GPIO_13: U2.10 (~{CS}/SHDN)
- net +3V3: now also R4.1, R5.1, R6.1, R7.1, R8.1, R2.1, R3.1; no longer R4.2, R5.2, R6.2, R7.2
- net 3v3_enable: no longer R13.1
- net A0: no longer R4.1
- net A1: no longer R6.1
- net BCLK: no longer S1.12 (NO_6)
- net DATA_IN: no longer S1.8 (NO_4)
- net GND: now also U3.2 (speaker-), U5.2 (VSS), D2.1 (K), D3.1 (K), D4.1 (K), SW1.2 (B)
- net GPIO_06: now also U3.9 (SD_/_MODE)
- net GPIO_09: now also U3.5 (LRC_(Left/Right_Clock)
- net GPIO_10: now also U2.13 (CLK)
- net GPIO_11: now also U2.12 (Dout)
- net GPIO_12: now also U2.11 (Din)
- net GPIO_14: now also R12.2
- net GPIO_36: now also J2.P7 (DAT0), R3.2
- net GPIO_37: now also R4.2
- net GPIO_38: now also R5.2
- net GPIO_39: now also J2.P2 (CD/DAT3), R6.2
- net GPIO_40: now also J2.P3 (CMD), R7.2
- net GPIO_41: now also J2.MP2, R2.2
- net GPIO_42: now also R8.2
- net P3: no longer IC1.7 (P3)
- net POWER_MEASUREMENTS/ADC_CH0: now also U2.1 (CH0)
- net POWER_MEASUREMENTS/ADC_CH1: now also U2.2 (CH1)
- net POWER_MEASUREMENTS/ADC_CH2: now also U2.3 (CH2)
- net POWER_MEASUREMENTS/ADC_CH3: now also U2.4 (CH3)
- net POWER_MEASUREMENTS/ADC_CH5: now also U2.6 (CH5)
- net POWER_MEASUREMENTS/ADC_CH6: now also U2.7 (CH6)
- net VBUS: now also U5.5 (VCC)
- net at IC1.3 (RESET#), R14.1: now also SW1.1 (A)
- net at U3.1 (speaker+): now also J1.2, J1.5
- net at R11.1: now also D3.2 (A)
- net at R10.1: now also D2.2 (A)
- net DATA0 renamed GPIO0
- net GPIO0: no longer J2.P7 (DAT0)
- removed net DATA3: IC1.5 (P1), J2.P2 (CD/DAT3), R5.1
- net GPIO10: no longer names the net of S1.14 (NO_7)
- net GPIO10: no longer S1.15 (COM_8)
- removed net GPIO2: J2.P3 (CMD), R7.1
- net GPIO5 renamed IRQ
- net GPIO8: no longer names the net of S1.6 (NO_3)
- net GPIO8: no longer S1.7 (COM_4)
- net GPIO9: no longer names the net of S1.10 (NO_5)
- net GPIO9: no longer S1.11 (COM_6)
- net LRC: no longer names the net of S1.16 (NO_8)
- net LRC: no longer U3.5 (LRC_(Left/Right_Clock)
- net SD_sense: no longer names the net of IC1.6 (P2)
- net SD_sense: no longer J2.MP2
- net SPI1_CLK: no longer names the net of S1.9 (COM_5)
- net SPI1_CLK: no longer U2.13 (CLK)
- net SPI1_MISO: no longer names the net of S1.5 (COM_3)
- net SPI1_MISO: no longer U2.12 (Dout)
- net SPI1_MOSI: no longer names the net of S1.13 (COM_7)
- net SPI1_MOSI: no longer U2.11 (Din)
- net SPI2_SS1: no longer names the net of IC1.4 (P0)
- removed net on/off+mode: R8.1, U3.9 (SD_/_MODE)
- new net: D4.2 (A), R12.1
- no-connect marks 24 -> 12
Other:
- note added: "ESP32-S3 has four strapping pins: • GPIO0 / BOOT • GPIO45 • GPIO46 • GPIO3 GPIO0, GPIO45 and GPIO46 are connected to the chip's internal weak pull-up/pull-down during the chip reset. GPIO3 is floating by default"
- note removed: "ADC ON SIDE"
- note removed: "AUDIO ON SIDE"
- note removed: "DIP SWITCHES"
- note removed: "ESP32-S3 has four strapping pins: • GPIO0 • GPIO45 • GPIO46 • GPIO3 GPIO0, GPIO45 and GPIO46 are connected to the chip's internal weak pull-up/pull-down during the chip reset. GPIO3 is floating by default"
- note removed: "I2C bus"
- note removed: "I2S pins/ SPI1 for ADC"
- note removed: "Pull ups"
- note removed: "SD +SPI2"
- note removed: "pull down since this way it is by default off and it doent draw power as oposed to a pull up that is turned off when tied to GND"
- note removed: "test points for bodges later one"
- moved on the sheet: C1, C5, C6, C7, C8, D1, IC1, J2, R1, R10, R11, R13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

Commit message: f
Parts:
- removed J3: SS-52100-001, SamacSys_Parts:SS52100001, symbol SamacSys_Parts:SS-52100-001
- removed R13: 20k, Resistor_SMD:R_0603_1608Metric_Pad0.98x0.95mm_HandSolder, symbol Device:R
- added J3: USB_A, Connector_USB:USB_A_Molex_67643_Horizontal, symbol Connector:USB_A
- added R15: 10k, Resistor_SMD:R_0603_1608Metric_Pad0.98x0.95mm_HandSolder, symbol Device:R_Small
- added R16, R17: 100k, Resistor_SMD:R_0603_1608Metric_Pad0.98x0.95mm_HandSolder, symbol Device:R_Small
- C1: value 100n -> 10u; footprint Capacitor_SMD:C_0603_1608Metric_Pad1.08x0.95mm_HandSolder -> Capacitor_SMD:C_0805_2012Metric
- C12: value 15n -> 100n
- C4: footprint Capacitor_SMD:C_0603_1608Metric_Pad1.08x0.95mm_HandSolder -> Capacitor_SMD:C_0805_2012Metric
- F1: footprint Fuse:Fuse_0603_1608Metric_Pad1.05x0.95mm_HandSolder -> Fuse:Fuse_1812_4532Metric
- FB1: footprint SamacSys_Parts:BEADC4516X185N -> BEADC4516X185N
- IC1: footprint SamacSys_Parts:SOP65P640X120-24N -> SOP65P640X120-24N
- J1: footprint SamacSys_Parts:STX31205B -> STX31205B
- J2: footprint SamacSys_Parts:MEM20510019500A -> MEM20510019500A
- R20: renamed from R18; value 10k -> 100k
- S1: footprint SamacSys_Parts:DS01C254S08BE -> DS01C254S08BE
- U5: footprint Package_TO_SOT_SMD:SOT-23-5 -> Package_TO_SOT_SMD:SOT-23-5_HandSoldering
- renumbered R14 to R13, R15 to R14, R16 to R18, R17 to R19, R19 to R21
Connections:
- net GPIO0 is gone; now on net EN: J4.5 (Pin_5)
- net RX is gone; now on net UART0_RX: J4.3 (Pin_3)
- net TX is gone; now on net UART0_TX: J4.2 (Pin_2)
- net reset is gone; now on net BOOT: J4.4 (Pin_4)
- net +3V3: no longer C7.1, C8.2, IC1.24 (VCC), J2.P4 (VDD), J4.6 (Pin_6), R10.2, R13.2, R14.2, R2.1, R3.1, R4.1, R5.1, R6.1, R7.1, R8.1
- net +VDC: now also C4.2, S1.2 (NO_1), S1.4 (NO_2), S1.6 (NO_3); no longer C4.1
- net 3v3_enable: now also R15.1
- net D+: now also U5.3 (CH1), J3.2 (D-); no longer U5.4 (CH2)
- net D-: now also U5.4 (CH2), J3.3 (D+); no longer U5.3 (CH1)
- net GND: now also C4.1, H1.1, H2.1, H3.1, H4.1, S1.8 (NO_4), J3.4 (GND); no longer C4.2
- net VBUS: now also J3.1 (VBUS)
- net gain: now also S1.5 (COM_3), R16.1, R17.2
- net at S1.1 (COM_1): now also R15.2
- net at S1.3 (COM_2): now also R16.2
- net at S1.7 (COM_4): now also R17.1
- new net +3.3V: C7.1, C8.2, IC1.24 (VCC), J2.P4 (VDD), J4.6 (Pin_6), R10.2, R13.2, R14.2, R2.1, R3.1, R4.1, R5.1, R6.1, R7.1, R8.1
- no-connect marks 12 -> 9
Other:
- moved on the sheet: C12, C4, F1, J1, J4, S1

Commit message: f
Parts:
- removed Q1: BC847BS, Package_TO_SOT_SMD:SOT-363_SC-70-6_Handsoldering, symbol Device:Q_Dual_NPN_NPN_E1B1C2E2B2C1
- removed R18, R21: 10k, Resistor_SMD:R_0603_1608Metric_Pad0.98x0.95mm_HandSolder, symbol Device:R_Small
- R9: value 4.7k -> 4k7; footprint Resistor_SMD:R_0805_2012Metric -> Resistor_SMD:R_0603_1608Metric_Pad0.98x0.95mm_HandSolder
Connections:
- net USB_OTG_D+ is gone; now on net D+: U4.14 (GPIO20/U1CTS/ADC2_CH9/CLK_OUT1/USB_D+)
- net USB_OTG_D- is gone; now on net D-: U4.13 (GPIO19/U1RTS/ADC2_CH8/CLK_OUT2/USB_D-)
- net UART0_RX: no longer U4.36 (U0RXD/GPIO44/CLK_OUT2)
- net UART0_TX: no longer U4.37 (U0TXD/GPIO43/CLK_OUT1)
