File: ESP32_power_meter_MP3_player_WIFI_radio_V2/ESP32_power_meter_MP3_player_WIFI_radio_V2.kicad_sch (KiCad schematic)
At the start: 64 parts, among them IC1 XRA1203IG24TR-F, J1 STX-3120-5B, J14 Conn_02x10_Odd_Even, J15 I2C, J16 I2C, J2 MEM2051-00-195-00-A, J3 USB_A, J4 Conn_01x06, SW1 GPIO_RESET, SW2 MCU_RESET, U1 LM4040DBZ-3, U2 MCP3208, U3 Adafruit_MAX98357, U4 ESP32-S3-WROOM-1, U5 D1213A-02SM

Commit message: y
Parts:
- added R45, R46, R47, R48: 10k, Resistor_SMD:R_0603_1608Metric_Pad0.98x0.95mm_HandSolder, symbol Device:R_Small
- added TP10, TP4, TP5, TP6, TP7, TP8, TP9: TestPoint, TestPoint:TestPoint_Pad_1.5x1.5mm, symbol Connector:TestPoint
- added TP11, TP12, TP13: TestPoint, TestPoint:TestPoint_THTPad_D2.0mm_Drill1.0mm, symbol Connector:TestPoint
Connections:
- net A0 is gone; now on net GND: IC1.21 (A0)
- net A1 is gone; now on net +3V3: IC1.2 (A1)
- net 3v3_enable: now also R15.2, S1.1 (COM_1); no longer R15.1
- net GND: now also R15.1, R45.1, R46.1, R47.1, R48.1
- net GPIO_01: now also TP12.1
- net GPIO_02: now also TP13.1
- net GPIO_04: now also TP9.1
- net GPIO_05: now also TP10.1
- net GPIO_06: now also S1.10 (NO_5), TP5.1
- net GPIO_07: now also S1.12 (NO_6), TP6.1
- net GPIO_13: now also TP4.1
- net GPIO_15: now also S1.14 (NO_7), TP7.1
- net GPIO_16: now also S1.16 (NO_8), TP8.1
- net GPIO_35: now also TP11.1
- net at S1.11 (COM_6): now also R46.2
- net at S1.13 (COM_7): now also R47.2
- net at S1.15 (COM_8): now also R48.2
- net at S1.9 (COM_5): now also R45.2
Other:
- note added: "I2C"
- note added: "IO"
- moved on the sheet: J14, J15, J16, R15, R16, R17, R18, R21, S1

Commit message: f
Parts:
- removed R45, R46, R47, R48: 10k, Resistor_SMD:R_0603_1608Metric_Pad0.98x0.95mm_HandSolder, symbol Device:R_Small
- added C31: 100n, Capacitor_SMD:C_0603_1608Metric_Pad1.08x0.95mm_HandSolder, symbol Device:C_Small
- added L2: L_Small, Inductor_SMD:L_1206_3216Metric, symbol Device:L_Small
- added R22, R23, R24, R25: 10k, Resistor_SMD:R_0603_1608Metric, symbol Device:R_Small
- added R49, R50: 0, Resistor_SMD:R_0603_1608Metric_Pad0.98x0.95mm_HandSolder, symbol Device:R_Small
- R13, R14, R15, R18, R19, R2, R21, R3, R4, R5, R6, R7, R8: footprint Resistor_SMD:R_0603_1608Metric_Pad0.98x0.95mm_HandSolder -> Resistor_SMD:R_0603_1608Metric; LCSC (none) -> C25804
Connections:
- net +3V3: now also R13.1, R14.1, C31.1, R23.2, R24.2, R25.2; no longer R13.2, R14.2, R18.1, R19.2, R21.1
- net +VDC: now also L2.1; no longer C1.1, C2.2, U2.16 (Vdd)
- net 3v3_enable: now also R15.1; no longer R15.2
- net BOOT: now also R25.1; no longer R19.1
- net D+: now also J3.3 (D+), U5.4 (CH2), R49.2; no longer J3.2 (D-), U4.14 (GPIO20/U1CTS/ADC2_CH9/CLK_OUT1/USB_D+), U5.3 (CH1)
- net D-: now also J3.2 (D-), U5.3 (CH1), R50.1; no longer J3.3 (D+), U4.13 (GPIO19/U1RTS/ADC2_CH8/CLK_OUT2/USB_D-), U5.4 (CH2)
- net GND: now also R15.2, R18.1, R19.1, R21.1, C31.2, R22.1; no longer R15.1
- net IRQ: now also R14.2; no longer R14.1
- net SCL: now also R23.1; no longer R18.2
- net SDA: now also R24.1; no longer R21.2
- net at IC1.3 (RESET#), SW1.1 (A): now also R13.2; no longer R13.1
- net at S1.13 (COM_7): now also R21.2
- net at S1.11 (COM_6): now also R19.2
- net at S1.9 (COM_5): now also R18.2
- net at S1.15 (COM_8): now also R22.2
- new net: C1.1, C2.2, L2.2, U2.16 (Vdd)
- new net: R49.1, U4.14 (GPIO20/U1CTS/ADC2_CH9/CLK_OUT1/USB_D+)
- new net: R50.2, U4.13 (GPIO19/U1RTS/ADC2_CH8/CLK_OUT2/USB_D-)

Commit message: n
Parts:
- removed U5: D1213A-02SM, Package_TO_SOT_SMD:SOT-23-5_HandSoldering, symbol My_custom_lib:D1213A-02SM
- added SW3: MCU_RESET, SamacSys_Parts:PTS526SK15SMTR2LFS, symbol Switch:SW_SPST
- added U5: SRV05-4, Package_TO_SOT_SMD:SOT-23-6, symbol Power_Protection:SRV05-4
- C1, C4, C5, C7, C9: LCSC (none) -> C45783
- C10, C12, C2, C3, C31, C6, C8: LCSC (none) -> C1623
- D1, D2, D3, D4: LCSC (none) -> C72043
- R1: LCSC (none) -> C21190
- R10, R11, R12: LCSC (none) -> C23025
- R16, R17, R20: LCSC (none) -> C25803
- R49, R50: LCSC (none) -> C22936
- R9: LCLS (none) -> C23162
- SW1, SW2: LCSC (none) -> C318884
Connections:
- net BOOT: now also SW3.1 (A)
- net D+: now also U5.1 (IO1)
- net D-: now also U5.6 (IO4)
- net GND: now also SW3.2 (B), U5.2 (VN)
- net VBUS: now also U5.5 (VP)
- no-connect marks 9 -> 10
Other:
- note removed: "ESD protection IC"
