File: ESP32_power_meter_MP3_player_WIFI_radio_V2/_autosave-ESP32_power_meter_MP3_player_WIFI_radio_V2.kicad_sch (KiCad schematic)
At the start: 64 parts, among them IC1 XRA1203IG24TR-F, J1 STX-3120-5B, J14 Conn_02x10_Odd_Even, J15 I2C, J16 I2C, J2 MEM2051-00-195-00-A, J3 USB_A, J4 Conn_01x06, SW1 GPIO_RESET, SW2 MCU_RESET, U1 LM4040DBZ-3, U2 MCP3208, U3 Adafruit_MAX98357, U4 ESP32-S3-WROOM-1, U5 D1213A-02SM

Commit message: t
Parts:
- added R?: 10k, Resistor_SMD:R_0603_1608Metric_Pad0.98x0.95mm_HandSolder, symbol Device:R_Small
- added TP10, TP4, TP5, TP6, TP7, TP8, TP9: TestPoint, TestPoint:TestPoint_Pad_1.5x1.5mm, symbol Connector:TestPoint
- added TP11, TP12, TP13: TestPoint, TestPoint:TestPoint_THTPad_D2.0mm_Drill1.0mm, symbol Connector:TestPoint
Connections:
- net 3v3_enable: now also R15.2, S1.1 (COM_1); no longer R15.1
- net GND: now also R15.1
- net GPIO_01: now also TP12.1
- net GPIO_02: now also TP13.1
- net GPIO_04: now also TP9.1
- net GPIO_05: now also TP10.1
- net GPIO_06: now also TP5.1
- net GPIO_07: now also TP6.1
- net GPIO_13: now also TP4.1
- net GPIO_15: now also TP7.1
- net GPIO_16: now also TP8.1
- net GPIO_35: now also TP11.1
Other:
- note added: "I2C"
- note added: "IO"
- moved on the sheet: J14, J15, J16, R15, R16, R17, R18, R21, S1
