File: ESP32_power_meter_MP3_player_WIFI_radio_V2/_autosave-ESP32_power_meter_MP3_player_WIFI_radio_V2.kicad_pcb (KiCad board)
At the start: 2 copper layers, 99.9 x 100 mm, 136 parts, among them IC1 XRA1203IG24TR-F, IC2 INA2181A4QDGSRQ1, IC3 AP2112M-3.3TRG1, IC4 MCP73834T-FCI_UN, J1 STX-3120-5B, J10 Conn_01x02, J11 USB_A, J12 Conn_01x03, J13 Conn_01x02, J14 Conn_02x10_Odd_Even, J15 I2C, J16 I2C, J2 MEM2051-00-195-00-A, J3 USB_A, J4 Conn_01x06, J5 Barrel_Jack_Switch, J6 Conn_01x02, J7 Barrel_Jack_Switch, J8 USB_A, J9 Conn_01x03, Q2 DMG9933USD-13, SW1 GPIO_RESET, SW2 MCU_RESET, U1 LM4040DBZ-3, U2 MCP3208, U3 Adafruit_MAX98357, U4 ESP32-S3-WROOM-1, U5 D1213A-02SM, U6 LM324, U7 1043, U8 APX810S05, U9 DIO6012BCST6

Commit message: t
Parts:
- added TP10: TestPoint, TestPoint:TestPoint_Pad_1.5x1.5mm, F.Cu at (83.2, 51.8)
- added TP11: TestPoint, TestPoint:TestPoint_THTPad_D2.0mm_Drill1.0mm, F.Cu at (113.8, 69.8)
- added TP12: TestPoint, TestPoint:TestPoint_THTPad_D2.0mm_Drill1.0mm, B.Cu at (112.4, 51.8)
- added TP13: TestPoint, TestPoint:TestPoint_THTPad_D2.0mm_Drill1.0mm, B.Cu at (114.4, 55.0)
- added TP4: TestPoint, TestPoint:TestPoint_Pad_1.5x1.5mm, F.Cu at (100.6, 72.8)
- added TP5: TestPoint, TestPoint:TestPoint_Pad_1.5x1.5mm, F.Cu at (79.8, 51.8)
- added TP6: TestPoint, TestPoint:TestPoint_Pad_1.5x1.5mm, B.Cu at (190.6, 96.6)
- added TP7: TestPoint, TestPoint:TestPoint_Pad_1.5x1.5mm, F.Cu at (81.6, 57.9)
- added TP8: TestPoint, TestPoint:TestPoint_Pad_1.5x1.5mm, B.Cu at (190.6, 93.2)
- added TP9: TestPoint, TestPoint:TestPoint_Pad_1.5x1.5mm, F.Cu at (78.5, 55.0)
- moved R15 0.86 mm to (99.8, 99.2)
Connections:
- R15 pad 1: 3v3_enable -> GND
- R15 pad 2: Net-(R15-Pad2) -> 3v3_enable
- S1 pad 1: Net-(R15-Pad2) -> 3v3_enable
Routing:
- net /GPIO_35: track 0.00 -> 6.17 mm
- net /GPIO_02: track 0.00 -> 5.90 mm
- net 3v3_enable: track 63.8 -> 68.7 mm
- net /GPIO_01: track 0.00 -> 4.20 mm
- net Net-(R15-Pad2): track 3.27 -> 0.00 mm
- net /GPIO_13: track 0.00 -> 3.19 mm
- net GND: track 154.8 -> 156.2 mm, vias 101 -> 102

Commit message: Update _autosave-ESP32_power_meter_MP3_player_WIFI_radio_V2.kicad_pcb
Parts:
- moved TP6 109.9 mm to (87.7, 58.1), turned to 0 degrees
- moved TP8 107.7 mm to (87.7, 61.5), turned to 0 degrees
- moved TP9 5.94 mm to (83.5, 51.8), turned to 180 degrees
- moved TP5 3.32 mm to (77.4, 54.1)
- moved TP10 3.26 mm to (80.0, 51.5)
Routing:
- net /GPIO_06: track 0.00 -> 15.6 mm
- net /GPIO_05: track 0.00 -> 13.5 mm
- net /GPIO_15: track 0.00 -> 10.8 mm
- net /GPIO_04: track 0.00 -> 10.2 mm
- net /GPIO_07: track 0.00 -> 4.12 mm, vias 0 -> 1
- net /GPIO_16: track 0.00 -> 3.90 mm, vias 0 -> 1
Changed lines of the file:
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@@
   )
   (footprint "TestPoint:TestPoint_Pad_1.5x1.5mm" (layer "F.Cu")
-    (at 78.5 55 90)
+    (at 83.5 51.8 180)
     (descr "SMD rectangular pad as test Point, square 1.5mm side length")
     (tags "test point SMD pad rectangle square")
@@
     (property "exclude_from_bom" "")
     (attr exclude_from_pos_files exclude_from_bom)
-    (fp_text reference "TP9" (at 0 -1.648 90) (layer "F.SilkS")
+    (fp_text reference "TP9" (at 0.3 -1.9) (layer "F.SilkS")
       (effects (font (size 1 1) (thickness 0.15)))
     )
-    (fp_text value "TestPoint" (at 0 1.75 90) (layer "F.Fab")
+    (fp_text value "TestPoint" (at 0 1.75) (layer "F.Fab")
       (effects (font (size 1 1) (thickness 0.15)))
     )
-    (fp_text user "${REFERENCE}" (at 0 -1.65 90) (layer "F.Fab")
+    (fp_text user "${REFERENCE}" (at 0 -1.65) (layer "F.Fab")
       (effects (font (size 1 1) (thickness 0.15)))
     )
@@
     (fp_line (start 1.25 1.25) (end 1.25 -1.25) (layer "F.CrtYd") (width 0.05))
     (fp_line (start 1.25 1.25) (end -1.25 1.25) (layer "F.CrtYd") (width 0.05))
-    (pad "1" smd rect (at 0 0 90) (size 1.5 1.5) (layers "F.Cu" "F.Mask")
+    (pad "1" smd rect (at 0 0 180) (size 1.5 1.5) (layers "F.Cu" "F.Mask")
       (net 136 "/GPIO_04") (pinfunction "1") (pintype "passive"))
   )
@@
   )
   (footprint "TestPoint:TestPoint_Pad_1.5x1.5mm" (layer "F.Cu")
-    (at 83.25 51.8 180)
+    (at 80 51.5 180)
     (descr "SMD rectangular pad as test Point, square 1.5mm side length")
     (tags "test point SMD pad rectangle square")
@@
     (property "exclude_from_bom" "")
     (attr exclude_from_pos_files exclude_from_bom)
-    (fp_text reference "TP10" (at 0 -1.648) (layer "F.SilkS")
+    (fp_text reference "TP10" (at 2.9 -0.1) (layer "F.SilkS")
       (effects (font (size 1 1) (thickness 0.15)))
     )
@@
   )
   (footprint "TestPoint:TestPoint_Pad_1.5x1.5mm" (layer "F.Cu")
-    (at 79.8 51.8 90)
+    (at 77.4 54.1 90)
     (descr "SMD rectangular pad as test Point, square 1.5mm side length")
     (tags "test point SMD pad rectangle square")
@@
     (property "exclude_from_bom" "")
     (attr exclude_from_pos_files exclude_from_bom)
-    (fp_text reference "TP5" (at 0 -1.648 90) (layer "F.SilkS")
+    (fp_text reference "TP5" (at -2.2 0.8 180) (layer "F.SilkS")
       (effects (font (size 1 1) (thickness 0.15)))
     )
@@
   )
   (footprint "TestPoint:TestPoint_Pad_1.5x1.5mm" (layer "B.Cu")
-    (at 190.6 96.6 180)
+    (at 87.7 58.1)
     (descr "SMD rectangular pad as test Point, square 1.5mm side length")
     (tags "test point SMD pad rectangle square")
@@
     (fp_line (start 1.25 -1.25) (end -1.25 -1.25) (layer "B.CrtYd") (width 0.05))
     (fp_line (start -1.25 1.25) (end -1.25 -1.25) (layer "B.CrtYd") (width 0.05))
-    (pad "1" smd rect (at 0 0 180) (size 1.5 1.5) (layers "B.Cu" "B.Mask")
+    (pad "1" smd rect (at 0 0) (size 1.5 1.5) (layers "B.Cu" "B.Mask")
       (net 140 "/GPIO_07") (pinfunction "1") (pintype "passive"))
   )
@@
   )
   (footprint "TestPoint:TestPoint_Pad_1.5x1.5mm" (layer "B.Cu")
-    (at 190.55 93.25 180)
+    (at 87.65 61.45)
     (descr "SMD rectangular pad as test Point, square 1.5mm side length")
     (tags "test point SMD pad rectangle square")
@@
     (fp_line (start 1.25 -1.25) (end 1.25 1.25) (layer "B.CrtYd") (width 0.05))
     (fp_line (start -1.25 1.25) (end -1.25 -1.25) (layer "B.CrtYd") (width 0.05))
-    (pad "1" smd rect (at 0 0 180) (size 1.5 1.5) (layers "B.Cu" "B.Mask")
+    (pad "1" smd rect (at 0 0) (size 1.5 1.5) (layers "B.Cu" "B.Mask")
       (net 53 "/GPIO_16") (pinfunction "1") (pintype "passive"))
   )
@@
   (segment (start 122.195 135.7) (end 122.195 136.995) (width 0.2) (layer "F.Cu") (net 50))
   (segment (start 125.4 137.3) (end 126.005 136.695) (width 0.2) (layer "F.Cu") (net 50))
+  (segment (start 77.9 54.6) (end 77.4 54.1) (width 0.2) (layer "F.Cu") (net 51))
+  (segment (start 91.04 58) (end 86 58) (width 0.2) (layer "F.Cu") (net 51))
+  (segment (start 82.6 54.6) (end 77.9 54.6) (width 0.2) (layer "F.Cu") (net 51))
+  (segment (start 86 58) (end 82.6 54.6) (width 0.2) (layer "F.Cu") (net 51))
+  (segment (start 91.25 58.21) (end 91.04 58) (width 0.2) (layer "F.Cu") (net 51))
+  (segment (start 91.25 60.75) (end 89.35 60.75) (width 0.2) (layer "F.Cu") (net 52))
+  (segment (start 83.4125 59.7125) (end 81.6 57.9) (width 0.2) (layer "F.Cu") (net 52))
+  (segment (start 89.35 60.75) (end 88.3125 59.7125) (width 0.2) (layer "F.Cu") (net 52))
+  (segment (start 88.3125 59.7125) (end 83.4125 59.7125) (width 0.2) (layer "F.Cu") (net 52))
+  (segment (start 91.25 62.02) (end 89.78 62.02) (width 0.2) (layer "F.Cu") (net 53))
+  (segment (start 89.78 62.02) (end 89.7 62.1) (width 0.2) (layer "F.Cu") (net 53))
+  (via (at 89.7 62.1) (size 0.7) (drill 0.4) (layers "F.Cu" "B.Cu") (net 53))
+  (segment (start 89.7 62.1) (end 89.05 61.45) (width 0.2) (layer "B.Cu") (net 53))
+  (segment (start 89.05 61.45) (end 87.65 61.45) (width 0.2) (layer "B.Cu") (net 53))
   (segment (start 130.6 95.8505) (end 130.6 86.4) (width 0.2) (layer "F.Cu") (net 54))
   (segment (start 123.665686 112.6) (end 119.4 116.865686) (width 0.2) (layer "F.Cu") (net 54))
@@
   (segment (start 69.1 119.8) (end 69.1 135.25) (width 0.2) (layer "B.Cu") (net 135))
   (segment (start 70.25 118.65) (end 69.1 119.8) (width 0.2) (layer "B.Cu") (net 135))
+  (segment (start 86.5 55.9) (end 91.02 55.9) (width 0.2) (layer "F.Cu") (net 136))
+  (segment (start 91.02 55.9) (end 91.25 55.67) (width 0.2) (layer "F.Cu") (net 136))
+  (segment (start 83.5 52.9) (end 86.5 55.9) (width 0.2) (layer "F.Cu") (net 136))
+  (segment (start 83.5 51.8) (end 83.5 52.9) (width 0.2) (layer "F.Cu") (net 136))
+  (segment (start 85.9 56.7) (end 91.01 56.7) (width 0.2) (layer "F.Cu") (net 137))
+  (segment (start 91.01 56.7) (end 91.25 56.94) (width 0.2) (layer "F.Cu") (net 137))
+  (segment (start 80 51.5) (end 80.7 51.5) (width 0.2) (layer "F.Cu") (net 137))
+  (segment (start 80.7 51.5) (end 85.9 56.7) (width 0.2) (layer "F.Cu") (net 137))
   (segment (start 109.27 119.075) (end 109.4 119.205) (width 0.2) (layer "F.Cu") (net 138))
   (segment (start 109.4 119.205) (end 109.4 122.3) (width 0.2) (layer "F.Cu") (net 138))
@@
   (segment (start 112.6505 118.9) (end 113.8495 118.9) (width 0.2) (layer "B.Cu") (net 139))
   (segment (start 113.8495 118.9) (end 113.9495 118.8) (width 0.2) (layer "B.Cu") (net 139))
+  (segment (start 91.25 59.48) (end 89.88 59.48) (width 0.2) (layer "F.Cu") (net 140))
+  (segment (start 89.88 59.48) (end 89.7 59.3) (width 0.2) (layer "F.Cu") (net 140))
+  (via (at 89.7 59.3) (size 0.7) (drill 0.4) (layers "F.Cu" "B.Cu") (net 140))
+  (segment (start 88.5 58.1) (end 87.7 58.1) (width 0.2) (layer "B.Cu") (net 140))
+  (segment (start 89.7 59.3) (end 88.5 58.1) (width 0.2) (layer "B.Cu") (net 140))
   (segment (start 87.13 65.83) (end 85.425 64.125) (width 0.2) (layer "F.Cu") (net 141))
   (segment (start 91.25 65.83) (end 87.13 65.83) (width 0.2) (layer "F.Cu") (net 141))

Commit message: y
Parts:
- added R45: 10k, Resistor_SMD:R_0603_1608Metric_Pad0.98x0.95mm_HandSolder, B.Cu at (99.7, 87.8)
- added R46: 10k, Resistor_SMD:R_0603_1608Metric_Pad0.98x0.95mm_HandSolder, B.Cu at (99.7, 86.3)
- added R47: 10k, Resistor_SMD:R_0603_1608Metric_Pad0.98x0.95mm_HandSolder, B.Cu at (99.7, 84.7)
- added R48: 10k, Resistor_SMD:R_0603_1608Metric_Pad0.98x0.95mm_HandSolder, B.Cu at (99.7, 83.1)
Connections:
- IC1 pad 2: /A1 -> +3V3
- IC1 pad 21: /A0 -> GND
- S1 pad 10: unconnected-(S1-Pad10) -> /GPIO_06
- S1 pad 11: unconnected-(S1-Pad11) -> Net-(S1-Pad11)
- S1 pad 12: unconnected-(S1-Pad12) -> /GPIO_07
- S1 pad 13: unconnected-(S1-Pad13) -> Net-(S1-Pad13)
- S1 pad 14: unconnected-(S1-Pad14) -> /GPIO_15
- S1 pad 15: unconnected-(S1-Pad15) -> Net-(S1-Pad15)
- S1 pad 16: unconnected-(S1-Pad16) -> /GPIO_16
- S1 pad 9: unconnected-(S1-Pad9) -> Net-(S1-Pad9)
Routing:
- net /GPIO_07: track 4.12 -> 37.4 mm, vias 1 -> 2
- net /GPIO_15: track 10.8 -> 40.0 mm, vias 0 -> 1
- net /GPIO_16: track 3.90 -> 29.1 mm, vias 1 -> 2
- net GND: track 156.2 -> 164.2 mm, vias 102 -> 103
- net +3V3: track 268.5 -> 273.2 mm
- net Net-(S1-Pad9): track 0.00 -> 4.29 mm
- net Net-(S1-Pad15): track 0.00 -> 4.08 mm
- net Net-(S1-Pad11): track 0.00 -> 3.88 mm
- net Net-(S1-Pad13): track 0.00 -> 3.69 mm
