File: ESP32_power_meter_MP3_player_WIFI_radio_V2/Power-IN-OUT-BMS.kicad_sch (KiCad schematic)
At the start: 25 parts, among them IC3 MCP73834T-FCI_UN, IC4 AP2112M-3.3TRG1, J13 Conn_01x02, Q1 DMG9933USD-13, U6 LM324A, U7 1043, U8 APX810S05

Commit message: m
Parts:
- renumbered C17 to C18, C18 to C19, C15 to C20, C16 to C21, D2 to D5, D3 to D6, D4 to D7, IC4 to IC3, IC3 to IC4, Q1 to Q2, R36 to R33, R38 to R34, R41 to R35, R37 to R36, R42 to R37, R39 to R38, R40 to R39, R43 to R40, S3 to S2

Commit message: f
Parts:
- removed R37, R40: 1Meg, Resistor_SMD:R_0603_1608Metric_Pad0.98x0.95mm_HandSolder, symbol Device:R_Small
- removed U6: LM324A, Package_SO:SOIC-14_3.9x8.7mm_P1.27mm, symbol Amplifier_Operational:LM324A
- F2: footprint Fuse:Fuse_0603_1608Metric_Pad1.05x0.95mm_HandSolder -> Fuse:Fuse_1812_4532Metric
- IC3: footprint SamacSys_Parts:SOIC127P600X170-8N -> SOIC127P600X170-8N
- IC4: footprint SamacSys_Parts:SOP50P490X110-10N -> SOP50P490X110-10N
- Q2: footprint SamacSys_Parts:SOIC127P600X175-8N -> SOIC127P600X175-8N
- S2: footprint SamacSys_Parts:EG1224 -> EG1224
- U7: footprint SamacSys_Parts:1043 -> 1043
- renumbered C18 to C22, C19 to C23, C20 to C24, C21 to C25, R33 to R39, R34 to R40, R36 to R41, R35 to R42, R38 to R43, R39 to R44
Connections:
- net GND: now also J13.1 (Pin_1); no longer J13.2 (Pin_2)
- net at RV1.1: now also J13.2 (Pin_2); no longer J13.1 (Pin_1)
- net +3V3 renamed +3.3V
Other:
- moved on the sheet: D7, F2, J13, Q2, R42, RV1

Commit message: t
Parts:
- C25: value 4.7u -> 22u; footprint Capacitor_SMD:C_0603_1608Metric_Pad1.08x0.95mm_HandSolder -> Capacitor_SMD:C_0805_2012Metric_Pad1.18x1.45mm_HandSolder
Connections:
- net +3.3V renamed +3V3
Changed lines of the file:
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@@
     )
-  )
-  (hierarchical_label "5v" (shape input) (at 27.94 62.23 90)
-    (effects (font (size 1.27 1.27)) (justify left))
   )
   (symbol (lib_id "Device:R") (at 187.96 105.41 0) (mirror x) (unit 1)
@@
     (pin "2")
   )
+  (symbol (lib_id "power:+3V3") (at 327.66 86.36 0) (unit 1)
+    (in_bom yes) (on_board yes) (fields_autoplaced)
+    (property "Reference" "#PWR0107" (id 0) (at 327.66 90.17 0)
+      (effects (font (size 1.27 1.27)) hide)
+    )
+    (property "Value" "+3V3" (id 1) (at 327.66 81.28 0))
+    (property "Footprint" "" (id 2) (at 327.66 86.36 0)
+      (effects (font (size 1.27 1.27)) hide)
+    )
+    (property "Datasheet" "" (id 3) (at 327.66 86.36 0)
+      (effects (font (size 1.27 1.27)) hide)
+    )
+    (pin "1")
+  )
   (symbol (lib_id "Device:R_Potentiometer") (at 86.36 104.14 270) (unit 1)
     (in_bom yes) (on_board yes)
@@
     (pin "2")
     (pin "3")
+  )
+  (symbol (lib_id "Device:C_Small") (at 104.14 85.09 0) (mirror y) (unit 1)
+    (in_bom yes) (on_board yes)
+    (property "Reference" "C25" (id 0) (at 110.49 83.82 0)
+      (effects (font (size 1.27 1.27)) (justify left))
+    )
+    (property "Value" "22u" (id 1) (at 110.49 86.36 0)
+      (effects (font (size 1.27 1.27)) (justify left))
+    )
+    (property "Footprint" "Capacitor_SMD:C_0805_2012Metric_Pad1.18x1.45mm_HandSolder" (id 2) (at 104.14 85.09 0)
+      (effects (font (size 1.27 1.27)) hide)
+    )
+    (property "Datasheet" "~" (id 3) (at 104.14 85.09 0)
+      (effects (font (size 1.27 1.27)) hide)
+    )
+    (pin "1")
+    (pin "2")
   )
   (symbol (lib_id "Connector_Generic:Conn_01x02") (at 97.79 106.68 0) (mirror x) (unit 1)
@@
     (pin "9")
   )
-  (symbol (lib_id "Device:C_Small") (at 104.14 85.09 0) (mirror y) (unit 1)
-    (in_bom yes) (on_board yes)
-    (property "Reference" "C25" (id 0) (at 112.395 86.995 0)
-      (effects (font (size 1.27 1.27)) (justify left))
-    )
-    (property "Value" "4.7u" (id 1) (at 111.76 84.455 0)
-      (effects (font (size 1.27 1.27)) (justify left))
-    )
-    (property "Footprint" "Capacitor_SMD:C_0603_1608Metric_Pad1.08x0.95mm_HandSolder" (id 2) (at 104.14 85.09 0)
-      (effects (font (size 1.27 1.27)) hide)
-    )
-    (property "Datasheet" "~" (id 3) (at 104.14 85.09 0)
-      (effects (font (size 1.27 1.27)) hide)
-    )
-    (pin "1")
-    (pin "2")
-  )
   (symbol (lib_id "power:+VDC") (at 232.41 78.74 0) (unit 1)
     (in_bom yes) (on_board yes) (fields_autoplaced)
@@
       (effects (font (size 1.27 1.27)) hide)
     )
-    (pin "1")
-  )
-  (symbol (lib_id "power:+3.3V") (at 327.66 86.36 0) (unit 1)
-    (in_bom yes) (on_board yes) (fields_autoplaced)
-    (property "Reference" "#PWR082" (id 0) (at 327.66 90.17 0)
-      (effects (font (size 1.27 1.27)) hide)
-    )
-    (property "Value" "+3.3V" (id 1) (at 327.66 81.28 0))
-    (property "Footprint" "" (id 2) (at 327.66 86.36 0)
-      (effects (font (size 1.27 1.27)) hide)
-    )
-    (property "Datasheet" "" (id 3) (at 327.66 86.36 0)
-      (effects (font (size 1.27 1.27)) hide)
-    )

Commit message: f
Parts:
- removed R40: 10k, Resistor_SMD:R_0603_1608Metric_Pad0.98x0.95mm_HandSolder, symbol Device:R_Small
- removed R43, R44: 10k, Resistor_SMD:R_0603_1608Metric_Pad0.98x0.95mm_HandSolder, symbol Device:R
- added R46, R48, R51: 10k, Resistor_SMD:R_0603_1608Metric, symbol Device:R_Small
Connections:
- net +5V: now also R51.1
- net GND: now also R46.1, R48.2, R51.2
- net low_batt_shutoff: now also R48.1
- net at IC4.8 (THERM): now also R46.2
Changed lines of the file:
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@@
     (stroke (width 0) (type default) (color 0 0 0 0))
   )
-  (wire (pts (xy 187.96 96.52) (xy 187.96 101.6))
+  (wire (pts (xy 187.96 96.52) (xy 187.96 104.14))
     (stroke (width 0) (type default) (color 0 0 0 0))
   )
@@
     (stroke (width 0) (type default) (color 0 0 0 0))
   )
-  (wire (pts (xy 193.04 96.52) (xy 193.04 101.6))
+  (wire (pts (xy 193.04 96.52) (xy 193.04 104.14))
     (stroke (width 0) (type default) (color 0 0 0 0))
   )
@@
     )
   )
-  (symbol (lib_id "Device:R") (at 187.96 105.41 0) (mirror x) (unit 1)
-    (in_bom yes) (on_board yes)
-    (property "Reference" "R43" (id 0) (at 184.15 104.14 0))
-    (property "Value" "10k" (id 1) (at 184.15 106.68 0))
-    (property "Footprint" "Resistor_SMD:R_0603_1608Metric_Pad0.98x0.95mm_HandSolder" (id 2) (at 186.182 105.41 90)
-      (effects (font (size 1.27 1.27)) hide)
-    )
-    (property "Datasheet" "~" (id 3) (at 187.96 105.41 0)
-      (effects (font (size 1.27 1.27)) hide)
-    )
-    (pin "1")
-    (pin "2")
-  )
   (symbol (lib_id "power:+3V3") (at 327.66 86.36 0) (unit 1)
     (in_bom yes) (on_board yes) (fields_autoplaced)
@@
     )
     (property "Datasheet" "~" (id 3) (at 350.52 55.88 0)
+      (effects (font (size 1.27 1.27)) hide)
+    )
+    (pin "1")
+    (pin "2")
+  )
+  (symbol (lib_id "Device:R_Small") (at 187.96 106.68 0) (mirror y) (unit 1)
+    (in_bom yes) (on_board yes)
+    (property "Reference" "R48" (id 0) (at 186.055 104.14 0)
+      (effects (font (size 1.27 1.27)) (justify left))
+    )
+    (property "Value" "10k" (id 1) (at 186.055 106.68 0)
+      (effects (font (size 1.27 1.27)) (justify left))
+    )
+    (property "Footprint" "Resistor_SMD:R_0603_1608Metric" (id 2) (at 187.96 106.68 0)
+      (effects (font (size 1.27 1.27)) hide)
+    )
+    (property "Datasheet" "~" (id 3) (at 187.96 106.68 0)
+      (effects (font (size 1.27 1.27)) hide)
+    )
+    (property "LCSC" "C25804" (id 4) (at 187.96 106.68 0)
       (effects (font (size 1.27 1.27)) hide)
     )
@@
     )
     (pin "1")
-  )
-  (symbol (lib_id "Device:R") (at 193.04 105.41 0) (mirror x) (unit 1)
-    (in_bom yes) (on_board yes)
-    (property "Reference" "R44" (id 0) (at 196.85 104.14 0))
-    (property "Value" "10k" (id 1) (at 196.85 106.68 0))
-    (property "Footprint" "Resistor_SMD:R_0603_1608Metric_Pad0.98x0.95mm_HandSolder" (id 2) (at 191.262 105.41 90)
-      (effects (font (size 1.27 1.27)) hide)
-    )
-    (property "Datasheet" "~" (id 3) (at 193.04 105.41 0)
-      (effects (font (size 1.27 1.27)) hide)
-    )
-    (pin "1")
-    (pin "2")
   )
   (symbol (lib_id "Device:LED_Small") (at 27.94 82.55 180) (unit 1)
@@
     (pin "1")
   )
+  (symbol (lib_id "Device:R_Small") (at 193.04 106.68 0) (mirror y) (unit 1)
+    (in_bom yes) (on_board yes)
+    (property "Reference" "R51" (id 0) (at 198.12 104.14 0)
+      (effects (font (size 1.27 1.27)) (justify left))
+    )
+    (property "Value" "10k" (id 1) (at 198.12 106.68 0)
+      (effects (font (size 1.27 1.27)) (justify left))
+    )
+    (property "Footprint" "Resistor_SMD:R_0603_1608Metric" (id 2) (at 193.04 106.68 0)
+      (effects (font (size 1.27 1.27)) hide)
+    )
+    (property "Datasheet" "~" (id 3) (at 193.04 106.68 0)
+      (effects (font (size 1.27 1.27)) hide)
+    )
+    (property "LCSC" "C25804" (id 4) (at 193.04 106.68 0)
+      (effects (font (size 1.27 1.27)) hide)
+    )
+    (pin "1")
+    (pin "2")
+  )
   (symbol (lib_id "SamacSys_Parts:EG1224") (at 325.12 93.98 90) (mirror x) (unit 1)
     (in_bom yes) (on_board yes) (fields_autoplaced)
@@
     (pin "1")
   )
+  (symbol (lib_id "Device:R_Small") (at 88.9 80.01 270) (mirror x) (unit 1)
+    (in_bom yes) (on_board yes)
+    (property "Reference" "R46" (id 0) (at 91.44 76.2 90)
+      (effects (font (size 1.27 1.27)) (justify left))
+    )
+    (property "Value" "10k" (id 1) (at 91.44 78.74 90)
+      (effects (font (size 1.27 1.27)) (justify left))
+    )
+    (property "Footprint" "Resistor_SMD:R_0603_1608Metric" (id 2) (at 88.9 80.01 0)
+      (effects (font (size 1.27 1.27)) hide)
+    )
+    (property "Datasheet" "~" (id 3) (at 88.9 80.01 0)
+      (effects (font (size 1.27 1.27)) hide)
+    )
+    (property "LCSC" "C25804" (id 4) (at 88.9 80.01 0)
+      (effects (font (size 1.27 1.27)) hide)
+    )
+    (pin "1")
+    (pin "2")
+  )
   (symbol (lib_id "Device:C_Small") (at 40.64 66.04 0) (mirror y) (unit 1)
     (in_bom yes) (on_board yes)
@@
     (pin "1")
   )
-  (symbol (lib_id "Device:R_Small") (at 88.9 80.01 270) (mirror x) (unit 1)
-    (in_bom yes) (on_board yes)
-    (property "Reference" "R40" (id 0) (at 92.075 76.2 90)
-      (effects (font (size 1.27 1.27)) (justify right))
-    )
-    (property "Value" "10k" (id 1) (at 90.805 78.105 90)
-      (effects (font (size 1.27 1.27)) (justify right))
-    )
-    (property "Footprint" "Resistor_SMD:R_0603_1608Metric_Pad0.98x0.95mm_HandSolder" (id 2) (at 88.9 80.01 0)
-      (effects (font (size 1.27 1.27)) hide)
-    )
-    (property "Datasheet" "~" (id 3) (at 88.9 80.01 0)
-      (effects (font (size 1.27 1.27)) hide)
-    )
-    (pin "1")
-    (pin "2")
-  )
   (symbol (lib_id "Device:C_Small") (at 290.83 55.88 0) (unit 1)

Commit message: n
Parts:
- C22, C23, C25: LCSC (none) -> C45783
- C24: LCSC (none) -> C1623
- D5: LCSC (none) -> C2286
- D6: LCSC (none) -> C72043
- R39, R41: value 470 -> 1K; LCSC (none) -> C21190
Changed lines of the file:
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@@
+      (effects (font (size 1.27 1.27)) hide)
+    )
+    (property "LCSC" "C45783" (id 4) (at 350.52 55.88 0)
       (effects (font (size 1.27 1.27)) hide)
     )
@@
       (effects (font (size 1.27 1.27)) hide)
     )
+    (property "LCSC" "C45783" (id 4) (at 104.14 85.09 0)
+      (effects (font (size 1.27 1.27)) hide)
+    )
     (pin "1")
     (pin "2")
@@
       (effects (font (size 1.27 1.27)) (justify right))
     )
-    (property "Value" "470" (id 1) (at 34.925 85.09 90)
+    (property "Value" "1K" (id 1) (at 34.925 85.09 90)
       (effects (font (size 1.27 1.27)) (justify right))
     )
@@
     )
     (property "Datasheet" "~" (id 3) (at 35.56 82.55 0)
+      (effects (font (size 1.27 1.27)) hide)
+    )
+    (property "LCSC" "C21190" (id 4) (at 35.56 82.55 90)
       (effects (font (size 1.27 1.27)) hide)
     )
@@
     )
     (property "Datasheet" "~" (id 3) (at 27.94 82.55 90)
+      (effects (font (size 1.27 1.27)) hide)
+    )
+    (property "LCSC" "C72043" (id 4) (at 27.94 82.55 0)
       (effects (font (size 1.27 1.27)) hide)
     )
@@
       (effects (font (size 1.27 1.27)) (justify right))
     )
-    (property "Value" "470" (id 1) (at 34.29 74.93 90)
+    (property "Value" "1K" (id 1) (at 34.29 74.93 90)
       (effects (font (size 1.27 1.27)) (justify right))
     )
@@
     )
     (property "Datasheet" "~" (id 3) (at 35.56 80.01 0)
+      (effects (font (size 1.27 1.27)) hide)
+    )
+    (property "LCSC" "C21190" (id 4) (at 35.56 80.01 90)
       (effects (font (size 1.27 1.27)) hide)
     )
@@
       (effects (font (size 1.27 1.27)) hide)
     )
+    (property "LCSC" "C1623" (id 4) (at 40.64 66.04 0)
+      (effects (font (size 1.27 1.27)) hide)
+    )
     (pin "1")
     (pin "2")
@@
     )
     (property "Datasheet" "~" (id 3) (at 290.83 55.88 0)
+      (effects (font (size 1.27 1.27)) hide)
+    )
+    (property "LCSC" "C45783" (id 4) (at 290.83 55.88 0)
       (effects (font (size 1.27 1.27)) hide)
     )
@@
       (effects (font (size 1.27 1.27)) hide)
     )
+    (property "LCSC" "C2286" (id 4) (at 27.94 80.01 0)
+      (effects (font (size 1.27 1.27)) hide)
+    )
