File: ESP32_power_meter_MP3_player_WIFI_radio_V2/buck.kicad_sch (KiCad schematic)
At the start: 11 parts, among them U10 DIO6012BCST6

Commit message: m
Parts:
- renumbered C19 to C22, C20 to C23, C21 to C24, C22 to C25, C24 to C26, C25 to C27, U10 to U9
Changed lines of the file:
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@@
   (symbol (lib_id "power:GND") (at 140.335 83.82 0) (unit 1)
     (in_bom yes) (on_board yes) (fields_autoplaced)
-    (property "Reference" "#PWR083" (id 0) (at 140.335 90.17 0)
+    (property "Reference" "#PWR091" (id 0) (at 140.335 90.17 0)
       (effects (font (size 1.27 1.27)) hide)
     )
@@
   (symbol (lib_id "power:GND") (at 61.595 74.93 0) (unit 1)
     (in_bom yes) (on_board yes) (fields_autoplaced)
-    (property "Reference" "#PWR081" (id 0) (at 61.595 81.28 0)
+    (property "Reference" "#PWR085" (id 0) (at 61.595 81.28 0)
       (effects (font (size 1.27 1.27)) hide)
     )
@@
   (symbol (lib_id "My_custom_lib:DIO6012BCST6") (at 84.455 66.675 0) (unit 1)
     (in_bom yes) (on_board yes) (fields_autoplaced)
-    (property "Reference" "U10" (id 0) (at 84.455 55.88 0))
+    (property "Reference" "U9" (id 0) (at 84.455 55.88 0))
     (property "Value" "DIO6012BCST6" (id 1) (at 84.455 58.42 0))
     (property "Footprint" "Package_TO_SOT_SMD:SOT-23-6_Handsoldering" (id 2) (at 81.915 59.055 0)
@@
   (symbol (lib_id "Device:C_Small") (at 154.305 74.93 0) (unit 1)
     (in_bom yes) (on_board yes) (fields_autoplaced)
-    (property "Reference" "C21" (id 0) (at 157.48 73.6662 0)
+    (property "Reference" "C24" (id 0) (at 157.48 73.6662 0)
       (effects (font (size 1.27 1.27)) (justify left))
     )
@@
   (symbol (lib_id "power:GND") (at 81.915 77.47 0) (unit 1)
     (in_bom yes) (on_board yes) (fields_autoplaced)
-    (property "Reference" "#PWR082" (id 0) (at 81.915 83.82 0)
+    (property "Reference" "#PWR086" (id 0) (at 81.915 83.82 0)
       (effects (font (size 1.27 1.27)) hide)
     )
@@
   (symbol (lib_id "power:GND") (at 165.735 81.915 0) (unit 1)
     (in_bom yes) (on_board yes) (fields_autoplaced)
-    (property "Reference" "#PWR085" (id 0) (at 165.735 88.265 0)
+    (property "Reference" "#PWR088" (id 0) (at 165.735 88.265 0)
       (effects (font (size 1.27 1.27)) hide)
     )
@@
   (symbol (lib_id "Device:C_Small") (at 61.595 70.485 0) (unit 1)
     (in_bom yes) (on_board yes) (fields_autoplaced)
-    (property "Reference" "C19" (id 0) (at 64.135 69.2212 0)
+    (property "Reference" "C22" (id 0) (at 64.135 69.2212 0)
       (effects (font (size 1.27 1.27)) (justify left))
     )
@@
   (symbol (lib_id "Device:C_Small") (at 187.96 74.93 0) (unit 1)
     (in_bom yes) (on_board yes) (fields_autoplaced)
-    (property "Reference" "C25" (id 0) (at 190.5 73.6662 0)
+    (property "Reference" "C27" (id 0) (at 190.5 73.6662 0)
       (effects (font (size 1.27 1.27)) (justify left))
     )
@@
   (symbol (lib_id "Device:C_Small") (at 165.735 74.93 0) (unit 1)
     (in_bom yes) (on_board yes) (fields_autoplaced)
-    (property "Reference" "C22" (id 0) (at 168.275 73.6662 0)
+    (property "Reference" "C25" (id 0) (at 168.275 73.6662 0)
       (effects (font (size 1.27 1.27)) (justify left))
     )
@@
   (symbol (lib_id "Device:C_Small") (at 131.445 70.485 0) (unit 1)
     (in_bom yes) (on_board yes)
-    (property "Reference" "C20" (id 0) (at 121.285 69.215 0)
+    (property "Reference" "C23" (id 0) (at 121.285 69.215 0)
       (effects (font (size 1.27 1.27)) (justify left))
     )
@@
   (symbol (lib_id "power:GND") (at 154.305 81.915 0) (unit 1)
     (in_bom yes) (on_board yes) (fields_autoplaced)
-    (property "Reference" "#PWR084" (id 0) (at 154.305 88.265 0)
+    (property "Reference" "#PWR087" (id 0) (at 154.305 88.265 0)
       (effects (font (size 1.27 1.27)) hide)
     )
@@
   (symbol (lib_id "Device:C_Small") (at 176.53 74.93 0) (unit 1)
     (in_bom yes) (on_board yes) (fields_autoplaced)
-    (property "Reference" "C24" (id 0) (at 179.07 73.6662 0)
-      (effects (font (size 1.27 1.27)) (justify left))
-    )
+    (property "Reference" "C26" (id 0) (at 179.07 73.6662 0)
+      (effects (font (size 1.27 1.27)) (justify left))
+    )

Commit message: f
Parts:
- removed C22: 22u, Capacitor_THT:CP_Radial_D5.0mm_P2.00mm, symbol Device:C_Small
- removed C27: 10u, Capacitor_SMD:C_0805_2012Metric, symbol Device:C_Small
- added C26: 22u, Capacitor_SMD:C_0805_2012Metric, symbol Device:C_Small
- C28: renamed from C24; value 10u -> 22u
- C29: renamed from C25; value 10u -> 22u
- C30: renamed from C26; value 10u -> 100n; footprint Capacitor_SMD:C_0805_2012Metric -> Capacitor_SMD:C_0603_1608Metric
- FB2: footprint Resistor_SMD:R_0402_1005Metric_Pad0.72x0.64mm_HandSolder -> Resistor_SMD:R_0603_1608Metric_Pad0.98x0.95mm_HandSolder
- L1: footprint SamacSys_Parts:NRH3012T220MNV -> NRH3012T220MNV
- renumbered C23 to C27
Connections:
- net GND: now also C26.2
- net buck_input_filtered: now also C26.1
Other:
- moved on the sheet: C27, C28, C29, FB2, L1, RR1, RR2

Commit message: n
Parts:
- C26, C28, C29: LCSC (none) -> C45783
- C30: LCSC (none) -> C14663
- RR1: LCSC (none) -> C23265
- RR2: LCSC (none) -> C4184
Changed lines of the file:
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@@
+      (effects (font (size 1.27 1.27)) hide)
+    )
+    (property "LCSC" "C45783" (id 4) (at 62.23 71.12 0)
       (effects (font (size 1.27 1.27)) hide)
     )
@@
     )
     (property "Datasheet" "~" (id 3) (at 140.97 71.12 0)
+      (effects (font (size 1.27 1.27)) hide)
+    )
+    (property "LCSC" "C23265" (id 4) (at 140.97 71.12 0)
       (effects (font (size 1.27 1.27)) hide)
     )
@@
       (effects (font (size 1.27 1.27)) hide)
     )
+    (property "LCSC" "C45783" (id 4) (at 154.94 74.93 0)
+      (effects (font (size 1.27 1.27)) hide)
+    )
     (pin "1")
     (pin "2")
@@
       (effects (font (size 1.27 1.27)) hide)
     )
+    (property "LCSC" "C4184" (id 4) (at 140.97 80.01 0)
+      (effects (font (size 1.27 1.27)) hide)
+    )
     (pin "1")
     (pin "2")
@@
     )
     (property "Datasheet" "~" (id 3) (at 166.37 74.93 0)
+      (effects (font (size 1.27 1.27)) hide)
+    )
+    (property "LCSC" "C45783" (id 4) (at 166.37 74.93 0)
       (effects (font (size 1.27 1.27)) hide)
     )
@@
       (effects (font (size 1.27 1.27)) hide)
     )
+    (property "LCSC" "C14663" (id 4) (at 176.53 74.93 0)
+      (effects (font (size 1.27 1.27)) hide)
+    )
