File: ESP32_power_meter_MP3_player_WIFI_radio_V2/untitled.kicad_sch (KiCad schematic)
At the start: 29 parts, among them IC2 INA2181A4QDGSRQ1, J10 10033527-N3112MLF, J11 Conn_01x02, J12 Conn_01x02, J4 Barrel_Jack_Switch, J5 Barrel_Jack_Switch, J6 Conn_01x03, J7 Conn_01x03, J9 USB_A, U6 LM324A

Commit message: m
Parts:
- renumbered C10 to C13, C13 to C14, C14 to C15, C11 to C16, C12 to C17, J9 to J10, J7 to J11, J4 to J5, J11 to J6, J10 to J7, J5 to J8, J6 to J9, JP2 to JP1, R33 to R20, R34 to R21, R28 to R22, R29 to R23, R31 to R24, R35 to R25, R32 to R26, R24 to R27, R27 to R28, R25 to R29, R22 to R30, R26 to R31, R23 to R32

Commit message: f
Parts:
- removed J7: 10033527-N3112MLF, SamacSys_Parts:10033527N3112MLF, symbol SamacSys_Parts:10033527-N3112MLF
- removed U6: LM324A, Package_SO:SOIC-14_3.9x8.7mm_P1.27mm, symbol Amplifier_Operational:LM324A
- added C13, C14, C18, C21: 100n, Capacitor_SMD:C_0603_1608Metric_Pad1.08x0.95mm_HandSolder, symbol Device:C_Small
- added J8: USB_A, Connector_USB:USB_A_Molex_67643_Horizontal, symbol Connector:USB_A
- added R24, R27, R33, R37: 10k, Resistor_SMD:R_0603_1608Metric_Pad0.98x0.95mm_HandSolder, symbol Device:R_Small
- added U6: LM324, symbol Amplifier_Operational:LM324
- C15: renamed from C13; value 0.1u -> 100n
- renumbered C14 to C16, C15 to C17, C16 to C19, C17 to C20, J12 to J10, J10 to J11, J11 to J12, J8 to J7, R20 to R22, R21 to R23, R22 to R25, R23 to R26, R24 to R28, R25 to R29, R26 to R30, R27 to R31, R28 to R32, R29 to R34, R30 to R35, R31 to R36, R32 to R38
Connections:
- net +VDC: now also U6.4 (V+)
- net ADC_CH0: now also C13.1, R24.2
- net ADC_CH2: now also C14.1, R27.2
- net ADC_CH5: now also C18.1, R33.2; no longer R32.2
- net ADC_CH6: now also C21.1, R37.2; no longer R35.1, R38.2
- net D2+: now also J8.2 (D-)
- net D2-: now also J8.3 (D+)
- net GND: now also J6.1 (Pin_1), C13.2, C14.2, C18.2, C21.2, J8.4 (GND), U6.11 (V-); no longer J6.2 (Pin_2)
- net ext_5v: now also J6.2 (Pin_2), J8.1 (VBUS); no longer J6.1 (Pin_1)
- net at R34.2, R36.2: now also U6.9 (-)
- net at R25.2, R26.1: now also U6.5 (+)
- net at R22.2, R23.1: now also U6.3 (+)
- net at R31.2, R32.1: now also U6.10 (+)
- new net: R32.2, R33.1, U6.8
- new net: R35.1, R37.1, R38.2
- new net: R24.1, U6.1, U6.2 (-)
- new net: R27.1, U6.6 (-), U6.7
Other:
- moved on the sheet: C16, C19, C20, IC2, J10, J11, J12, J5, J6, J7, J9, R28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

Commit message: t
Parts:
- added TP1, TP2, TP3: TestPoint, TestPoint:TestPoint_Pad_1.5x1.5mm, symbol Connector:TestPoint
- R29: footprint Resistor_SMD:R_0402_1005Metric_Pad0.72x0.64mm_HandSolder -> Resistor_SMD:R_0805_2012Metric
Connections:
- net at U6.12 (+): now also TP1.1
- net at U6.13 (-): now also TP3.1
- net at U6.14: now also TP2.1
Other:
- note added: "5m 100gain 2A 1V 200mA 0.1V 20mA 0.01V"
Changed lines of the file:
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@@
+    (stroke (width 0) (type default) (color 0 0 0 0))
+  )
+  (wire (pts (xy 181.61 200.66) (xy 187.96 200.66))
     (stroke (width 0) (type default) (color 0 0 0 0))
   )
@@
     (stroke (width 0) (type default) (color 0 0 0 0))
   )
+  (wire (pts (xy 203.2 203.2) (xy 208.28 203.2))
+    (stroke (width 0) (type default) (color 0 0 0 0))
+  )
   (wire (pts (xy 384.81 24.13) (xy 381 24.13))
     (stroke (width 0) (type default) (color 0 0 0 0))
@@
     (stroke (width 0) (type default) (color 0 0 0 0))
   )
+  (wire (pts (xy 176.53 205.74) (xy 187.96 205.74))
+    (stroke (width 0) (type default) (color 0 0 0 0))
+  )
   (wire (pts (xy 50.8 64.77) (xy 54.61 64.77))
     (stroke (width 0) (type default) (color 0 0 0 0))
@@
   (wire (pts (xy 120.65 205.74) (xy 129.54 205.74))
     (stroke (width 0) (type default) (color 0 0 0 0))
+  )
+  (text "5m  100gain\n2A  1V\n200mA 0.1V\n20mA   0.01V" (at 143.51 208.28 0)
+    (effects (font (size 1.27 1.27)) (justify left bottom))
   )
   (text "USB input for power only" (at 260.858 48.387 0)
@@
     )
     (property "Datasheet" "" (id 3) (at 256.54 132.08 0)
+      (effects (font (size 1.27 1.27)) hide)
+    )
+    (pin "1")
+  )
+  (symbol (lib_id "Connector:TestPoint") (at 181.61 200.66 0) (unit 1)
+    (in_bom no) (on_board yes)
+    (property "Reference" "TP1" (id 0) (at 180.34 194.31 0)
+      (effects (font (size 1.27 1.27)) (justify left))
+    )
+    (property "Value" "TestPoint" (id 1) (at 184.15 198.6279 0)
+      (effects (font (size 1.27 1.27)) (justify left) hide)
+    )
+    (property "Footprint" "TestPoint:TestPoint_Pad_1.5x1.5mm" (id 2) (at 186.69 200.66 0)
+      (effects (font (size 1.27 1.27)) hide)
+    )
+    (property "Datasheet" "~" (id 3) (at 186.69 200.66 0)
       (effects (font (size 1.27 1.27)) hide)
     )
@@
       (effects (font (size 1.27 1.27)) (justify right))
     )
-    (property "Footprint" "Resistor_SMD:R_0402_1005Metric_Pad0.72x0.64mm_HandSolder" (id 2) (at 380.238 76.2 90)
+    (property "Footprint" "Resistor_SMD:R_0805_2012Metric" (id 2) (at 380.238 76.2 90)
       (effects (font (size 1.27 1.27)) hide)
     )
@@
     (pin "1")
     (pin "2")
+  )
+  (symbol (lib_id "Connector:TestPoint") (at 176.53 205.74 0) (unit 1)
+    (in_bom no) (on_board yes)
+    (property "Reference" "TP3" (id 0) (at 175.26 199.39 0)
+      (effects (font (size 1.27 1.27)) (justify left))
+    )
+    (property "Value" "TestPoint" (id 1) (at 179.07 203.7079 0)
+      (effects (font (size 1.27 1.27)) (justify left) hide)
+    )
+    (property "Footprint" "TestPoint:TestPoint_Pad_1.5x1.5mm" (id 2) (at 181.61 205.74 0)
+      (effects (font (size 1.27 1.27)) hide)
+    )
+    (property "Datasheet" "~" (id 3) (at 181.61 205.74 0)
+      (effects (font (size 1.27 1.27)) hide)
+    )
+    (pin "1")
   )
   (symbol (lib_id "Device:C_Small") (at 370.84 200.66 0) (unit 1)
@@
       (effects (font (size 1.27 1.27)) hide)
     )
+    (pin "1")
+  )
+  (symbol (lib_id "Connector:TestPoint") (at 208.28 203.2 0) (unit 1)
+    (in_bom no) (on_board yes)
+    (property "Reference" "TP2" (id 0) (at 207.01 196.85 0)
+      (effects (font (size 1.27 1.27)) (justify left))
+    )
+    (property "Value" "TestPoint" (id 1) (at 210.82 201.1679 0)
+      (effects (font (size 1.27 1.27)) (justify left) hide)
+    )
+    (property "Footprint" "TestPoint:TestPoint_Pad_1.5x1.5mm" (id 2) (at 213.36 203.2 0)
+      (effects (font (size 1.27 1.27)) hide)
+    )
+    (property "Datasheet" "~" (id 3) (at 213.36 203.2 0)
+      (effects (font (size 1.27 1.27)) hide)
+    )

Commit message: f
Parts:
- removed R22, R23, R24, R25: 10k, Resistor_SMD:R_0603_1608Metric_Pad0.98x0.95mm_HandSolder, symbol Device:R_Small
- added R40, R43, R44, R45: 10k, Resistor_SMD:R_0603_1608Metric, symbol Device:R_Small
- R27, R33, R35, R37, R38: footprint Resistor_SMD:R_0603_1608Metric_Pad0.98x0.95mm_HandSolder -> Resistor_SMD:R_0603_1608Metric; LCSC (none) -> C25804
Connections:
- net ADC_CH0: now also R35.2
- net ADC_CH2: now also R38.2; no longer R27.2
- net ADC_CH5: now also R40.1; no longer R33.2
- net ADC_CH6: now also R44.2; no longer R37.2
- net GND: now also R27.2, R37.2, TP1.1, U6.12 (+), R45.1; no longer R38.1
- net Power_in+: now also R43.2; no longer R35.2
- net mini_power_source: now also R33.1
- net at U6.3 (+): now also R27.1, R33.2
- net at R32.2, U6.8: now also R40.2; no longer R33.1
- net at R26.1, U6.5 (+): now also R37.1
- net at TP3.1, U6.13 (-): now also TP2.1, U6.14
- net at U6.1, U6.2 (-): now also R35.1
- net at U6.6 (-), U6.7: now also R38.1; no longer R27.1
- new net: R43.1, R44.1, R45.2
Other:
- moved on the sheet: TP2

Commit message: n
Parts:
- C13: LCSCC (none) -> C14663
- C14, C15, C18, C21: LCSC (none) -> C14663
- C16, C17, C20: LCSC (none) -> C1623
- R31, R34: LCSC (none) -> C21190
- R32, R36: LCSC (none) -> C25803
- U6: footprint (none) -> Package_SO:SOIC-14_3.9x8.7mm_P1.27mm; LCSC (none) -> C71035
- U6: LCSC (none) -> C71035
Changed lines of the file:
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@@
+      (effects (font (size 1.27 1.27)) hide)
+    )
+    (property "LCSC" "C25803" (id 4) (at 82.55 214.63 0)
       (effects (font (size 1.27 1.27)) hide)
     )
@@
       (effects (font (size 1.27 1.27)) hide)
     )
+    (property "LCSC" "C1623" (id 4) (at 367.03 200.66 0)
+      (effects (font (size 1.27 1.27)) hide)
+    )
     (pin "1")
     (pin "2")
@@
     (property "Reference" "U6" (id 0) (at 95.25 210.82 0))
     (property "Value" "LM324" (id 1) (at 95.25 213.36 0))
-    (property "Footprint" "" (id 2) (at 91.44 203.2 0)
+    (property "Footprint" "Package_SO:SOIC-14_3.9x8.7mm_P1.27mm" (id 2) (at 91.44 203.2 0)
       (effects (font (size 1.27 1.27)) hide)
     )
     (property "Datasheet" "http://www.ti.com/lit/ds/symlink/lm2902-n.pdf" (id 3) (at 93.98 200.66 0)
+      (effects (font (size 1.27 1.27)) hide)
+    )
+    (property "LCSC" "C71035" (id 4) (at 92.71 205.74 0)
       (effects (font (size 1.27 1.27)) hide)
     )
@@
       (effects (font (size 1.27 1.27)) hide)
     )
+    (property "LCSC" "C14663" (id 4) (at 52.07 224.79 0)
+      (effects (font (size 1.27 1.27)) hide)
+    )
     (pin "1")
     (pin "2")
@@
     )
     (property "Datasheet" "~" (id 3) (at 246.38 137.16 0)
+      (effects (font (size 1.27 1.27)) hide)
+    )
+    (property "LCSC" "C14663" (id 4) (at 246.38 137.16 0)
       (effects (font (size 1.27 1.27)) hide)
     )
@@
       (effects (font (size 1.27 1.27)) hide)
     )
+    (property "LCSC" "C1623" (id 4) (at 283.21 213.36 0)
+      (effects (font (size 1.27 1.27)) hide)
+    )
     (pin "1")
     (pin "2")
@@
       (effects (font (size 1.27 1.27)) hide)
     )
+    (property "LCSC" "C1623" (id 4) (at 370.84 200.66 0)
+      (effects (font (size 1.27 1.27)) hide)
+    )
     (pin "1")
     (pin "2")
@@
     (property "Reference" "U6" (id 0) (at 358.14 35.56 0))
     (property "Value" "LM324" (id 1) (at 358.14 38.1 0))
-    (property "Footprint" "" (id 2) (at 363.22 29.21 0)
+    (property "Footprint" "Package_SO:SOIC-14_3.9x8.7mm_P1.27mm" (id 2) (at 363.22 29.21 0)
       (effects (font (size 1.27 1.27)) hide)
     )
     (property "Datasheet" "http://www.ti.com/lit/ds/symlink/lm2902-n.pdf" (id 3) (at 360.68 26.67 0)
+      (effects (font (size 1.27 1.27)) hide)
+    )
+    (property "LCSC" "C71035" (id 4) (at 361.95 31.75 0)
       (effects (font (size 1.27 1.27)) hide)
     )
@@
       (effects (font (size 1.27 1.27)) hide)
     )
+    (property "LCSC" "C14663" (id 4) (at 120.65 210.82 0)
+      (effects (font (size 1.27 1.27)) hide)
+    )
     (pin "1")
     (pin "2")
@@
       (effects (font (size 1.27 1.27)) hide)
     )
+    (property "LCSC" "C21190" (id 4) (at 77.47 195.58 90)
+      (effects (font (size 1.27 1.27)) hide)
+    )
     (pin "1")
     (pin "2")
@@
       (effects (font (size 1.27 1.27)) hide)
     )
+    (property "LCSC" "C21190" (id 4) (at 74.93 208.28 90)
+      (effects (font (size 1.27 1.27)) hide)
+    )
     (pin "1")
     (pin "2")
@@
       (effects (font (size 1.27 1.27)) (justify left))
     )
-    (property "Footprint" "" (id 2) (at 289.56 210.82 0)
+    (property "Footprint" "Package_SO:SOIC-14_3.9x8.7mm_P1.27mm" (id 2) (at 289.56 210.82 0)
       (effects (font (size 1.27 1.27)) hide)
     )
     (property "Datasheet" "http://www.ti.com/lit/ds/symlink/lm2902-n.pdf" (id 3) (at 292.1 208.28 0)
+      (effects (font (size 1.27 1.27)) hide)
+    )
+    (property "LCSC" "C71035" (id 4) (at 290.83 213.36 0)
       (effects (font (size 1.27 1.27)) hide)
     )
@@
     (property "Reference" "U6" (id 0) (at 111.76 59.69 0))
     (property "Value" "LM324" (id 1) (at 111.76 62.23 0))
-    (property "Footprint" "" (id 2) (at 118.11 53.34 0)
+    (property "Footprint" "Package_SO:SOIC-14_3.9x8.7mm_P1.27mm" (id 2) (at 118.11 53.34 0)
       (effects (font (size 1.27 1.27)) hide)
     )
     (property "Datasheet" "http://www.ti.com/lit/ds/symlink/lm2902-n.pdf" (id 3) (at 115.57 50.8 0)
+      (effects (font (size 1.27 1.27)) hide)
+    )
+    (property "LCSC" "C71035" (id 4) (at 116.84 55.88 0)
       (effects (font (size 1.27 1.27)) hide)
     )
@@
       (effects (font (size 1.27 1.27)) hide)
     )
+    (property "LCSC" "C25803" (id 4) (at 90.17 195.58 90)
+      (effects (font (size 1.27 1.27)) hide)
+    )
     (pin "1")
     (pin "2")
@@
     )
     (property "Datasheet" "http://www.ti.com/lit/ds/symlink/lm2902-n.pdf" (id 3) (at 196.85 198.12 0)
+      (effects (font (size 1.27 1.27)) hide)
+    )
+    (property "LCSC" "C71035" (id 4) (at 195.58 203.2 0)
       (effects (font (size 1.27 1.27)) hide)
     )
@@
       (effects (font (size 1.27 1.27)) hide)
     )
+    (property "LCSC" "C14663" (id 4) (at 91.44 60.96 0)
+      (effects (font (size 1.27 1.27)) hide)
+    )
     (pin "1")
     (pin "2")
@@
       (effects (font (size 1.27 1.27)) hide)
     )
+    (property "LCSCC" "C14663" (id 4) (at 336.55 36.83 0)
+      (effects (font (size 1.27 1.27)) hide)
+    )
